Commit message: fixed xacro error, move property outside macro

File: tor_description/urdf/leg/leg.urdf.xacro (robot description, xacro)
@@ -1,57 +1,9 @@
 <?xml version="1.0"?>
-<robot xmlns:xacro="http://ros.org/wiki/xacro" name="tor">
-    <!--
-    <link name="base_link">
-      <inertial>
-        <origin xyz="0.0 0.0 0.36" rpy="0 0 0"/>
-        <mass value="34.0" />
-         <inertia ixx="0.1"  ixy="0.0"  ixz="0.0" iyy="0.1" iyz="0.0" izz="0.1" />
-      </inertial>
-      <visual>
-        <origin rpy="0 0 0" xyz="0 0 0"/>
-        <geometry>
-          <mesh filename="package://tor_description/meshes/torso_dummy.stl" scale="1 1 1"/>
-        </geometry>
-      </visual>
-      <collision>
-       <origin rpy="0 0 0" xyz="0 0 0.05"/>
-	    <geometry>
-           <box size="0.1 0.3 0.1"/>
-        </geometry>
-      </collision>
-     </link>
-     -->
-   <!--
-    <link name="torso_link">
-      <inertial>
-        <origin xyz="0.0 0.0 0.4" rpy="0 0 0"/>
-        <mass value="50.0" />
-         <inertia ixx="0.03"  ixy="0.0"  ixz="0.0" iyy="0.03" iyz="0.0" izz="0.03" />
-      </inertial>
-      <visual>
-        <origin rpy="0 0 0" xyz="0 0 0.3"/>
-	<geometry>
-           <box size="0.1 0.1 0.45"/>
-        </geometry>
-      </visual>
-      <collision>
-       <origin rpy="0 0 0" xyz="0 0 0.3"/>
-	<geometry>
-           <box size="0.1 0.1 0.45"/>
-        </geometry>
-      </collision>
-     </link>
-    <joint name="torso_fixed_joint" type="fixed">
-      <parent link="base_link" />
-      <child link="torso_link" />
-      <origin xyz="0.0 0.0 0.0" rpy="0 0 0" />
-      <axis xyz="0 0 1" />
-     </joint>
-    -->
-    <xacro:include filename="$(find tor_description)/urdf/leg/leg.transmission.xacro" />
-    <xacro:property name="leg_reduction"      value="1.0" />
+<robot name="tor" xmlns:xacro="http://ros.org/wiki/xacro" >
+   <xacro:include filename="$(find tor_description)/urdf/leg/leg.transmission.xacro" />
+   <xacro:property name="leg_reduction"      value="1.0" />
+   <xacro:property name="leg_friction"       value="0.0" />
+   <xacro:property name="leg_damping"        value="0.0" />
    <xacro:macro name="tor_leg" params="prefix reflect">
-  <xacro:property name="leg_friction"       value="0.0" />
-  <xacro:property name="leg_damping"        value="0.0" />
     <link name="leg_${prefix}_1_link">
       <inertial>

Commit message: Added correct joint limit for Z leg

File: tor_description/urdf/leg/leg.urdf.xacro (robot description, xacro)
@@ -141,5 +141,10 @@
       <!-- <limit lower="-0.5236" upper="1.571" effort="49" velocity="3.87" /> -->
       <!-- peak -->
-      <limit lower="-0.5236" upper="1.571" effort="100" velocity="3.87" />
+      <xacro:if value="${reflect == 1}">
+        <limit lower="-0.5236" upper="1.571" effort="100" velocity="3.87" />
+      </xacro:if>
+      <xacro:if value="${reflect == -1}">
+        <limit lower="-1.571" upper="0.5236" effort="100" velocity="3.87" />
+      </xacro:if>
       <dynamics friction="${leg_friction}" damping="${leg_damping}"/>
      </joint>
