Commit message: Added simmetry in v2

File: tor_description/urdf/leg/leg_v2.urdf.xacro (robot description, xacro)
@@ -79,5 +79,5 @@
     <link name="leg_${prefix}_3_link">
       <inertial>
-        <origin xyz="0.00658 0.06563 -0.17278" rpy="0.00000 0.00000 0.00000"/>
+        <origin xyz="0.00658 ${reflect*0.06563} -0.17278" rpy="0.00000 0.00000 0.00000"/>
         <mass value="6.82734"/>
         <inertia ixx="0.12390600000" ixy="${reflect*-0.00041200000}" ixz="-0.00205900000"
@@ -111,8 +111,8 @@
     <link name="leg_${prefix}_4_link">
       <inertial>
-        <origin xyz="0.01520 0.02331 -0.12063" rpy="0.00000 0.00000 0.00000"/>
+        <origin xyz="0.01520 ${reflect*0.02331} -0.12063" rpy="0.00000 0.00000 0.00000"/>
         <mass value="3.63668"/>
-        <inertia ixx="0.03531500000" ixy="0.00002900000" ixz="-0.00016600000"
-                 iyy="0.02933600000" iyz="-0.00130500000"
+        <inertia ixx="0.03531500000" ixy="${reflect*0.00002900000}" ixz="-0.00016600000"
+                 iyy="0.02933600000" iyz="${reflect*-0.00130500000}"
                  izz="0.01174000000"/>
       </inertial>
@@ -145,6 +145,6 @@
         <origin xyz="-0.01106 ${reflect*0.04708} 0.05271" rpy="0.00000 0.00000 0.00000"/>
         <mass value="1.24433"/>
-        <inertia ixx="0.01148700000" ixy="-0.00068600000" ixz="-0.00052600000"
-                 iyy="0.00952600000" iyz="0.00263300000"
+        <inertia ixx="0.01148700000" ixy="${reflect*-0.00068600000}" ixz="-0.00052600000"
+                 iyy="0.00952600000" iyz="${reflect*0.00263300000}"
                  izz="0.00390800000"/>
       </inertial>

Commit message: Added tor leg v2

File: tor_description/urdf/leg/leg_v2.urdf.xacro (robot description, xacro)
@@ -38,8 +38,10 @@
               rpy="${0.00000 * deg_to_rad} ${0.00000 * deg_to_rad} ${0.00000 * deg_to_rad}"/>
       <axis xyz="0 0 1" />
-      <!-- trick to use reflect (left=1, right=-1)
-           to make ranges -30 to 90 and -90 to 30 respectively
-           as (reflect-1.0) will be either 0.0 or -2.0 -->
-      <limit lower="${(-30.0 + (reflect-1.0)*30.0) * deg_to_rad}" upper="${(90.0 + (reflect-1.0)*30.0) * deg_to_rad}" effort="160" velocity="5.8"/>
+     <xacro:if value="${reflect == 1}">
+        <limit lower="-0.5236" upper="1.571" effort="100" velocity="3.87" />
+      </xacro:if>
+      <xacro:if value="${reflect == -1}">
+        <limit lower="-1.571" upper="0.5236" effort="100" velocity="3.87" />
+      </xacro:if>
       <dynamics friction="${leg_friction}" damping="${leg_damping}"/>
     </joint>
@@ -73,5 +75,5 @@
               rpy="${0.00000 * deg_to_rad} ${0.00000 * deg_to_rad} ${0.00000 * deg_to_rad}"/>
       <axis xyz="1 0 0" />
-      <limit lower="${reflect*-30.00000 * deg_to_rad}" upper="${reflect*30.00000 * deg_to_rad}" effort="160" velocity="5.8"/>
+      <limit lower="-0.524" upper="0.5236" effort="160" velocity="5.8" />
       <dynamics friction="${leg_friction}" damping="${leg_damping}"/>
     </joint>
@@ -105,5 +107,5 @@
               rpy="${0.00000 * deg_to_rad} ${0.00000 * deg_to_rad} ${0.00000 * deg_to_rad}"/>
       <axis xyz="0 1 0" />
-      <limit lower="${-120.00000 * deg_to_rad}" upper="${45.00000 * deg_to_rad}" effort="160" velocity="5.8"/>
+      <limit lower="-2.095" upper="0.7" effort="160" velocity="5.8" />
       <dynamics friction="${leg_friction}" damping="${leg_damping}"/>
     </joint>
@@ -137,5 +139,5 @@
               rpy="${0.00000 * deg_to_rad} ${0.00000 * deg_to_rad} ${0.00000 * deg_to_rad}"/>
       <axis xyz="0 1 0" />
-      <limit lower="${0.00000 * deg_to_rad}" upper="${150.00000 * deg_to_rad}" effort="300" velocity="7" />
+      <limit lower="0" upper="2.618" effort="300" velocity="7" />
       <dynamics friction="${leg_friction}" damping="${leg_damping}"/>
     </joint>
@@ -169,5 +171,5 @@
               rpy="${0.00000 * deg_to_rad} ${0.00000 * deg_to_rad} ${0.00000 * deg_to_rad}"/>
       <axis xyz="0 1 0" />
-      <limit lower="${-75.00000 * deg_to_rad}" upper="${45.00000 * deg_to_rad}" effort="160" velocity="5.8"/>
+      <limit lower="-1.309" upper="0.768" effort="160" velocity="5.8" />
       <dynamics friction="${leg_friction}" damping="${leg_damping}"/>
     </joint>
@@ -201,5 +203,5 @@
               rpy="${0.00000 * deg_to_rad} ${0.00000 * deg_to_rad} ${0.00000 * deg_to_rad}"/>
       <axis xyz="1 0 0" />
-      <limit lower="${-30.00000 * deg_to_rad}" upper="${30.00000 * deg_to_rad}" effort="100" velocity="4.8"/>
+      <limit lower="-0.524" upper="0.524" effort="100" velocity="4.8" />
       <dynamics friction="${leg_friction}" damping="${leg_damping}"/>
     </joint>
