Commit message: Copied joint limits from v1 to v2

File: tor_description/robots/tor_lower_body_v1.urdf.xacro (robot description, xacro)
@@ -11,27 +11,24 @@
         xmlns:controller="http://playerstage.sourceforge.net/gazebo/xmlschema/#controller"
         xmlns:interface="http://playerstage.sourceforge.net/gazebo/xmlschema/#interface">
-  <xacro:include filename="$(find tor_description)/urdf/leg/leg_v2.urdf.xacro" />
+  <xacro:include filename="$(find tor_description)/urdf/leg/leg.urdf.xacro" />
     <link name="base_link">
       <inertial>
-        <origin xyz="-0.06071 0.00861 0.06368" rpy="0.00000 0.00000 0.00000"/>
-        <mass value="13.34865"/>
-        <inertia ixx="0.06652900000" ixy="-0.00035700000" ixz="0.00027600000"
-                 iyy="0.03746500000" iyz="-0.00125400000"
-                 izz="0.07895100000"/>
+        <origin xyz="0.0 0.0 0.36" rpy="0 0 0"/>
+        <mass value="34.0" />
+         <inertia ixx="0.529688470"  ixy="0.0"  ixz="0.0" iyy="0.34860507904" iyz="0.0" izz="0.23865908621" />
       </inertial>
       <visual>
         <origin rpy="0 0 0" xyz="0 0 0"/>
         <geometry>
-          <mesh filename="package://tor_description/meshes/v2/base_link_lo_res.stl" scale="1 1 1"/>
+          <mesh filename="package://tor_description/meshes/torso_dummy.stl" scale="1 1 1"/>
         </geometry>
-        <material name="DarkGrey" />
       </visual>
       <collision>
-        <origin rpy="0 0 0" xyz="0 0 0"/>
-        <geometry>
-          <mesh filename="package://tor_description/meshes/v2/base_link_collision.stl" scale="1 1 1"/>
+       <origin rpy="0 0 0" xyz="0 0 0.05"/>
+	    <geometry>
+           <box size="0.1 0.3 0.1"/>
         </geometry>
       </collision>
-    </link>
+     </link>
    <xacro:tor_leg prefix="left"  reflect="1" />
    <xacro:tor_leg prefix="right" reflect="-1" />
@@ -40,3 +37,8 @@
   <!-- Materials for visualization -->
   <xacro:include filename="$(find tor_description)/urdf/materials.urdf.xacro" />
+  <xacro:include filename="$(find tor_description)/urdf/sensors/imu.urdf.xacro" />
+    <!-- imu -->
+  <xacro:tor_imu name="imu" parent="base_link" update_rate="100.0">
+    <origin xyz="0 0 0" rpy="0 0 0"/>
+  </xacro:tor_imu>
 </robot>
