Commit message: Updating links from the arm 7 to the gripper (provisional dummy gripper

File: tor_description/robots/tor_full.urdf.xacro (robot description, xacro)
@@ -14,4 +14,5 @@
   <xacro:include filename="$(find tor_description)/urdf/head/head.urdf.xacro" />
   <xacro:include filename="$(find tor_description)/urdf/arm/arm.urdf.xacro" />
+  <xacro:include filename="$(find tor_description)/urdf/sensors/ftsensor.urdf.xacro" />
   <xacro:include filename="$(find tor_description)/urdf/gripper/gripper.urdf.xacro" />
   <xacro:include filename="$(find tor_description)/urdf/leg/leg_v2.urdf.xacro" />
@@ -20,6 +21,8 @@
   <xacro:tor_arm name="arm" parent="torso_2_link" side="left" reflect="1"/>
   <xacro:tor_arm name="arm" parent="torso_2_link" side="right" reflect="-1"/>
-  <xacro:tor_gripper name="left_gripper" parent="arm_left_7_link"/>
-  <xacro:tor_gripper name="right_gripper" parent="arm_right_7_link"/>
+  <xacro:ft_sensor name="wrist" parent="arm_right_7_link" side="right" reflect="1"  />
+  <xacro:ft_sensor name="wrist" parent="arm_left_7_link"  side="left"  reflect="-1" />
+  <xacro:tor_gripper name="left_gripper" parent="wrist_left_ft_tool_link"/>
+  <xacro:tor_gripper name="right_gripper" parent="wrist_right_ft_tool_link"/>
   <xacro:tor_leg prefix="left"  reflect="1" />
   <xacro:tor_leg prefix="right" reflect="-1" />

File: tor_description/urdf/arm/arm.urdf.xacro (robot description, xacro)
@@ -217,5 +217,5 @@
     <!--        TOOL           -->
     <!--***********************-->
-    <link name="${name}_${side}_tool_link">
+<!--     <link name="${name}_${side}_tool_link">
       <inertial>
         <mass value="0.1" />
@@ -239,6 +239,12 @@
       <parent link="${name}_${side}_7_link" />
       <child link="${name}_${side}_tool_link" />
-      <origin xyz="0 0 ${reflect * 0.046}" rpy="${90.0 * deg_to_rad} ${-90.0 * reflect * deg_to_rad} 0" />
-    </joint>
+      <xacro:if value="${reflect == 1}">
+        <origin xyz="0 0 -0.051" rpy="0 ${90.0 * deg_to_rad} 0" />
+      </xacro:if>
+      <xacro:if value="${reflect == -1}">
+        <origin xyz="0 0 -0.051" rpy="${180.0 * deg_to_rad} ${90.0 * deg_to_rad} ${0.0 * deg_to_rad}" />
+      </xacro:if>
+    </joint>
+ -->
     <!-- extensions -->
     <xacro:tor_arm_simple_transmission name="${name}" side="${side}" number="1" reduction="1.0" />

File: tor_description/urdf/gripper/gripper.urdf.xacro (robot description, xacro)
@@ -6,5 +6,5 @@
   <xacro:include filename="$(find tor_description)/urdf/gripper.gazebo.xacro" /> -->
   <xacro:macro name="tor_gripper" params="name parent">
-  <link name="${name}_link">
+  <link name="${name}_base_link">
     <inertial>
       <origin xyz="0.01507 -0.01177 -0.02788" rpy="0.00000 0.00000 0.00000"/>
@@ -17,5 +17,33 @@
       <origin rpy="0 0 0" xyz="0 0 0" />
       <geometry>
-        <mesh filename="package://tor_description/meshes/gripper/gripper.STL"/>
+        <mesh filename="package://tor_description/meshes/gripper/base_link.STL"/>
+      </geometry>
+      <material name="DarkGrey"/>
+    </visual>
+    <collision>
+      <origin rpy="0 0 0" xyz="0 0 0" />
+      <geometry>
+        <mesh filename="package://tor_description/meshes/gripper/base_link_collision.STL"/>
+      </geometry>
+    </collision>
+  </link>
+  <joint name="${name}_base_joint" type="fixed">
+    <parent link="${parent}" />
+    <child link="${name}_base_link" />
+    <axis xyz="0 0 0" />
+    <origin xyz="0 0 0" rpy="0 0 0" />
+  </joint>
+  <link name="${name}_link">
+    <inertial>
+      <origin xyz="0.01507 -0.01177 -0.02788" rpy="0.00000 0.00000 0.00000"/>
+      <mass value="0.3"/>
+      <inertia ixx="0.00195600000" ixy="-0.00007300000" ixz="0.00026500000"
+               iyy="0.00139500000" iyz="-0.00015700000"
+               izz="0.00170400000"/>
+    </inertial>
+    <visual>
+      <origin rpy="0 0 0" xyz="0 0 0" />
+      <geometry>
+        <mesh filename="package://tor_description/meshes/gripper/gripper_simple.STL"/>
       </geometry>
       <material name="Orange"/>
@@ -24,13 +52,13 @@
       <origin rpy="0 0 0" xyz="0 0 0" />
       <geometry>
-        <mesh filename="package://tor_description/meshes/gripper/gripper_collision.STL"/>
+        <mesh filename="package://tor_description/meshes/gripper/gripper_simple_collision.STL"/>
       </geometry>
     </collision>
   </link>
   <joint name="${name}_joint" type="fixed">
-    <parent link="${parent}" />
+    <parent link="${name}_base_link" />
     <child link="${name}_link" />
     <axis xyz="0 0 0" />
-    <origin xyz="0 0.02 -0.10975" rpy="0 0 0" />
+    <origin xyz="0 0.02025 -0.02875" rpy="0 0 0" />
   </joint>
  </xacro:macro>

File: tor_description/urdf/sensors/ftsensor.urdf.xacro (robot description, xacro)
@@ -34,5 +34,5 @@
       <parent link="${parent}" />
       <child link="${name}_${side}_ft_link" />
-      <origin xyz="${0.0157*0.5} 0 0" rpy="${90.0 * deg_to_rad} 0 ${90.0 * deg_to_rad}" />
+      <origin xyz="0 0 -0.051" rpy="${0.0 * deg_to_rad} 0 ${-90.0 * deg_to_rad}" />
     </joint>
     <!--***********************-->
@@ -45,5 +45,5 @@
       </inertial>
       <visual>
-        <origin xyz="0.0 0 0" rpy="0 ${90.0 * deg_to_rad} 0" />
+        <origin xyz="0.0 0 0" rpy="0 ${0.0 * deg_to_rad} 0" />
         <geometry>
           <cylinder radius="${0.05*0.5}" length="0.00975"/>
@@ -52,5 +52,5 @@
       </visual>
       <collision>
-        <origin xyz="0.0 0 0" rpy="0 ${90.0 * deg_to_rad} 0" />
+        <origin xyz="0.0 0 0" rpy="0 ${0.0 * deg_to_rad} 0" />
         <geometry>
           <cylinder radius="${0.05*0.5}" length="0.00975"/>
@@ -61,5 +61,5 @@
       <parent link="${name}_${side}_ft_link" />
       <child link="${name}_${side}_ft_tool_link" />
-      <origin xyz="0 0 ${0.0157*0.5 + 0.00975*0.5}" rpy="${-90.0 * deg_to_rad} ${-90.0 * deg_to_rad} 0" />
+      <origin xyz="0 0 ${-1.0 * (0.0157*0.5 + 0.00975*0.5)}" rpy="0 0 ${-90.0 * reflect * deg_to_rad}" />
     </joint>
 </xacro:macro>
