Commit message: Full model

File: tor_description/urdf/head/head.urdf.xacro (robot description, xacro)
@@ -34,5 +34,5 @@
           <mesh filename="package://tor_description/meshes/head/head_1.stl" scale="1 1 1"/>
         </geometry>
-        <material name="LightGrey" />
+        <material name="DarkGrey" />
       </visual>
       <collision>

File: tor_description/urdf/materials.urdf.xacro (robot description, xacro)
@@ -29,3 +29,6 @@
     <color rgba="1.0 1.0 1.0 1.0"/>
   </material>
+  <material name="Orange">
+    <color rgba="1.0 0.5 0.0 1.0"/>
+  </material>
 </robot>
