Commit message: Mirrowed com position shoulder

File: tor_description/urdf/arm/arm.urdf.xacro (robot description, xacro)
@@ -31,5 +31,5 @@
       <!-- TODO: Missing reflects of inertias -->
       <inertial>
-        <origin xyz="-0.01346 0.09130 0.04812" rpy="0.00000 0.00000 0.00000"/>
+        <origin xyz="-0.01346 ${reflect*0.09130} 0.04812" rpy="0.00000 0.00000 0.00000"/>
         <mass value="1.52896"/>
         <inertia ixx="0.00555100000" ixy="-0.00073100000" ixz="0.00000800000"
