Commit message: Added imu

File: tor_description/gazebo/gazebo.urdf.xacro (robot description, xacro)
@@ -15,5 +15,5 @@
     </plugin>
   </gazebo>
-  <gazebo reference="base_link">
+  <gazebo reference="imu_link">
     <!-- this is expected to be reparented to pelvis with appropriate offset
          when imu_link is reduced by fixed joint reduction -->
@@ -53,4 +53,18 @@
             <bias_stddev>0.001</bias_stddev>
           </accel>
+          <!--
+          <rate>
+            <mean>0.0</mean>
+            <stddev>0</stddev>
+            <bias_mean>0.000000</bias_mean>
+            <bias_stddev>0.0000008</bias_stddev>
+          </rate>
+          <accel>
+            <mean>0.0</mean>
+            <stddev>0</stddev>
+            <bias_mean>0.0</bias_mean>
+            <bias_stddev>0.000</bias_stddev>
+          </accel>
+          -->
         </noise>
       </imu>

File: tor_description/robots/tor_lower_body.urdf.xacro (robot description, xacro)
@@ -37,3 +37,8 @@
   <!-- Materials for visualization -->
   <xacro:include filename="$(find tor_description)/urdf/materials.urdf.xacro" />
+  <xacro:include filename="$(find tor_description)/urdf/sensors/imu.urdf.xacro" />
+    <!-- imu -->
+  <xacro:tor_imu name="imu" parent="base_link" update_rate="100.0">
+    <origin xyz="0 0 0" rpy="0 0 0"/>
+  </xacro:tor_imu>
 </robot>

Commit message: Fixed gazebo contact model

File: tor_description/gazebo/gazebo.urdf.xacro (robot description, xacro)
@@ -10,5 +10,5 @@
   </gazebo>
   <gazebo>
-    <plugin filename="libgazebo_world_odometry.so" name="gazebo_ros_force">
+    <plugin filename="libgazebo_world_odometry.so" name="gazebo_ros_odometry">
       <frameName>base_link</frameName>
       <topicName>floating_base_pose</topicName>
@@ -41,5 +41,4 @@
                bias means and stddevs to produce biases close to the provided
                data. -->
-          <!--
           <rate>
             <mean>0.0</mean>
@@ -54,8 +53,8 @@
             <bias_stddev>0.001</bias_stddev>
           </accel>
-          -->
+          <!--
           <rate>
             <mean>0.0</mean>
-            <stddev>2e-3</stddev>
+            <stddev>0.0</stddev>
             <bias_mean>0.000000</bias_mean>
             <bias_stddev>0.0000008</bias_stddev>
@@ -63,8 +62,9 @@
           <accel>
             <mean>0.0</mean>
-            <stddev>1.7e-1</stddev>
+            <stddev>0.0</stddev>
             <bias_mean>0.0</bias_mean>
             <bias_stddev>0.000</bias_stddev>
           </accel>
+          -->
         </noise>
       </imu>

File: tor_description/robots/tor_lower_body.urdf.xacro (robot description, xacro)
@@ -31,4 +31,25 @@
       </collision>
      </link>
+     <!--
+      <link name="base_link">
+      <inertial>
+        <origin xyz="0.0 0.0 0.05" rpy="0 0 0"/>
+        <mass value="5.0" />
+         <inertia ixx="0.01"  ixy="0.0"  ixz="0.0" iyy="0.01" iyz="0.0" izz="0.01" />
+      </inertial>
+      <visual>
+        <origin rpy="0 0 0" xyz="0 0 0"/>
+        <geometry>
+          <mesh filename="package://tor_description/meshes/torso_dummy.stl" scale="1 1 1"/>
+        </geometry>
+      </visual>
+      <collision>
+       <origin rpy="0 0 0" xyz="0 0 0.05"/>
+	    <geometry>
+           <box size="0.1 0.3 0.1"/>
+        </geometry>
+      </collision>
+     </link>
+   -->
    <xacro:tor_leg prefix="left"  reflect="1" />
    <xacro:tor_leg prefix="right" reflect="-1" />
@@ -40,5 +61,5 @@
     <!-- imu -->
   <xacro:tor_imu name="imu" parent="base_link" update_rate="100.0">
-    <origin xyz="0 0 0" rpy="0 0 0"/>
+    <origin xyz="0.069 0 0.14647" rpy="3.14 0.0 1.57"/>
   </xacro:tor_imu>
 </robot>

File: tor_description/urdf/leg/leg.urdf.xacro (robot description, xacro)
@@ -231,5 +231,5 @@
      <mu2>0.9</mu2>
    </gazebo>
-   <!-- contact model for foot surface -->
+   <!--
    <gazebo reference="leg_${prefix}_6_link">
      <kp>1000000.0</kp>
@@ -242,4 +242,14 @@
      <implicitSpringDamper>1</implicitSpringDamper>
    </gazebo>
+   -->
+   <gazebo reference="leg_${prefix}_6_link">
+    <kp>1000000.0</kp>
+    <kd>100.0</kd>
+    <mu1>1.5</mu1>
+    <mu2>1.5</mu2>
+    <fdir1>1 0 0</fdir1>
+    <maxVel>1.0</maxVel>
+    <minDepth>0.00</minDepth>
+   </gazebo>
    <gazebo reference="leg_${prefix}_1_joint">
       <implicitSpringDamper>0.1</implicitSpringDamper>

Commit message: Changed tor v2 leg contact parameters

File: tor_description/gazebo/gazebo.urdf.xacro (robot description, xacro)
@@ -11,5 +11,5 @@
   <gazebo>
     <plugin filename="libgazebo_world_odometry.so" name="gazebo_ros_odometry">
-      <frameName>base_link</frameName>
+      <frameName>torso_2_link</frameName>
       <topicName>floating_base_pose</topicName>
     </plugin>

File: tor_description/urdf/arm/wrist.transmission.xacro (robot description, xacro)
@@ -16,4 +16,5 @@
       <joint name="${name}_${side}_${number}_joint">
         <hardwareInterface>hardware_interface/PositionJointInterface</hardwareInterface>
+        <hardwareInterface>hardware_interface/EffortJointInterface</hardwareInterface>
       </joint>
     </transmission>
@@ -36,4 +37,5 @@
         <mechanicalReduction>${jnt_reduction_1}</mechanicalReduction>
         <hardwareInterface>hardware_interface/PositionJointInterface</hardwareInterface>
+        <hardwareInterface>hardware_interface/EffortJointInterface</hardwareInterface>
       </joint>
       <joint name="${name}_${side}_${number_2}_joint">
@@ -42,4 +44,5 @@
         <mechanicalReduction>${jnt_reduction_2}</mechanicalReduction>
         <hardwareInterface>hardware_interface/PositionJointInterface</hardwareInterface>
+        <hardwareInterface>hardware_interface/EffortJointInterface</hardwareInterface>
       </joint>
     </transmission>

File: tor_description/urdf/leg/leg_v2.urdf.xacro (robot description, xacro)
@@ -190,8 +190,16 @@
         <material name="Grey" />
       </visual>
+      <!--
       <collision>
         <origin xyz="0 0 0" rpy="0 0 0" />
         <geometry>
           <mesh filename="package://tor_description/meshes/v2/ankle_X_collision.stl" scale="1 ${reflect*1} 1"/>
+        </geometry>
+      </collision>
+      -->
+       <collision>
+        <origin xyz="0 0 -0.1" rpy="0 0 0" />
+        <geometry>
+           <box size="0.21 0.13 0.02"/>
         </geometry>
       </collision>
@@ -249,12 +257,11 @@
    <!-- contact model for foot surface -->
    <gazebo reference="leg_${prefix}_6_link">
-     <kp>1000000.0</kp>
-     <kd>100.0</kd>
-     <mu1>1.0</mu1>
-     <mu2>1.0</mu2>
-     <fdir1>0 0 1</fdir1>
-     <maxVel>1.0</maxVel>
-     <minDepth>0.003</minDepth>
-     <implicitSpringDamper>1</implicitSpringDamper>
+    <kp>1000000.0</kp>
+    <kd>100.0</kd>
+    <mu1>1.5</mu1>
+    <mu2>1.5</mu2>
+    <fdir1>1 0 0</fdir1>
+    <maxVel>1.0</maxVel>
+    <minDepth>0.00</minDepth>
    </gazebo>
    <gazebo reference="leg_${prefix}_1_joint">
