Commit message: Add new gripper model

File: talos_description/urdf/gripper/gripper_v2.urdf.xacro (robot description, xacro)
@@ -2,6 +2,6 @@
 <robot xmlns:xacro="http://ros.org/wiki/xacro">
   <!--File includes-->
-  <!-- <xacro:include filename="$(find talos_description)/urdf/deg_to_rad.urdf.xacro" />
-  <xacro:include filename="$(find talos_description)/urdf/gripper.transmission.xacro" />
+  <xacro:include filename="$(find talos_description)/urdf/deg_to_rad.xacro" />
+  <!-- <xacro:include filename="$(find talos_description)/urdf/gripper.transmission.xacro" />
   <xacro:include filename="$(find talos_description)/urdf/gripper.gazebo.xacro" /> -->
   <xacro:macro name="talos_gripper" params="name parent">
@@ -19,4 +19,5 @@
                   <mesh filename="package://talos_description/meshes/gripper/base_link.STL" scale="1 1 1"/>
                 </geometry>
+                <material name="DarkGrey"/>
               </visual>
               <collision>
@@ -34,5 +35,4 @@
               <axis xyz="0 0 0" />
             </joint>
-            <!-- Joint gripper_motor_double (None) : child link -- -> parent link gripper_base_link -->
             <link name="${name}_motor_double_link">
               <inertial>
@@ -48,4 +48,5 @@
                   <mesh filename="package://talos_description/meshes/gripper/gripper_motor_double.STL" scale="1 1 1"/>
                 </geometry>
+              <material name="Orange"/>
               </visual>
               <collision>
@@ -59,9 +60,8 @@
               <parent link="${name}_base_link"/>
               <child link="${name}_motor_double_link"/>
-              <origin xyz="0.00000 0.02025 -0.03000"
-                      rpy="${0.00000 * deg_to_rad} ${0.00000 * deg_to_rad} ${0.00000 * deg_to_rad}"/>
-              <!-- You may want to change axis -->
-              <axis xyz="0 0 1" />
-              <limit lower="${0.00000 * deg_to_rad}" upper="${60.00000 * deg_to_rad}" effort="1.0" velocity="1.0" />
+              <origin xyz="0.0 0.02025 -0.03"
+                      rpy="${0.0 * deg_to_rad} ${0.0 * deg_to_rad} ${0.0 * deg_to_rad}"/>
+              <axis xyz="1 0 0" />
+              <limit lower="${-60.0 * deg_to_rad}" upper="${0.0 * deg_to_rad}" effort="1.0" velocity="1.0" />
               <dynamics friction="1.0" damping="1.0"/>
             </joint>
@@ -79,4 +79,5 @@
                   <mesh filename="package://talos_description/meshes/gripper/inner_double.STL" scale="1 1 1"/>
                 </geometry>
+              <material name="Orange"/>
               </visual>
               <collision>
@@ -92,8 +93,162 @@
               <origin xyz="0.00000 0.00525 -0.05598"
                       rpy="${0.00000 * deg_to_rad} ${0.00000 * deg_to_rad} ${0.00000 * deg_to_rad}"/>
-              <!-- You may want to change axis -->
-              <axis xyz="0 0 1" />
+              <axis xyz="1 0 0" />
               <limit lower="${0.00000 * deg_to_rad}" upper="${0.00000 * deg_to_rad}" effort="1.0" velocity="1.0" />
               <mimic joint="${name}_motor_double_joint" multiplier="${1.0}" offset="0.0" />
+            </joint>
+            <link name="${name}_fingertip_1_link">
+              <inertial>
+                <origin xyz="0.00000 0.00460 -0.00254" rpy="0.00000 0.00000 0.00000"/>
+                <mass value="0.02630"/>
+                <inertia ixx="0.00000800000" ixy="0.00000000000" ixz="0.00000000000"
+                         iyy="0.00000900000" iyz="0.00000100000"
+                         izz="0.00000200000"/>
+              </inertial>
+              <visual>
+                <origin xyz="0 0 0" rpy="0 0 0" />
+                <geometry>
+                  <mesh filename="package://talos_description/meshes/gripper/fingertip.STL" scale="1 1 1"/>
+                </geometry>
+              <material name="DarkGrey"/>
+              </visual>
+              <collision>
+                <origin xyz="0 0 0" rpy="0 0 0" />
+                <geometry>
+                  <mesh filename="package://talos_description/meshes/gripper/fingertip_collision.STL" scale="1 1 1"/>
+                </geometry>
+              </collision>
+            </link>
+            <joint name="fingertip_1_joint" type="revolute">
+              <parent link="${name}_inner_double_link"/>
+              <child link="${name}_fingertip_1_link"/>
+              <origin xyz="0.03200 0.04589 -0.06553"
+                      rpy="${0.00000 * deg_to_rad} ${0.00000 * deg_to_rad} ${0.00000 * deg_to_rad}"/>
+              <axis xyz="1 0 0" />
+              <limit lower="${0.00000 * deg_to_rad}" upper="${0.00000 * deg_to_rad}" effort="1.0" velocity="1.0" />
+              <mimic joint="${name}_motor_double_joint" multiplier="${-1.0}" offset="0.0" />
+            </joint>
+            <link name="${name}_fingertip_2_link">
+              <inertial>
+                <origin xyz="0.00000 0.00460 -0.00254" rpy="0.00000 0.00000 0.00000"/>
+                <mass value="0.02630"/>
+                <inertia ixx="0.00000800000" ixy="0.00000000000" ixz="0.00000000000"
+                         iyy="0.00000900000" iyz="0.00000100000"
+                         izz="0.00000200000"/>
+              </inertial>
+              <visual>
+                <origin xyz="0 0 0" rpy="0 0 0" />
+                <geometry>
+                  <mesh filename="package://talos_description/meshes/gripper/fingertip.STL" scale="1 1 1"/>
+                </geometry>
+                <material name="DarkGrey"/>
+              </visual>
+              <collision>
+                <origin xyz="0 0 0" rpy="0 0 0" />
+                <geometry>
+                  <mesh filename="package://talos_description/meshes/gripper/fingertip_collision.STL" scale="1 1 1"/>
+                </geometry>
+              </collision>
+            </link>
+            <joint name="${name}_fingertip_2_joint" type="revolute">
+              <parent link="${name}_inner_double_link"/>
+              <child link="${name}_fingertip_2_link"/>
+              <origin xyz="-0.03200 0.04589 -0.06553"
+                      rpy="${0.00000 * deg_to_rad} ${0.00000 * deg_to_rad} ${0.00000 * deg_to_rad}"/>
+              <axis xyz="1 0 0" />
+              <limit lower="${0.00000 * deg_to_rad}" upper="${0.00000 * deg_to_rad}" effort="1.0" velocity="1.0" />
+              <mimic joint="${name}_motor_double_joint" multiplier="${-1.0}" offset="0.0" />
+            </joint>
+            <link name="${name}_motor_single_link">
+              <inertial>
+                <origin xyz="0.02589 -0.01284 -0.00640" rpy="0.00000 0.00000 0.00000"/>
+                <mass value="0.14765"/>
+                <inertia ixx="0.00011500000" ixy="0.00005200000" ixz="0.00002500000"
+                         iyy="0.00015300000" iyz="0.00003400000"
+                         izz="0.00019000000"/>
+              </inertial>
+              <visual>
+                <origin xyz="0 0 0" rpy="0 0 0" />
+                <geometry>
+                  <mesh filename="package://talos_description/meshes/gripper/gripper_motor_single.STL" scale="1 1 1"/>
+                </geometry>
+              <material name="Orange"/>
+              </visual>
+              <collision>
+                <origin xyz="0 0 0" rpy="0 0 0" />
+                <geometry>
+                  <mesh filename="package://talos_description/meshes/gripper/gripper_motor_single_collision.STL" scale="1 1 1"/>
+                </geometry>
+              </collision>
+            </link>
+            <joint name="${name}_motor_single_joint" type="revolute">
+              <parent link="${name}_base_link"/>
+              <child link="${name}_motor_single_link"/>
+              <origin xyz="0.00000 -0.02025 -0.03000"
+                      rpy="${0.00000 * deg_to_rad} ${0.00000 * deg_to_rad} ${0.00000 * deg_to_rad}"/>
+              <axis xyz="1 0 0" />
+              <limit lower="${0.00000 * deg_to_rad}" upper="${0.00000 * deg_to_rad}" effort="1.0" velocity="1.0" />
+              <mimic joint="${name}_motor_double_joint" multiplier="${-1.0}" offset="0.0" />
+            </joint>
+          <link name="${name}_inner_single_link">
+              <inertial>
+                <origin xyz="0.00000 -0.03253 -0.01883" rpy="0.00000 0.00000 0.00000"/>
+                <mass value="0.05356"/>
+                <inertia ixx="0.00004700000" ixy="-0.00000000000" ixz="-0.00000000000"
+                         iyy="0.00003500000" iyz="0.00001700000"
+                         izz="0.00002400000"/>
+              </inertial>
+              <visual>
+                <origin xyz="0 0 0" rpy="0 0 0" />
+                <geometry>
+                  <mesh filename="package://talos_description/meshes/gripper/inner_single.STL" scale="1 1 1"/>
+                </geometry>
+              <material name="Orange"/>
+              </visual>
+              <collision>
+                <origin xyz="0 0 0" rpy="0 0 0" />
+                <geometry>
+                  <mesh filename="package://talos_description/meshes/gripper/inner_single_collision.STL" scale="1 1 1"/>
+                </geometry>
+              </collision>
+            </link>
+            <joint name="${name}_inner_single_joint" type="revolute">
+              <parent link="${name}_base_link"/>
+              <child link="${name}_inner_single_link"/>
+              <origin xyz="0.00000 -0.00525 -0.05598"
+                      rpy="${0.00000 * deg_to_rad} ${0.00000 * deg_to_rad} ${0.00000 * deg_to_rad}"/>
+              <axis xyz="1 0 0" />
+              <limit lower="${0.00000 * deg_to_rad}" upper="${0.00000 * deg_to_rad}" effort="1.0" velocity="1.0" />
+              <mimic joint="${name}_motor_double_joint" multiplier="${-1.0}" offset="0.0" />
+            </joint>
+            <link name="${name}_fingertip_3_link">
+              <inertial>
+                <origin xyz="0.00000 0.00460 -0.00254" rpy="0.00000 0.00000 0.00000"/>
+                <mass value="0.02630"/>
+                <inertia ixx="0.00000800000" ixy="0.00000000000" ixz="0.00000000000"
+                         iyy="0.00000900000" iyz="0.00000100000"
+                         izz="0.00000200000"/>
+              </inertial>
+              <visual>
+                <origin xyz="0 0 0" rpy="0 0 0" />
+                <geometry>
+                  <mesh filename="package://talos_description/meshes/gripper/fingertip.STL" scale="1 1 1"/>
+                </geometry>
+              <material name="DarkGrey"/>
+              </visual>
+              <collision>
+                <origin xyz="0 0 0" rpy="0 0 0" />
+                <geometry>
+                  <mesh filename="package://talos_description/meshes/gripper/fingertip_collision.STL" scale="1 1 1"/>
+                </geometry>
+              </collision>
+            </link>
+            <joint name="${name}_fingertip_3_joint" type="revolute">
+              <parent link="${name}_inner_single_link"/>
+              <child link="${name}_fingertip_3_link"/>
+              <origin xyz="0.00000 -0.04589 -0.06553"
+                      rpy="${0.00000 * deg_to_rad} ${0.00000 * deg_to_rad} ${180.00000 * deg_to_rad}"/>
+              <axis xyz="1 0 0" />
+              <limit lower="${0.00000 * deg_to_rad}" upper="${0.00000 * deg_to_rad}" effort="1.0" velocity="1.0" />
+              <mimic joint="${name}_motor_double_joint" multiplier="${-1.0}" offset="0.0" />
             </joint>
  </xacro:macro>

Commit message: Change gripper motor joint to just side_gripper_joint

File: talos_description/urdf/gripper/gripper_v2.urdf.xacro (robot description, xacro)
@@ -3,6 +3,6 @@
   <!--File includes-->
   <xacro:include filename="$(find talos_description)/urdf/deg_to_rad.xacro" />
-  <!-- <xacro:include filename="$(find talos_description)/urdf/gripper.transmission.xacro" />
-  <xacro:include filename="$(find talos_description)/urdf/gripper.gazebo.xacro" /> -->
+  <xacro:include filename="$(find talos_description)/urdf/gripper/gripper.transmission.xacro" />
+  <xacro:include filename="$(find talos_description)/urdf/gripper/gripper.gazebo.xacro" />
   <xacro:macro name="talos_gripper" params="name parent">
            <link name="${name}_base_link">
@@ -39,7 +39,9 @@
                 <origin xyz="0.02270 0.01781 -0.00977" rpy="0.00000 0.00000 0.00000"/>
                 <mass value="0.16889"/>
-                <inertia ixx="0.00015900000" ixy="-0.00007000000" ixz="0.00003800000"
-                         iyy="0.00022100000" iyz="-0.00005300000"
-                         izz="0.00026800000"/>
+                <!-- In order for Gazebo not to explode we needed to add these 0.001 values to the diagonal,
+                also the tool pal_dynamics InertiaMassVisualization gave NaN on the computation of the inertia box -->
+                <inertia ixx="${0.00015900000 + 0.001}" ixy="-0.00007000000" ixz="0.00003800000"
+                         iyy="${0.00022100000 + 0.001}" iyz="-0.00005300000"
+                         izz="${0.00026800000 + 0.001}"/>
               </inertial>
               <visual>
@@ -57,5 +59,5 @@
               </collision>
             </link>
-            <joint name="${name}_motor_double_joint" type="revolute">
+             <joint name="${name}_joint" type="revolute">
               <parent link="${name}_base_link"/>
               <child link="${name}_motor_double_link"/>
@@ -95,5 +97,5 @@
               <axis xyz="1 0 0" />
               <limit lower="${0.00000 * deg_to_rad}" upper="${0.00000 * deg_to_rad}" effort="1.0" velocity="1.0" />
-              <mimic joint="${name}_motor_double_joint" multiplier="${1.0}" offset="0.0" />
+              <mimic joint="${name}_joint" multiplier="${1.0}" offset="0.0" />
             </joint>
             <link name="${name}_fingertip_1_link">
@@ -126,5 +128,5 @@
               <axis xyz="1 0 0" />
               <limit lower="${0.00000 * deg_to_rad}" upper="${0.00000 * deg_to_rad}" effort="1.0" velocity="1.0" />
-              <mimic joint="${name}_motor_double_joint" multiplier="${-1.0}" offset="0.0" />
+              <mimic joint="${name}_joint" multiplier="${-1.0}" offset="0.0" />
             </joint>
             <link name="${name}_fingertip_2_link">
@@ -157,7 +159,7 @@
               <axis xyz="1 0 0" />
               <limit lower="${0.00000 * deg_to_rad}" upper="${0.00000 * deg_to_rad}" effort="1.0" velocity="1.0" />
-              <mimic joint="${name}_motor_double_joint" multiplier="${-1.0}" offset="0.0" />
-            </joint>
-            <link name="${name}_motor_single_link">
+              <mimic joint="${name}_joint" multiplier="${-1.0}" offset="0.0" />
+            </joint>
+             <link name="${name}_motor_single_link">
               <inertial>
                 <origin xyz="0.02589 -0.01284 -0.00640" rpy="0.00000 0.00000 0.00000"/>
@@ -188,5 +190,5 @@
               <axis xyz="1 0 0" />
               <limit lower="${0.00000 * deg_to_rad}" upper="${0.00000 * deg_to_rad}" effort="1.0" velocity="1.0" />
-              <mimic joint="${name}_motor_double_joint" multiplier="${-1.0}" offset="0.0" />
+              <mimic joint="${name}_joint" multiplier="${-1.0}" offset="0.0" />
             </joint>
           <link name="${name}_inner_single_link">
@@ -219,5 +221,5 @@
               <axis xyz="1 0 0" />
               <limit lower="${0.00000 * deg_to_rad}" upper="${0.00000 * deg_to_rad}" effort="1.0" velocity="1.0" />
-              <mimic joint="${name}_motor_double_joint" multiplier="${-1.0}" offset="0.0" />
+              <mimic joint="${name}_joint" multiplier="${-1.0}" offset="0.0" />
             </joint>
             <link name="${name}_fingertip_3_link">
@@ -250,6 +252,8 @@
               <axis xyz="1 0 0" />
               <limit lower="${0.00000 * deg_to_rad}" upper="${0.00000 * deg_to_rad}" effort="1.0" velocity="1.0" />
-              <mimic joint="${name}_motor_double_joint" multiplier="${-1.0}" offset="0.0" />
-            </joint>
+              <mimic joint="${name}_joint" multiplier="${-1.0}" offset="0.0" />
+            </joint>
+        <xacro:finger_mimics name="${name}" />
+        <xacro:gripper_transmission name="${name}" reduction="1.0" />
  </xacro:macro>
 </robot>
