Commit message: Updated dynamic parameters of the grippers.
Note: sensor between the wrist and gripper is split into two links, I
set inertial parameters of the first one, considering the second one
negligible. This must be reviewed.

File: talos_description/urdf/gripper/gripper.urdf.xacro (robot description, xacro)
@@ -8,9 +8,9 @@
            <link name="${name}_base_link">
               <inertial>
-                <origin xyz="-0.00534 0.00362 -0.02357" rpy="0.00000 0.00000 0.00000"/>
-                <mass value="0.61585"/>
-                <inertia ixx="0.00047200000" ixy="-0.00000800000" ixz="0.00003500000"
-                         iyy="0.00052100000" iyz="0.00000000000"
-                         izz="0.00069000000"/>
+                <origin xyz="0.00002800000 0.00539400000 -0.02365400000" rpy="0.00000000000 0.00000000000 0.00000000000"/>
+                <mass value="0.63753400000"/>
+                <inertia ixx="0.00058496920" ixy="0.00000437159" ixz="-0.00001258900"
+                         iyy="0.00067076439" iyz="0.00002824361"
+                         izz="0.00085526645"/>
               </inertial>
               <visual>
@@ -37,11 +37,9 @@
             <link name="${name}_motor_double_link">
               <inertial>
-                <origin xyz="0.02270 0.01781 -0.00977" rpy="0.00000 0.00000 0.00000"/>
-                <mass value="0.16889"/>
-                <!-- In order for Gazebo not to explode we needed to add these 0.001 values to the diagonal,
-                also the tool pal_dynamics InertiaMassVisualization gave NaN on the computation of the inertia box -->
-                <inertia ixx="${0.00015900000 + 0.001}" ixy="-0.00007000000" ixz="0.00003800000"
-                         iyy="${0.00022100000 + 0.001}" iyz="-0.00005300000"
-                         izz="${0.00026800000 + 0.001}"/>
+                <origin xyz="0.01965400000 0.01857200000 -0.01199800000" rpy="0.00000000000 0.00000000000 0.00000000000"/>
+                <mass value="0.13435600000"/>
+                <inertia ixx="0.00013479919" ixy="0.00006184429" ixz="-0.00003079800"
+                         iyy="0.00019602207" iyz="0.00004707722"
+                         izz="0.00024217879"/>
               </inertial>
               <visual>
@@ -59,5 +57,5 @@
               </collision>
             </link>
-             <joint name="${name}_joint" type="revolute">
+            <joint name="${name}_joint" type="revolute">
               <parent link="${name}_base_link"/>
               <child link="${name}_motor_double_link"/>
@@ -70,9 +68,9 @@
             <link name="${name}_inner_double_link">
               <inertial>
-                <origin xyz="-0.00056 0.03358 -0.01741" rpy="0.00000 0.00000 0.00000"/>
-                <mass value="0.11922"/>
-                <inertia ixx="0.00009100000" ixy="0.00000100000" ixz="-0.00000100000"
-                         iyy="0.00015600000" iyz="-0.00003200000"
-                         izz="0.00012600000"/>
+                <origin xyz="-0.01328300000 0.03685200000 -0.02315300000" rpy="0.00000000000 0.00000000000 0.00000000000"/>
+                <mass value="0.08798600000"/>
+                <inertia ixx="0.00007410642" ixy="-0.00000074773" ixz="0.00000101536"
+                         iyy="0.00012794180" iyz="0.00002504083"
+                         izz="0.00010495175"/>
               </inertial>
               <visual>
@@ -101,9 +99,9 @@
             <link name="${name}_fingertip_1_link">
               <inertial>
-                <origin xyz="0.00000 0.00460 -0.00254" rpy="0.00000 0.00000 0.00000"/>
-                <mass value="0.02630"/>
+                <origin xyz="0.00000000000 0.00460400000 -0.00253700000" rpy="0.00000000000 0.00000000000 0.00000000000"/>
+                <mass value="0.02630100000"/>
                 <inertia ixx="0.00000800000" ixy="0.00000000000" ixz="0.00000000000"
-                         iyy="0.00000900000" iyz="0.00000100000"
-                         izz="0.00000200000"/>
+                         iyy="0.00000869179" iyz="-0.00000143612"
+                         izz="0.00000230820"/>
               </inertial>
               <visual>
@@ -129,12 +127,12 @@
               <limit lower="${0.0 * deg_to_rad}" upper="${60.0 * deg_to_rad}" effort="100.0" velocity="1.0" />
               <mimic joint="${name}_joint" multiplier="${-1.0}" offset="0.0" />
-           </joint>
+            </joint>
             <link name="${name}_fingertip_2_link">
               <inertial>
-                <origin xyz="0.00000 0.00460 -0.00254" rpy="0.00000 0.00000 0.00000"/>
-                <mass value="0.02630"/>
+                <origin xyz="0.00000000000 0.00460400000 -0.00253700000" rpy="0.00000000000 0.00000000000 0.00000000000"/>
+                <mass value="0.02630100000"/>
                 <inertia ixx="0.00000800000" ixy="0.00000000000" ixz="0.00000000000"
-                         iyy="0.00000900000" iyz="0.00000100000"
-                         izz="0.00000200000"/>
+                         iyy="0.00000869179" iyz="-0.00000143612"
+                         izz="0.00000230820"/>
               </inertial>
               <visual>
@@ -160,12 +158,12 @@
               <limit lower="${0.0 * deg_to_rad}" upper="${60.0 * deg_to_rad}" effort="100.0" velocity="1.0" />
               <mimic joint="${name}_joint" multiplier="${-1.0}" offset="0.0" />
-           </joint>
+            </joint>
             <link name="${name}_motor_single_link">
               <inertial>
-                <origin xyz="0.02589 -0.01284 -0.00640" rpy="0.00000 0.00000 0.00000"/>
-                <mass value="0.14765"/>
-                <inertia ixx="0.00011500000" ixy="0.00005200000" ixz="0.00002500000"
-                         iyy="0.00015300000" iyz="0.00003400000"
-                         izz="0.00019000000"/>
+                <origin xyz="0.02523700000 -0.01123100000 -0.00815800000" rpy="0.00000000000 0.00000000000 0.00000000000"/>
+                <mass value="0.10792300000"/>
+                <inertia ixx="0.00008973662" ixy="-0.00004082027" ixz="-0.00001927099"
+                         iyy="0.00011957255" iyz="-0.00002873284"
+                         izz="0.00015469079"/>
               </inertial>
               <visual>
@@ -191,12 +189,12 @@
               <limit lower="${0.0 * deg_to_rad}" upper="${60.0 * deg_to_rad}" effort="100.0" velocity="1.0" />
               <mimic joint="${name}_joint" multiplier="${-1.0}" offset="0.0" />
-           </joint>
+            </joint>
             <link name="${name}_inner_single_link">
               <inertial>
-                <origin xyz="0.00000 -0.03253 -0.01883" rpy="0.00000 0.00000 0.00000"/>
-                <mass value="0.05356"/>
-                <inertia ixx="0.00004700000" ixy="-0.00000000000" ixz="-0.00000000000"
-                         iyy="0.00003500000" iyz="0.00001700000"
-                         izz="0.00002400000"/>
+                <origin xyz="0.00000000000 -0.03456500000 -0.02141200000" rpy="0.00000000000 0.00000000000 0.00000000000"/>
+                <mass value="0.04717700000"/>
+                <inertia ixx="0.00004199818" ixy="0.00000013418" ixz="0.00000019358"
+                         iyy="0.00003231338" iyz="-0.00001509136"
+                         izz="0.00002168842"/>
               </inertial>
               <visual>
@@ -222,12 +220,12 @@
               <limit lower="${0.0 * deg_to_rad}" upper="${60.0 * deg_to_rad}" effort="100.0" velocity="1.0" />
               <mimic joint="${name}_joint" multiplier="${-1.0}" offset="0.0" />
-           </joint>
+            </joint>
             <link name="${name}_fingertip_3_link">
               <inertial>
-                <origin xyz="0.00000 0.00460 -0.00254" rpy="0.00000 0.00000 0.00000"/>
-                <mass value="0.02630"/>
+                <origin xyz="0.00000000000 0.00460400000 -0.00253700000" rpy="0.00000000000 0.00000000000 0.00000000000"/>
+                <mass value="0.02630100000"/>
                 <inertia ixx="0.00000800000" ixy="0.00000000000" ixz="0.00000000000"
-                         iyy="0.00000900000" iyz="0.00000100000"
-                         izz="0.00000200000"/>
+                         iyy="0.00000869179" iyz="-0.00000143612"
+                         izz="0.00000230820"/>
               </inertial>
               <visual>
@@ -253,5 +251,5 @@
               <limit lower="${0.0 * deg_to_rad}" upper="${60.0 * deg_to_rad}" effort="100.0" velocity="1.0" />
               <mimic joint="${name}_joint" multiplier="${-1.0}" offset="0.0" />
-           </joint>
+            </joint>
         <xacro:virtual_joints name="${name}" />
         <xacro:gripper_transmission name="${name}" reduction="1.0" />

File: talos_description/urdf/sensors/ftsensor.urdf.xacro (robot description, xacro)
@@ -14,6 +14,9 @@
     <link name="${name}_${side}_ft_link">
       <inertial>
-        <mass value="0.1" />
-        <inertia ixx="0.0" ixy="0.0" ixz="0.0" iyy="0.0" iyz="0.0" izz="0.0" />
+        <mass value="0.09500000000" />
+        <inertia ixx="0.00001108502" ixy="0.00000099077" ixz="-0.00000023811"
+                 iyy="0.00001092725" iyz="0.00000023137"
+                 izz="0.00001898772"/>
+        <origin xyz="-0.00100100000 0.00099500000 -0.00810800000" rpy="0.00000000000 0.00000000000 0.00000000000"/>
       </inertial>
       <visual>
@@ -41,5 +44,5 @@
     <link name="${name}_${side}_ft_tool_link">
       <inertial>
-        <mass value="0.1" />
+        <mass value="0.001" />
         <inertia ixx="0.0" ixy="0.0" ixz="0.0" iyy="0.0" iyz="0.0" izz="0.0" />
       </inertial>

Commit message: Add visual offset of 7mm to the meshes

File: talos_description/urdf/gripper/gripper.urdf.xacro (robot description, xacro)
@@ -6,8 +6,9 @@
   <xacro:include filename="$(find talos_description)/urdf/gripper/gripper.gazebo.xacro" />
   <xacro:macro name="talos_gripper" params="name parent reflect">
+            <xacro:property name="gripper_visual_offset_y"       value="0.007" />
             <link name="${name}_base_link">
               <xacro:call macro="${name}_base_link_inertial" />
               <visual>
-                <origin xyz="0 0 0" rpy="0 0 0" />
+                <origin xyz="0 ${gripper_visual_offset_y} 0" rpy="0 0 0" />
                 <geometry>
                   <mesh filename="package://talos_description/meshes/gripper/base_link.STL" scale="1 1 1"/>
@@ -16,5 +17,5 @@
               </visual>
               <collision>
-                <origin xyz="0 0 0" rpy="0 0 0" />
+                <origin xyz="0 ${gripper_visual_offset_y} 0" rpy="0 0 0" />
                 <geometry>
                   <mesh filename="package://talos_description/meshes/gripper/base_link_collision.STL" scale="1 1 1"/>
@@ -25,5 +26,5 @@
               <parent link="${parent}"/>
               <child link="${name}_base_link"/>
-              <origin xyz="0.00000 0.00000 -0.02875"
+              <origin xyz="0.00000 0.0 -0.02875"
                       rpy="${0.00000 * deg_to_rad} ${0.00000 * deg_to_rad} ${0.00000 * deg_to_rad}"/>
               <axis xyz="0 0 0" />
@@ -32,5 +33,5 @@
               <xacro:call macro="${name}_motor_double_link_inertial" />
               <visual>
-                <origin xyz="0 0 0" rpy="0 0 0" />
+                <origin xyz="0 ${gripper_visual_offset_y} 0" rpy="0 0 0" />
                 <geometry>
                   <mesh filename="package://talos_description/meshes/gripper/gripper_motor_double.STL" scale="1 1 1"/>
@@ -39,5 +40,5 @@
               </visual>
               <collision>
-                <origin xyz="0 0 0" rpy="0 0 0" />
+                <origin xyz="0 ${gripper_visual_offset_y} 0" rpy="0 0 0" />
                 <geometry>
                   <mesh filename="package://talos_description/meshes/gripper/gripper_motor_double_collision.STL" scale="1 1 1"/>
@@ -57,5 +58,5 @@
               <xacro:call macro="${name}_inner_double_link_inertial" />
               <visual>
-                <origin xyz="0 0 0" rpy="0 0 0" />
+                <origin xyz="0 ${gripper_visual_offset_y} 0" rpy="0 0 0" />
                 <geometry>
                   <mesh filename="package://talos_description/meshes/gripper/inner_double.STL" scale="1 1 1"/>
@@ -64,5 +65,5 @@
               </visual>
               <collision>
-                <origin xyz="0 0 0" rpy="0 0 0" />
+                <origin xyz="0 ${gripper_visual_offset_y} 0" rpy="0 0 0" />
                 <geometry>
                   <mesh filename="package://talos_description/meshes/gripper/inner_double_collision.STL" scale="1 1 1"/>
@@ -82,5 +83,5 @@
               <xacro:call macro="${name}_fingertip_1_link_inertial" />
               <visual>
-                <origin xyz="0 0 0" rpy="0 0 0" />
+                <origin xyz="0 ${gripper_visual_offset_y} 0" rpy="0 0 0" />
                 <geometry>
                   <mesh filename="package://talos_description/meshes/gripper/fingertip.STL" scale="1 1 1"/>
@@ -89,5 +90,5 @@
               </visual>
               <collision>
-                <origin xyz="0 0 0" rpy="0 0 0" />
+                <origin xyz="0 ${gripper_visual_offset_y} 0" rpy="0 0 0" />
                 <geometry>
                   <mesh filename="package://talos_description/meshes/gripper/fingertip_collision.STL" scale="1 1 1"/>
@@ -107,5 +108,5 @@
               <xacro:call macro="${name}_fingertip_2_link_inertial" />
               <visual>
-                <origin xyz="0 0 0" rpy="0 0 0" />
+                <origin xyz="0 ${gripper_visual_offset_y} 0" rpy="0 0 0" />
                 <geometry>
                   <mesh filename="package://talos_description/meshes/gripper/fingertip.STL" scale="1 1 1"/>
@@ -114,5 +115,5 @@
               </visual>
               <collision>
-                <origin xyz="0 0 0" rpy="0 0 0" />
+                <origin xyz="0 ${gripper_visual_offset_y} 0" rpy="0 0 0" />
                 <geometry>
                   <mesh filename="package://talos_description/meshes/gripper/fingertip_collision.STL" scale="1 1 1"/>
@@ -132,5 +133,5 @@
               <xacro:call macro="${name}_motor_single_link_inertial" />
               <visual>
-                <origin xyz="0 0 0" rpy="0 0 0" />
+                <origin xyz="0 ${gripper_visual_offset_y} 0" rpy="0 0 0" />
                 <geometry>
                   <mesh filename="package://talos_description/meshes/gripper/gripper_motor_single.STL" scale="1 1 1"/>
@@ -139,5 +140,5 @@
               </visual>
               <collision>
-                <origin xyz="0 0 0" rpy="0 0 0" />
+                <origin xyz="0 ${gripper_visual_offset_y} 0" rpy="0 0 0" />
                 <geometry>
                   <mesh filename="package://talos_description/meshes/gripper/gripper_motor_single_collision.STL" scale="1 1 1"/>
@@ -157,5 +158,5 @@
               <xacro:call macro="${name}_inner_single_link_inertial" />
               <visual>
-                <origin xyz="0 0 0" rpy="0 0 0" />
+                <origin xyz="0 ${gripper_visual_offset_y} 0" rpy="0 0 0" />
                 <geometry>
                   <mesh filename="package://talos_description/meshes/gripper/inner_single.STL" scale="1 1 1"/>
@@ -164,5 +165,5 @@
               </visual>
               <collision>
-                <origin xyz="0 0 0" rpy="0 0 0" />
+                <origin xyz="0 ${gripper_visual_offset_y} 0" rpy="0 0 0" />
                 <geometry>
                   <mesh filename="package://talos_description/meshes/gripper/inner_single_collision.STL" scale="1 1 1"/>
@@ -182,5 +183,5 @@
               <xacro:call macro="${name}_fingertip_3_link_inertial" />
               <visual>
-                <origin xyz="0 0 0" rpy="0 0 0" />
+                <origin xyz="0 ${gripper_visual_offset_y} 0" rpy="0 0 0" />
                 <geometry>
                   <mesh filename="package://talos_description/meshes/gripper/fingertip.STL" scale="1 1 1"/>
@@ -189,5 +190,5 @@
               </visual>
               <collision>
-                <origin xyz="0 0 0" rpy="0 0 0" />
+                <origin xyz="0 ${gripper_visual_offset_y} 0" rpy="0 0 0" />
                 <geometry>
                   <mesh filename="package://talos_description/meshes/gripper/fingertip_collision.STL" scale="1 1 1"/>

Commit message: update new detachable gripper link information

File: talos_description/urdf/gripper/gripper.urdf.xacro (robot description, xacro)
@@ -6,5 +6,5 @@
   <xacro:include filename="$(find talos_description)/urdf/gripper/gripper.gazebo.xacro" />
   <xacro:macro name="talos_gripper" params="name parent reflect">
-            <xacro:property name="gripper_visual_offset_y"       value="0.007" />
+            <xacro:property name="gripper_visual_offset_y"       value="0.00" />
             <link name="${name}_base_link">
               <xacro:call macro="${name}_base_link_inertial" />

File: talos_description_inertial/urdf/inertial.xacro (robot description, xacro)
@@ -60,7 +60,7 @@
     <xacro:if value="${gripper_type == 'detachable'}">
       <inertial>
-        <origin xyz="-0.002117 -0.000722 -0.066129" rpy="0 0 0" />
-        <mass value="0.656327" />
-        <inertia ixx="0.003723" ixy="-0.000004" ixz="0.000111" iyy="0.003611" iyz="-0.000049" izz="0.000536" />
+        <origin xyz="0.0020157 -0.00071287 -0.064959" rpy="0 0 0" />
+        <mass value="0.58111" />
+        <inertia ixx="0.00034987" ixy="-4.826E-06" ixz="6.9606E-06" iyy="0.00027237" iyz="-5.6115E-06" izz="0.00034699" />
       </inertial>
     </xacro:if>
@@ -118,7 +118,7 @@
     <xacro:if value="${gripper_type == 'detachable'}">
       <inertial>
-        <origin xyz="-0.002117 0.000722 -0.066129" rpy="0 0 0" />
-        <mass value="0.656327" />
-        <inertia ixx="0.003723" ixy="0.000004" ixz="0.000111" iyy="0.003611" iyz="0.000049" izz="0.000536" />
+        <origin xyz="0.0020157 0.00071287 -0.064959" rpy="0 0 0" />
+        <mass value="0.58111" />
+        <inertia ixx="0.00034987" ixy="4.826E-06" ixz="6.9606E-06" iyy="0.00027237" iyz="5.6115E-06" izz="0.00034699" />
       </inertial>
     </xacro:if>
