Commit message: Remove gripper_visual_offset_y fix to meshes as fixed with new 180º rotated meshes

File: talos_description/urdf/gripper/gripper.urdf.xacro (robot description, xacro)
@@ -6,9 +6,8 @@
   <xacro:include filename="$(find talos_description)/urdf/gripper/gripper.gazebo.xacro" />
   <xacro:macro name="talos_gripper" params="name parent reflect">
-            <xacro:property name="gripper_visual_offset_y"       value="0.00" />
             <link name="${name}_base_link">
               <xacro:call macro="${name}_base_link_inertial" />
               <visual>
-                <origin xyz="0 ${gripper_visual_offset_y} 0" rpy="0 0 0" />
+                <origin xyz="0 0 0" rpy="0 0 0" />
                 <geometry>
                   <mesh filename="package://talos_description/meshes/gripper/base_link.STL" scale="1 1 1"/>
@@ -17,5 +16,5 @@
               </visual>
               <collision>
-                <origin xyz="0 ${gripper_visual_offset_y} 0" rpy="0 0 0" />
+                <origin xyz="0 0 0" rpy="0 0 0" />
                 <geometry>
                   <mesh filename="package://talos_description/meshes/gripper/base_link_collision.STL" scale="1 1 1"/>
@@ -33,5 +32,5 @@
               <xacro:call macro="${name}_motor_double_link_inertial" />
               <visual>
-                <origin xyz="0 ${gripper_visual_offset_y} 0" rpy="0 0 0" />
+                <origin xyz="0 0 0" rpy="0 0 0" />
                 <geometry>
                   <mesh filename="package://talos_description/meshes/gripper/gripper_motor_double.STL" scale="1 1 1"/>
@@ -40,5 +39,5 @@
               </visual>
               <collision>
-                <origin xyz="0 ${gripper_visual_offset_y} 0" rpy="0 0 0" />
+                <origin xyz="0 0 0" rpy="0 0 0" />
                 <geometry>
                   <mesh filename="package://talos_description/meshes/gripper/gripper_motor_double_collision.STL" scale="1 1 1"/>
@@ -58,5 +57,5 @@
               <xacro:call macro="${name}_inner_double_link_inertial" />
               <visual>
-                <origin xyz="0 ${gripper_visual_offset_y} 0" rpy="0 0 0" />
+                <origin xyz="0 0 0" rpy="0 0 0" />
                 <geometry>
                   <mesh filename="package://talos_description/meshes/gripper/inner_double.STL" scale="1 1 1"/>
@@ -65,5 +64,5 @@
               </visual>
               <collision>
-                <origin xyz="0 ${gripper_visual_offset_y} 0" rpy="0 0 0" />
+                <origin xyz="0 0 0" rpy="0 0 0" />
                 <geometry>
                   <mesh filename="package://talos_description/meshes/gripper/inner_double_collision.STL" scale="1 1 1"/>
@@ -83,5 +82,5 @@
               <xacro:call macro="${name}_fingertip_1_link_inertial" />
               <visual>
-                <origin xyz="0 ${gripper_visual_offset_y} 0" rpy="0 0 0" />
+                <origin xyz="0 0 0" rpy="0 0 0" />
                 <geometry>
                   <mesh filename="package://talos_description/meshes/gripper/fingertip.STL" scale="1 1 1"/>
@@ -90,5 +89,5 @@
               </visual>
               <collision>
-                <origin xyz="0 ${gripper_visual_offset_y} 0" rpy="0 0 0" />
+                <origin xyz="0 0 0" rpy="0 0 0" />
                 <geometry>
                   <mesh filename="package://talos_description/meshes/gripper/fingertip_collision.STL" scale="1 1 1"/>
@@ -108,5 +107,5 @@
               <xacro:call macro="${name}_fingertip_2_link_inertial" />
               <visual>
-                <origin xyz="0 ${gripper_visual_offset_y} 0" rpy="0 0 0" />
+                <origin xyz="0 0 0" rpy="0 0 0" />
                 <geometry>
                   <mesh filename="package://talos_description/meshes/gripper/fingertip.STL" scale="1 1 1"/>
@@ -115,5 +114,5 @@
               </visual>
               <collision>
-                <origin xyz="0 ${gripper_visual_offset_y} 0" rpy="0 0 0" />
+                <origin xyz="0 0 0" rpy="0 0 0" />
                 <geometry>
                   <mesh filename="package://talos_description/meshes/gripper/fingertip_collision.STL" scale="1 1 1"/>
@@ -133,5 +132,5 @@
               <xacro:call macro="${name}_motor_single_link_inertial" />
               <visual>
-                <origin xyz="0 ${gripper_visual_offset_y} 0" rpy="0 0 0" />
+                <origin xyz="0 0 0" rpy="0 0 0" />
                 <geometry>
                   <mesh filename="package://talos_description/meshes/gripper/gripper_motor_single.STL" scale="1 1 1"/>
@@ -140,5 +139,5 @@
               </visual>
               <collision>
-                <origin xyz="0 ${gripper_visual_offset_y} 0" rpy="0 0 0" />
+                <origin xyz="0 0 0" rpy="0 0 0" />
                 <geometry>
                   <mesh filename="package://talos_description/meshes/gripper/gripper_motor_single_collision.STL" scale="1 1 1"/>
@@ -158,5 +157,5 @@
               <xacro:call macro="${name}_inner_single_link_inertial" />
               <visual>
-                <origin xyz="0 ${gripper_visual_offset_y} 0" rpy="0 0 0" />
+                <origin xyz="0 0 0" rpy="0 0 0" />
                 <geometry>
                   <mesh filename="package://talos_description/meshes/gripper/inner_single.STL" scale="1 1 1"/>
@@ -165,5 +164,5 @@
               </visual>
               <collision>
-                <origin xyz="0 ${gripper_visual_offset_y} 0" rpy="0 0 0" />
+                <origin xyz="0 0 0" rpy="0 0 0" />
                 <geometry>
                   <mesh filename="package://talos_description/meshes/gripper/inner_single_collision.STL" scale="1 1 1"/>
@@ -183,5 +182,5 @@
               <xacro:call macro="${name}_fingertip_3_link_inertial" />
               <visual>
-                <origin xyz="0 ${gripper_visual_offset_y} 0" rpy="0 0 0" />
+                <origin xyz="0 0 0" rpy="0 0 0" />
                 <geometry>
                   <mesh filename="package://talos_description/meshes/gripper/fingertip.STL" scale="1 1 1"/>
@@ -190,5 +189,5 @@
               </visual>
               <collision>
-                <origin xyz="0 ${gripper_visual_offset_y} 0" rpy="0 0 0" />
+                <origin xyz="0 0 0" rpy="0 0 0" />
                 <geometry>
                   <mesh filename="package://talos_description/meshes/gripper/fingertip_collision.STL" scale="1 1 1"/>

Commit message: change the camera orientation to have the USB ports exterior

File: talos_description/urdf/gripper/gripper.urdf.xacro (robot description, xacro)
@@ -31,5 +31,5 @@
               </link>
               <joint name="support_${name}_${side}_wrist_camera_joint" type="fixed">
-                <origin xyz="0.11239 0 -0.12048" rpy="-3.1415925371051 1.0472025163988 -3.14159251909337" />
+                <origin xyz="0.11239 0 -0.12048" rpy="${-180.0 * deg_to_rad} ${60.0 * deg_to_rad} ${-180.0 * deg_to_rad}" />
                 <parent link="arm_${side}_7_link"/>
                 <child link="support_${name}_${side}_camera_link" />
@@ -42,7 +42,12 @@
                 use_nominal_extrinsics="${simulation}"
                 disable_gazebo_camera="${disable_gazebo_camera}">
-                <origin
-                  xyz="0.0 0.0 0.0"
-                  rpy="0.0 0.0 0.0"/>
+                <xacro:if value="${reflect == 1}">
+                  <origin xyz="0.0 0.0 0.0" rpy="0.0 0.0 0.0"/>
+                </xacro:if>
+                <xacro:if value="${reflect == -1}">
+                  <!-- there is a difference of 0.042 m due to the fact that the screw hole is on different direction
+                  the screw hole to the center of camera is 0.021 m  -->
+                  <origin xyz="0.0 0.0 0.042" rpy="${180.0 * deg_to_rad} 0.0 0.0"/>
+                </xacro:if>
               </xacro:sensor_d405>
             </xacro:if>

File: talos_description/urdf/leg/leg.urdf.xacro (robot description, xacro)
@@ -241,6 +241,12 @@
         <parent link="leg_${prefix}_6_link"/>
         <child link="support_front_${prefix}_camera_link"/>
-        <origin xyz="0.1125 0 -0.064"
-                rpy="0.0 0.0 0.0"/>
+        <xacro:if value="${reflect == 1}">
+          <!-- there is a difference of 0.025 m due to the fact that the screw hole is on different direction
+          the screw hole to the center of camera is 0.0125 m  -->
+          <origin xyz="0.1125 0.0 -0.039" rpy="${180.0 * deg_to_rad} 0.0 0.0"/>
+        </xacro:if>
+        <xacro:if value="${reflect == -1}">
+          <origin xyz="0.1125 0.0 -0.064" rpy="0.0 0.0 0.0"/>
+        </xacro:if>
         <axis xyz="1 0 0" />
       </joint>
@@ -251,6 +257,12 @@
         <parent link="leg_${prefix}_6_link"/>
         <child link="support_rear_${prefix}_camera_link"/>
-        <origin xyz="-0.1313 0 -0.064"
-                rpy="0.0 0.0 3.14"/>
+        <xacro:if value="${reflect == 1}">
+          <origin xyz="-0.1313 0 -0.064" rpy="0.0 0.0 ${180.0 * deg_to_rad}"/>
+        </xacro:if>
+        <xacro:if value="${reflect == -1}">
+          <!-- there is a difference of 0.025 m due to the fact that the screw hole is on different direction
+          the screw hole to the center of camera is 0.0125 m  -->
+          <origin xyz="-0.1313 0 -0.039" rpy="${180.0 * deg_to_rad} 0.0 ${180.0 * deg_to_rad}"/>
+        </xacro:if>
         <axis xyz="1 0 0" />
       </joint>
