Commit message: Finished renaming

File: talos_description/gazebo/gazebo.urdf.xacro (robot description, xacro)
@@ -1,4 +1,4 @@
 <?xml version="1.0"?>
-<robot name="starleth">
+<robot name="talos">
   <gazebo>
     <plugin filename="libgazebo_ros_control.so" name="gazebo_ros_control">
@@ -11,5 +11,5 @@
   <gazebo>
     <plugin filename="libgazebo_world_odometry.so" name="gazebo_ros_odometry">
-      <frameName>talos_2_link</frameName>
+      <frameName>torso_2_link</frameName>
       <topicName>floating_base_pose</topicName>
     </plugin>
@@ -72,4 +72,4 @@
   </gazebo>
   <!-- define global properties -->
-  <property name="M_PI" value="3.1415926535897931" />
+  <!-- <xacro:property name="M_PI" value="3.1415926535897931" /> -->
 </robot>

File: talos_description/robots/talos_full.urdf.xacro (robot description, xacro)
@@ -17,5 +17,5 @@
   <xacro:include filename="$(find talos_description)/urdf/gripper/gripper.urdf.xacro" />
   <xacro:include filename="$(find talos_description)/urdf/leg/leg_v2.urdf.xacro" />
-  <xacro:talos_talos name="talos" />
+  <xacro:talos_torso name="torso" />
   <xacro:talos_head name="head" parent="torso_2_link"/>
   <xacro:talos_arm name="arm" parent="torso_2_link" side="left" reflect="1"/>

File: talos_description/robots/talos_torso.urdf.xacro (robot description, xacro)
@@ -11,6 +11,6 @@
         xmlns:controller="http://playerstage.sourceforge.net/gazebo/xmlschema/#controller"
         xmlns:interface="http://playerstage.sourceforge.net/gazebo/xmlschema/#interface">
-  <xacro:include filename="$(find talos_description)/urdf/talos/talos.urdf.xacro" />
-  <xacro:talos_talos name="talos" />
+  <xacro:include filename="$(find talos_description)/urdf/torso/torso.urdf.xacro" />
+  <xacro:talos_torso name="torso" />
   <!-- Generic simulatalos_gazebo plugins -->
   <xacro:include filename="$(find talos_description)/gazebo/gazebo.urdf.xacro" />

File: talos_description/urdf/deg_to_rad.xacro (robot description, xacro)
@@ -1,3 +1,3 @@
 <robot xmlns:xacro="http://ros.org/wiki/xacro">
-    <property name="deg_to_rad" value="0.01745329251994329577" />
+    <xacro:property name="deg_to_rad" value="0.01745329251994329577" />
 </robot>

File: talos_description/urdf/sensors/back_camera.urdf.xacro (robot description, xacro)
@@ -14,5 +14,5 @@
   <xacro:macro name="reemc_back_camera" params="name parent focal_length hfov image_format image_width image_height *origin">
     <joint name="${name}_frame_joint" type="fixed">
-      <insert_block name="origin" />
+      <xacro:insert_block name="origin" />
       <parent link="${parent}"/>
       <child link="${name}_link"/>

File: talos_description/urdf/sensors/calibration.xacro (robot description, xacro)
@@ -9,14 +9,14 @@
 -->
 <robot>
-  <property name="M_PI" value="3.1415926535897931" />
+  <xacro:property name="M_PI" value="3.1415926535897931" />
   <!-- Head-mounted ASUS Xtion Pro Live -->
   <!-- These calibration values affect 2 frames:
          (name)_xtion_ir_optical_frame
          (name)_xtion_rgb_optical_frame              -->
-  <property name="cal_head_mount_xtion_x"     value="0.0" />
-  <property name="cal_head_mount_xtion_y"     value="0.0" />
-  <property name="cal_head_mount_xtion_z"     value="0.0" />
-  <property name="cal_head_mount_xtion_roll"  value="0.0" />
-  <property name="cal_head_mount_xtion_pitch" value="0.0" />
-  <property name="cal_head_mount_xtion_yaw"   value="0.0" />
+  <xacro:property name="cal_head_mount_xtion_x"     value="0.0" />
+  <xacro:property name="cal_head_mount_xtion_y"     value="0.0" />
+  <xacro:property name="cal_head_mount_xtion_z"     value="0.0" />
+  <xacro:property name="cal_head_mount_xtion_roll"  value="0.0" />
+  <xacro:property name="cal_head_mount_xtion_pitch" value="0.0" />
+  <xacro:property name="cal_head_mount_xtion_yaw"   value="0.0" />
 </robot>

File: talos_description/urdf/sensors/imu.urdf.xacro (robot description, xacro)
@@ -23,5 +23,5 @@
     </link>
     <joint name="imu_joint" type="fixed">
-      <insert_block name="origin"/>
+      <xacro:insert_block name="origin"/>
       <parent link="${parent}"/>
       <child link="${name}_link"/>

File: talos_description/urdf/sensors/laser.urdf.xacro (robot description, xacro)
@@ -27,5 +27,5 @@
     <joint name="${name}_joint" type="fixed">
       <axis xyz="0 1 0" />
-      <insert_block name="origin" />
+      <xacro:insert_block name="origin" />
       <parent link="${parent}"/>
       <child link="${name}_link"/>

File: talos_description/urdf/sensors/mvbluefox_camera.urdf.xacro (robot description, xacro)
@@ -11,5 +11,5 @@
   <xacro:macro name="mvbluefox_camera" params="name parent *origin">
     <joint name="${name}_frame_joint" type="fixed">
-      <insert_block name="origin" />
+      <xacro:insert_block name="origin" />
       <parent link="${parent}"/>
       <child link="${name}_link"/>

File: talos_description/urdf/sensors/orbbec_astra_pro.urdf.xacro (robot description, xacro)
@@ -23,5 +23,5 @@
     <!-- frames in the center of the camera -->
     <joint name="${name}_joint" type="fixed">
-      <insert_block name="origin"/>
+      <xacro:insert_block name="origin"/>
       <axis xyz="0 0 1"/>
       <!-- <limit lower="0" upper="0.001" effort="100" velocity="0.01"/> -->
@@ -55,5 +55,5 @@
     </link>
     <joint name="${name}_optical_joint" type="fixed">
-      <insert_block name="optical_origin" />
+      <xacro:insert_block name="optical_origin" />
       <parent link="${name}_link"/>
       <child link="${name}_optical_frame"/>

File: talos_description/urdf/sensors/prosilicaGC655C_camera.urdf.xacro (robot description, xacro)
@@ -11,5 +11,5 @@
   <xacro:macro name="prosilicaGC655C_camera" params="name parent *origin">
     <joint name="${name}_frame_joint" type="fixed">
-      <insert_block name="origin" />
+      <xacro:insert_block name="origin" />
       <parent link="${parent}"/>
       <child link="${name}_link"/>

File: talos_description/urdf/sensors/range.urdf.xacro (robot description, xacro)
@@ -18,5 +18,5 @@
     </link>
     <joint name="${name}_joint" type="fixed">
-      <insert_block name="origin" />
+      <xacro:insert_block name="origin" />
       <axis xyz="0 0 1"/>
       <parent link="${parent}_link"/>

File: talos_description/urdf/sensors/stereo_camera.urdf.xacro (robot description, xacro)
@@ -10,14 +10,14 @@
   <xacro:include filename="$(find reemc_description)/urdf/sensors/prosilica_stereo_camera.gazebo.xacro" />
   <xacro:include filename="$(find reemc_description)/urdf/sensors/prosilicaGC655C_camera.urdf.xacro" />
-  <property name="stereo_dx" value="0.00" />
-  <property name="stereo_dy" value="-0.073" /> <!-- stereo baseline according to base_link which has X pointing forward, Y leftwards and Z upwards (required by Gazebo for a camera sensor) -->
-  <property name="stereo_dz" value="0.00" />
-  <property name="stereo_rx" value="0.00" />
-  <property name="stereo_ry" value="0.00" />
-  <property name="stereo_rz" value="0.00" />
+  <xacro:property name="stereo_dx" value="0.00" />
+  <xacro:property name="stereo_dy" value="-0.073" /> <!-- stereo baseline according to base_link which has X pointing forward, Y leftwards and Z upwards (required by Gazebo for a camera sensor) -->
+  <xacro:property name="stereo_dz" value="0.00" />
+  <xacro:property name="stereo_rx" value="0.00" />
+  <xacro:property name="stereo_ry" value="0.00" />
+  <xacro:property name="stereo_rz" value="0.00" />
   <!-- this macro is used for creating wide and narrow double stereo camera links -->
   <xacro:macro name="reemc_stereo_camera" params="name parent focal_length hfov image_format image_width image_height *origin">
     <joint name="${name}_frame_joint" type="fixed">
-      <insert_block name="origin" />
+      <xacro:insert_block name="origin" />
       <parent link="${parent}"/>
       <child link="${name}_link"/>

File: talos_description/urdf/sensors/xtion_pro_live.urdf.xacro (robot description, xacro)
@@ -20,10 +20,10 @@
   <xacro:include filename="$(find reemc)/urdf/sensors/calibration.xacro" />
   <xacro:include filename="$(find reemc)/urdf/sensors/openni.gazebo.xacro" />
-  <property name="M_PI" value="3.1415926535897931" />
+  <xacro:property name="M_PI" value="3.1415926535897931" />
   <!-- Macro -->
   <xacro:macro name="xtion_pro_live" params="name parent *origin *calibration_origin">
     <!-- base link -->
     <joint name="${name}_joint" type="fixed">
-      <insert_block name="origin" />
+      <xacro:insert_block name="origin" />
       <parent link="${parent}"/>
       <child link="${name}_link"/>
@@ -73,5 +73,5 @@
     <!-- Xtion IR sensor frame -->
     <joint name="${name}_ir_optical_frame_joint" type="fixed">
-      <insert_block name="calibration_origin" /> <!-- macro argument -->
+      <xacro:insert_block name="calibration_origin" /> <!-- macro argument -->
       <parent link="${name}_ir_link"/>
       <child link="${name}_ir_optical_frame"/>
@@ -107,5 +107,5 @@
     <!-- Xtion RGB sensor frame -->
     <joint name="${name}_rgb_optical_frame_joint" type="fixed">
-      <insert_block name="calibration_origin" /> <!-- macro argument -->
+      <xacro:insert_block name="calibration_origin" /> <!-- macro argument -->
       <parent link="${name}_rgb_link"/>
       <child link="${name}_rgb_optical_frame"/>

File: talos_description/urdf/torso/torso.urdf.xacro (robot description, xacro)
@@ -113,5 +113,5 @@
       <axis xyz="0 0 1" />
       <limit lower="${-75.00000 * deg_to_rad}" upper="${75.00000 * deg_to_rad}"
-             effort="${talos_max_effort}" velocity="${torso_max_vel}" />
+             effort="${torso_max_effort}" velocity="${torso_max_vel}" />
       <dynamics friction="1.0" damping="1.0"/>
       <!-- <safety_controller k_position="20"
