Commit message: Fix gripper movement in simulation. Add colors to model

File: talos_description/gazebo/gazebo.urdf.xacro (robot description, xacro)
@@ -13,4 +13,5 @@
       <frameName>torso_2_link</frameName>
       <topicName>floating_base_pose</topicName>
+      <updateRate>100.0</updateRate>
     </plugin>
   </gazebo>

File: talos_description/urdf/arm/arm.urdf.xacro (robot description, xacro)
@@ -185,16 +185,20 @@
      <mu1>0.9</mu1>
      <mu2>0.9</mu2>
+     <material>Gazebo/FlatBlack</material>
    </gazebo>
    <gazebo reference="${name}_${side}_2_link">
      <mu1>0.9</mu1>
      <mu2>0.9</mu2>
+     <material>Gazebo/FlatBlack</material>
    </gazebo>
    <gazebo reference="${name}_${side}_3_link">
      <mu1>0.9</mu1>
      <mu2>0.9</mu2>
+     <material>Gazebo/FlatBlack</material>
    </gazebo>
    <gazebo reference="${name}_${side}_4_link">
      <mu1>0.9</mu1>
      <mu2>0.9</mu2>
+     <material>Gazebo/FlatBlack</material>
    </gazebo>
    <gazebo reference="${name}_${side}_1_joint">

File: talos_description/urdf/arm/wrist.urdf.xacro (robot description, xacro)
@@ -147,4 +147,5 @@
       <mu1>0.9</mu1>
       <mu2>0.9</mu2>
+      <material>Gazebo/FlatBlack</material>
     </gazebo>
     <gazebo reference="${name}_${side}_5_joint">

File: talos_description/urdf/gripper/gripper.gazebo.xacro (robot description, xacro)
@@ -8,41 +8,121 @@
 -->
 <robot xmlns:xacro="http://ros.org/wiki/xacro">
-  <!-- MACROS FOR MIMIC JOINTS -->
-  <xacro:macro name="finger_mimics" params="name">
-    <plugin name="mimic_${name}_inner_double_joint" filename="libroboticsgroup_gazebo_mimic_joint_plugin.so">
-      <joint>${name}_joint</joint>
-      <mimicJoint>${name}_inner_double_joint</mimicJoint>
-      <multiplier>1.0</multiplier>
-      <offset>0.0</offset>
-      <hasPID/>
-    </plugin>
-    <plugin name="mimic_${name}_fingertip_1_joint" filename="libroboticsgroup_gazebo_mimic_joint_plugin.so">
-      <joint>${name}_joint</joint>
-      <mimicJoint>${name}_fingertip_1_joint</mimicJoint>
-      <multiplier>-1.0</multiplier>
-      <offset>0.0</offset>
-      <hasPID/>
-    </plugin>
-    <plugin name="mimic_${name}_fingertip_2_joint" filename="libroboticsgroup_gazebo_mimic_joint_plugin.so">
-      <joint>${name}_joint</joint>
-      <mimicJoint>${name}_fingertip_2_joint</mimicJoint>
-      <multiplier>-1.0</multiplier>
-      <offset>0.0</offset>
-      <hasPID/>
-    </plugin>
-    <plugin name="mimic_${name}_motor_single_joint" filename="libroboticsgroup_gazebo_mimic_joint_plugin.so">
-      <joint>${name}_joint</joint>
-      <mimicJoint>${name}_motor_single_joint</mimicJoint>
-      <multiplier>1.0</multiplier>
-      <offset>0.0</offset>
-      <hasPID/>
-    </plugin>
-    <plugin name="mimic_${name}_fingertip_3_joint" filename="libroboticsgroup_gazebo_mimic_joint_plugin.so">
-      <joint>${name}_joint</joint>
-      <mimicJoint>${name}_fingertip_3_joint</mimicJoint>
-      <multiplier>-1.0</multiplier>
-      <offset>0.0</offset>
-      <hasPID/>
-    </plugin>
+  <!-- VIRTUAL (mimic) JOINTS -->
+  <xacro:macro name="virtual_joints" params="name">
+    <gazebo>
+      <plugin name="mimic_${name}_inner_double_joint" filename="libroboticsgroup_gazebo_mimic_joint_plugin.so">
+        <joint>${name}_joint</joint>
+        <mimicJoint>${name}_inner_double_joint</mimicJoint>
+        <multiplier>1.0</multiplier>
+        <offset>0.0</offset>
+        <!-- <hasPID/> -->
+      </plugin>
+      <plugin name="mimic_${name}_fingertip_1_joint" filename="libroboticsgroup_gazebo_mimic_joint_plugin.so">
+        <joint>${name}_joint</joint>
+        <mimicJoint>${name}_fingertip_1_joint</mimicJoint>
+        <multiplier>-1.0</multiplier>
+        <offset>0.0</offset>
+        <!-- <hasPID/> -->
+      </plugin>
+      <plugin name="mimic_${name}_fingertip_2_joint" filename="libroboticsgroup_gazebo_mimic_joint_plugin.so">
+        <joint>${name}_joint</joint>
+        <mimicJoint>${name}_fingertip_2_joint</mimicJoint>
+        <multiplier>-1.0</multiplier>
+        <offset>0.0</offset>
+        <!-- <hasPID/> -->
+      </plugin>
+      <plugin name="mimic_${name}_inner_single_joint" filename="libroboticsgroup_gazebo_mimic_joint_plugin.so">
+        <joint>${name}_joint</joint>
+        <mimicJoint>${name}_inner_single_joint</mimicJoint>
+        <multiplier>-1.0</multiplier>
+        <offset>0.0</offset>
+        <!-- <hasPID/> -->
+      </plugin>
+      <plugin name="mimic_${name}_motor_single_joint" filename="libroboticsgroup_gazebo_mimic_joint_plugin.so">
+        <joint>${name}_joint</joint>
+        <mimicJoint>${name}_motor_single_joint</mimicJoint>
+        <multiplier>-1.0</multiplier>
+        <offset>0.0</offset>
+        <!-- <hasPID/> -->
+      </plugin>
+      <plugin name="mimic_${name}_fingertip_3_joint" filename="libroboticsgroup_gazebo_mimic_joint_plugin.so">
+        <joint>${name}_joint</joint>
+        <mimicJoint>${name}_fingertip_3_joint</mimicJoint>
+        <multiplier>-1.0</multiplier>
+        <offset>0.0</offset>
+       <!-- <hasPID/> -->
+      </plugin>
+  </gazebo>
+<!--     <plugin filename="libgazebo_underactuated_finger.so" name="gazebo_${name}_underactuated">
+      <actuatedJoint>${name}_joint</actuatedJoint>
+      <virtualJoint>
+        <name>${name}_inner_double_joint</name>
+        <scale_factor>1.0</scale_factor>
+      </virtualJoint> -->
+<!--       <virtualJoint>
+        <name>${name}_fingertip_1_joint</name>
+        <scale_factor>-1.0</scale_factor>
+      </virtualJoint>
+      <virtualJoint>
+        <name>${name}_fingertip_2_joint</name>
+        <scale_factor>-1.0</scale_factor>
+      </virtualJoint>
+      <virtualJoint>
+        <name>${name}_motor_single_joint</name>
+        <scale_factor>1.0</scale_factor>
+      </virtualJoint>
+      <virtualJoint>
+        <name>${name}_fingertip_3_joint</name>
+        <scale_factor>-1.0</scale_factor>
+      </virtualJoint> -->
+<!--     </plugin> -->
+  <gazebo reference="${name}_joint">
+    <implicitSpringDamper>1</implicitSpringDamper>
+    <provideFeedback>1</provideFeedback>
+  </gazebo>
+  <gazebo reference="${name}_inner_double_joint">
+    <implicitSpringDamper>1</implicitSpringDamper>
+    <provideFeedback>1</provideFeedback>
+  </gazebo>
+  <gazebo reference="${name}_fingertip_1_joint">
+    <implicitSpringDamper>1</implicitSpringDamper>
+    <provideFeedback>1</provideFeedback>
+  </gazebo>
+  <gazebo reference="${name}_fingertip_2_joint">
+    <implicitSpringDamper>1</implicitSpringDamper>
+    <provideFeedback>1</provideFeedback>
+  </gazebo>
+  <gazebo reference="${name}_motor_single_joint">
+    <implicitSpringDamper>1</implicitSpringDamper>
+    <provideFeedback>1</provideFeedback>
+  </gazebo>
+  <gazebo reference="${name}_fingertip_3_joint">
+    <implicitSpringDamper>1</implicitSpringDamper>
+    <provideFeedback>1</provideFeedback>
+  </gazebo>
+  <gazebo reference="${name}_base_link">
+    <material>Gazebo/FlatBlack</material>
+  </gazebo>
+  <gazebo reference="${name}_motor_double_link">
+    <material>Gazebo/Orange</material>
+  </gazebo>
+  <gazebo reference="${name}_inner_double_link">
+    <material>Gazebo/Orange</material>
+  </gazebo>
+  <gazebo reference="${name}_fingertip_1_link">
+    <material>Gazebo/FlatBlack</material>
+  </gazebo>
+  <gazebo reference="${name}_motor_single_link">
+    <material>Gazebo/Orange</material>
+  </gazebo>
+  <gazebo reference="${name}_inner_single_link">
+    <material>Gazebo/Orange</material>
+  </gazebo>
+  <gazebo reference="${name}_fingertip_2_link">
+    <material>Gazebo/FlatBlack</material>
+  </gazebo>
+  <gazebo reference="${name}_fingertip_3_link">
+    <material>Gazebo/FlatBlack</material>
+  </gazebo>
   </xacro:macro>
 </robot>

File: talos_description/urdf/gripper/gripper.transmission.xacro (robot description, xacro)
@@ -19,3 +19,14 @@
     </transmission>
   </xacro:macro>
+  <xacro:macro name="gripper_virtual_transmission" params="name reduction" >
+    <transmission name="${name}_trans">
+      <type>transmission_interface/SimpleTransmission</type>
+      <actuator name="${name}_motor" >
+        <mechanicalReduction>${reduction}</mechanicalReduction>
+      </actuator>
+      <joint name="${name}_joint" >
+        <hardwareInterface>hardware_interface/JointStateInterface</hardwareInterface>
+      </joint>
+    </transmission>
+  </xacro:macro>
 </robot>

File: talos_description/urdf/gripper/gripper_v2.urdf.xacro (robot description, xacro)
@@ -96,5 +96,5 @@
                       rpy="${0.00000 * deg_to_rad} ${0.00000 * deg_to_rad} ${0.00000 * deg_to_rad}"/>
               <axis xyz="1 0 0" />
-              <limit lower="${0.00000 * deg_to_rad}" upper="${0.00000 * deg_to_rad}" effort="1.0" velocity="1.0" />
+              <limit lower="${-60.0 * deg_to_rad}" upper="${0.0 * deg_to_rad}" effort="100.0" velocity="1.0" />
               <mimic joint="${name}_joint" multiplier="${1.0}" offset="0.0" />
             </joint>
@@ -127,7 +127,7 @@
                       rpy="${0.00000 * deg_to_rad} ${0.00000 * deg_to_rad} ${0.00000 * deg_to_rad}"/>
               <axis xyz="1 0 0" />
-              <limit lower="${0.00000 * deg_to_rad}" upper="${0.00000 * deg_to_rad}" effort="1.0" velocity="1.0" />
-              <mimic joint="${name}_joint" multiplier="${-1.0}" offset="0.0" />
-            </joint>
+              <limit lower="${0.0 * deg_to_rad}" upper="${60.0 * deg_to_rad}" effort="100.0" velocity="1.0" />
+              <mimic joint="${name}_joint" multiplier="${-1.0}" offset="0.0" />
+           </joint>
             <link name="${name}_fingertip_2_link">
               <inertial>
@@ -158,8 +158,8 @@
                       rpy="${0.00000 * deg_to_rad} ${0.00000 * deg_to_rad} ${0.00000 * deg_to_rad}"/>
               <axis xyz="1 0 0" />
-              <limit lower="${0.00000 * deg_to_rad}" upper="${0.00000 * deg_to_rad}" effort="1.0" velocity="1.0" />
-              <mimic joint="${name}_joint" multiplier="${-1.0}" offset="0.0" />
-            </joint>
-             <link name="${name}_motor_single_link">
+              <limit lower="${0.0 * deg_to_rad}" upper="${60.0 * deg_to_rad}" effort="100.0" velocity="1.0" />
+              <mimic joint="${name}_joint" multiplier="${-1.0}" offset="0.0" />
+           </joint>
+            <link name="${name}_motor_single_link">
               <inertial>
                 <origin xyz="0.02589 -0.01284 -0.00640" rpy="0.00000 0.00000 0.00000"/>
@@ -189,8 +189,8 @@
                       rpy="${0.00000 * deg_to_rad} ${0.00000 * deg_to_rad} ${0.00000 * deg_to_rad}"/>
               <axis xyz="1 0 0" />
-              <limit lower="${0.00000 * deg_to_rad}" upper="${0.00000 * deg_to_rad}" effort="1.0" velocity="1.0" />
-              <mimic joint="${name}_joint" multiplier="${-1.0}" offset="0.0" />
-            </joint>
-          <link name="${name}_inner_single_link">
+              <limit lower="${0.0 * deg_to_rad}" upper="${60.0 * deg_to_rad}" effort="100.0" velocity="1.0" />
+              <mimic joint="${name}_joint" multiplier="${-1.0}" offset="0.0" />
+           </joint>
+            <link name="${name}_inner_single_link">
               <inertial>
                 <origin xyz="0.00000 -0.03253 -0.01883" rpy="0.00000 0.00000 0.00000"/>
@@ -220,7 +220,7 @@
                       rpy="${0.00000 * deg_to_rad} ${0.00000 * deg_to_rad} ${0.00000 * deg_to_rad}"/>
               <axis xyz="1 0 0" />
-              <limit lower="${0.00000 * deg_to_rad}" upper="${0.00000 * deg_to_rad}" effort="1.0" velocity="1.0" />
-              <mimic joint="${name}_joint" multiplier="${-1.0}" offset="0.0" />
-            </joint>
+              <limit lower="${0.0 * deg_to_rad}" upper="${60.0 * deg_to_rad}" effort="100.0" velocity="1.0" />
+              <mimic joint="${name}_joint" multiplier="${-1.0}" offset="0.0" />
+           </joint>
             <link name="${name}_fingertip_3_link">
               <inertial>
@@ -251,9 +251,16 @@
                       rpy="${0.00000 * deg_to_rad} ${0.00000 * deg_to_rad} ${180.00000 * deg_to_rad}"/>
               <axis xyz="1 0 0" />
-              <limit lower="${0.00000 * deg_to_rad}" upper="${0.00000 * deg_to_rad}" effort="1.0" velocity="1.0" />
-              <mimic joint="${name}_joint" multiplier="${-1.0}" offset="0.0" />
-            </joint>
-        <xacro:finger_mimics name="${name}" />
+              <limit lower="${0.0 * deg_to_rad}" upper="${60.0 * deg_to_rad}" effort="100.0" velocity="1.0" />
+              <mimic joint="${name}_joint" multiplier="${-1.0}" offset="0.0" />
+           </joint>
+        <xacro:virtual_joints name="${name}" />
         <xacro:gripper_transmission name="${name}" reduction="1.0" />
+        <!-- virtual mimic joints -->
+        <xacro:gripper_virtual_transmission name="${name}_inner_double" reduction="1.0"/>
+        <xacro:gripper_virtual_transmission name="${name}_fingertip_1" reduction="1.0"/>
+        <xacro:gripper_virtual_transmission name="${name}_fingertip_2" reduction="1.0"/>
+        <xacro:gripper_virtual_transmission name="${name}_inner_single" reduction="1.0"/>
+        <xacro:gripper_virtual_transmission name="${name}_motor_single" reduction="1.0"/>
+        <xacro:gripper_virtual_transmission name="${name}_fingertip_3" reduction="1.0"/>
  </xacro:macro>
 </robot>

File: talos_description/urdf/head/head.urdf.xacro (robot description, xacro)
@@ -63,4 +63,7 @@
        <implicitSpringDamper>1</implicitSpringDamper>
     </gazebo>
+    <gazebo reference="${name}_link">
+      <material>Gazebo/FlatBlack</material>
+    </gazebo>
   </xacro:macro>
   <!--************************-->
@@ -110,4 +113,7 @@
        <implicitSpringDamper>1</implicitSpringDamper>
     </gazebo>
+    <gazebo reference="${name}_link">
+      <material>Gazebo/White</material>
+    </gazebo>
   </xacro:macro>
   <xacro:macro name="talos_head" params="name parent">

File: talos_description/urdf/leg/leg_v2.urdf.xacro (robot description, xacro)
@@ -284,4 +284,22 @@
      <provideFeedback>1</provideFeedback>
    </gazebo>
+  <gazebo reference="leg_${prefix}_1_link">
+    <material>Gazebo/FlatBlack</material>
+  </gazebo>
+  <gazebo reference="leg_${prefix}_2_link">
+    <material>Gazebo/FlatBlack</material>
+  </gazebo>
+  <gazebo reference="leg_${prefix}_3_link">
+    <material>Gazebo/FlatBlack</material>
+  </gazebo>
+  <gazebo reference="leg_${prefix}_4_link">
+    <material>Gazebo/FlatBlack</material>
+  </gazebo>
+  <gazebo reference="leg_${prefix}_5_link">
+    <material>Gazebo/White</material>
+  </gazebo>
+  <gazebo reference="leg_${prefix}_6_link">
+    <material>Gazebo/White</material>
+  </gazebo>
  </xacro:macro>
 </robot>

File: talos_description/urdf/sensors/xtion_pro_live.gazebo.xacro (robot description, xacro)
@@ -85,4 +85,5 @@
         </plugin>
       </sensor>
+      <material>Gazebo/FlatBlack</material>
     </gazebo>
   </xacro:macro>
