Commit message: Added sub models to debug gazebo and added implicit tag simulation to 1.0

File: talos_description/robots/talos_full_no_lower_arm.urdf.xacro (robot description, xacro)
@@ -17,29 +17,8 @@
   <xacro:include filename="$(find talos_description)/urdf/gripper/gripper_v2.urdf.xacro" />
   <xacro:include filename="$(find talos_description)/urdf/leg/leg_v2.urdf.xacro" />
-    <!--************************-->
-    <!--        BASE_LINK       -->
-    <!--************************-->
-    <link name="base_link">
-      <inertial>
-        <origin xyz="-0.08222 0.00838 -0.07261" rpy="0.00000 0.00000 0.00000"/>
-        <mass value="13.53810"/>
-        <inertia ixx="0.06989000000" ixy="-0.00011700000" ixz="0.00023000000"
-                 iyy="0.03998200000" iyz="-0.00132500000"
-                 izz="0.08234500000"/>
-      </inertial>
-      <visual>
-        <origin xyz="0 0 0" rpy="0 0 0" />
-        <geometry>
-          <mesh filename="package://talos_description/meshes/torso/base_link.STL" scale="1 1 1"/>
-        </geometry>
-        <material name="LightGrey" />
-      </visual>
-      <collision>
-        <origin xyz="0 0 0" rpy="0 0 0" />
-        <geometry>
-          <mesh filename="package://talos_description/meshes/torso/base_link_collision.STL" scale="1 1 1"/>
-        </geometry>
-      </collision>
-    </link>
+  <xacro:talos_torso name="torso" />
+  <xacro:talos_head name="head" parent="torso_2_link"/>
+  <xacro:talos_arm name="arm" parent="torso_2_link" side="left" reflect="1"/>
+  <xacro:talos_arm name="arm" parent="torso_2_link" side="right" reflect="-1"/>
   <xacro:talos_leg prefix="left"  reflect="1" />
   <xacro:talos_leg prefix="right" reflect="-1" />
@@ -48,8 +27,3 @@
   <!-- Materials for visualization -->
   <xacro:include filename="$(find talos_description)/urdf/materials.urdf.xacro" />
-  <xacro:include filename="$(find talos_description)/urdf/sensors/imu.urdf.xacro" />
-    <!-- imu -->
-  <xacro:talos_imu name="imu" parent="base_link" update_rate="100.0">
-    <origin xyz="0 0 0" rpy="0 0 0"/>
-  </xacro:talos_imu>
 </robot>

File: talos_description/robots/talos_lower_body_with_torso.urdf.xacro (robot description, xacro)
@@ -17,29 +17,6 @@
   <xacro:include filename="$(find talos_description)/urdf/gripper/gripper_v2.urdf.xacro" />
   <xacro:include filename="$(find talos_description)/urdf/leg/leg_v2.urdf.xacro" />
-    <!--************************-->
-    <!--        BASE_LINK       -->
-    <!--************************-->
-    <link name="base_link">
-      <inertial>
-        <origin xyz="-0.08222 0.00838 -0.07261" rpy="0.00000 0.00000 0.00000"/>
-        <mass value="13.53810"/>
-        <inertia ixx="0.06989000000" ixy="-0.00011700000" ixz="0.00023000000"
-                 iyy="0.03998200000" iyz="-0.00132500000"
-                 izz="0.08234500000"/>
-      </inertial>
-      <visual>
-        <origin xyz="0 0 0" rpy="0 0 0" />
-        <geometry>
-          <mesh filename="package://talos_description/meshes/torso/base_link.STL" scale="1 1 1"/>
-        </geometry>
-        <material name="LightGrey" />
-      </visual>
-      <collision>
-        <origin xyz="0 0 0" rpy="0 0 0" />
-        <geometry>
-          <mesh filename="package://talos_description/meshes/torso/base_link_collision.STL" scale="1 1 1"/>
-        </geometry>
-      </collision>
-    </link>
+  <xacro:talos_torso name="torso" />
+  <xacro:talos_head name="head" parent="torso_2_link"/>
   <xacro:talos_leg prefix="left"  reflect="1" />
   <xacro:talos_leg prefix="right" reflect="-1" />
@@ -48,8 +25,3 @@
   <!-- Materials for visualization -->
   <xacro:include filename="$(find talos_description)/urdf/materials.urdf.xacro" />
-  <xacro:include filename="$(find talos_description)/urdf/sensors/imu.urdf.xacro" />
-    <!-- imu -->
-  <xacro:talos_imu name="imu" parent="base_link" update_rate="100.0">
-    <origin xyz="0 0 0" rpy="0 0 0"/>
-  </xacro:talos_imu>
 </robot>

File: talos_description/urdf/arm/arm.urdf.xacro (robot description, xacro)
@@ -217,5 +217,5 @@
     <!--        WRIST           -->
     <!--************************-->
-    <xacro:talos_wrist name="arm" parent="${name}_${side}_4_link" side="${side}" reflect="${reflect}" />
+     <xacro:talos_wrist name="arm" parent="${name}_${side}_4_link" side="${side}" reflect="${reflect}" />
     <!--***********************-->
     <!--        TOOL           -->

File: talos_description/urdf/leg/leg_v2.urdf.xacro (robot description, xacro)
@@ -259,27 +259,28 @@
     <kp>1000000.0</kp>
     <kd>100.0</kd>
-    <mu1>1.5</mu1>
-    <mu2>1.5</mu2>
+    <mu1>1.0</mu1>
+    <mu2>1.0</mu2>
     <fdir1>1 0 0</fdir1>
     <maxVel>1.0</maxVel>
     <minDepth>0.00</minDepth>
+    <implicitSpringDamper>1</implicitSpringDamper>
    </gazebo>
    <gazebo reference="leg_${prefix}_1_joint">
-      <implicitSpringDamper>0.1</implicitSpringDamper>
+      <implicitSpringDamper>1</implicitSpringDamper>
    </gazebo>
    <gazebo reference="leg_${prefix}_2_joint">
-      <implicitSpringDamper>0.1</implicitSpringDamper>
+      <implicitSpringDamper>1</implicitSpringDamper>
    </gazebo>
    <gazebo reference="leg_${prefix}_3_joint">
-      <implicitSpringDamper>0.1</implicitSpringDamper>
+      <implicitSpringDamper>1</implicitSpringDamper>
    </gazebo>
    <gazebo reference="leg_${prefix}_4_joint">
-      <implicitSpringDamper>0.1</implicitSpringDamper>
+      <implicitSpringDamper>1</implicitSpringDamper>
    </gazebo>
    <gazebo reference="leg_${prefix}_5_joint">
-      <implicitSpringDamper>0.1</implicitSpringDamper>
+      <implicitSpringDamper>1</implicitSpringDamper>
    </gazebo>
    <gazebo reference="leg_${prefix}_6_joint">
-     <implicitSpringDamper>0.1</implicitSpringDamper>
+     <implicitSpringDamper>1</implicitSpringDamper>
      <provideFeedback>1</provideFeedback>
    </gazebo>
