Commit message: Fixing

File: talos_description/robots/talos_full.urdf.xacro (robot description, xacro)
@@ -11,5 +11,5 @@
         xmlns:controller="http://playerstage.sourceforge.net/gazebo/xmlschema/#controller"
         xmlns:interface="http://playerstage.sourceforge.net/gazebo/xmlschema/#interface">
-  <xacro:include filename="$(find talos_description)/urdf/talos/talos.urdf.xacro" />
+  <xacro:include filename="$(find talos_description)/urdf/torso/torso.urdf.xacro" />
   <xacro:include filename="$(find talos_description)/urdf/head/head.urdf.xacro" />
   <xacro:include filename="$(find talos_description)/urdf/arm/arm.urdf.xacro" />
@@ -18,7 +18,7 @@
   <xacro:include filename="$(find talos_description)/urdf/leg/leg_v2.urdf.xacro" />
   <xacro:talos_talos name="talos" />
-  <xacro:talos_head name="head" parent="talos_2_link"/>
-  <xacro:talos_arm name="arm" parent="talos_2_link" side="left" reflect="1"/>
-  <xacro:talos_arm name="arm" parent="talos_2_link" side="right" reflect="-1"/>
+  <xacro:talos_head name="head" parent="torso_2_link"/>
+  <xacro:talos_arm name="arm" parent="torso_2_link" side="left" reflect="1"/>
+  <xacro:talos_arm name="arm" parent="torso_2_link" side="right" reflect="-1"/>
   <xacro:ft_sensor name="wrist" parent="arm_right_7_link" side="right" reflect="1"  />
   <xacro:ft_sensor name="wrist" parent="arm_left_7_link"  side="left"  reflect="-1" />

File: talos_description/urdf/arm/arm.transmission.xacro (robot description, xacro)
@@ -11,7 +11,7 @@
     <transmission name="${name}_${side}_${number}_trans">
       <type>transmission_interface/SimpleTransmission</type>
-      <actuatalos name="${name}_${side}_${number}_motalos" >
+      <actuator name="${name}_${side}_${number}_motor" >
         <mechanicalReduction>${reduction}</mechanicalReduction>
-      </actuatalos>
+      </actuator>
       <joint name="${name}_${side}_${number}_joint">
         <hardwareInterface>hardware_interface/PositionJointInterface</hardwareInterface>

File: talos_description/urdf/arm/wrist.transmission.xacro (robot description, xacro)
@@ -11,7 +11,7 @@
     <transmission name="${name}_${side}_${number}_trans">
       <type>transmission_interface/SimpleTransmission</type>
-      <actuatalos name="${name}_${side}_${number}_motalos" >
+      <actuator name="${name}_${side}_${number}_motor" >
         <mechanicalReduction>${reduction}</mechanicalReduction>
-      </actuatalos>
+      </actuator>
       <joint name="${name}_${side}_${number}_joint">
         <hardwareInterface>hardware_interface/PositionJointInterface</hardwareInterface>
@@ -24,12 +24,12 @@
     <transmission name="wrist_${side}_trans">
       <type>transmission_interface/DifferentialTransmission</type>
-      <actuatalos name="${name}_${side}_${number_1}_motalos">
-        <role>actuatalos1</role>
+      <actuator name="${name}_${side}_${number_1}_motor">
+        <role>actuator1</role>
         <mechanicalReduction>${act_reduction_1}</mechanicalReduction>
-      </actuatalos>
-      <actuatalos name="${name}_${side}_${number_2}_motalos">
-        <role>actuatalos2</role>
+      </actuator>
+      <actuator name="${name}_${side}_${number_2}_motor">
+        <role>actuator2</role>
         <mechanicalReduction>${act_reduction_2}</mechanicalReduction>
-      </actuatalos>
+      </actuator>
       <joint name="${name}_${side}_${number_1}_joint">
         <role>joint1</role>

File: talos_description/urdf/gripper/gripper_v2.urdf.xacro (robot description, xacro)
@@ -34,6 +34,6 @@
               <axis xyz="0 0 0" />
             </joint>
-            <!-- Joint gripper_motalos_double (None) : child link -- -> parent link gripper_base_link -->
-            <link name="${name}_motalos_double_link">
+            <!-- Joint gripper_motor_double (None) : child link -- -> parent link gripper_base_link -->
+            <link name="${name}_motor_double_link">
               <inertial>
                 <origin xyz="0.02270 0.01781 -0.00977" rpy="0.00000 0.00000 0.00000"/>
@@ -46,5 +46,5 @@
                 <origin xyz="0 0 0" rpy="0 0 0" />
                 <geometry>
-                  <mesh filename="package://talos_description/meshes/gripper/gripper_motalos_double.STL" scale="1 1 1"/>
+                  <mesh filename="package://talos_description/meshes/gripper/gripper_motor_double.STL" scale="1 1 1"/>
                 </geometry>
               </visual>
@@ -52,11 +52,11 @@
                 <origin xyz="0 0 0" rpy="0 0 0" />
                 <geometry>
-                  <mesh filename="package://talos_description/meshes/gripper/gripper_motalos_double_collision.STL" scale="1 1 1"/>
+                  <mesh filename="package://talos_description/meshes/gripper/gripper_motor_double_collision.STL" scale="1 1 1"/>
                 </geometry>
               </collision>
             </link>
-            <joint name="${name}_motalos_double_joint" type="revolute">
+            <joint name="${name}_motor_double_joint" type="revolute">
               <parent link="${name}_base_link"/>
-              <child link="${name}_motalos_double_link"/>
+              <child link="${name}_motor_double_link"/>
               <origin xyz="0.00000 0.02025 -0.03000"
                       rpy="${0.00000 * deg_to_rad} ${0.00000 * deg_to_rad} ${0.00000 * deg_to_rad}"/>
@@ -95,5 +95,5 @@
               <axis xyz="0 0 1" />
               <limit lower="${0.00000 * deg_to_rad}" upper="${0.00000 * deg_to_rad}" effort="1.0" velocity="1.0" />
-              <mimic joint="${name}_motalos_double_joint" multiplier="${1.0}" offset="0.0" />
+              <mimic joint="${name}_motor_double_joint" multiplier="${1.0}" offset="0.0" />
             </joint>
  </xacro:macro>

File: talos_description/urdf/head/head.transmission.xacro (robot description, xacro)
@@ -12,12 +12,12 @@
     <transmission name="talos_trans">
       <type>transmission_interface/DifferentialTransmission</type>
-      <actuatalos name="${name}_${number1}_motalos">
-        <role>actuatalos1</role>
+      <actuator name="${name}_${number1}_motor">
+        <role>actuator1</role>
         <mechanicalReduction>${act_reduction1}</mechanicalReduction>
-      </actuatalos>
-      <actuatalos name="${name}_${number2}_motalos">
-        <role>actuatalos2</role>
+      </actuator>
+      <actuator name="${name}_${number2}_motor">
+        <role>actuator2</role>
         <mechanicalReduction>${act_reduction2}</mechanicalReduction>
-      </actuatalos>
+      </actuator>
       <joint name="${name}_${number1}_joint">
         <role>joint1</role>

File: talos_description/urdf/leg/leg.transmission.xacro (robot description, xacro)
@@ -11,7 +11,7 @@
     <transmission name="leg_${side}_${number}_trans">
       <type>transmission_interface/SimpleTransmission</type>
-      <actuatalos name="leg_${side}_${number}_motalos" >
+      <actuator name="leg_${side}_${number}_motor" >
         <mechanicalReduction>${reduction}</mechanicalReduction>
-      </actuatalos>
+      </actuator>
       <joint name="leg_${side}_${number}_joint">
         <hardwareInterface>hardware_interface/PositionJointInterface</hardwareInterface>

File: talos_description/urdf/torso/torso.transmission.xacro (robot description, xacro)
@@ -8,16 +8,16 @@
 -->
 <robot xmlns:xacro="http://ros.org/wiki/xacro">
-  <xacro:macro name="talos_talos_differential_transmission"
+  <xacro:macro name="talos_torso_differential_transmission"
                params="name number1 number2 act_reduction1 act_reduction2 jnt_reduction1 jnt_reduction2" >
-    <transmission name="talos_trans">
+    <transmission name="talos_torso_trans">
       <type>transmission_interface/DifferentialTransmission</type>
-      <actuatalos name="${name}_${number1}_motalos">
-        <role>actuatalos1</role>
+      <actuator name="${name}_${number1}_motor">
+        <role>actuator1</role>
         <mechanicalReduction>${act_reduction1}</mechanicalReduction>
-      </actuatalos>
-      <actuatalos name="${name}_${number2}_motalos">
-        <role>actuatalos2</role>
+      </actuator>
+      <actuator name="${name}_${number2}_motor">
+        <role>actuator2</role>
         <mechanicalReduction>${act_reduction2}</mechanicalReduction>
-      </actuatalos>
+      </actuator>
       <joint name="${name}_${number1}_joint">
         <role>joint1</role>

File: talos_description/urdf/torso/torso.urdf.xacro (robot description, xacro)
@@ -10,11 +10,11 @@
   <!--File includes-->
   <xacro:include filename="$(find talos_description)/urdf/deg_to_rad.xacro" />
-  <xacro:include filename="$(find talos_description)/urdf/talos/talos.transmission.xacro" />
+  <xacro:include filename="$(find talos_description)/urdf/torso/torso.transmission.xacro" />
   <xacro:include filename="$(find talos_description)/urdf/sensors/imu.urdf.xacro" />
  <!--Constant parameters-->
-  <xacro:property name="talos_max_vel"  value="5.4" />
-  <xacro:property name="talos_max_effort"  value="78.0" />
-  <xacro:property name="talos_eps"      value="0.02" />
-  <xacro:macro name="talos_talos" params="name">
+  <xacro:property name="torso_max_vel"  value="5.4" />
+  <xacro:property name="torso_max_effort"  value="78.0" />
+  <xacro:property name="torso_eps"      value="0.02" />
+  <xacro:macro name="talos_torso" params="name">
     <!--************************-->
     <!--        TORSO_2  (TILT) -->
@@ -31,5 +31,5 @@
         <origin xyz="0 0 0" rpy="0 0 0" />
         <geometry>
-          <mesh filename="package://talos_description/meshes/talos/talos_2.STL" scale="1 1 1"/>
+          <mesh filename="package://talos_description/meshes/torso/torso_2.STL" scale="1 1 1"/>
         </geometry>
         <material name="LightGrey" />
@@ -38,5 +38,5 @@
         <origin xyz="0 0 0" rpy="0 0 0" />
         <geometry>
-          <mesh filename="package://talos_description/meshes/talos/talos_2_collision.STL" scale="1 1 1"/>
+          <mesh filename="package://talos_description/meshes/torso/torso_2_collision.STL" scale="1 1 1"/>
         </geometry>
       </collision>
@@ -56,5 +56,5 @@
         <origin xyz="0 0 0" rpy="0 0 0" />
         <geometry>
-          <mesh filename="package://talos_description/meshes/talos/talos_1.STL" scale="1 1 1"/>
+          <mesh filename="package://talos_description/meshes/torso/torso_1.STL" scale="1 1 1"/>
         </geometry>
         <material name="LightGrey" />
@@ -63,5 +63,5 @@
         <origin xyz="0 0 0" rpy="0 0 0" />
         <geometry>
-          <mesh filename="package://talos_description/meshes/talos/talos_1.STL" scale="1 1 1"/>
+          <mesh filename="package://talos_description/meshes/torso/torso_1.STL" scale="1 1 1"/>
         </geometry>
       </collision>
@@ -74,10 +74,10 @@
       <axis xyz="0 1 0" />
       <limit lower="${-45.0 * deg_to_rad}" upper="${15.0 * deg_to_rad}"
-             effort="${talos_max_effort}" velocity="${talos_max_vel}"/>
+             effort="${torso_max_effort}" velocity="${torso_max_vel}"/>
       <dynamics damping="1.0" friction="1.0"/>
       <!-- <safety_controller k_position="20"
                          k_velocity="20"
-                         soft_lower_limit="${-15.0 * deg_to_rad + talos_eps}"
-                         soft_upper_limit="${ 45.0 * deg_to_rad - talos_eps}" /> -->
+                         soft_lower_limit="${-15.0 * deg_to_rad + torso_eps}"
+                         soft_upper_limit="${ 45.0 * deg_to_rad - torso_eps}" /> -->
     </joint>
     <!--************************-->
@@ -95,5 +95,5 @@
         <origin xyz="0 0 0" rpy="0 0 0" />
         <geometry>
-          <mesh filename="package://talos_description/meshes/talos/base_link.STL" scale="1 1 1"/>
+          <mesh filename="package://talos_description/meshes/torso/base_link.STL" scale="1 1 1"/>
         </geometry>
         <material name="LightGrey" />
@@ -102,5 +102,5 @@
         <origin xyz="0 0 0" rpy="0 0 0" />
         <geometry>
-          <mesh filename="package://talos_description/meshes/talos/base_link_collision.STL" scale="1 1 1"/>
+          <mesh filename="package://talos_description/meshes/torso/base_link_collision.STL" scale="1 1 1"/>
         </geometry>
       </collision>
@@ -113,5 +113,5 @@
       <axis xyz="0 0 1" />
       <limit lower="${-75.00000 * deg_to_rad}" upper="${75.00000 * deg_to_rad}"
-             effort="${talos_max_effort}" velocity="${talos_max_vel}" />
+             effort="${talos_max_effort}" velocity="${torso_max_vel}" />
       <dynamics friction="1.0" damping="1.0"/>
       <!-- <safety_controller k_position="20"
@@ -143,5 +143,5 @@
    </gazebo>
     <!-- extensions -->
-    <xacro:talos_talos_differential_transmission name="${name}" number1="1" number2="2"
+    <xacro:talos_torso_differential_transmission name="${name}" number1="1" number2="2"
                                                 act_reduction1="1.0" act_reduction2="1.0"
                                                 jnt_reduction1="1.0" jnt_reduction2="1.0" />

Commit message: Using new gripper

File: talos_description/robots/talos_full.urdf.xacro (robot description, xacro)
@@ -15,5 +15,5 @@
   <xacro:include filename="$(find talos_description)/urdf/arm/arm.urdf.xacro" />
   <xacro:include filename="$(find talos_description)/urdf/sensors/ftsensor.urdf.xacro" />
-  <xacro:include filename="$(find talos_description)/urdf/gripper/gripper.urdf.xacro" />
+  <xacro:include filename="$(find talos_description)/urdf/gripper/gripper_v2.urdf.xacro" />
   <xacro:include filename="$(find talos_description)/urdf/leg/leg_v2.urdf.xacro" />
   <xacro:talos_torso name="torso" />

File: talos_description/urdf/gripper/gripper_v2.urdf.xacro (robot description, xacro)
@@ -119,5 +119,5 @@
               </collision>
             </link>
-            <joint name="fingertip_1_joint" type="revolute">
+            <joint name="${name}_fingertip_1_joint" type="revolute">
               <parent link="${name}_inner_double_link"/>
               <child link="${name}_fingertip_1_link"/>

Commit message: Temporaly fixed arm dynamics

File: talos_description/robots/talos_full.urdf.xacro (robot description, xacro)
@@ -23,6 +23,6 @@
   <xacro:ft_sensor name="wrist" parent="arm_right_7_link" side="right" reflect="1"  />
   <xacro:ft_sensor name="wrist" parent="arm_left_7_link"  side="left"  reflect="-1" />
-  <xacro:talos_gripper name="gripper_left" parent="wrist_left_ft_tool_link"/>
-  <xacro:talos_gripper name="gripper_right" parent="wrist_right_ft_tool_link"/>
+  <xacro:talos_gripper name="gripper_left" parent="wrist_left_ft_tool_link" reflect="1" />
+  <xacro:talos_gripper name="gripper_right" parent="wrist_right_ft_tool_link" reflect="-1" />
   <xacro:talos_leg prefix="left"  reflect="1" />
   <xacro:talos_leg prefix="right" reflect="-1" />

File: talos_description/urdf/arm/arm.urdf.xacro (robot description, xacro)
@@ -32,5 +32,6 @@
       <inertial>
         <origin xyz="-0.01346 ${reflect*0.09130} 0.04812" rpy="0.00000 0.00000 0.00000"/>
-        <mass value="1.52896"/>
+        <!-- <mass value="1.52896"/> -->
+        <mass value="1.42896"/>
         <inertia ixx="0.00555100000" ixy="-0.00073100000" ixz="0.00000800000"
                  iyy="0.00167300000" iyz="-0.00006000000"
@@ -72,5 +73,6 @@
       <inertial>
         <origin xyz="0.02607 0.00049 -0.05209" rpy="0.00000 0.00000 0.00000"/>
-        <mass value="1.77729"/>
+        <!-- <mass value="1.77729"/> -->
+        <mass value="1.67729"/>
         <inertia ixx="0.00708700000" ixy="-0.00001400000" ixz="0.00214200000"
                  iyy="0.00793600000" iyz="0.00003000000"
@@ -112,5 +114,6 @@
       <inertial>
         <origin xyz="0.00841 0.01428 -0.22291" rpy="0.00000 0.00000 0.00000"/>
-        <mass value="1.57029"/>
+        <!-- <mass value="1.57029"/> -->
+        <mass value="1.47029"/>
         <inertia ixx="0.00433200000" ixy="0.00015300000" ixz="-0.00049600000"
                  iyy="0.00434000000" iyz="-0.00060900000"
@@ -150,5 +153,6 @@
       <inertial>
         <origin xyz="-0.00655 -0.02107 -0.02612" rpy="0.00000 0.00000 0.00000"/>
-        <mass value="1.20216"/>
+        <!-- <mass value="1.20216"/> -->
+        <mass value="1.10216"/>
         <inertia ixx="0.00221700000" ixy="-0.00010100000" ixz="0.00028800000"
                  iyy="0.00241800000" iyz="-0.00039300000"

File: talos_description/urdf/arm/wrist.urdf.xacro (robot description, xacro)
@@ -28,5 +28,6 @@
       <inertial>
         <origin xyz="-0.00006 0.00326 0.07963" rpy="0.00000 0.00000 0.00000"/>
-        <mass value="1.87792"/>
+        <!-- <mass value="1.87792"/> -->
+        <mass value="1.77792"/>
         <inertia ixx="0.00349500000" ixy="-0.00001300000" ixz="-0.00001000000"
                  iyy="0.00436800000" iyz="0.00009700000"
@@ -69,5 +70,6 @@
       <inertial>
         <origin xyz="0.00002 -0.00197 -0.00059" rpy="0.00000 0.00000 0.00000"/>
-        <mass value="0.40931"/>
+        <!-- <mass value="0.40931"/> -->
+        <mass value="0.30931"/>
         <inertia ixx="0.00010700000" ixy="0.00000000000" ixz="0.00000000000"
                  iyy="0.00014100000" iyz="-0.00000000000"
@@ -102,4 +104,5 @@
     </joint>
     <link name="${name}_${side}_7_link">
+      <!-- WRONG VALUES
       <inertial>
         <origin xyz="-0.00089 0.00365 -0.07824" rpy="0.00000 0.00000 0.00000"/>
@@ -108,4 +111,12 @@
                  iyy="0.00146400000" iyz="0.00001200000"
                  izz="0.00090300000"/>
+      </inertial>
+      -->
+      <inertial>
+        <origin xyz="0.007525 0.001378 -0.024630" rpy="0.00000 0.00000 0.00000"/>
+        <mass value="0.308441"/>
+        <inertia ixx="0.000309" ixy="0.000002" ixz="-0.000002"
+                 iyy="0.000219" iyz="0.000012"
+                 izz="0.000176"/>
       </inertial>
       <visual>

File: talos_description/urdf/gripper/gripper_v2.urdf.xacro (robot description, xacro)
@@ -5,5 +5,5 @@
   <xacro:include filename="$(find talos_description)/urdf/gripper/gripper.transmission.xacro" />
   <xacro:include filename="$(find talos_description)/urdf/gripper/gripper.gazebo.xacro" />
-  <xacro:macro name="talos_gripper" params="name parent">
+  <xacro:macro name="talos_gripper" params="name parent reflect">
            <link name="${name}_base_link">
               <inertial>
@@ -32,5 +32,5 @@
               <child link="${name}_base_link"/>
               <origin xyz="0.00000 0.00000 -0.02875"
-                      rpy="${0.00000 * deg_to_rad} ${0.00000 * deg_to_rad} ${90.00000 * deg_to_rad}"/>
+                      rpy="${0.00000 * deg_to_rad} ${0.00000 * deg_to_rad} ${(reflect -1)* 90.000000 * deg_to_rad}"/>
               <axis xyz="0 0 0" />
             </joint>
