Commit message: Foot collision object can now be specified as an option.

File: talos_description/robots/talos_full_no_grippers.urdf.xacro (robot description, xacro)
@@ -16,4 +16,5 @@
   <xacro:include filename="$(find talos_description)/urdf/sensors/ftsensor.urdf.xacro" />
   <xacro:include filename="$(find talos_description)/urdf/leg/leg.urdf.xacro" />
+  <xacro:include filename="$(find talos_description)/urdf/leg/foot_collision_$(arg foot_collision).urdf.xacro" />
   <xacro:talos_torso name="torso" />
   <xacro:talos_head name="head" parent="torso_2_link"/>

File: talos_description/robots/talos_full_v1.urdf.xacro (robot description, xacro)
@@ -18,4 +18,5 @@
   <xacro:include filename="$(find talos_description)/urdf/gripper/gripper.urdf.xacro" />
   <xacro:include filename="$(find talos_description)/urdf/leg/leg.urdf.xacro" />
+  <xacro:include filename="$(find talos_description)/urdf/leg/foot_collision_$(arg foot_collision).urdf.xacro" />
   <xacro:talos_torso name="torso" />
   <xacro:talos_head name="head" parent="torso_2_link"/>

File: talos_description/robots/talos_full_v2.urdf.xacro (robot description, xacro)
@@ -18,4 +18,5 @@
   <xacro:include filename="$(find talos_description)/urdf/gripper/gripper.urdf.xacro" />
   <xacro:include filename="$(find talos_description)/urdf/leg/leg.urdf.xacro" />
+  <xacro:include filename="$(find talos_description)/urdf/leg/foot_collision_$(arg foot_collision).urdf.xacro" />
   <xacro:talos_torso name="torso" />
   <xacro:talos_head name="head" parent="torso_2_link"/>

File: talos_description/robots/talos_lower_body.urdf.xacro (robot description, xacro)
@@ -13,4 +13,5 @@
   <xacro:include filename="$(find talos_description)/urdf/sensors/ftsensor.urdf.xacro" />
   <xacro:include filename="$(find talos_description)/urdf/leg/leg.urdf.xacro" />
+  <xacro:include filename="$(find talos_description)/urdf/leg/foot_collision_$(arg foot_collision).urdf.xacro" />
     <!--************************-->
     <!--        BASE_LINK       -->

File: talos_description/urdf/leg/leg.urdf.xacro (robot description, xacro)
@@ -185,18 +185,5 @@
         <material name="Grey" />
       </visual>
-      <!--
-      <collision>
-        <origin xyz="0 0 0" rpy="0 0 0" />
-        <geometry>
-          <mesh filename="package://talos_description/meshes/v2/ankle_X_collision.stl" scale="1 ${reflect*1} 1"/>
-        </geometry>
-      </collision>
-      -->
-       <collision>
-        <origin xyz="0 0 -0.1" rpy="0 0 0" />
-        <geometry>
-           <box size="0.21 0.13 0.02"/>
-        </geometry>
-      </collision>
+      <xacro:talos_foot_collision />
     </link>
     <joint name="leg_${prefix}_6_joint" type="revolute">
@@ -298,4 +285,4 @@
     <material>Gazebo/White</material>
   </gazebo>
- </xacro:macro>
+  </xacro:macro>
 </robot>

Commit message: Fix issues when replacing tor with talos

File: talos_description/robots/talos_full_no_grippers.urdf.xacro (robot description, xacro)
@@ -24,5 +24,5 @@
   <xacro:talos_leg prefix="left"  reflect="1" />
   <xacro:talos_leg prefix="right" reflect="-1" />
-  <!-- Generic simulatalos_gazebo plugins -->
+  <!-- Generic simulator_gazebo plugins -->
   <xacro:include filename="$(find talos_description)/gazebo/gazebo.urdf.xacro" />
   <!-- Materials for visualization -->

File: talos_description/robots/talos_full_v1.urdf.xacro (robot description, xacro)
@@ -28,5 +28,5 @@
   <xacro:talos_leg prefix="left"  reflect="1" />
   <xacro:talos_leg prefix="right" reflect="-1" />
-  <!-- Generic simulatalos_gazebo plugins -->
+  <!-- Generic simulator_gazebo plugins -->
   <xacro:include filename="$(find talos_description)/gazebo/gazebo.urdf.xacro" />
   <!-- Materials for visualization -->

File: talos_description/robots/talos_full_v2.urdf.xacro (robot description, xacro)
@@ -28,5 +28,5 @@
   <xacro:talos_leg prefix="left"  reflect="1" />
   <xacro:talos_leg prefix="right" reflect="-1" />
-  <!-- Generic simulatalos_gazebo plugins -->
+  <!-- Generic simulator_gazebo plugins -->
   <xacro:include filename="$(find talos_description)/gazebo/gazebo.urdf.xacro" />
   <!-- Materials for visualization -->

File: talos_description/robots/talos_lower_body.urdf.xacro (robot description, xacro)
@@ -40,5 +40,5 @@
   <xacro:talos_leg prefix="left"  reflect="1" />
   <xacro:talos_leg prefix="right" reflect="-1" />
-  <!-- Generic simulatalos_gazebo plugins -->
+  <!-- Generic simulator_gazebo plugins -->
   <xacro:include filename="$(find talos_description)/gazebo/gazebo.urdf.xacro" />
   <!-- Materials for visualization -->

File: talos_description/urdf/sensors/ftsensor.gazebo.xacro (robot description, xacro)
@@ -8,5 +8,5 @@
 -->
 <robot name="reemc" xmlns:xacro="http://ros.org/wiki/xacro">
-<xacro:macro name="reemc_force_talosque_sensor" params="name update_rate">
+<xacro:macro name="reemc_force_torque_sensor" params="name update_rate">
   <gazebo reference="${name}">
     <sensor name="${name}_contact_sensor" type="contact">

File: talos_description/urdf/sensors/openni.gazebo.xacro (robot description, xacro)
@@ -33,9 +33,9 @@
           <frameName>${frame_name}</frameName>
           <pointCloudCutoff>0.5</pointCloudCutoff>
-          <distalostionK1>0.00000001</distalostionK1>
-          <distalostionK2>0.00000001</distalostionK2>
-          <distalostionK3>0.00000001</distalostionK3>
-          <distalostionT1>0.00000001</distalostionT1>
-          <distalostionT2>0.00000001</distalostionT2>
+          <distortionK1>0.00000001</distortionK1>
+          <distortionK2>0.00000001</distortionK2>
+          <distortionK3>0.00000001</distortionK3>
+          <distortionT1>0.00000001</distortionT1>
+          <distortionT2>0.00000001</distortionT2>
         </controller:gazebo_ros_openni_kinect>
       </sensor:camera>
@@ -61,9 +61,9 @@
           <frameName>${frame_name}</frameName>
           <pointCloudCutoff>0.5</pointCloudCutoff>
-          <distalostionK1>0.00000001</distalostionK1>
-          <distalostionK2>0.00000001</distalostionK2>
-          <distalostionK3>0.00000001</distalostionK3>
-          <distalostionT1>0.00000001</distalostionT1>
-          <distalostionT2>0.00000001</distalostionT2>
+          <distortionK1>0.00000001</distortionK1>
+          <distortionK2>0.00000001</distortionK2>
+          <distortionK3>0.00000001</distortionK3>
+          <distortionT1>0.00000001</distortionT1>
+          <distortionT2>0.00000001</distortionT2>
         </controller:gazebo_ros_openni_kinect>
       </sensor:camera>

File: talos_description/urdf/sensors/orbbec_astra_pro.gazebo.xacro (robot description, xacro)
@@ -43,9 +43,9 @@
           <pointCloudCutoff>0.45</pointCloudCutoff>
           <rangeMax>10.0</rangeMax>
-          <distalostionK1>0.00000001</distalostionK1>
-          <distalostionK2>0.00000001</distalostionK2>
-          <distalostionK3>0.00000001</distalostionK3>
-          <distalostionT1>0.00000001</distalostionT1>
-          <distalostionT2>0.00000001</distalostionT2>
+          <distortionK1>0.00000001</distortionK1>
+          <distortionK2>0.00000001</distortionK2>
+          <distortionK3>0.00000001</distortionK3>
+          <distortionT1>0.00000001</distortionT1>
+          <distortionT2>0.00000001</distortionT2>
         </plugin>
       </sensor>
@@ -81,9 +81,9 @@
           <frameName>${name}_optical_frame</frameName>
           <hackBaseline>0.07</hackBaseline>
-          <distalostionK1>0.00000001</distalostionK1>
-          <distalostionK2>0.00000001</distalostionK2>
-          <distalostionK3>0.00000001</distalostionK3>
-          <distalostionT1>0.00000001</distalostionT1>
-          <distalostionT2>0.00000001</distalostionT2>
+          <distortionK1>0.00000001</distortionK1>
+          <distortionK2>0.00000001</distortionK2>
+          <distortionK3>0.00000001</distortionK3>
+          <distortionT1>0.00000001</distortionT1>
+          <distortionT2>0.00000001</distortionT2>
         </plugin>
       </sensor>

File: talos_description/urdf/sensors/xtion_pro_live.gazebo.xacro (robot description, xacro)
@@ -45,9 +45,9 @@
           <pointCloudCutoff>0.45</pointCloudCutoff>
           <rangeMax>10.0</rangeMax>
-          <distalostionK1>0.00000001</distalostionK1>
-          <distalostionK2>0.00000001</distalostionK2>
-          <distalostionK3>0.00000001</distalostionK3>
-          <distalostionT1>0.00000001</distalostionT1>
-          <distalostionT2>0.00000001</distalostionT2>
+          <distortionK1>0.00000001</distortionK1>
+          <distortionK2>0.00000001</distortionK2>
+          <distortionK3>0.00000001</distortionK3>
+          <distortionT1>0.00000001</distortionT1>
+          <distortionT2>0.00000001</distortionT2>
         </plugin>
       </sensor>
@@ -78,9 +78,9 @@
           <pointCloudCutoff>0.45</pointCloudCutoff>
           <rangeMax>10.0</rangeMax>
-          <distalostionK1>0.00000001</distalostionK1>
-          <distalostionK2>0.00000001</distalostionK2>
-          <distalostionK3>0.00000001</distalostionK3>
-          <distalostionT1>0.00000001</distalostionT1>
-          <distalostionT2>0.00000001</distalostionT2>
+          <distortionK1>0.00000001</distortionK1>
+          <distortionK2>0.00000001</distortionK2>
+          <distortionK3>0.00000001</distortionK3>
+          <distortionT1>0.00000001</distortionT1>
+          <distortionT2>0.00000001</distortionT2>
         </plugin>
       </sensor>
