Commit message: Inertials in a separate package. [dubnium compatibility is lost!]

File: talos_description/robots/talos_full_no_grippers.urdf.xacro (robot description, xacro)
@@ -20,4 +20,5 @@
   <xacro:include filename="$(find talos_description)/urdf/leg/leg.urdf.xacro" />
   <xacro:include filename="$(find talos_description)/urdf/leg/foot_collision_$(arg foot_collision).urdf.xacro" />
+  <xacro:include filename="$(find talos_description_inertial)/urdf/inertial.xacro" />
   <xacro:talos_torso name="torso" />
   <xacro:if value="$(arg enable_crane)">

File: talos_description/robots/talos_full_v1.urdf.xacro (robot description, xacro)
@@ -22,4 +22,5 @@
   <xacro:include filename="$(find talos_description)/urdf/leg/leg.urdf.xacro" />
   <xacro:include filename="$(find talos_description)/urdf/leg/foot_collision_$(arg foot_collision).urdf.xacro" />
+  <xacro:include filename="$(find talos_description_inertial)/urdf/inertial.xacro" />
   <xacro:talos_torso name="torso" />
   <xacro:if value="$(arg enable_crane)">

File: talos_description/robots/talos_full_v2.urdf.xacro (robot description, xacro)
@@ -22,4 +22,5 @@
   <xacro:include filename="$(find talos_description)/urdf/leg/leg.urdf.xacro" />
   <xacro:include filename="$(find talos_description)/urdf/leg/foot_collision_$(arg foot_collision).urdf.xacro" />
+  <xacro:include filename="$(find talos_description_inertial)/urdf/inertial.xacro" />
   <xacro:talos_torso name="torso" />
   <xacro:if value="$(arg enable_crane)">

File: talos_description/robots/talos_lower_body.urdf.xacro (robot description, xacro)
@@ -14,4 +14,5 @@
   <xacro:include filename="$(find talos_description)/urdf/leg/leg.urdf.xacro" />
   <xacro:include filename="$(find talos_description)/urdf/leg/foot_collision_$(arg foot_collision).urdf.xacro" />
+  <xacro:include filename="$(find talos_description_inertial)/urdf/inertial.xacro" />
     <!--************************-->
     <!--        BASE_LINK       -->

File: talos_description/urdf/arm/arm_v2.urdf.xacro (robot description, xacro)
@@ -29,11 +29,5 @@
     <!--************************-->
     <link name="${name}_${side}_1_link">
-      <inertial>
-        <origin xyz="-0.00027620000 ${reflect*0.10060223000} 0.04437419000" rpy="0.00000000000 0.00000000000 0.00000000000"/>
-        <mass value="2.71456700000"/>
-        <inertia ixx="0.01237818683" ixy="${reflect*-0.00003625571}" ixz="0.00007144720"
-                 iyy="0.00419137200" iyz="${reflect*-0.00023639064}"
-                 izz="0.01358161109"/>
-      </inertial>
+      <xacro:call macro="${name}_${side}_1_link_inertial" />
       <visual>
         <origin xyz="0 0 0" rpy="0 0 0" />
@@ -66,11 +60,5 @@
     </joint>
     <link name="${name}_${side}_2_link">
-      <inertial>
-        <origin xyz="0.01438831000 ${reflect*0.00092938000} -0.08684268000" rpy="0.00000000000 0.00000000000 0.00000000000"/>
-        <mass value="2.42508600000"/>
-        <inertia ixx="0.01297822101" ixy="${reflect*0.00001208791}" ixz="-0.00320370433"
-                 iyy="0.01380870278" iyz="${reflect*-0.00012770059}"
-                 izz="0.00478856621"/>
-      </inertial>
+      <xacro:call macro="${name}_${side}_2_link_inertial" />
       <visual>
         <origin xyz="0 0 0" rpy="0 0 0" />
@@ -101,11 +89,5 @@
     </joint>
     <link name="${name}_${side}_3_link">
-      <inertial>
-        <origin xyz="0.01360840000 ${reflect*0.01241619000} -0.24990040000" rpy="0.00000000000 0.00000000000 0.00000000000"/>
-        <mass value="2.20874100000"/>
-        <inertia ixx="0.00718831493" ixy="${reflect*-0.00011563551}" ixz="0.00075969733"
-                 iyy="0.00693528503" iyz="${reflect*0.00042134743}"
-                 izz="0.00388359007"/>
-      </inertial>
+      <xacro:call macro="${name}_${side}_3_link_inertial" />
       <visual>
         <origin xyz="0 0 0" rpy="0 0 0" />
@@ -139,11 +121,5 @@
     <!--************************-->
     <link name="${name}_${side}_4_link">
-      <inertial>
-        <origin xyz="-0.00742138000 ${reflect*-0.02138950000} -0.03312656000" rpy="0.00000000000 0.00000000000 0.00000000000"/>
-        <mass value="0.87734600000"/>
-        <inertia ixx="0.00251207716" ixy="${reflect*0.00010070062}" ixz="-0.00032788214"
-            iyy="0.00275869324" iyz="${reflect*0.00040022227}"
-                 izz="0.00120735959"/>
-      </inertial>
+      <xacro:call macro="${name}_${side}_4_link_inertial" />
       <visual>
         <origin xyz="0 0 0" rpy="0 0 0" />

File: talos_description/urdf/arm/wrist.urdf.xacro (robot description, xacro)
@@ -26,11 +26,5 @@
     <!--************************-->
     <link name="${name}_${side}_5_link">
-      <inertial>
-        <origin xyz="-0.00006000000 ${reflect*0.00326200000} 0.07962500000" rpy="0.00000000000 0.00000000000 0.00000000000"/>
-        <mass value="1.87792300000"/>
-        <inertia ixx="0.00349507283" ixy="${reflect*0.00001265489}" ixz="0.00001038286"
-                 iyy="0.00436830072" iyz="${reflect*-0.00009736042}"
-                 izz="0.00228263370"/>
-      </inertial>
+      <xacro:call macro="${name}_${side}_5_link_inertial" />
       <visual>
         <origin xyz="0 0 0" rpy="0 0 0" />
@@ -61,11 +55,5 @@
     </joint>
     <link name="${name}_${side}_6_link">
-      <inertial>
-        <origin xyz="0.00002100000 ${reflect*-0.00196500000} -0.00059100000" rpy="0.00000000000 0.00000000000 0.00000000000"/>
-        <mass value="0.40931000000"/>
-        <inertia ixx="0.00010700023" ixy="${reflect*-0.00000008899}" ixz="-0.00000004392"
-                 iyy="0.00014101316" iyz="${reflect*0.00000041702}"
-                 izz="0.00015398658"/>
-      </inertial>
+      <xacro:call macro="${name}_${side}_6_link_inertial" />
       <visual>
         <origin xyz="0 0 0" rpy="0 0 0" />
@@ -96,11 +84,5 @@
     </joint>
     <link name="${name}_${side}_7_link">
-      <inertial>
-        <origin xyz="0.00752500000 ${reflect*0.00137800000} -0.02463000000" rpy="0.00000000000 0.00000000000 0.00000000000"/>
-        <mass value="0.30844100000"/>
-        <inertia ixx="0.00030894317" ixy="${reflect*-0.00000158687}" ixz="0.00000173418"
-                 iyy="0.00021886181" iyz="${reflect*-0.00001221167}"
-                 izz="0.00017519492"/>
-      </inertial>
+      <xacro:call macro="${name}_${side}_7_link_inertial" />
       <visual>
         <origin xyz="0 0 0" rpy="0 0 0" />

File: talos_description/urdf/gripper/gripper.urdf.xacro (robot description, xacro)
@@ -6,12 +6,6 @@
   <xacro:include filename="$(find talos_description)/urdf/gripper/gripper.gazebo.xacro" />
   <xacro:macro name="talos_gripper" params="name parent reflect">
-           <link name="${name}_base_link">
-              <inertial>
-                <origin xyz="0.00002800000 0.00539400000 -0.02365400000" rpy="0.00000000000 0.00000000000 0.00000000000"/>
-                <mass value="0.63753400000"/>
-                <inertia ixx="0.00058496920" ixy="0.00000437159" ixz="-0.00001258900"
-                         iyy="0.00067076439" iyz="0.00002824361"
-                         izz="0.00085526645"/>
-              </inertial>
+            <link name="${name}_base_link">
+              <xacro:call macro="${name}_base_link_inertial" />
               <visual>
                 <origin xyz="0 0 0" rpy="0 0 0" />
@@ -36,11 +30,5 @@
             </joint>
             <link name="${name}_motor_double_link">
-              <inertial>
-                <origin xyz="0.01965400000 0.01857200000 -0.01199800000" rpy="0.00000000000 0.00000000000 0.00000000000"/>
-                <mass value="0.13435600000"/>
-                <inertia ixx="0.00013479919" ixy="0.00006184429" ixz="-0.00003079800"
-                         iyy="0.00019602207" iyz="0.00004707722"
-                         izz="0.00024217879"/>
-              </inertial>
+              <xacro:call macro="${name}_motor_double_link_inertial" />
               <visual>
                 <origin xyz="0 0 0" rpy="0 0 0" />
@@ -67,11 +55,5 @@
             </joint>
             <link name="${name}_inner_double_link">
-              <inertial>
-                <origin xyz="-0.01328300000 0.03685200000 -0.02315300000" rpy="0.00000000000 0.00000000000 0.00000000000"/>
-                <mass value="0.08798600000"/>
-                <inertia ixx="0.00007410642" ixy="-0.00000074773" ixz="0.00000101536"
-                         iyy="0.00012794180" iyz="0.00002504083"
-                         izz="0.00010495175"/>
-              </inertial>
+              <xacro:call macro="${name}_inner_double_link_inertial" />
               <visual>
                 <origin xyz="0 0 0" rpy="0 0 0" />
@@ -98,11 +80,5 @@
             </joint>
             <link name="${name}_fingertip_1_link">
-              <inertial>
-                <origin xyz="0.00000000000 0.00460400000 -0.00253700000" rpy="0.00000000000 0.00000000000 0.00000000000"/>
-                <mass value="0.02630100000"/>
-                <inertia ixx="0.00000800000" ixy="0.00000000000" ixz="0.00000000000"
-                         iyy="0.00000869179" iyz="-0.00000143612"
-                         izz="0.00000230820"/>
-              </inertial>
+              <xacro:call macro="${name}_fingertip_1_link_inertial" />
               <visual>
                 <origin xyz="0 0 0" rpy="0 0 0" />
@@ -129,11 +105,5 @@
             </joint>
             <link name="${name}_fingertip_2_link">
-              <inertial>
-                <origin xyz="0.00000000000 0.00460400000 -0.00253700000" rpy="0.00000000000 0.00000000000 0.00000000000"/>
-                <mass value="0.02630100000"/>
-                <inertia ixx="0.00000800000" ixy="0.00000000000" ixz="0.00000000000"
-                         iyy="0.00000869179" iyz="-0.00000143612"
-                         izz="0.00000230820"/>
-              </inertial>
+              <xacro:call macro="${name}_fingertip_2_link_inertial" />
               <visual>
                 <origin xyz="0 0 0" rpy="0 0 0" />
@@ -160,11 +130,5 @@
             </joint>
             <link name="${name}_motor_single_link">
-              <inertial>
-                <origin xyz="0.02523700000 -0.01123100000 -0.00815800000" rpy="0.00000000000 0.00000000000 0.00000000000"/>
-                <mass value="0.10792300000"/>
-                <inertia ixx="0.00008973662" ixy="-0.00004082027" ixz="-0.00001927099"
-                         iyy="0.00011957255" iyz="-0.00002873284"
-                         izz="0.00015469079"/>
-              </inertial>
+              <xacro:call macro="${name}_motor_single_link_inertial" />
               <visual>
                 <origin xyz="0 0 0" rpy="0 0 0" />
@@ -191,11 +155,5 @@
             </joint>
             <link name="${name}_inner_single_link">
-              <inertial>
-                <origin xyz="0.00000000000 -0.03456500000 -0.02141200000" rpy="0.00000000000 0.00000000000 0.00000000000"/>
-                <mass value="0.04717700000"/>
-                <inertia ixx="0.00004199818" ixy="0.00000013418" ixz="0.00000019358"
-                         iyy="0.00003231338" iyz="-0.00001509136"
-                         izz="0.00002168842"/>
-              </inertial>
+              <xacro:call macro="${name}_inner_single_link_inertial" />
               <visual>
                 <origin xyz="0 0 0" rpy="0 0 0" />
@@ -222,11 +180,5 @@
             </joint>
             <link name="${name}_fingertip_3_link">
-              <inertial>
-                <origin xyz="0.00000000000 0.00460400000 -0.00253700000" rpy="0.00000000000 0.00000000000 0.00000000000"/>
-                <mass value="0.02630100000"/>
-                <inertia ixx="0.00000800000" ixy="0.00000000000" ixz="0.00000000000"
-                         iyy="0.00000869179" iyz="-0.00000143612"
-                         izz="0.00000230820"/>
-              </inertial>
+              <xacro:call macro="${name}_fingertip_3_link_inertial" />
               <visual>
                 <origin xyz="0 0 0" rpy="0 0 0" />
@@ -261,4 +213,4 @@
         <xacro:gripper_virtual_transmission name="${name}_motor_single" reduction="1.0"/>
         <xacro:gripper_virtual_transmission name="${name}_fingertip_3" reduction="1.0"/> -->
- </xacro:macro>
+  </xacro:macro>
 </robot>

File: talos_description/urdf/head/head.urdf.xacro (robot description, xacro)
@@ -23,11 +23,5 @@
   <xacro:macro name="talos_head_1" params="name parent">
     <link name="${name}_link">
-      <inertial>
-        <origin xyz="-0.00157211000 -0.00157919000 0.02175767000" rpy="0.00000000000 0.00000000000 0.00000000000"/>
-        <mass value="0.73746000000"/>
-        <inertia ixx="0.00224878584" ixy="0.00000469375" ixz="0.00008555570"
-                 iyy="0.00111158492" iyz="-0.00004132536"
-                 izz="0.00205225921"/>
-      </inertial>
+      <xacro:call macro="${name}_link_inertial" />
       <visual>
         <origin xyz="0 0 0" rpy="0 0 0" />
@@ -73,11 +67,5 @@
   <xacro:macro name="talos_head_2" params="name parent">
     <link name="${name}_link">
-      <inertial>
-        <origin xyz="0.01002657000 0.00005218000 0.14136068000" rpy="0.00000000000 0.00000000000 0.00000000000"/>
-        <mass value="1.44395400000"/>
-        <inertia ixx="0.01084624339" ixy="0.00001050889" ixz="0.00041594252"
-                 iyy="0.01095691760" iyz="0.00002367831"
-                 izz="0.00571698895"/>
-      </inertial>
+      <xacro:call macro="${name}_link_inertial" />
       <visual>
         <origin xyz="0 0 0" rpy="0 0 0" />

File: talos_description/urdf/leg/leg.urdf.xacro (robot description, xacro)
@@ -11,11 +11,5 @@
     <!-- Joint hip_z (mesh link) : child link hip_x -> parent link base_link -->
     <link name="leg_${prefix}_1_link">
-      <inertial>
-        <origin xyz="0.02247868000 ${reflect*0.00106736000} 0.03130665000" rpy="0.00000000000 0.00000000000 0.00000000000"/>
-        <mass value="1.84559100000"/>
-        <inertia ixx="0.00541533521" ixy="${reflect*-0.00015428714}" ixz="0.00131612622"
-                 iyy="0.00848624936" iyz="${reflect*-0.00001906103}"
-                 izz="0.00474512541"/>
-      </inertial>
+      <xacro:call macro="leg_${prefix}_1_link_inertial" />
       <visual>
         <origin rpy="0 0 0" xyz="0 0 0"/>
@@ -43,11 +37,5 @@
     <!-- Joint hip_x (mesh link) : child link hip_y -> parent link hip_z -->
     <link name="leg_${prefix}_2_link">
-      <inertial>
-        <origin xyz="-0.00704703000 ${reflect*0.02592659000} 0.00273385000" rpy="0.00000000000 0.00000000000 0.00000000000"/>
-        <mass value="1.49095200000"/>
-        <inertia ixx="0.00497152259" ixy="${reflect*-0.00013113580}" ixz="-0.00000486648"
-                 iyy="0.00190550993" iyz="${reflect*0.00004585381}"
-                 izz="0.00474289754"/>
-      </inertial>
+      <xacro:call macro="leg_${prefix}_2_link_inertial" />
       <visual>
         <origin xyz="0 0 0.0" rpy="0  0  0" />
@@ -75,11 +63,5 @@
     <!-- Joint hip_y (mesh link) : child link knee -> parent link hip_x -->
     <link name="leg_${prefix}_3_link">
-      <inertial>
-        <origin xyz="0.00585230000 ${reflect*0.06369670000} -0.18339564000" rpy="0.00000000000 0.00000000000 0.00000000000"/>
-        <mass value="6.23987100000"/>
-        <inertia ixx="0.15337403915" ixy="${reflect*0.00068913396}" ixz="0.00168034366"
-                 iyy="0.13648139346" iyz="${reflect*-0.02187635445}"
-                 izz="0.03001594885"/>
-      </inertial>
+      <xacro:call macro="leg_${prefix}_3_link_inertial" />
       <visual>
         <origin rpy="0 0 0" xyz="0 0 0"/>
@@ -107,11 +89,5 @@
     <!-- Joint knee (mesh link) : child link ankle_y -> parent link hip_y -->
     <link name="leg_${prefix}_4_link">
-      <inertial>
-        <origin xyz="0.01317717000 ${reflect*0.02917508000} -0.11594602000" rpy="0.00000000000 0.00000000000 0.00000000000"/>
-        <mass value="3.75995100000"/>
-        <inertia ixx="0.04287677484" ixy="${reflect*0.00043705397}" ixz="0.00078292368"
-                 iyy="0.03598906971" iyz="${reflect*0.00037717694}"
-                 izz="0.01364791564"/>
-      </inertial>
+      <xacro:call macro="leg_${prefix}_4_link_inertial" />
       <visual>
         <origin rpy="0 0 0" xyz="0 0 0"/>
@@ -140,11 +116,5 @@
     <link name="leg_${prefix}_5_link">
       <!-- XXX AS: this link has moving lever and inertial parameters should slightly vary depending on configuration. XXX -->
-      <inertial>
-        <origin xyz="-0.01400838000 ${reflect*0.04180064000} 0.03820186000" rpy="0.00000000000 0.00000000000 0.00000000000"/>
-        <mass value="1.29096000000"/>
-        <inertia ixx="0.01143430819" ixy="${reflect*0.00096978273}" ixz="0.00039976581"
-                 iyy="0.00888974312" iyz="${reflect*-0.00277808667}"
-                 izz="0.00506373875"/>
-      </inertial>
+      <xacro:call macro="leg_${prefix}_5_link_inertial" />
       <visual>
         <origin xyz="0 0 0.0" rpy="0 0 0" />
@@ -172,11 +142,5 @@
     <!-- Joint ankle_x (mesh link) : child link None -> parent link ankle_y -->
     <link name="leg_${prefix}_6_link">
-      <inertial>
-        <origin xyz="-0.02034668000 ${reflect*-0.00051514000} -0.05987428000" rpy="0.00000000000 0.00000000000 0.00000000000"/>
-        <mass value="1.59777300000"/>
-        <inertia ixx="0.00439027267" ixy="${reflect*-0.00006743674}" ixz="0.00113816363"
-                 iyy="0.00743063029" iyz="${reflect*0.00003943143}"
-                 izz="0.00550906699"/>
-      </inertial>
+      <xacro:call macro="leg_${prefix}_6_link_inertial" />
       <visual>
         <origin rpy="0 0 0" xyz="0 0 0"/>
@@ -199,9 +163,5 @@
   <!-- from here is copy paste -->
     <link name="${prefix}_sole_link">
-      <inertial>
-        <origin xyz="0.0 0.0 0.0" rpy="0 0 0"/>
-        <mass value="0.01" />
-        <inertia ixx="0.0001"  ixy="0.0"  ixz="0.0" iyy="0.0001" iyz="0.0" izz="0.0001" />
-      </inertial>
+      <xacro:call macro="${prefix}_sole_link_inertial" />
     </link>
     <joint name="leg_${prefix}_sole_fix_joint" type="fixed">

File: talos_description/urdf/sensors/ftsensor.urdf.xacro (robot description, xacro)
@@ -13,11 +13,5 @@
     <!--************************-->
     <link name="${name}_${side}_ft_link">
-      <inertial>
-        <mass value="0.09500000000" />
-        <inertia ixx="0.00001108502" ixy="0.00000099077" ixz="-0.00000023811"
-                 iyy="0.00001092725" iyz="0.00000023137"
-                 izz="0.00001898772"/>
-        <origin xyz="-0.00100100000 0.00099500000 -0.00810800000" rpy="0.00000000000 0.00000000000 0.00000000000"/>
-      </inertial>
+      <xacro:call macro="${name}_${side}_ft_link_inertial" />
       <visual>
         <origin xyz="0 0 0" rpy="0 0 0" />
@@ -43,8 +37,5 @@
     <!--***********************-->
     <link name="${name}_${side}_ft_tool_link">
-      <inertial>
-        <mass value="0.001" />
-        <inertia ixx="0.0" ixy="0.0" ixz="0.0" iyy="0.0" iyz="0.0" izz="0.0" />
-      </inertial>
+      <xacro:call macro="${name}_${side}_ft_tool_link_inertial" />
       <visual>
         <origin xyz="0.0 0 0" rpy="0 ${0.0 * deg_to_rad} 0" />

File: talos_description/urdf/sensors/imu.urdf.xacro (robot description, xacro)
@@ -10,9 +10,5 @@
   <xacro:macro name="talos_imu" params="name parent update_rate *origin">
     <link name="${name}_link">
-      <inertial>
-        <mass value="0.01"/>
-        <origin xyz="0 0 0"/>
-        <inertia ixx="0.000001" ixy="0" ixz="0" iyy="0.000001" iyz="0" izz="0.000001"/>
-      </inertial>
+      <xacro:call macro="${name}_link_inertial" />
       <visual>
         <origin rpy="0 0 0" xyz="0 0 0"/>

File: talos_description/urdf/sensors/orbbec_astra_pro.urdf.xacro (robot description, xacro)
@@ -31,11 +31,5 @@
     <link name="${name}_link">
       <!-- inertia tensor computed analytically for a solid cuboid -->
-      <inertial>
-        <mass value="0.01" />
-        <origin xyz="-0.01 0.0025 0" rpy="0 0 0"/>
-        <inertia ixx="0.000030"  ixy="0.0"  ixz="0.0"
-                 iyy="0.000002"  iyz="0.0"
-                 izz="0.000030" />
-      </inertial>
+      <xacro:call macro="${name}_link_inertial" />
       <visual>
         <origin xyz="0 0 0" rpy="0 0 0"/>
@@ -60,11 +54,5 @@
     </joint>
     <link name="${name}_optical_frame">
-      <inertial>
-        <mass value="0.01" />
-        <origin xyz="0 0 0" rpy="0 0 0"/>
-        <inertia ixx="0.0"  ixy="0.0"  ixz="0.0"
-                 iyy="0.0"  iyz="0.0"
-                 izz="0.0" />
-      </inertial>
+      <xacro:call macro="${name}_optical_frame_inertial" />
     </link>
     <!-- frames of the depth sensor -->

File: talos_description/urdf/sensors/xtion_pro_live.urdf.xacro (robot description, xacro)
@@ -25,5 +25,5 @@
     <!-- base link -->
     <joint name="${name}_joint" type="fixed">
-      <xacro:insert_block name="origin" />
+      <xacro:call macro="origin" />
       <parent link="${parent}"/>
       <child link="${name}_link"/>
@@ -73,5 +73,5 @@
     <!-- Xtion IR sensor frame -->
     <joint name="${name}_ir_optical_frame_joint" type="fixed">
-      <xacro:insert_block name="calibration_origin" /> <!-- macro argument -->
+      <xacro:call macro="calibration_origin" /> <!-- macro argument -->
       <parent link="${name}_ir_link"/>
       <child link="${name}_ir_optical_frame"/>
@@ -107,5 +107,5 @@
     <!-- Xtion RGB sensor frame -->
     <joint name="${name}_rgb_optical_frame_joint" type="fixed">
-      <xacro:insert_block name="calibration_origin" /> <!-- macro argument -->
+      <xacro:call macro="calibration_origin" /> <!-- macro argument -->
       <parent link="${name}_rgb_link"/>
       <child link="${name}_rgb_optical_frame"/>
