Commit message: Inertials in a separate package. [dubnium compatibility is lost!]

File: talos_description/urdf/torso/torso.urdf.xacro (robot description, xacro)
@@ -21,11 +21,5 @@
     <!--************************-->
     <link name="${name}_2_link">
-      <inertial>
-        <origin xyz="-0.04635630000 -0.00099023000 0.14528050000" rpy="0.00000000000 0.00000000000 0.00000000000"/>
-        <mass value="16.97403000000"/>
-        <inertia ixx="0.44372633826" ixy="0.00069132133" ixz="-0.01218206353"
-                 iyy="0.29985760680" iyz="-0.00019623338"
-                 izz="0.32201554742"/>
-      </inertial>
+      <xacro:call macro="${name}_2_link_inertial" />
       <visual>
         <origin xyz="0 0 0" rpy="0 0 0" />
@@ -46,11 +40,5 @@
     <!--************************-->
     <link name="${name}_1_link">
-      <inertial>
-        <origin xyz="0.00078223000 0.00003528000 -0.01782457000" rpy="0.00000000000 0.00000000000 0.00000000000"/>
-        <mass value="2.29465800000"/>
-        <inertia ixx="0.00638508087" ixy="-0.00000007107" ixz="-0.00003065592"
-                 iyy="0.00410256102" iyz="-0.00000146946"
-                 izz="0.00622968815"/>
-      </inertial>
+      <xacro:call macro="${name}_1_link_inertial" />
       <visual>
         <origin xyz="0 0 0" rpy="0 0 0" />
@@ -86,11 +74,5 @@
     <!--************************-->
     <link name="base_link">
-      <inertial>
-        <origin xyz="-0.05709419000 0.00153054000 -0.07625210000" rpy="0.00000000000 0.00000000000 0.00000000000"/>
-        <mass value="15.36284000000"/>
-        <inertia ixx="0.20105075811" ixy="0.00023244734" ixz="0.00401677280"
-                 iyy="0.08411496729" iyz="-0.00087206649"
-                 izz="0.23189084140"/>
-      </inertial>
+      <xacro:call macro="base_link_inertial" />
       <visual>
         <origin xyz="0 0 0" rpy="0 0 0" />
