Commit message: merge talos versions, add tests.

File: talos_description/robots/talos_full_v1.urdf.xacro (robot description, xacro)
@@ -11,32 +11,5 @@
         xmlns:controller="http://playerstage.sourceforge.net/gazebo/xmlschema/#controller"
         xmlns:interface="http://playerstage.sourceforge.net/gazebo/xmlschema/#interface">
-  <xacro:if value="$(arg enable_crane)">
-    <xacro:include filename="$(find talos_description)/urdf/crane/crane.urdf.xacro" />
-  </xacro:if>
-  <xacro:include filename="$(find talos_description)/urdf/torso/torso.urdf.xacro" />
-  <xacro:include filename="$(find talos_description)/urdf/head/head.urdf.xacro" />
-  <!--arm_v1 loadded because of the different joint range for 1st DoF-->
-  <xacro:include filename="$(find talos_description)/urdf/arm/arm_v1.urdf.xacro" />
-  <xacro:include filename="$(find talos_description)/urdf/sensors/ftsensor.urdf.xacro" />
-  <xacro:include filename="$(find talos_description)/urdf/gripper/gripper.urdf.xacro" />
-  <xacro:include filename="$(find talos_description)/urdf/leg/leg.urdf.xacro" />
-  <xacro:include filename="$(find talos_description)/urdf/leg/foot_collision_$(arg foot_collision).urdf.xacro" />
-  <xacro:include filename="$(find talos_description_inertial)/urdf/inertial.xacro" />
-  <xacro:talos_torso name="torso" />
-  <xacro:if value="$(arg enable_crane)">
-    <xacro:crane parent="torso_2_link"/>
-  </xacro:if>
-  <xacro:talos_head name="head" parent="torso_2_link"/>
-  <xacro:talos_arm name="arm" parent="torso_2_link" side="left" reflect="1"/>
-  <xacro:talos_arm name="arm" parent="torso_2_link" side="right" reflect="-1"/>
-  <xacro:ft_sensor name="wrist" parent="arm_right_7_link" side="right" reflect="1"  />
-  <xacro:ft_sensor name="wrist" parent="arm_left_7_link"  side="left"  reflect="-1" />
-  <xacro:talos_gripper name="gripper_left" parent="wrist_left_ft_tool_link" reflect="1" />
-  <xacro:talos_gripper name="gripper_right" parent="wrist_right_ft_tool_link" reflect="-1" />
-  <xacro:talos_leg prefix="left"  reflect="1" />
-  <xacro:talos_leg prefix="right" reflect="-1" />
-  <!-- Generic simulator_gazebo plugins -->
-  <xacro:include filename="$(find talos_description)/gazebo/gazebo.urdf.xacro" />
-  <!-- Materials for visualization -->
-  <xacro:include filename="$(find talos_description)/urdf/materials.urdf.xacro" />
+  <xacro:include filename="$(find talos_description)/urdf/arm/arm_specifics_v1.urdf.xacro" />
+  <xacro:include filename="$(find talos_description)/urdf/talos_full_common.urdf.xacro" />
 </robot>

File: talos_description/robots/talos_full_v2.urdf.xacro (robot description, xacro)
@@ -11,32 +11,5 @@
         xmlns:controller="http://playerstage.sourceforge.net/gazebo/xmlschema/#controller"
         xmlns:interface="http://playerstage.sourceforge.net/gazebo/xmlschema/#interface">
-  <xacro:if value="$(arg enable_crane)">
-    <xacro:include filename="$(find talos_description)/urdf/crane/crane.urdf.xacro" />
-  </xacro:if>
-  <xacro:include filename="$(find talos_description)/urdf/torso/torso.urdf.xacro" />
-  <xacro:include filename="$(find talos_description)/urdf/head/head.urdf.xacro" />
-  <!--arm_v1 loadded because of the different joint range for 1st DoF-->
-  <xacro:include filename="$(find talos_description)/urdf/arm/arm_v2.urdf.xacro" />
-  <xacro:include filename="$(find talos_description)/urdf/sensors/ftsensor.urdf.xacro" />
-  <xacro:include filename="$(find talos_description)/urdf/gripper/gripper.urdf.xacro" />
-  <xacro:include filename="$(find talos_description)/urdf/leg/leg.urdf.xacro" />
-  <xacro:include filename="$(find talos_description)/urdf/leg/foot_collision_$(arg foot_collision).urdf.xacro" />
-  <xacro:include filename="$(find talos_description_inertial)/urdf/inertial.xacro" />
-  <xacro:talos_torso name="torso" />
-  <xacro:if value="$(arg enable_crane)">
-    <xacro:crane parent="torso_2_link"/>
-  </xacro:if>
-  <xacro:talos_head name="head" parent="torso_2_link"/>
-  <xacro:talos_arm name="arm" parent="torso_2_link" side="left" reflect="1"/>
-  <xacro:talos_arm name="arm" parent="torso_2_link" side="right" reflect="-1"/>
-  <xacro:ft_sensor name="wrist" parent="arm_right_7_link" side="right" reflect="1"  />
-  <xacro:ft_sensor name="wrist" parent="arm_left_7_link"  side="left"  reflect="-1" />
-  <xacro:talos_gripper name="gripper_left" parent="wrist_left_ft_tool_link" reflect="1" />
-  <xacro:talos_gripper name="gripper_right" parent="wrist_right_ft_tool_link" reflect="-1" />
-  <xacro:talos_leg prefix="left"  reflect="1" />
-  <xacro:talos_leg prefix="right" reflect="-1" />
-  <!-- Generic simulator_gazebo plugins -->
-  <xacro:include filename="$(find talos_description)/gazebo/gazebo.urdf.xacro" />
-  <!-- Materials for visualization -->
-  <xacro:include filename="$(find talos_description)/urdf/materials.urdf.xacro" />
+  <xacro:include filename="$(find talos_description)/urdf/arm/arm_specifics_v2.urdf.xacro" />
+  <xacro:include filename="$(find talos_description)/urdf/talos_full_common.urdf.xacro" />
 </robot>

File: talos_description/urdf/arm/arm.urdf.xacro (robot description, xacro)
@@ -29,12 +29,5 @@
     <!--************************-->
     <link name="${name}_${side}_1_link">
-      <inertial>
-        <origin xyz="-0.01346 ${reflect*0.09130} 0.04812" rpy="0.00000 0.00000 0.00000"/>
-        <!-- <mass value="1.52896"/> -->
-        <mass value="1.42896"/>
-        <inertia ixx="0.00555100000" ixy="-0.00073100000" ixz="0.00000800000"
-                 iyy="0.00167300000" iyz="-0.00006000000"
-                 izz="0.00582200000"/>
-      </inertial>
+      <xacro:call macro="${name}_${side}_1_link_inertial" />
       <visual>
         <origin xyz="0 0 0" rpy="0 0 0" />
@@ -57,5 +50,5 @@
               rpy="${0.0 * deg_to_rad} ${0.0 * deg_to_rad} ${0.0 * deg_to_rad}"/>
       <axis xyz="0 0 1" />
-      <limit lower="${(-60.0 - 30.0*reflect)* deg_to_rad}" upper="${(60.0 - 30.0*reflect)* deg_to_rad}" effort="${arm_1_max_effort}" velocity="${arm_1_max_vel}" />
+      <xacro:arm_1_joint_limits reflect="${reflect}" />
       <dynamics friction="${arm_friction}" damping="${arm_damping}"/>
 <!--        <safety_controller k_position="20"
@@ -64,13 +57,6 @@
                           soft_upper_limit="${30.00000 * deg_to_rad - arm_eps}" /> -->
     </joint>
-   <link name="${name}_${side}_2_link">
-      <inertial>
-        <origin xyz="0.02607 0.00049 -0.05209" rpy="0.00000 0.00000 0.00000"/>
-        <!-- <mass value="1.77729"/> -->
-        <mass value="1.67729"/>
-        <inertia ixx="0.00708700000" ixy="-0.00001400000" ixz="0.00214200000"
-                 iyy="0.00793600000" iyz="0.00003000000"
-                 izz="0.00378800000"/>
-      </inertial>
+    <link name="${name}_${side}_2_link">
+      <xacro:call macro="${name}_${side}_2_link_inertial" />
       <visual>
         <origin xyz="0 0 0" rpy="0 0 0" />
@@ -93,5 +79,5 @@
               rpy="${0.00000 * deg_to_rad} ${0.00000 * deg_to_rad} ${0.00000 * deg_to_rad}"/>
       <axis xyz="1 0 0" />
-      <limit lower="${(-82.0000 + 82.5000*reflect)* deg_to_rad}" upper="${(82.50000 + 82.0000*reflect)* deg_to_rad}" effort="${arm_2_max_effort}" velocity="${arm_2_max_vel}" />
+      <limit lower="${(-82.0000 + 82.5000*reflect)* deg_to_rad}" upper="${(82.50000*reflect + 82.0000)* deg_to_rad}" effort="${arm_2_max_effort}" velocity="${arm_2_max_vel}" />
       <dynamics friction="${arm_friction}" damping="${arm_damping}"/>
 <!--        <safety_controller k_position="20"
@@ -101,12 +87,5 @@
     </joint>
     <link name="${name}_${side}_3_link">
-      <inertial>
-        <origin xyz="0.00841 0.01428 -0.22291" rpy="0.00000 0.00000 0.00000"/>
-        <!-- <mass value="1.57029"/> -->
-        <mass value="1.47029"/>
-        <inertia ixx="0.00433200000" ixy="0.00015300000" ixz="-0.00049600000"
-                 iyy="0.00434000000" iyz="-0.00060900000"
-                 izz="0.00254300000"/>
-      </inertial>
+      <xacro:call macro="${name}_${side}_3_link_inertial" />
       <visual>
         <origin xyz="0 0 0" rpy="0 0 0" />
@@ -140,12 +119,5 @@
     <!--************************-->
     <link name="${name}_${side}_4_link">
-      <inertial>
-        <origin xyz="-0.00655 -0.02107 -0.02612" rpy="0.00000 0.00000 0.00000"/>
-        <!-- <mass value="1.20216"/> -->
-        <mass value="1.10216"/>
-        <inertia ixx="0.00221700000" ixy="-0.00010100000" ixz="0.00028800000"
-                 iyy="0.00241800000" iyz="-0.00039300000"
-                 izz="0.00111500000"/>
-      </inertial>
+      <xacro:call macro="${name}_${side}_4_link_inertial" />
       <visual>
         <origin xyz="0 0 0" rpy="0 0 0" />

File: talos_description/urdf/talos_full_common.urdf.xacro (robot description, xacro)
@@ -16,7 +16,7 @@
   <xacro:include filename="$(find talos_description)/urdf/torso/torso.urdf.xacro" />
   <xacro:include filename="$(find talos_description)/urdf/head/head.urdf.xacro" />
-  <xacro:include filename="$(find talos_description)/urdf/arm/arm_specifics_v2.urdf.xacro" />
   <xacro:include filename="$(find talos_description)/urdf/arm/arm.urdf.xacro" />
   <xacro:include filename="$(find talos_description)/urdf/sensors/ftsensor.urdf.xacro" />
+  <xacro:include filename="$(find talos_description)/urdf/gripper/gripper.urdf.xacro" />
   <xacro:include filename="$(find talos_description)/urdf/leg/leg.urdf.xacro" />
   <xacro:include filename="$(find talos_description)/urdf/leg/foot_collision_$(arg foot_collision).urdf.xacro" />
@@ -27,8 +27,10 @@
   </xacro:if>
   <xacro:talos_head name="head" parent="torso_2_link"/>
-  <xacro:talos_arm name="arm" parent="torso_2_link" side="left" reflect="1"/>
-  <xacro:talos_arm name="arm" parent="torso_2_link" side="right" reflect="-1"/>
+  <xacro:talos_arm name="arm" parent="torso_2_link" side="left" reflect="1" />
+  <xacro:talos_arm name="arm" parent="torso_2_link" side="right" reflect="-1" />
   <xacro:ft_sensor name="wrist" parent="arm_right_7_link" side="right" reflect="1"  />
   <xacro:ft_sensor name="wrist" parent="arm_left_7_link"  side="left"  reflect="-1" />
+  <xacro:talos_gripper name="gripper_left" parent="wrist_left_ft_tool_link" reflect="1" />
+  <xacro:talos_gripper name="gripper_right" parent="wrist_right_ft_tool_link" reflect="-1" />
   <xacro:talos_leg prefix="left"  reflect="1" />
   <xacro:talos_leg prefix="right" reflect="-1" />
