Commit message: camera leg integrationç

File: talos_description/robots/talos_full_fake_grippers.urdf.xacro (robot description, xacro)
@@ -32,6 +32,6 @@
   <xacro:ft_sensor name="wrist" parent="arm_right_7_link" side="right" reflect="1"  />
   <xacro:ft_sensor name="wrist" parent="arm_left_7_link"  side="left"  reflect="-1" />
-  <xacro:talos_leg prefix="left"  reflect="1" />
-  <xacro:talos_leg prefix="right" reflect="-1" />
+  <xacro:talos_leg prefix="left"  reflect="1" leg_camera="$(arg leg_camera)" disable_gazebo_camera="$(arg disable_gazebo_camera)"/>
+  <xacro:talos_leg prefix="right" reflect="-1" leg_camera="$(arg leg_camera)" disable_gazebo_camera="$(arg disable_gazebo_camera)"/>
   <!-- Macro to have the add-on links specific to each TALOS -->
   <xacro:talos_addons />

File: talos_description/robots/talos_full_no_grippers.urdf.xacro (robot description, xacro)
@@ -32,6 +32,6 @@
   <xacro:ft_sensor name="wrist" parent="arm_right_7_link" side="right" reflect="1" gripper_mount_type="$(arg gripper_mount_type)"/>
   <xacro:ft_sensor name="wrist" parent="arm_left_7_link"  side="left"  reflect="-1" gripper_mount_type="$(arg gripper_mount_type)"/>
-  <xacro:talos_leg prefix="left"  reflect="1" />
-  <xacro:talos_leg prefix="right" reflect="-1" />
+  <xacro:talos_leg prefix="left"  reflect="1" leg_camera="$(arg leg_camera)" disable_gazebo_camera="$(arg disable_gazebo_camera)"/>
+  <xacro:talos_leg prefix="right" reflect="-1" leg_camera="$(arg leg_camera)" disable_gazebo_camera="$(arg disable_gazebo_camera)"/>
   <!-- Macro to have the add-on links specific to each TALOS -->
   <xacro:talos_addons />

File: talos_description/robots/talos_lower_body.urdf.xacro (robot description, xacro)
@@ -41,6 +41,6 @@
       </collision>
     </link>
-  <xacro:talos_leg prefix="left"  reflect="1" />
-  <xacro:talos_leg prefix="right" reflect="-1" />
+  <xacro:talos_leg prefix="left"  reflect="1" leg_camera="$(arg leg_camera)" disable_gazebo_camera="$(arg disable_gazebo_camera)"/>
+  <xacro:talos_leg prefix="right" reflect="-1" leg_camera="$(arg leg_camera)" disable_gazebo_camera="$(arg disable_gazebo_camera)" />
   <!-- Macro to have the add-on links specific to each TALOS -->
   <xacro:talos_addons />

File: talos_description/robots/talos_lower_body_torso_head.urdf.xacro (robot description, xacro)
@@ -26,6 +26,6 @@
   <xacro:talos_torso name="torso" />
   <xacro:talos_head name="head" parent="torso_2_link" disable_gazebo_camera="$(arg disable_gazebo_camera)"/>
-  <xacro:talos_leg prefix="left"  reflect="1" />
-  <xacro:talos_leg prefix="right" reflect="-1" />
+  <xacro:talos_leg prefix="left"  reflect="1" leg_camera="$(arg leg_camera)" disable_gazebo_camera="$(arg disable_gazebo_camera)"/>
+  <xacro:talos_leg prefix="right" reflect="-1" leg_camera="$(arg leg_camera)" disable_gazebo_camera="$(arg disable_gazebo_camera)"/>
   <xacro:if value="$(arg enable_crane)">
     <xacro:crane parent="torso_2_link"/>

File: talos_description/urdf/leg/leg.urdf.xacro (robot description, xacro)
@@ -3,4 +3,5 @@
   <xacro:include filename="$(find talos_description)/urdf/leg/foot_frames.urdf.xacro" />
   <xacro:include filename="$(find talos_description)/urdf/leg/leg.transmission.xacro" />
+  <xacro:include filename="$(find realsense2_description)/urdf/_d435.urdf.xacro" />
   <xacro:property name="deg_to_rad"       value="0.01745329251994329577" />
   <xacro:property name="eps_radians"      value="0.008" /> <!-- 0.45deg -->
@@ -9,5 +10,5 @@
   <xacro:property name="leg_friction"     value="0.0" />
   <xacro:property name="leg_damping"      value="0.0" />
-  <xacro:macro name="talos_leg" params="prefix reflect flexibility:=false">
+  <xacro:macro name="talos_leg" params="prefix reflect flexibility:=false leg_camera:=false disable_gazebo_camera:=false">
     <xacro:unless value="$(arg test)">
       <xacro:include filename="$(find talos_description_calibration)/urdf/calibration/leg_${prefix}.xacro" />
@@ -212,7 +213,12 @@
       <visual>
         <origin rpy="0 0 0" xyz="0 0 0"/>
-        <geometry>
-          <mesh filename="package://talos_description/meshes/v2/ankle_X_lo_res.stl" scale="1 ${reflect*1} 1"/>
-        </geometry>
+          <geometry>
+          <xacro:if value="${leg_camera}">
+            <mesh filename="package://talos_description/meshes/v2/ankle_X_lo_res_camera.stl" scale="1 ${reflect*1} 1"/>
+          </xacro:if>
+          <xacro:unless value="${leg_camera}">
+            <mesh filename="package://talos_description/meshes/v2/ankle_X_lo_res.stl" scale="1 ${reflect*1} 1"/>
+          </xacro:unless>
+          </geometry>
         <material name="Grey" />
       </visual>
@@ -228,4 +234,44 @@
       <dynamics friction="${leg_friction}" damping="${leg_damping}"/>
     </joint>
+    <xacro:if value="${leg_camera}">
+      <link name="foot_front_${prefix}_link">
+        <origin rpy="0 0 0" xyz="0 0 0"/>
+      </link>
+      <joint name="foot_front_${prefix}_joint" type="fixed">
+        <parent link="leg_${prefix}_5_link"/>
+        <child link="foot_front_${prefix}_link"/>
+        <origin xyz="0.1125 0 -0.064"
+                rpy="0.0 0.0 0.0"/>
+        <axis xyz="1 0 0" />
+      </joint>
+      <link name="foot_rear_${prefix}_link">
+        <origin rpy="0 0 0" xyz="0 0 0"/>
+      </link>
+      <joint name="foot_rear_${prefix}_joint" type="fixed">
+        <parent link="leg_${prefix}_5_link"/>
+        <child link="foot_rear_${prefix}_link"/>
+        <origin xyz="-0.1313 0 -0.064"
+                rpy="0.0 0.0 3.14"/>
+        <axis xyz="1 0 0" />
+      </joint>
+      <xacro:unless value="${disable_gazebo_camera}">
+        <xacro:sensor_d435
+          name="foot_front_${prefix}_camera"
+          parent="foot_front_${prefix}_link"
+          topics_ns="foot_front_${prefix}_camera_rgbd">
+          <origin
+            xyz="0.0 0.0 0.0"
+            rpy="0.0 0.0 0.0"/>
+        </xacro:sensor_d435>
+        <xacro:sensor_d435
+          name="foot_rer_${prefix}_camera"
+          parent="foot_rear_${prefix}_link"
+          topics_ns="foot_rear_${prefix}_camera_rgbd">
+          <origin
+            xyz="0.0 0.0 0.0"
+            rpy="0.0 0.0 0.0"/>
+        </xacro:sensor_d435>
+      </xacro:unless>
+    </xacro:if>
   <!-- from here is copy paste -->
     <link name="${prefix}_sole_link">

File: talos_description/urdf/talos_full_common.urdf.xacro (robot description, xacro)
@@ -34,6 +34,6 @@
   <xacro:talos_gripper name="gripper" side="left" parent="wrist_left_ft_tool_link" reflect="1"  gripper_camera="$(arg gripper_camera)" simulation="$(arg simulation)" />
   <xacro:talos_gripper name="gripper" side="right" parent="wrist_right_ft_tool_link" reflect="-1"  gripper_camera="$(arg gripper_camera)" simulation="$(arg simulation)" />
-  <xacro:talos_leg prefix="left"  reflect="1" flexibility="$(arg flexibility)"/>
-  <xacro:talos_leg prefix="right" reflect="-1" flexibility="$(arg flexibility)"/>
+  <xacro:talos_leg prefix="left"  reflect="1" flexibility="$(arg flexibility)" leg_camera="$(arg leg_camera)" disable_gazebo_camera="$(arg disable_gazebo_camera)"/>
+  <xacro:talos_leg prefix="right" reflect="-1" flexibility="$(arg flexibility)" leg_camera="$(arg leg_camera)" disable_gazebo_camera="$(arg disable_gazebo_camera)"/>
   <!-- Macro to have the add-on links specific to each TALOS -->
   <xacro:talos_addons />

Commit message: added simulaton arg for use nominal extrinsic and renamed link of the support of cameras

File: talos_description/robots/talos_full_fake_grippers.urdf.xacro (robot description, xacro)
@@ -32,6 +32,6 @@
   <xacro:ft_sensor name="wrist" parent="arm_right_7_link" side="right" reflect="1"  />
   <xacro:ft_sensor name="wrist" parent="arm_left_7_link"  side="left"  reflect="-1" />
-  <xacro:talos_leg prefix="left"  reflect="1" leg_camera="$(arg leg_camera)" disable_gazebo_camera="$(arg disable_gazebo_camera)"/>
-  <xacro:talos_leg prefix="right" reflect="-1" leg_camera="$(arg leg_camera)" disable_gazebo_camera="$(arg disable_gazebo_camera)"/>
+  <xacro:talos_leg prefix="left"  reflect="1" leg_camera="$(arg leg_camera)" disable_gazebo_camera="$(arg disable_gazebo_camera)" simulation="$(arg simulation)"/>
+  <xacro:talos_leg prefix="right" reflect="-1" leg_camera="$(arg leg_camera)" disable_gazebo_camera="$(arg disable_gazebo_camera)" simulation="$(arg simulation)"/>
   <!-- Macro to have the add-on links specific to each TALOS -->
   <xacro:talos_addons />

File: talos_description/robots/talos_full_no_grippers.urdf.xacro (robot description, xacro)
@@ -32,6 +32,6 @@
   <xacro:ft_sensor name="wrist" parent="arm_right_7_link" side="right" reflect="1" gripper_mount_type="$(arg gripper_mount_type)"/>
   <xacro:ft_sensor name="wrist" parent="arm_left_7_link"  side="left"  reflect="-1" gripper_mount_type="$(arg gripper_mount_type)"/>
-  <xacro:talos_leg prefix="left"  reflect="1" leg_camera="$(arg leg_camera)" disable_gazebo_camera="$(arg disable_gazebo_camera)"/>
-  <xacro:talos_leg prefix="right" reflect="-1" leg_camera="$(arg leg_camera)" disable_gazebo_camera="$(arg disable_gazebo_camera)"/>
+  <xacro:talos_leg prefix="left"  reflect="1" leg_camera="$(arg leg_camera)" disable_gazebo_camera="$(arg disable_gazebo_camera)" simulation="$(arg simulation)"/>
+  <xacro:talos_leg prefix="right" reflect="-1" leg_camera="$(arg leg_camera)" disable_gazebo_camera="$(arg disable_gazebo_camera)" simulation="$(arg simulation)"/>
   <!-- Macro to have the add-on links specific to each TALOS -->
   <xacro:talos_addons />

File: talos_description/robots/talos_lower_body.urdf.xacro (robot description, xacro)
@@ -41,6 +41,6 @@
       </collision>
     </link>
-  <xacro:talos_leg prefix="left"  reflect="1" leg_camera="$(arg leg_camera)" disable_gazebo_camera="$(arg disable_gazebo_camera)"/>
-  <xacro:talos_leg prefix="right" reflect="-1" leg_camera="$(arg leg_camera)" disable_gazebo_camera="$(arg disable_gazebo_camera)" />
+  <xacro:talos_leg prefix="left"  reflect="1" leg_camera="$(arg leg_camera)" disable_gazebo_camera="$(arg disable_gazebo_camera)" simulation="$(arg simulation)"/>
+  <xacro:talos_leg prefix="right" reflect="-1" leg_camera="$(arg leg_camera)" disable_gazebo_camera="$(arg disable_gazebo_camera)" simulation="$(arg simulation)"/>
   <!-- Macro to have the add-on links specific to each TALOS -->
   <xacro:talos_addons />

File: talos_description/robots/talos_lower_body_torso_head.urdf.xacro (robot description, xacro)
@@ -26,6 +26,6 @@
   <xacro:talos_torso name="torso" />
   <xacro:talos_head name="head" parent="torso_2_link" disable_gazebo_camera="$(arg disable_gazebo_camera)"/>
-  <xacro:talos_leg prefix="left"  reflect="1" leg_camera="$(arg leg_camera)" disable_gazebo_camera="$(arg disable_gazebo_camera)"/>
-  <xacro:talos_leg prefix="right" reflect="-1" leg_camera="$(arg leg_camera)" disable_gazebo_camera="$(arg disable_gazebo_camera)"/>
+  <xacro:talos_leg prefix="left"  reflect="1" leg_camera="$(arg leg_camera)" disable_gazebo_camera="$(arg disable_gazebo_camera)" simulation="$(arg simulation)"/>
+  <xacro:talos_leg prefix="right" reflect="-1" leg_camera="$(arg leg_camera)" disable_gazebo_camera="$(arg disable_gazebo_camera)" simulation="$(arg simulation)"/>
   <xacro:if value="$(arg enable_crane)">
     <xacro:crane parent="torso_2_link"/>

File: talos_description/urdf/leg/leg.urdf.xacro (robot description, xacro)
@@ -10,5 +10,5 @@
   <xacro:property name="leg_friction"     value="0.0" />
   <xacro:property name="leg_damping"      value="0.0" />
-  <xacro:macro name="talos_leg" params="prefix reflect flexibility:=false leg_camera:=false disable_gazebo_camera:=false">
+  <xacro:macro name="talos_leg" params="prefix reflect flexibility:=false leg_camera:=false disable_gazebo_camera:=false simulation:=false">
     <xacro:unless value="$(arg test)">
       <xacro:include filename="$(find talos_description_calibration)/urdf/calibration/leg_${prefix}.xacro" />
@@ -235,20 +235,20 @@
     </joint>
     <xacro:if value="${leg_camera}">
-      <link name="foot_front_${prefix}_link">
+      <link name="support_front_${prefix}_camera_link">
         <origin rpy="0 0 0" xyz="0 0 0"/>
       </link>
-      <joint name="foot_front_${prefix}_joint" type="fixed">
+      <joint name="support_front_${prefix}_joint" type="fixed">
         <parent link="leg_${prefix}_5_link"/>
-        <child link="foot_front_${prefix}_link"/>
+        <child link="support_front_${prefix}_camera_link"/>
         <origin xyz="0.1125 0 -0.064"
                 rpy="0.0 0.0 0.0"/>
         <axis xyz="1 0 0" />
       </joint>
-      <link name="foot_rear_${prefix}_link">
+      <link name="support_rear_${prefix}_camera_link">
         <origin rpy="0 0 0" xyz="0 0 0"/>
       </link>
-      <joint name="foot_rear_${prefix}_joint" type="fixed">
+      <joint name="support_rear_${prefix}_joint" type="fixed">
         <parent link="leg_${prefix}_5_link"/>
-        <child link="foot_rear_${prefix}_link"/>
+        <child link="support_rear_${prefix}_camera_link"/>
         <origin xyz="-0.1313 0 -0.064"
                 rpy="0.0 0.0 3.14"/>
@@ -257,7 +257,8 @@
       <xacro:unless value="${disable_gazebo_camera}">
         <xacro:sensor_d435
-          name="foot_front_${prefix}_camera"
-          parent="foot_front_${prefix}_link"
-          topics_ns="foot_front_${prefix}_rgbd_camera">
+          name="foot_front_${prefix}_rgbd_camera"
+          parent="support_front_${prefix}_camera_link"
+          topics_ns="foot_front_${prefix}_rgbd_camera"
+          use_nominal_extrinsics="${simulation}">
           <origin
             xyz="0.0 0.0 0.0"
@@ -265,7 +266,8 @@
         </xacro:sensor_d435>
         <xacro:sensor_d435
-          name="foot_rear_${prefix}_camera"
-          parent="foot_rear_${prefix}_link"
-          topics_ns="foot_rear_${prefix}_rgbd_camera">
+          name="foot_rear_${prefix}_rgbd_camera"
+          parent="support_rear_${prefix}_camera_link"
+          topics_ns="foot_rear_${prefix}_rgbd_camera"
+          use_nominal_extrinsics="${simulation}">
           <origin
             xyz="0.0 0.0 0.0"

File: talos_description/urdf/talos_full_common.urdf.xacro (robot description, xacro)
@@ -34,6 +34,6 @@
   <xacro:talos_gripper name="gripper" side="left" parent="wrist_left_ft_tool_link" reflect="1"  gripper_camera="$(arg gripper_camera)" simulation="$(arg simulation)" />
   <xacro:talos_gripper name="gripper" side="right" parent="wrist_right_ft_tool_link" reflect="-1"  gripper_camera="$(arg gripper_camera)" simulation="$(arg simulation)" />
-  <xacro:talos_leg prefix="left"  reflect="1" flexibility="$(arg flexibility)" leg_camera="$(arg leg_camera)" disable_gazebo_camera="$(arg disable_gazebo_camera)"/>
-  <xacro:talos_leg prefix="right" reflect="-1" flexibility="$(arg flexibility)" leg_camera="$(arg leg_camera)" disable_gazebo_camera="$(arg disable_gazebo_camera)"/>
+  <xacro:talos_leg prefix="left"  reflect="1" flexibility="$(arg flexibility)" leg_camera="$(arg leg_camera)" disable_gazebo_camera="$(arg disable_gazebo_camera)" simulation="$(arg simulation)"/>
+  <xacro:talos_leg prefix="right" reflect="-1" flexibility="$(arg flexibility)" leg_camera="$(arg leg_camera)" disable_gazebo_camera="$(arg disable_gazebo_camera)" simulation="$(arg simulation)"/>
   <!-- Macro to have the add-on links specific to each TALOS -->
   <xacro:talos_addons />
