Commit message: Rename base link of detached arm

File: talos_description/robots/talos_arm_right.urdf.xacro (robot description, xacro)
@@ -19,5 +19,5 @@
   <!--     FAKE BASE_LINK     -->
   <!--************************-->
-  <link name="base_link">
+  <link name="arm_base_link">
     <inertial>
       <origin xyz="0.0 0.0 0.0" rpy="0.00000 0.00000 0.00000"/>
@@ -46,5 +46,5 @@
     <color rgba="0.7 0.7 0.7 1.0"/>
   </material>
-  <xacro:talos_arm name="arm" parent="base_link" side="right" reflect="-1" />
+  <xacro:talos_arm name="arm" parent="arm_base_link" side="right" reflect="-1" />
   <xacro:ft_sensor name="wrist" parent="arm_right_7_link" side="right" reflect="1"  />
   <xacro:talos_gripper name="gripper_right" parent="wrist_right_ft_tool_link" reflect="-1" />

Commit message: added d405, simulation arg for use nominal extrinsic and renamed link

File: talos_description/robots/talos_arm_right.urdf.xacro (robot description, xacro)
@@ -48,5 +48,5 @@
   <xacro:talos_arm name="arm" parent="arm_base_link" side="right" reflect="-1" />
   <xacro:ft_sensor name="wrist" parent="arm_right_7_link" side="right" reflect="1"  />
-  <xacro:talos_gripper name="gripper_right" parent="wrist_right_ft_tool_link" reflect="-1" />
+  <xacro:talos_gripper name="gripper_right" parent="wrist_right_ft_tool_link" reflect="-1" gripper_camera="$(arg gripper_camera)" simulation="$(arg simulation)" />
   <!-- Generic simulator_gazebo plugins -->
   <xacro:include filename="$(find talos_description)/gazebo/gazebo.urdf.xacro" />

File: talos_description/urdf/gripper/gripper.urdf.xacro (robot description, xacro)
@@ -5,7 +5,8 @@
   <xacro:include filename="$(find talos_description)/urdf/gripper/gripper.transmission.xacro" />
   <xacro:include filename="$(find talos_description)/urdf/gripper/gripper.gazebo.xacro" />
-  <xacro:macro name="talos_gripper" params="name side parent reflect gripper_camera">
+  <xacro:include filename="$(find realsense2_description)/urdf/_d405.urdf.xacro" />
+  <xacro:macro name="talos_gripper" params="name side parent reflect gripper_camera simulation">
             <xacro:if value="${gripper_camera}">
-              <link name="${name}_${side}_gripper_camera_link">
+              <link name="support_${name}_${side}_camera_link">
                 <inertial>
                   <origin xyz="0.01021 -0.00042075 -0.00034305" rpy="0 0 0" />
@@ -29,10 +30,19 @@
                 </collision>
               </link>
-              <joint name="${name}_${side}_wrist_left_camera_joint" type="fixed">
+              <joint name="support_${name}_${side}_wrist_camera_joint" type="fixed">
                 <origin xyz="0.11239 0 -0.12048" rpy="-3.1415925371051 1.0472025163988 -3.14159251909337" />
                 <parent link="arm_${side}_7_link"/>
-                <child link="${name}_${side}_gripper_camera_link" />
+                <child link="support_${name}_${side}_camera_link" />
                 <axis xyz="0 0 0" />
               </joint>
+              <xacro:sensor_d405
+                name="${name}_${side}_rgbd_camera_"
+                parent="support_${name}_${side}_camera_link"
+                topics_ns="${name}_${side}_rgbd_camera"
+                use_nominal_extrinsics="${simulation}">
+                <origin
+                  xyz="0.0 0.0 0.0"
+                  rpy="0.0 0.0 0.0"/>
+              </xacro:sensor_d405>
             </xacro:if>
             <link name="${name}_${side}_base_link">

File: talos_description/urdf/talos_full_common.urdf.xacro (robot description, xacro)
@@ -32,6 +32,6 @@
   <xacro:ft_sensor name="wrist" parent="arm_right_7_link" side="right" reflect="1" gripper_mount_type="$(arg gripper_mount_type)" />
   <xacro:ft_sensor name="wrist" parent="arm_left_7_link"  side="left"  reflect="-1" gripper_mount_type="$(arg gripper_mount_type)" />
-  <xacro:talos_gripper name="gripper" side="left" parent="wrist_left_ft_tool_link" reflect="1"  gripper_camera="$(arg gripper_camera)"/>
-  <xacro:talos_gripper name="gripper" side="right" parent="wrist_right_ft_tool_link" reflect="-1"  gripper_camera="$(arg gripper_camera)"/>
+  <xacro:talos_gripper name="gripper" side="left" parent="wrist_left_ft_tool_link" reflect="1"  gripper_camera="$(arg gripper_camera)" simulation="$(arg simulation)" />
+  <xacro:talos_gripper name="gripper" side="right" parent="wrist_right_ft_tool_link" reflect="-1"  gripper_camera="$(arg gripper_camera)" simulation="$(arg simulation)" />
   <xacro:talos_leg prefix="left"  reflect="1" flexibility="$(arg flexibility)"/>
   <xacro:talos_leg prefix="right" reflect="-1" flexibility="$(arg flexibility)"/>

Commit message: update disable_gazebo camera strategy and created realsense xacro

File: talos_description/robots/talos_arm_right.urdf.xacro (robot description, xacro)
@@ -48,5 +48,5 @@
   <xacro:talos_arm name="arm" parent="arm_base_link" side="right" reflect="-1" gripper_mount_type="$(arg gripper_mount_type)"/>
   <xacro:ft_sensor name="wrist" parent="arm_right_7_link" side="right" reflect="1" gripper_mount_type="$(arg gripper_mount_type)"/>
-  <xacro:talos_gripper name="gripper" side="right" parent="wrist_right_ft_tool_link" reflect="-1" gripper_camera="$(arg gripper_camera)" simulation="$(arg simulation)"/>
+  <xacro:talos_gripper name="gripper" side="right" parent="wrist_right_ft_tool_link" reflect="-1" gripper_camera="$(arg gripper_camera)" simulation="$(arg simulation)" disable_gazebo_camera="$(arg disable_gazebo_camera)"/>
   <!-- Generic simulator_gazebo plugins -->
   <xacro:include filename="$(find talos_description)/gazebo/gazebo.urdf.xacro" />

File: talos_description/urdf/gripper/gripper.urdf.xacro (robot description, xacro)
@@ -5,6 +5,6 @@
   <xacro:include filename="$(find talos_description)/urdf/gripper/gripper.transmission.xacro" />
   <xacro:include filename="$(find talos_description)/urdf/gripper/gripper.gazebo.xacro" />
-  <xacro:include filename="$(find realsense2_description)/urdf/_d405.urdf.xacro" />
-  <xacro:macro name="talos_gripper" params="name side parent reflect gripper_camera simulation">
+  <xacro:include filename="$(find talos_description)/urdf/sensors/realsense_d405_urdf.xacro" />
+  <xacro:macro name="talos_gripper" params="name side parent reflect gripper_camera simulation disable_gazebo_camera">
             <xacro:if value="${gripper_camera}">
               <link name="support_${name}_${side}_camera_link">
@@ -40,5 +40,6 @@
                 parent="support_${name}_${side}_camera_link"
                 topics_ns="${name}_${side}_rgbd_camera"
-                use_nominal_extrinsics="${simulation}">
+                use_nominal_extrinsics="${simulation}"
+                disable_gazebo_camera="${disable_gazebo_camera}">
                 <origin
                   xyz="0.0 0.0 0.0"

File: talos_description/urdf/leg/leg.urdf.xacro (robot description, xacro)
@@ -3,5 +3,5 @@
   <xacro:include filename="$(find talos_description)/urdf/leg/foot_frames.urdf.xacro" />
   <xacro:include filename="$(find talos_description)/urdf/leg/leg.transmission.xacro" />
-  <xacro:include filename="$(find realsense2_description)/urdf/_d435.urdf.xacro" />
+  <xacro:include filename="$(find talos_description)/urdf/sensors/realsense_d435_urdf.xacro" />
   <xacro:property name="deg_to_rad"       value="0.01745329251994329577" />
   <xacro:property name="eps_radians"      value="0.008" /> <!-- 0.45deg -->
@@ -255,10 +255,10 @@
         <axis xyz="1 0 0" />
       </joint>
-      <xacro:unless value="${disable_gazebo_camera}">
         <xacro:sensor_d435
           name="foot_front_${prefix}_rgbd_camera"
           parent="support_front_${prefix}_camera_link"
           topics_ns="foot_front_${prefix}_rgbd_camera"
-          use_nominal_extrinsics="${simulation}">
+          use_nominal_extrinsics="${simulation}"
+          disable_gazebo_camera="${disable_gazebo_camera}">
           <origin
             xyz="0.0 0.0 0.0"
@@ -269,10 +269,10 @@
           parent="support_rear_${prefix}_camera_link"
           topics_ns="foot_rear_${prefix}_rgbd_camera"
-          use_nominal_extrinsics="${simulation}">
+          use_nominal_extrinsics="${simulation}"
+          disable_gazebo_camera="${disable_gazebo_camera}">
           <origin
             xyz="0.0 0.0 0.0"
             rpy="0.0 0.0 0.0"/>
         </xacro:sensor_d435>
-      </xacro:unless>
     </xacro:if>
   <!-- from here is copy paste -->

File: talos_description/urdf/talos_full_common.urdf.xacro (robot description, xacro)
@@ -32,6 +32,6 @@
   <xacro:ft_sensor name="wrist" parent="arm_right_7_link" side="right" reflect="1" gripper_mount_type="$(arg gripper_mount_type)" />
   <xacro:ft_sensor name="wrist" parent="arm_left_7_link"  side="left"  reflect="-1" gripper_mount_type="$(arg gripper_mount_type)" />
-  <xacro:talos_gripper name="gripper" side="left" parent="wrist_left_ft_tool_link" reflect="1"  gripper_camera="$(arg gripper_camera)" simulation="$(arg simulation)" />
-  <xacro:talos_gripper name="gripper" side="right" parent="wrist_right_ft_tool_link" reflect="-1"  gripper_camera="$(arg gripper_camera)" simulation="$(arg simulation)" />
+  <xacro:talos_gripper name="gripper" side="left" parent="wrist_left_ft_tool_link" reflect="1"  gripper_camera="$(arg gripper_camera)" simulation="$(arg simulation)" disable_gazebo_camera="$(arg disable_gazebo_camera)" />
+  <xacro:talos_gripper name="gripper" side="right" parent="wrist_right_ft_tool_link" reflect="-1"  gripper_camera="$(arg gripper_camera)" simulation="$(arg simulation)" disable_gazebo_camera="$(arg disable_gazebo_camera)" />
   <xacro:talos_leg prefix="left"  reflect="1" flexibility="$(arg flexibility)" leg_camera="$(arg leg_camera)" disable_gazebo_camera="$(arg disable_gazebo_camera)" simulation="$(arg simulation)"/>
   <xacro:talos_leg prefix="right" reflect="-1" flexibility="$(arg flexibility)" leg_camera="$(arg leg_camera)" disable_gazebo_camera="$(arg disable_gazebo_camera)" simulation="$(arg simulation)"/>
