Commit message: Fix frame for wrist ft sensors

File: talos_description/urdf/sensors/ftsensor.urdf.xacro (robot description, xacro)
@@ -34,5 +34,5 @@
       <parent link="${parent}" />
       <child link="${name}_${side}_ft_link" />
-      <origin xyz="0 0 -0.051" rpy="${0.0 * deg_to_rad} 0 ${-90.0 * deg_to_rad}" />
+      <origin xyz="0 0 -0.051" rpy="${0.0 * deg_to_rad} 0 ${(-60 + 90.0*reflect) * deg_to_rad}" />
     </joint>
     <!--***********************-->
@@ -61,5 +61,5 @@
       <parent link="${name}_${side}_ft_link" />
       <child link="${name}_${side}_ft_tool_link" />
-      <origin xyz="0 0 ${-1.0 * (0.0157*0.5 + 0.00975*0.5)}" rpy="0 0 ${-90.0 * reflect * deg_to_rad}" />
+      <origin xyz="0 0 ${-1.0 * (0.0157*0.5 + 0.00975*0.5)}" rpy="0 0 ${(-30 - 180.0 * reflect) * deg_to_rad}" />
     </joint>
 </xacro:macro>

Commit message: Added motions, and ft sensor signs fixed

File: talos_description/urdf/sensors/ftsensor.urdf.xacro (robot description, xacro)
@@ -34,5 +34,5 @@
       <parent link="${parent}" />
       <child link="${name}_${side}_ft_link" />
-      <origin xyz="0 0 -0.051" rpy="${0.0 * deg_to_rad} 0 ${(-60 + 90.0*reflect) * deg_to_rad}" />
+      <origin xyz="0 0 -0.051" rpy="${0.0 * deg_to_rad} 0 ${(-180.0 + 90.0*reflect)* deg_to_rad}" />
     </joint>
     <!--***********************-->
@@ -61,5 +61,5 @@
       <parent link="${name}_${side}_ft_link" />
       <child link="${name}_${side}_ft_tool_link" />
-      <origin xyz="0 0 ${-1.0 * (0.0157*0.5 + 0.00975*0.5)}" rpy="0 0 ${(-30 - 180.0 * reflect) * deg_to_rad}" />
+      <origin xyz="0 0 ${-1.0 * (0.0157*0.5 + 0.00975*0.5)}" rpy="0 0 ${(90.0 -180.0* reflect) * deg_to_rad}" />
     </joint>
 </xacro:macro>
