Commit message: Minor fix in inertial parameters of orbbec_astra_pro.

File: talos_description/urdf/sensors/orbbec_astra_pro.urdf.xacro (robot description, xacro)
@@ -30,11 +30,11 @@
     </joint>
     <link name="${name}_link">
+      <!-- inertia tensor computed analytically for a solid cuboid -->
       <inertial>
         <mass value="0.01" />
-        <origin xyz="0 0 0" rpy="0 0 0"/>
-        <!-- inertia tensor computed analytically for a solid cuboid -->
+        <origin xyz="-0.01 0.0025 0" rpy="0 0 0"/>
         <inertia ixx="0.000030"  ixy="0.0"  ixz="0.0"
-                 iyy="0.000030"  iyz="0.0"
-                 izz="0.000002" />
+                 iyy="0.000002"  iyz="0.0"
+                 izz="0.000030" />
       </inertial>
       <visual>

Commit message: Fix wrong optical frame

File: talos_description/urdf/sensors/orbbec_astra_pro.urdf.xacro (robot description, xacro)
@@ -50,4 +50,5 @@
     <joint name="${name}_optical_joint" type="fixed">
       <xacro:insert_block name="optical_origin" />
+       <origin xyz="0 0 0" rpy="${-90.0 * deg_to_rad} 0.0 ${-90.0 * deg_to_rad}" />
       <parent link="${name}_link"/>
       <child link="${name}_optical_frame"/>
