Commit message: Fix type in arm_v2 and rename arm_v1 urdf

File: talos_description/urdf/arm/arm_v2.urdf.xacro (robot description, xacro)
@@ -60,5 +60,5 @@
       <!-- v1 TALOS has 1st arm left joint (-90,30) and right joint (-30,90) -->
       <!-- v2 TALOS has 1st arm left joint (-90,50) and right joint (-50,90) -->
-      <limit lower="${((-70.0 - 20.0*reflect)* deg_to_rad}" upper="${(70.0 - 20.0*reflect)* deg_to_rad}" effort="${arm_1_max_effort}" velocity="${arm_1_max_vel}" />
+      <limit lower="${(-70.0 - 20.0*reflect)* deg_to_rad}" upper="${(70.0 - 20.0*reflect)* deg_to_rad}" effort="${arm_1_max_effort}" velocity="${arm_1_max_vel}" />
       <dynamics friction="${arm_friction}" damping="${arm_damping}"/>
 <!--        <safety_controller k_position="20"

Commit message: modified limits of gripper, leg 5 joint,  and arm v2 1 joint

File: talos_description/urdf/arm/arm_v2.urdf.xacro (robot description, xacro)
@@ -60,5 +60,5 @@
       <!-- v1 TALOS has 1st arm left joint (-90,30) and right joint (-30,90) -->
       <!-- v2 TALOS has 1st arm left joint (-90,50) and right joint (-50,90) -->
-      <limit lower="${(-70.0 - 20.0*reflect)* deg_to_rad}" upper="${(70.0 - 20.0*reflect)* deg_to_rad}" effort="${arm_1_max_effort}" velocity="${arm_1_max_vel}" />
+      <limit lower="${(-67,5.0 - 22.5*reflect)* deg_to_rad}" upper="${(67,5 - 22,5*reflect)* deg_to_rad}" effort="${arm_1_max_effort}" velocity="${arm_1_max_vel}" />
       <dynamics friction="${arm_friction}" damping="${arm_damping}"/>
 <!--        <safety_controller k_position="20"

File: talos_description/urdf/gripper/gripper.urdf.xacro (robot description, xacro)
@@ -65,5 +65,5 @@
                       rpy="${0.0 * deg_to_rad} ${0.0 * deg_to_rad} ${0.0 * deg_to_rad}"/>
               <axis xyz="1 0 0" />
-              <limit lower="${-60.0 * deg_to_rad}" upper="${0.0 * deg_to_rad}" effort="1.0" velocity="1.0" />
+              <limit lower="${-55.0 * deg_to_rad}" upper="${0.0 * deg_to_rad}" effort="1.0" velocity="1.0" />
               <dynamics friction="1.0" damping="1.0"/>
             </joint>

File: talos_description/urdf/leg/leg.urdf.xacro (robot description, xacro)
@@ -166,5 +166,5 @@
               rpy="${0.00000 * deg_to_rad} ${0.00000 * deg_to_rad} ${0.00000 * deg_to_rad}"/>
       <axis xyz="0 1 0" />
-      <limit lower="-1.309" upper="0.768" effort="160" velocity="5.8" />
+      <limit lower="-1.27" upper="0.68" effort="160" velocity="5.8" />
       <dynamics friction="${leg_friction}" damping="${leg_damping}"/>
     </joint>

Commit message: fixed type in urdf model

File: talos_description/urdf/arm/arm_v2.urdf.xacro (robot description, xacro)
@@ -60,5 +60,5 @@
       <!-- v1 TALOS has 1st arm left joint (-90,30) and right joint (-30,90) -->
       <!-- v2 TALOS has 1st arm left joint (-90,50) and right joint (-50,90) -->
-      <limit lower="${(-67,5.0 - 22.5*reflect)* deg_to_rad}" upper="${(67,5 - 22,5*reflect)* deg_to_rad}" effort="${arm_1_max_effort}" velocity="${arm_1_max_vel}" />
+      <limit lower="${(-67.5 - 22.5*reflect)* deg_to_rad}" upper="${(67.5 - 22.5*reflect)* deg_to_rad}" effort="${arm_1_max_effort}" velocity="${arm_1_max_vel}" />
       <dynamics friction="${arm_friction}" damping="${arm_damping}"/>
 <!--        <safety_controller k_position="20"

Commit message: Various fixes in the model.

File: talos_description/urdf/arm/arm_v2.urdf.xacro (robot description, xacro)
@@ -31,10 +31,9 @@
       <!-- TODO: Missing reflects of inertias -->
       <inertial>
-        <origin xyz="-0.01346 ${reflect*0.09130} 0.04812" rpy="0.00000 0.00000 0.00000"/>
-        <!-- <mass value="1.52896"/> -->
-        <mass value="1.42896"/>
-        <inertia ixx="0.00555100000" ixy="-0.00073100000" ixz="0.00000800000"
-                 iyy="0.00167300000" iyz="-0.00006000000"
-                 izz="0.00582200000"/>
+        <origin xyz="-0.00064789000 ${reflect*0.10043599000} 0.04424260000" rpy="0.00000000000 0.00000000000 0.00000000000"/>
+        <mass value="2.73980200000"/>
+        <inertia ixx="0.01265548000" ixy="${reflect*0.00000054000}" ixz="-0.00007347000"
+                 iyy="0.00414615000" iyz="${reflect*0.00027675000}"
+                 izz="0.01365466000"/>
       </inertial>
       <visual>
@@ -96,5 +95,5 @@
               rpy="${0.00000 * deg_to_rad} ${0.00000 * deg_to_rad} ${0.00000 * deg_to_rad}"/>
       <axis xyz="1 0 0" />
-      <limit lower="${(-82.0000 + 82.5000*reflect)* deg_to_rad}" upper="${(82.50000 + 82.0000*reflect)* deg_to_rad}" effort="${arm_2_max_effort}" velocity="${arm_2_max_vel}" />
+      <limit lower="${(-82.0000 + 82.5000*reflect)* deg_to_rad}" upper="${(82.50000*reflect + 82.0000)* deg_to_rad}" effort="${arm_2_max_effort}" velocity="${arm_2_max_vel}" />
       <dynamics friction="${arm_friction}" damping="${arm_damping}"/>
 <!--        <safety_controller k_position="20"
@@ -144,5 +143,5 @@
     <link name="${name}_${side}_4_link">
       <inertial>
-        <origin xyz="-0.00655 -0.02107 -0.02612" rpy="0.00000 0.00000 0.00000"/>
+        <origin xyz="-0.00655 ${reflect*-0.02107} -0.02612" rpy="0.00000 0.00000 0.00000"/>
         <!-- <mass value="1.20216"/> -->
         <mass value="1.10216"/>

File: talos_description/urdf/leg/leg.urdf.xacro (robot description, xacro)
@@ -12,8 +12,8 @@
     <link name="leg_${prefix}_1_link">
       <inertial>
-        <origin xyz="0.02320 -0.00009 0.04949" rpy="0.00000 0.00000 0.00000"/>
+        <origin xyz="0.02320 ${reflect*-0.00009} 0.04949" rpy="0.00000 0.00000 0.00000"/>
         <mass value="1.88569"/>
-        <inertia ixx="0.00384800000" ixy="0.00003200000" ixz="-0.00082600000"
-                 iyy="0.00599400000" iyz="0.00007800000"
+        <inertia ixx="0.00384800000" ixy="${reflect*0.00003200000}" ixz="-0.00082600000"
+                 iyy="0.00599400000" iyz="${reflect*0.00007800000}"
                  izz="0.00322200000"/>
       </inertial>
@@ -46,6 +46,6 @@
         <origin xyz="0.01583 -0.00021 0.00619" rpy="0.00000 0.00000 0.00000"/>
         <mass value="2.37607"/>
-        <inertia ixx="0.00342100000" ixy="-0.00011300000" ixz="-0.00022500000"
-                 iyy="0.00402400000" iyz="-0.00003100000"
+        <inertia ixx="0.00342100000" ixy="${reflect*-0.00011300000}" ixz="-0.00022500000"
+                 iyy="0.00402400000" iyz="${reflect*-0.00003100000}"
                  izz="0.00416400000"/>
       </inertial>
@@ -172,8 +172,8 @@
     <link name="leg_${prefix}_6_link">
       <inertial>
-        <origin xyz="-0.02087 -0.00019 -0.06059" rpy="0.00000 0.00000 0.00000"/>
+        <origin xyz="-0.02087 ${reflect*-0.00019} -0.06059" rpy="0.00000 0.00000 0.00000"/>
         <mass value="1.59457"/>
-        <inertia ixx="0.00383800000" ixy="0.00001600000" ixz="-0.00104100000"
-                 iyy="0.00657200000" iyz="-0.00001700000"
+        <inertia ixx="0.00383800000" ixy="${reflect*0.00001600000}" ixz="-0.00104100000"
+                 iyy="0.00657200000" iyz="${reflect*-0.00001700000}"
                  izz="0.00504400000"/>
       </inertial>

File: talos_description/urdf/torso/torso.urdf.xacro (robot description, xacro)
@@ -14,5 +14,5 @@
  <!--Constant parameters-->
   <xacro:property name="torso_max_vel"  value="5.4" />
-  <xacro:property name="torso_max_effort"  value="78.0" />
+  <xacro:property name="torso_max_effort"  value="200.0" />
   <xacro:property name="torso_eps"      value="0.02" />
   <xacro:macro name="talos_torso" params="name">

Commit message: New inertial parameters of links 1 and 2 in the arm (2 seems to be wrong).

File: talos_description/urdf/arm/arm_v2.urdf.xacro (robot description, xacro)
@@ -31,9 +31,9 @@
       <!-- TODO: Missing reflects of inertias -->
       <inertial>
-        <origin xyz="-0.00064789000 ${reflect*0.10043599000} 0.04424260000" rpy="0.00000000000 0.00000000000 0.00000000000"/>
-        <mass value="2.73980200000"/>
-        <inertia ixx="0.01265548000" ixy="${reflect*0.00000054000}" ixz="-0.00007347000"
-                 iyy="0.00414615000" iyz="${reflect*0.00027675000}"
-                 izz="0.01365466000"/>
+        <origin xyz="-0.00027620000 ${reflect*0.10060223000} 0.04437419000" rpy="0.00000000000 0.00000000000 0.00000000000"/>
+        <mass value="2.71456700000"/>
+        <inertia ixx="0.01237819000" ixy="${reflect*0.00003626000}" ixz="-0.00007145000"
+                 iyy="0.00419138000" iyz="${reflect*0.00023639000}"
+                 izz="0.01358161000"/>
       </inertial>
       <visual>
@@ -66,12 +66,11 @@
                           soft_upper_limit="${30.00000 * deg_to_rad - arm_eps}" /> -->
     </joint>
-   <link name="${name}_${side}_2_link">
-      <inertial>
-        <origin xyz="0.02607 0.00049 -0.05209" rpy="0.00000 0.00000 0.00000"/>
-        <!-- <mass value="1.77729"/> -->
-        <mass value="1.67729"/>
-        <inertia ixx="0.00708700000" ixy="-0.00001400000" ixz="0.00214200000"
-                 iyy="0.00793600000" iyz="0.00003000000"
-                 izz="0.00378800000"/>
+    <link name="${name}_${side}_2_link">
+      <inertial>
+        <origin xyz="0.01438831000 0.00092938000 -0.08684268000" rpy="0.00000000000 0.00000000000 0.00000000000"/>
+        <mass value="2.42508600000"/>
+        <inertia ixx="0.01297822000" ixy="-0.00001209000" ixz="0.00320371000"
+                 iyy="0.01380870000" iyz="0.00012770000"
+                 izz="0.00478857000"/>
       </inertial>
       <visual>

Commit message: Updated inertial parameters of the arms (they look ok now)

File: talos_description/urdf/arm/arm_v2.urdf.xacro (robot description, xacro)
@@ -29,11 +29,10 @@
     <!--************************-->
     <link name="${name}_${side}_1_link">
-      <!-- TODO: Missing reflects of inertias -->
       <inertial>
         <origin xyz="-0.00027620000 ${reflect*0.10060223000} 0.04437419000" rpy="0.00000000000 0.00000000000 0.00000000000"/>
         <mass value="2.71456700000"/>
-        <inertia ixx="0.01237819000" ixy="${reflect*0.00003626000}" ixz="-0.00007145000"
-                 iyy="0.00419138000" iyz="${reflect*0.00023639000}"
-                 izz="0.01358161000"/>
+        <inertia ixx="0.01237818683" ixy="${reflect*-0.00003625571}" ixz="0.00007144720"
+                 iyy="0.00419137200" iyz="${reflect*-0.00023639064}"
+                 izz="0.01358161109"/>
       </inertial>
       <visual>
@@ -68,9 +67,9 @@
     <link name="${name}_${side}_2_link">
       <inertial>
-        <origin xyz="0.01438831000 0.00092938000 -0.08684268000" rpy="0.00000000000 0.00000000000 0.00000000000"/>
+        <origin xyz="0.01438831000 ${reflect*0.00092938000} -0.08684268000" rpy="0.00000000000 0.00000000000 0.00000000000"/>
         <mass value="2.42508600000"/>
-        <inertia ixx="0.01297822000" ixy="-0.00001209000" ixz="0.00320371000"
-                 iyy="0.01380870000" iyz="0.00012770000"
-                 izz="0.00478857000"/>
+        <inertia ixx="0.01297822101" ixy="${reflect*0.00001208791}" ixz="-0.00320370433"
+                 iyy="0.01380870278" iyz="${reflect*-0.00012770059}"
+                 izz="0.00478856621"/>
       </inertial>
       <visual>
@@ -103,10 +102,9 @@
     <link name="${name}_${side}_3_link">
       <inertial>
-        <origin xyz="0.00841 0.01428 -0.22291" rpy="0.00000 0.00000 0.00000"/>
-        <!-- <mass value="1.57029"/> -->
-        <mass value="1.47029"/>
-        <inertia ixx="0.00433200000" ixy="0.00015300000" ixz="-0.00049600000"
-                 iyy="0.00434000000" iyz="-0.00060900000"
-                 izz="0.00254300000"/>
+        <origin xyz="0.01360840000 ${reflect*0.01241619000} -0.24990040000" rpy="0.00000000000 0.00000000000 0.00000000000"/>
+        <mass value="2.20874100000"/>
+        <inertia ixx="0.00718831493" ixy="${reflect*-0.00011563551}" ixz="0.00075969733"
+                 iyy="0.00693528503" iyz="${reflect*0.00042134743}"
+                 izz="0.00388359007"/>
       </inertial>
       <visual>
@@ -142,10 +140,9 @@
     <link name="${name}_${side}_4_link">
       <inertial>
-        <origin xyz="-0.00655 ${reflect*-0.02107} -0.02612" rpy="0.00000 0.00000 0.00000"/>
-        <!-- <mass value="1.20216"/> -->
-        <mass value="1.10216"/>
-        <inertia ixx="0.00221700000" ixy="-0.00010100000" ixz="0.00028800000"
-                 iyy="0.00241800000" iyz="-0.00039300000"
-                 izz="0.00111500000"/>
+        <origin xyz="-0.00742138000 ${reflect*-0.02138950000} -0.03312656000" rpy="0.00000000000 0.00000000000 0.00000000000"/>
+        <mass value="0.87734600000"/>
+        <inertia ixx="0.00251207716" ixy="${reflect*0.00010070062}" ixz="-0.00032788214"
+            iyy="0.00275869324" iyz="${reflect*0.00040022227}"
+                 izz="0.00120735959"/>
       </inertial>
       <visual>

File: talos_description/urdf/arm/wrist.urdf.xacro (robot description, xacro)
@@ -27,10 +27,9 @@
     <link name="${name}_${side}_5_link">
       <inertial>
-        <origin xyz="-0.00006 0.00326 0.07963" rpy="0.00000 0.00000 0.00000"/>
-        <!-- <mass value="1.87792"/> -->
-        <mass value="1.77792"/>
-        <inertia ixx="0.00349500000" ixy="-0.00001300000" ixz="-0.00001000000"
-                 iyy="0.00436800000" iyz="0.00009700000"
-                 izz="0.00228300000"/>
+        <origin xyz="-0.00006000000 ${reflect*0.00326200000} 0.07962500000" rpy="0.00000000000 0.00000000000 0.00000000000"/>
+        <mass value="1.87792300000"/>
+        <inertia ixx="0.00349507283" ixy="${reflect*0.00001265489}" ixz="0.00001038286"
+                 iyy="0.00436830072" iyz="${reflect*-0.00009736042}"
+                 izz="0.00228263370"/>
       </inertial>
       <visual>
@@ -63,10 +62,9 @@
     <link name="${name}_${side}_6_link">
       <inertial>
-        <origin xyz="0.00002 -0.00197 -0.00059" rpy="0.00000 0.00000 0.00000"/>
-        <!-- <mass value="0.40931"/> -->
-        <mass value="0.30931"/>
-        <inertia ixx="0.00010700000" ixy="0.00000000000" ixz="0.00000000000"
-                 iyy="0.00014100000" iyz="-0.00000000000"
-                 izz="0.00015400000"/>
+        <origin xyz="0.00002100000 ${reflect*-0.00196500000} -0.00059100000" rpy="0.00000000000 0.00000000000 0.00000000000"/>
+        <mass value="0.40931000000"/>
+        <inertia ixx="0.00010700023" ixy="${reflect*-0.00000008899}" ixz="-0.00000004392"
+                 iyy="0.00014101316" iyz="${reflect*0.00000041702}"
+                 izz="0.00015398658"/>
       </inertial>
       <visual>
@@ -98,19 +96,10 @@
     </joint>
     <link name="${name}_${side}_7_link">
-      <!-- WRONG VALUES
       <inertial>
-        <origin xyz="-0.00089 0.00365 -0.07824" rpy="0.00000 0.00000 0.00000"/>
-        <mass value="1.02604"/>
-        <inertia ixx="0.00151400000" ixy="0.00000600000" ixz="0.00006600000"
-                 iyy="0.00146400000" iyz="0.00001200000"
-                 izz="0.00090300000"/>
-      </inertial>
-      -->
-      <inertial>
-        <origin xyz="0.007525 0.001378 -0.024630" rpy="0.00000 0.00000 0.00000"/>
-        <mass value="0.308441"/>
-        <inertia ixx="0.000309" ixy="0.000002" ixz="-0.000002"
-                 iyy="0.000219" iyz="0.000012"
-                 izz="0.000176"/>
+        <origin xyz="0.00752500000 ${reflect*0.00137800000} -0.02463000000" rpy="0.00000000000 0.00000000000 0.00000000000"/>
+        <mass value="0.30844100000"/>
+        <inertia ixx="0.00030894317" ixy="${reflect*-0.00000158687}" ixz="0.00000173418"
+                 iyy="0.00021886181" iyz="${reflect*-0.00001221167}"
+                 izz="0.00017519492"/>
       </inertial>
       <visual>
