Commit message: Fix orientation of IMU, delete TODO comments.

File: talos_description/urdf/arm/arm_v1.urdf.xacro (robot description, xacro)
@@ -29,5 +29,4 @@
     <!--************************-->
     <link name="${name}_${side}_1_link">
-      <!-- TODO: Missing reflects of inertias -->
       <inertial>
         <origin xyz="-0.01346 ${reflect*0.09130} 0.04812" rpy="0.00000 0.00000 0.00000"/>

File: talos_description/urdf/torso/torso.urdf.xacro (robot description, xacro)
@@ -122,7 +122,5 @@
     </joint>
     <xacro:talos_imu name="imu" parent="${name}_2_link" update_rate="100.0">
-        <!-- TODO AS: match model & sensor -->
-        <!-- <origin xyz="0.04925 0 0.078" rpy="${180.0*deg_to_rad} 0 ${-90.0*deg_to_rad}"/>-->
-        <origin xyz="0.04925 0 0.078" rpy="${180.0*deg_to_rad} 0 ${0.0*deg_to_rad}"/>
+        <origin xyz="0.04925 0 0.078" rpy="${180.0*deg_to_rad} 0 ${-90.0*deg_to_rad}"/>
     </xacro:talos_imu>
     <gazebo reference="${name}_1_link">
