Commit message: Talos arms will use description_calibration

File: talos_description/urdf/arm/arm.transmission.xacro (robot description, xacro)
@@ -8,5 +8,5 @@
 -->
 <robot xmlns:xacro="http://ros.org/wiki/xacro">
-  <xacro:macro name="talos_arm_simple_transmission" params="name side number reduction" >
+  <xacro:macro name="talos_arm_simple_transmission" params="name side number reduction offset_value" >
     <transmission name="${name}_${side}_${number}_trans">
       <type>transmission_interface/SimpleTransmission</type>
@@ -15,4 +15,5 @@
       </actuator>
       <joint name="${name}_${side}_${number}_joint">
+        <offset>${offset_value}</offset>
         <hardwareInterface>hardware_interface/PositionJointInterface</hardwareInterface>
         <hardwareInterface>hardware_interface/EffortJointInterface</hardwareInterface>

File: talos_description/urdf/arm/arm_v1.urdf.xacro (robot description, xacro)
@@ -213,8 +213,5 @@
      <xacro:talos_wrist name="arm" parent="${name}_${side}_4_link" side="${side}" reflect="${reflect}" />
     <!-- extensions -->
-    <xacro:talos_arm_simple_transmission name="${name}" side="${side}" number="1" reduction="1.0" />
-    <xacro:talos_arm_simple_transmission name="${name}" side="${side}" number="2" reduction="1.0" />
-    <xacro:talos_arm_simple_transmission name="${name}" side="${side}" number="3" reduction="1.0" />
-    <xacro:talos_arm_simple_transmission name="${name}" side="${side}" number="4" reduction="1.0" />
+    <xacro:include filename="$(find talos_description)/urdf/arm/${side}_arm.transmissions.urdf.xacro" />
   </xacro:macro>
 </robot>

File: talos_description/urdf/arm/arm_v2.urdf.xacro (robot description, xacro)
@@ -215,8 +215,5 @@
      <xacro:talos_wrist name="arm" parent="${name}_${side}_4_link" side="${side}" reflect="${reflect}" />
     <!-- extensions -->
-    <xacro:talos_arm_simple_transmission name="${name}" side="${side}" number="1" reduction="1.0" />
-    <xacro:talos_arm_simple_transmission name="${name}" side="${side}" number="2" reduction="1.0" />
-    <xacro:talos_arm_simple_transmission name="${name}" side="${side}" number="3" reduction="1.0" />
-    <xacro:talos_arm_simple_transmission name="${name}" side="${side}" number="4" reduction="1.0" />
+    <xacro:include filename="$(find talos_description)/urdf/arm/${side}_arm.transmissions.urdf.xacro" />
   </xacro:macro>
 </robot>

File: talos_description/urdf/arm/wrist.transmission.xacro (robot description, xacro)
@@ -8,5 +8,5 @@
 -->
 <robot xmlns:xacro="http://ros.org/wiki/xacro">
-  <xacro:macro name="talos_wrist_simple_transmission" params="name side number reduction" >
+  <xacro:macro name="talos_wrist_simple_transmission" params="name side number reduction offset_value" >
     <transmission name="${name}_${side}_${number}_trans">
       <type>transmission_interface/SimpleTransmission</type>
@@ -15,4 +15,5 @@
       </actuator>
       <joint name="${name}_${side}_${number}_joint">
+        <offset>${offset_value}</offset>
         <hardwareInterface>hardware_interface/PositionJointInterface</hardwareInterface>
         <hardwareInterface>hardware_interface/EffortJointInterface</hardwareInterface>
@@ -21,5 +22,5 @@
   </xacro:macro>
   <xacro:macro name="talos_wrist_differential_transmission"
-               params="name side number_1 number_2 act_reduction_1 act_reduction_2 jnt_reduction_1 jnt_reduction_2" >
+               params="name side number_1 number_2 act_reduction_1 act_reduction_2 jnt_reduction_1 jnt_reduction_2 offset_value_1 offset_value_2" >
     <transmission name="wrist_${side}_trans">
       <type>transmission_interface/DifferentialTransmission</type>
@@ -34,5 +35,5 @@
       <joint name="${name}_${side}_${number_1}_joint">
         <role>joint1</role>
-        <offset>0.0</offset>
+        <offset>${offset_value_1}</offset>
         <mechanicalReduction>${jnt_reduction_1}</mechanicalReduction>
         <hardwareInterface>hardware_interface/PositionJointInterface</hardwareInterface>
@@ -41,5 +42,5 @@
       <joint name="${name}_${side}_${number_2}_joint">
         <role>joint2</role>
-        <offset>0.0</offset>
+        <offset>${offset_value_2}</offset>
         <mechanicalReduction>${jnt_reduction_2}</mechanicalReduction>
         <hardwareInterface>hardware_interface/PositionJointInterface</hardwareInterface>

File: talos_description/urdf/arm/wrist.urdf.xacro (robot description, xacro)
@@ -165,8 +165,5 @@
     </gazebo>
     <!-- extensions -->
-    <xacro:talos_wrist_simple_transmission name="${name}" side="${side}" number="5" reduction="1.0" />
-    <xacro:talos_wrist_differential_transmission name="${name}" side="${side}" number_1="6" number_2="7"
-                                                act_reduction_1="-1.0" act_reduction_2="1.0"
-                                                jnt_reduction_1="-1.0" jnt_reduction_2="-1.0" />
+    <xacro:include filename="$(find talos_description)/urdf/arm/${side}_wrist.transmissions.urdf.xacro" />
   </xacro:macro>
 </robot>
