Commit message: Fix right wrist and gripper rotations

File: talos_description/urdf/arm/wrist.urdf.xacro (robot description, xacro)
@@ -37,5 +37,5 @@
         <origin xyz="0 0 0" rpy="0 0 0" />
         <geometry>
-          <mesh filename="package://talos_description/meshes/arm/arm_5.STL" scale="1 1 1"/>
+          <mesh filename="package://talos_description/meshes/arm/arm_5.STL" scale="1 ${reflect} 1"/>
         </geometry>
         <material name="LightGrey" />
@@ -44,5 +44,5 @@
         <origin xyz="0 0 0" rpy="0 0 0" />
         <geometry>
-          <mesh filename="package://talos_description/meshes/arm/arm_5_collision.STL" scale="1 1 1"/>
+          <mesh filename="package://talos_description/meshes/arm/arm_5_collision.STL" scale="1 ${reflect} 1"/>
         </geometry>
       </collision>
@@ -51,12 +51,6 @@
       <parent link="${parent}" />
       <child link="${name}_${side}_5_link" />
-      <xacro:if value="${reflect == 1}">
-        <origin xyz="-0.02000 0.00000 -0.26430"
-              rpy="${0.00000 * deg_to_rad} ${0.00000 * deg_to_rad} ${0.00000 * deg_to_rad}"/>
-      </xacro:if>
-      <xacro:if value="${reflect == -1}">
-        <origin xyz="-0.02000 0.00000 -0.26430"
-              rpy="${0.00000 * deg_to_rad} ${0.00000 * deg_to_rad} ${180.00000 * deg_to_rad}"/>
-      </xacro:if>
+      <origin xyz="-0.02000 0.00000 -0.26430"
+                rpy="${0.00000 * deg_to_rad} ${0.00000 * deg_to_rad} ${0.00000 * deg_to_rad}"/>
       <axis xyz="0 0 1" />
       <limit lower="${-145.0 * deg_to_rad}" upper="${145.0 * deg_to_rad}" effort="${wrist_1_max_effort}" velocity="${wrist_1_max_vel}" />
@@ -123,5 +117,5 @@
         <origin xyz="0 0 0" rpy="0 0 0" />
         <geometry>
-          <mesh filename="package://talos_description/meshes/arm/arm_7.STL" scale="1 1 1"/>
+          <mesh filename="package://talos_description/meshes/arm/arm_7.STL" scale="1 ${reflect} 1"/>
         </geometry>
         <material name="DarkGrey" />
@@ -130,5 +124,5 @@
         <origin xyz="0 0 0" rpy="0 0 0" />
         <geometry>
-          <mesh filename="package://talos_description/meshes/arm/arm_7_collision.STL" scale="1 1 1"/>
+          <mesh filename="package://talos_description/meshes/arm/arm_7_collision.STL" scale="1 ${reflect} 1"/>
         </geometry>
       </collision>

File: talos_description/urdf/gripper/gripper_v2.urdf.xacro (robot description, xacro)
@@ -32,5 +32,5 @@
               <child link="${name}_base_link"/>
               <origin xyz="0.00000 0.00000 -0.02875"
-                      rpy="${0.00000 * deg_to_rad} ${0.00000 * deg_to_rad} ${(reflect -1)* 90.000000 * deg_to_rad}"/>
+                      rpy="${0.00000 * deg_to_rad} ${0.00000 * deg_to_rad} ${0.00000 * deg_to_rad}"/>
               <axis xyz="0 0 0" />
             </joint>

Commit message: Fix max wrist effort

File: talos_description/urdf/arm/wrist.urdf.xacro (robot description, xacro)
@@ -17,7 +17,7 @@
   <xacro:property name="wrist_2_max_vel"      value="1.76" />
   <xacro:property name="wrist_3_max_vel"      value="1.76" />
-  <xacro:property name="wrist_1_max_effort"   value="3" />
-  <xacro:property name="wrist_2_max_effort"   value="6.6" />
-  <xacro:property name="wrist_3_max_effort"   value="6.6" />
+  <xacro:property name="wrist_1_max_effort"   value="20.0" />
+  <xacro:property name="wrist_2_max_effort"   value="8.0" />
+  <xacro:property name="wrist_3_max_effort"   value="8.0" />
   <xacro:property name="wrist_eps"          value="0.02" />
   <xacro:macro name="talos_wrist" params="name parent side reflect">
