Commit message: Fix wrong transformations / meshes in the camera

File: talos_description/urdf/arm/left_arm.transmissions.urdf.xacro (robot description, xacro)
@@ -10,5 +10,4 @@
   <!--File includes-->
   <xacro:include filename="$(find talos_description)/urdf/arm/arm.transmission.xacro" />
-  <xacro:include filename="$(find talos_description_calibration)/urdf/calibration/calibration_constants.urdf.xacro" />
   <!-- extensions -->
   <xacro:talos_arm_simple_transmission name="${name}" side="left" number="1" reduction="1.0" offset_value="${arm_left_1_joint_offset}" />

File: talos_description/urdf/arm/left_wrist.transmissions.urdf.xacro (robot description, xacro)
@@ -10,5 +10,4 @@
   <!--File includes-->
   <xacro:include filename="$(find talos_description)/urdf/arm/wrist.transmission.xacro" />
-  <xacro:include filename="$(find talos_description_calibration)/urdf/calibration/calibration_constants.urdf.xacro" />
   <!-- extensions -->
   <xacro:talos_wrist_simple_transmission name="${name}" side="${side}" number="5" reduction="1.0"

File: talos_description/urdf/arm/right_arm.transmissions.urdf.xacro (robot description, xacro)
@@ -10,5 +10,4 @@
   <!--File includes-->
   <xacro:include filename="$(find talos_description)/urdf/arm/arm.transmission.xacro" />
-  <xacro:include filename="$(find talos_description_calibration)/urdf/calibration/calibration_constants.urdf.xacro" />
   <!-- extensions -->
   <xacro:talos_arm_simple_transmission name="${name}" side="right" number="1" reduction="1.0" offset_value="${arm_right_1_joint_offset}" />

File: talos_description/urdf/arm/right_wrist.transmissions.urdf.xacro (robot description, xacro)
@@ -10,5 +10,4 @@
   <!--File includes-->
   <xacro:include filename="$(find talos_description)/urdf/arm/wrist.transmission.xacro" />
-  <xacro:include filename="$(find talos_description_calibration)/urdf/calibration/calibration_constants.urdf.xacro" />
   <!-- extensions -->
   <xacro:talos_wrist_simple_transmission name="${name}" side="${side}" number="5" reduction="1.0"

File: talos_description/urdf/head/head.urdf.xacro (robot description, xacro)
@@ -12,10 +12,4 @@
   <xacro:include filename="$(find talos_description)/urdf/head/head.transmission.xacro" />
   <xacro:include filename="$(find talos_description)/urdf/sensors/orbbec_astra_pro.urdf.xacro" />
-  <xacro:unless value="$(arg test)">
-    <xacro:include filename="$(find talos_description_calibration)/urdf/calibration/calibration_constants.urdf.xacro" />
-  </xacro:unless>
-  <xacro:if value="$(arg test)">
-    <xacro:include filename="$(find talos_description)/test/calibration/calibration_constants.urdf.xacro" />
-  </xacro:if>
   <!--Constant parameters-->
   <xacro:property name="head_friction" value="1.0" />
@@ -119,5 +113,5 @@
         <origin xyz="${camera_position_x} ${camera_position_y} ${camera_position_z}" rpy="${camera_orientation_r} ${camera_orientation_p} ${camera_orientation_y}" />
         <!-- Pose of optical frame wrt to sensor -->
-        <origin xyz="0 0 0" rpy="${-90 * deg_to_rad} 0 ${-90 * deg_to_rad}"/>
+        <optical_origin xyz="0 0 0" rpy="${-90 * deg_to_rad} 0 ${-90 * deg_to_rad}"/>
       </xacro:orbbec_astra_pro>
     </xacro:if>

File: talos_description/urdf/sensors/orbbec_astra_pro.urdf.xacro (robot description, xacro)
@@ -71,5 +71,5 @@
     <!-- frames of the rgb sensor -->
     <joint name="${name}_rgb_joint" type="fixed">
-      <origin xyz="0.033 -0.025 0.0" rpy="0 0 0" />
+      <origin xyz="0.0033 -0.025 0.0" rpy="0 0 0" />
       <parent link="${name}_link" />
       <child link="${name}_rgb_frame"/>
