Commit message: Removed xacro if

File: talos_description/urdf/arm/arm.urdf.xacro (robot description, xacro)
@@ -58,11 +58,6 @@
               rpy="${0.0 * deg_to_rad} ${0.0 * deg_to_rad} ${0.0 * deg_to_rad}"/>
       <axis xyz="0 0 1" />
-      <xacro:if value="${reflect == 1}">
-        <limit lower="${-90.0 * deg_to_rad}" upper="${30.0 * deg_to_rad}" effort="${arm_1_max_effort}" velocity="${arm_1_max_vel}" />
-      </xacro:if>
-      <xacro:if value="${reflect == -1}">
-        <limit lower="${-30.0 * deg_to_rad}" upper="${90.0 * deg_to_rad}" effort="${arm_1_max_effort}" velocity="${arm_1_max_vel}" />
-      </xacro:if>
-       <dynamics friction="${arm_friction}" damping="${arm_damping}"/>
+      <limit lower="${(-60.0 - 30.0*reflect)* deg_to_rad}" upper="${(60.0 - 30.0*reflect)* deg_to_rad}" effort="${arm_1_max_effort}" velocity="${arm_1_max_vel}" />
+      <dynamics friction="${arm_friction}" damping="${arm_damping}"/>
 <!--        <safety_controller k_position="20"
                           k_velocity="20"
@@ -99,10 +94,5 @@
               rpy="${0.00000 * deg_to_rad} ${0.00000 * deg_to_rad} ${0.00000 * deg_to_rad}"/>
       <axis xyz="1 0 0" />
-      <xacro:if value="${reflect == 1}">
-        <limit lower="${0.00000 * deg_to_rad}" upper="${165.00000 * deg_to_rad}" effort="${arm_2_max_effort}" velocity="${arm_2_max_vel}" />
-      </xacro:if>
-      <xacro:if value="${reflect == -1}">
-        <limit lower="${-165.00000 * deg_to_rad}" upper="${0.00000 * deg_to_rad}" effort="${arm_2_max_effort}" velocity="${arm_2_max_vel}" />
-      </xacro:if>
+      <limit lower="${(-82.50000 + 82.5*reflect)* deg_to_rad}" upper="${(82.50000 + 82.5000*reflect)* deg_to_rad}" effort="${arm_2_max_effort}" velocity="${arm_2_max_vel}" />
       <dynamics friction="${arm_friction}" damping="${arm_damping}"/>
 <!--        <safety_controller k_position="20"
@@ -222,37 +212,4 @@
     <!--************************-->
      <xacro:talos_wrist name="arm" parent="${name}_${side}_4_link" side="${side}" reflect="${reflect}" />
-    <!--***********************-->
-    <!--        TOOL           -->
-    <!--***********************-->
-<!--     <link name="${name}_${side}_tool_link">
-      <inertial>
-        <mass value="0.1" />
-        <inertia ixx="0.0" ixy="0.0" ixz="0.0" iyy="0.0" iyz="0.0" izz="0.0" />
-      </inertial>
-      <visual>
-        <origin xyz="0.001 0 0" rpy="0 ${90.0 * deg_to_rad} 0" />
-        <geometry>
-          <cylinder radius="0.005" length="0.005"/>
-        </geometry>
-        <material name="LightGrey" />
-      </visual>
-      <collision>
-        <origin xyz="0.001 0 0" rpy="0 ${90.0 * deg_to_rad} 0" />
-        <geometry>
-          <cylinder radius="0.005" length="0.005"/>
-        </geometry>
-      </collision>
-    </link>
-    <joint name="${name}_${side}_tool_joint" type="fixed">
-      <parent link="${name}_${side}_7_link" />
-      <child link="${name}_${side}_tool_link" />
-      <xacro:if value="${reflect == 1}">
-        <origin xyz="0 0 -0.051" rpy="0 ${90.0 * deg_to_rad} 0" />
-      </xacro:if>
-      <xacro:if value="${reflect == -1}">
-        <origin xyz="0 0 -0.051" rpy="${180.0 * deg_to_rad} ${90.0 * deg_to_rad} ${0.0 * deg_to_rad}" />
-      </xacro:if>
-    </joint>
- -->
     <!-- extensions -->
     <xacro:talos_arm_simple_transmission name="${name}" side="${side}" number="1" reduction="1.0" />

File: talos_description/urdf/leg/leg_v2.urdf.xacro (robot description, xacro)
@@ -38,10 +38,5 @@
               rpy="${0.00000 * deg_to_rad} ${0.00000 * deg_to_rad} ${0.00000 * deg_to_rad}"/>
       <axis xyz="0 0 1" />
-     <xacro:if value="${reflect == 1}">
-        <limit lower="-0.5236" upper="1.571" effort="100" velocity="3.87" />
-      </xacro:if>
-      <xacro:if value="${reflect == -1}">
-        <limit lower="-1.571" upper="0.5236" effort="100" velocity="3.87" />
-      </xacro:if>
+      <limit lower="${(-55.0 + 35.0*reflect)*deg_to_rad}" upper="${(55.0 + 35.0*reflect)*deg_to_rad}" effort="100" velocity="3.87" />
       <dynamics friction="${leg_friction}" damping="${leg_damping}"/>
     </joint>
@@ -75,5 +70,5 @@
               rpy="${0.00000 * deg_to_rad} ${0.00000 * deg_to_rad} ${0.00000 * deg_to_rad}"/>
       <axis xyz="1 0 0" />
-      <limit lower="-0.524" upper="0.5236" effort="160" velocity="5.8" />
+      <limit lower="-0.5236" upper="0.5236" effort="160" velocity="5.8" />
       <dynamics friction="${leg_friction}" damping="${leg_damping}"/>
     </joint>
@@ -211,5 +206,5 @@
               rpy="${0.00000 * deg_to_rad} ${0.00000 * deg_to_rad} ${0.00000 * deg_to_rad}"/>
       <axis xyz="1 0 0" />
-      <limit lower="-0.524" upper="0.524" effort="100" velocity="4.8" />
+      <limit lower="-0.5236" upper="0.5236" effort="100" velocity="4.8" />
       <dynamics friction="${leg_friction}" damping="${leg_damping}"/>
     </joint>

Commit message: Safe range of motion for upper body

File: talos_description/urdf/arm/arm.urdf.xacro (robot description, xacro)
@@ -19,8 +19,8 @@
   <xacro:property name="arm_3_max_vel"      value="4.58" />
   <xacro:property name="arm_4_max_vel"      value="4.58" />
-  <xacro:property name="arm_1_max_effort"   value="44.64" />
-  <xacro:property name="arm_2_max_effort"   value="22.32" />
-  <xacro:property name="arm_3_max_effort"   value="17.86" />
-  <xacro:property name="arm_4_max_effort"   value="17.86" />
+  <xacro:property name="arm_1_max_effort"   value="100.0" />
+  <xacro:property name="arm_2_max_effort"   value="100.0" />
+  <xacro:property name="arm_3_max_effort"   value="70.0" />
+  <xacro:property name="arm_4_max_effort"   value="70.0" />
   <xacro:property name="arm_eps"            value="0.02" />
   <xacro:macro name="talos_arm" params="name parent side reflect">
@@ -94,5 +94,5 @@
               rpy="${0.00000 * deg_to_rad} ${0.00000 * deg_to_rad} ${0.00000 * deg_to_rad}"/>
       <axis xyz="1 0 0" />
-      <limit lower="${(-82.50000 + 82.5*reflect)* deg_to_rad}" upper="${(82.50000 + 82.5000*reflect)* deg_to_rad}" effort="${arm_2_max_effort}" velocity="${arm_2_max_vel}" />
+      <limit lower="${(-82.0000 + 82.5000*reflect)* deg_to_rad}" upper="${(82.50000 + 82.0000*reflect)* deg_to_rad}" effort="${arm_2_max_effort}" velocity="${arm_2_max_vel}" />
       <dynamics friction="${arm_friction}" damping="${arm_damping}"/>
 <!--        <safety_controller k_position="20"
@@ -130,5 +130,5 @@
               rpy="${0.00000 * deg_to_rad} ${0.00000 * deg_to_rad} ${0.00000 * deg_to_rad}"/>
       <axis xyz="0 0 1" />
-      <limit lower="${-140.0 * deg_to_rad}" upper="${140.0 * deg_to_rad}" effort="${arm_3_max_effort}" velocity="${arm_3_max_vel}" />
+      <limit lower="${-139.0 * deg_to_rad}" upper="${139.0 * deg_to_rad}" effort="${arm_3_max_effort}" velocity="${arm_3_max_vel}" />
       <dynamics friction="${arm_friction}" damping="${arm_damping}"/>
 <!--       <safety_controller k_position="20"
@@ -169,5 +169,5 @@
               rpy="${0.00000 * deg_to_rad} ${0.00000 * deg_to_rad} ${0.00000 * deg_to_rad}"/>
       <axis xyz="0 1 0" />
-      <limit lower="${-135.0 * deg_to_rad}" upper="${0.0 * deg_to_rad}" effort="${arm_4_max_effort}" velocity="${arm_4_max_vel}" />
+      <limit lower="${-128.0 * deg_to_rad}" upper="${0.2 * deg_to_rad}" effort="${arm_4_max_effort}" velocity="${arm_4_max_vel}" />
       <dynamics friction="${arm_friction}" damping="${arm_damping}"/>
 <!--       <safety_controller k_position="20"

File: talos_description/urdf/arm/wrist.urdf.xacro (robot description, xacro)
@@ -54,5 +54,5 @@
                 rpy="${0.00000 * deg_to_rad} ${0.00000 * deg_to_rad} ${0.00000 * deg_to_rad}"/>
       <axis xyz="0 0 1" />
-      <limit lower="${-145.0 * deg_to_rad}" upper="${145.0 * deg_to_rad}" effort="${wrist_1_max_effort}" velocity="${wrist_1_max_vel}" />
+      <limit lower="${-144.0 * deg_to_rad}" upper="${144.0 * deg_to_rad}" effort="${wrist_1_max_effort}" velocity="${wrist_1_max_vel}" />
       <dynamics friction="${wrist_friction}" damping="${wrist_damping}"/>
 <!--       <safety_controller k_position="20"
@@ -90,5 +90,5 @@
               rpy="${0.00000 * deg_to_rad} ${0.00000 * deg_to_rad} ${0.00000 * deg_to_rad}"/>
       <axis xyz="1 0 0" />
-      <limit lower="${-80.0 * deg_to_rad}" upper="${80.0 * deg_to_rad}" effort="${wrist_2_max_effort}" velocity="${wrist_2_max_vel}" />
+      <limit lower="${-78.5 * deg_to_rad}" upper="${78.5 * deg_to_rad}" effort="${wrist_2_max_effort}" velocity="${wrist_2_max_vel}" />
       <dynamics friction="${wrist_friction}" damping="${wrist_damping}"/>
 <!--       <safety_controller k_position="20"
@@ -134,5 +134,5 @@
                 rpy="${0.0 * deg_to_rad} ${0.0 * deg_to_rad} ${0.0 * deg_to_rad}"/>
       <axis xyz="0 1 0" />
-      <limit lower="${-40.0 * deg_to_rad}" upper="${40.0 * deg_to_rad}" effort="${wrist_3_max_effort}" velocity="${wrist_3_max_vel}"/>
+      <limit lower="${-39.0 * deg_to_rad}" upper="${39.0 * deg_to_rad}" effort="${wrist_3_max_effort}" velocity="${wrist_3_max_vel}"/>
       <dynamics friction="${wrist_friction}" damping="${wrist_damping}"/>
 <!--       <safety_controller k_position="20"

File: talos_description/urdf/head/head.urdf.xacro (robot description, xacro)
@@ -49,5 +49,5 @@
               rpy="${0.00000 * deg_to_rad} ${0.00000 * deg_to_rad} ${0.00000 * deg_to_rad}"/>
       <axis xyz="0 1 0" />
-      <limit lower="${-15.00000 * deg_to_rad}" upper="${45.00000 * deg_to_rad}" effort="8.0" velocity="1.0" />
+      <limit lower="${-12.00000 * deg_to_rad}" upper="${45.00000 * deg_to_rad}" effort="8.0" velocity="1.0" />
       <dynamics damping="${head_damping}" friction="${head_friction}"/>
        <!-- <safety_controller k_position="20"

File: talos_description/urdf/torso/torso.urdf.xacro (robot description, xacro)
@@ -73,5 +73,5 @@
               rpy="${0.00000 * deg_to_rad} ${0.00000 * deg_to_rad} ${0.00000 * deg_to_rad}"/>
       <axis xyz="0 0 1" />
-      <limit lower="${-75.00000 * deg_to_rad}" upper="${75.00000 * deg_to_rad}"
+      <limit lower="${-72.00000 * deg_to_rad}" upper="${72.00000 * deg_to_rad}"
              effort="${torso_max_effort}" velocity="${torso_max_vel}" />
       <dynamics damping="1.0" friction="1.0"/>
@@ -112,5 +112,5 @@
               rpy="${0.00000 * deg_to_rad} ${0.00000 * deg_to_rad} ${0.00000 * deg_to_rad}"/>
       <axis xyz="0 1 0" />
-      <limit lower="${-15.0 * deg_to_rad}" upper="${45.0 * deg_to_rad}"
+      <limit lower="${-13.0 * deg_to_rad}" upper="${42.0 * deg_to_rad}"
              effort="${torso_max_effort}" velocity="${torso_max_vel}"/>
       <dynamics friction="1.0" damping="1.0"/>

Commit message: Fix upper limit for arm_*_4_joint.

File: talos_description/urdf/arm/arm.urdf.xacro (robot description, xacro)
@@ -140,5 +140,5 @@
               rpy="${0.00000 * deg_to_rad} ${0.00000 * deg_to_rad} ${0.00000 * deg_to_rad}"/>
       <axis xyz="0 1 0" />
-      <limit lower="${-128.0 * deg_to_rad}" upper="${0.2 * deg_to_rad}" effort="${arm_4_max_effort}" velocity="${arm_4_max_vel}" />
+      <limit lower="${-128.0 * deg_to_rad}" upper="${-0.2 * deg_to_rad}" effort="${arm_4_max_effort}" velocity="${arm_4_max_vel}" />
       <dynamics friction="${arm_friction}" damping="${arm_damping}"/>
 <!--       <safety_controller k_position="20"
