Commit message: Use DAE with texture for color

File: talos_description/urdf/arm/arm.urdf.xacro (robot description, xacro)
@@ -33,12 +33,12 @@
         <origin xyz="0 0 0" rpy="0 0 0" />
         <geometry>
-          <mesh filename="package://talos_description/meshes/arm/arm_1.STL" scale="1 ${reflect} 1"/>
+          <mesh filename="package://talos_description/meshes/arm/arm_1.dae" scale="1 ${reflect} 1"/>
         </geometry>
-        <material name="DarkGrey" />
+        <material name="Black" />
       </visual>
       <collision>
        <origin xyz="0 0 0" rpy="0 0 0" />
         <geometry>
-          <mesh filename="package://talos_description/meshes/arm/arm_1_collision.STL" scale="1 ${reflect} 1"/>
+          <mesh filename="package://talos_description/meshes/arm/arm_1_collision.dae" scale="1 ${reflect} 1"/>
         </geometry>
       </collision>
@@ -62,12 +62,12 @@
         <origin xyz="0 0 0" rpy="0 0 0" />
         <geometry>
-          <mesh filename="package://talos_description/meshes/arm/arm_2.STL" scale="1 ${reflect} 1"/>
+          <mesh filename="package://talos_description/meshes/arm/arm_2.dae" scale="1 ${reflect} 1"/>
         </geometry>
-        <material name="DarkGrey" />
+        <material name="Black" />
       </visual>
       <collision>
         <origin xyz="0 0 0" rpy="0 0 0" />
         <geometry>
-          <mesh filename="package://talos_description/meshes/arm/arm_2_collision.STL" scale="1 ${reflect} 1"/>
+          <mesh filename="package://talos_description/meshes/arm/arm_2_collision.dae" scale="1 ${reflect} 1"/>
         </geometry>
       </collision>
@@ -91,12 +91,12 @@
         <origin xyz="0 0 0" rpy="0 0 0" />
         <geometry>
-          <mesh filename="package://talos_description/meshes/arm/arm_3.STL" scale="1 ${reflect} 1"/>
+          <mesh filename="package://talos_description/meshes/arm/arm_3.dae" scale="1 ${reflect} 1"/>
         </geometry>
-        <material name="DarkGrey" />
+        <material name="Black" />
       </visual>
       <collision>
         <origin xyz="0 0 0" rpy="0 0 0" />
         <geometry>
-          <mesh filename="package://talos_description/meshes/arm/arm_3_collision.STL" scale="1 ${reflect} 1"/>
+          <mesh filename="package://talos_description/meshes/arm/arm_3_collision.dae" scale="1 ${reflect} 1"/>
         </geometry>
       </collision>
@@ -123,12 +123,12 @@
         <origin xyz="0 0 0" rpy="0 0 0" />
         <geometry>
-          <mesh filename="package://talos_description/meshes/arm/arm_4.STL" scale="1 ${reflect} 1"/>
+          <mesh filename="package://talos_description/meshes/arm/arm_4.dae" scale="1 ${reflect} 1"/>
         </geometry>
-        <material name="DarkGrey" />
+        <material name="Black" />
       </visual>
       <collision>
         <origin xyz="0 0 0" rpy="0 0 0" />
         <geometry>
-          <mesh filename="package://talos_description/meshes/arm/arm_4_collision.STL" scale="1 ${reflect} 1"/>
+          <mesh filename="package://talos_description/meshes/arm/arm_4_collision.dae" scale="1 ${reflect} 1"/>
         </geometry>
       </collision>

File: talos_description/urdf/arm/wrist.urdf.xacro (robot description, xacro)
@@ -30,12 +30,12 @@
         <origin xyz="0 0 0" rpy="0 0 0" />
         <geometry>
-          <mesh filename="package://talos_description/meshes/arm/arm_5.STL" scale="1 ${reflect} 1"/>
+          <mesh filename="package://talos_description/meshes/arm/arm_5.dae" scale="1 ${reflect} 1"/>
         </geometry>
-        <material name="LightGrey" />
+        <material name="White" />
       </visual>
       <collision>
         <origin xyz="0 0 0" rpy="0 0 0" />
         <geometry>
-          <mesh filename="package://talos_description/meshes/arm/arm_5_collision.STL" scale="1 ${reflect} 1"/>
+          <mesh filename="package://talos_description/meshes/arm/arm_5_collision.dae" scale="1 ${reflect} 1"/>
         </geometry>
       </collision>
@@ -59,12 +59,12 @@
         <origin xyz="0 0 0" rpy="0 0 0" />
         <geometry>
-          <mesh filename="package://talos_description/meshes/arm/arm_6.STL" scale="1 ${reflect} 1"/>
+          <mesh filename="package://talos_description/meshes/arm/arm_6.dae" scale="1 ${reflect} 1"/>
         </geometry>
-        <material name="LightGrey" />
+        <material name="White" />
       </visual>
       <collision>
         <origin xyz="0 0 0" rpy="0 0 0" />
         <geometry>
-          <mesh filename="package://talos_description/meshes/arm/arm_6_collision.STL" scale="1 ${reflect} 1"/>
+          <mesh filename="package://talos_description/meshes/arm/arm_6_collision.dae" scale="1 ${reflect} 1"/>
         </geometry>
       </collision>
@@ -88,12 +88,12 @@
         <origin xyz="0 0 0" rpy="0 0 0" />
         <geometry>
-          <mesh filename="package://talos_description/meshes/arm/arm_7.STL" scale="1 ${reflect} 1"/>
+          <mesh filename="package://talos_description/meshes/arm/arm_7.dae" scale="1 ${reflect} 1"/>
         </geometry>
-        <material name="DarkGrey" />
+        <material name="Black" />
       </visual>
       <collision>
         <origin xyz="0 0 0" rpy="0 0 0" />
         <geometry>
-          <mesh filename="package://talos_description/meshes/arm/arm_7_collision.STL" scale="1 ${reflect} 1"/>
+          <mesh filename="package://talos_description/meshes/arm/arm_7_collision.dae" scale="1 ${reflect} 1"/>
         </geometry>
       </collision>
@@ -115,8 +115,10 @@
       <mu1>0.9</mu1>
       <mu2>0.9</mu2>
+      <material>Gazebo/White</material>
     </gazebo>
     <gazebo reference="${name}_${side}_6_link">
       <mu1>0.9</mu1>
       <mu2>0.9</mu2>
+      <material>Gazebo/White</material>
     </gazebo>
     <gazebo reference="${name}_${side}_7_link">

File: talos_description/urdf/gripper/gripper.urdf.xacro (robot description, xacro)
@@ -11,12 +11,12 @@
                 <origin xyz="0 0 0" rpy="0 0 0" />
                 <geometry>
-                  <mesh filename="package://talos_description/meshes/gripper/base_link.STL" scale="1 1 1"/>
-                </geometry>
-                <material name="DarkGrey"/>
-              </visual>
-              <collision>
-                <origin xyz="0 0 0" rpy="0 0 0" />
-                <geometry>
-                  <mesh filename="package://talos_description/meshes/gripper/base_link_collision.STL" scale="1 1 1"/>
+                  <mesh filename="package://talos_description/meshes/gripper/base_link.dae" scale="1 1 1"/>
+                </geometry>
+                <material name="Black"/>
+              </visual>
+              <collision>
+                <origin xyz="0 0 0" rpy="0 0 0" />
+                <geometry>
+                  <mesh filename="package://talos_description/meshes/gripper/base_link_collision.dae" scale="1 1 1"/>
                 </geometry>
               </collision>
@@ -34,5 +34,5 @@
                 <origin xyz="0 0 0" rpy="0 0 0" />
                 <geometry>
-                  <mesh filename="package://talos_description/meshes/gripper/gripper_motor_double.STL" scale="1 1 1"/>
+                  <mesh filename="package://talos_description/meshes/gripper/gripper_motor_double.dae" scale="1 1 1"/>
                 </geometry>
               <material name="Orange"/>
@@ -41,5 +41,5 @@
                 <origin xyz="0 0 0" rpy="0 0 0" />
                 <geometry>
-                  <mesh filename="package://talos_description/meshes/gripper/gripper_motor_double_collision.STL" scale="1 1 1"/>
+                  <mesh filename="package://talos_description/meshes/gripper/gripper_motor_double_collision.dae" scale="1 1 1"/>
                 </geometry>
               </collision>
@@ -59,5 +59,5 @@
                 <origin xyz="0 0 0" rpy="0 0 0" />
                 <geometry>
-                  <mesh filename="package://talos_description/meshes/gripper/inner_double.STL" scale="1 1 1"/>
+                  <mesh filename="package://talos_description/meshes/gripper/inner_double.dae" scale="1 1 1"/>
                 </geometry>
               <material name="Orange"/>
@@ -66,5 +66,5 @@
                 <origin xyz="0 0 0" rpy="0 0 0" />
                 <geometry>
-                  <mesh filename="package://talos_description/meshes/gripper/inner_double_collision.STL" scale="1 1 1"/>
+                  <mesh filename="package://talos_description/meshes/gripper/inner_double_collision.dae" scale="1 1 1"/>
                 </geometry>
               </collision>
@@ -84,12 +84,12 @@
                 <origin xyz="0 0 0" rpy="0 0 0" />
                 <geometry>
-                  <mesh filename="package://talos_description/meshes/gripper/fingertip.STL" scale="1 1 1"/>
-                </geometry>
-              <material name="DarkGrey"/>
-              </visual>
-              <collision>
-                <origin xyz="0 0 0" rpy="0 0 0" />
-                <geometry>
-                  <mesh filename="package://talos_description/meshes/gripper/fingertip_collision.STL" scale="1 1 1"/>
+                  <mesh filename="package://talos_description/meshes/gripper/fingertip.dae" scale="1 1 1"/>
+                </geometry>
+                <material name="Black"/>
+              </visual>
+              <collision>
+                <origin xyz="0 0 0" rpy="0 0 0" />
+                <geometry>
+                  <mesh filename="package://talos_description/meshes/gripper/fingertip_collision.dae" scale="1 1 1"/>
                 </geometry>
               </collision>
@@ -109,12 +109,12 @@
                 <origin xyz="0 0 0" rpy="0 0 0" />
                 <geometry>
-                  <mesh filename="package://talos_description/meshes/gripper/fingertip.STL" scale="1 1 1"/>
-                </geometry>
-                <material name="DarkGrey"/>
-              </visual>
-              <collision>
-                <origin xyz="0 0 0" rpy="0 0 0" />
-                <geometry>
-                  <mesh filename="package://talos_description/meshes/gripper/fingertip_collision.STL" scale="1 1 1"/>
+                  <mesh filename="package://talos_description/meshes/gripper/fingertip.dae" scale="1 1 1"/>
+                </geometry>
+                <material name="Black"/>
+              </visual>
+              <collision>
+                <origin xyz="0 0 0" rpy="0 0 0" />
+                <geometry>
+                  <mesh filename="package://talos_description/meshes/gripper/fingertip_collision.dae" scale="1 1 1"/>
                 </geometry>
               </collision>
@@ -134,12 +134,12 @@
                 <origin xyz="0 0 0" rpy="0 0 0" />
                 <geometry>
-                  <mesh filename="package://talos_description/meshes/gripper/gripper_motor_single.STL" scale="1 1 1"/>
-                </geometry>
-              <material name="Orange"/>
-              </visual>
-              <collision>
-                <origin xyz="0 0 0" rpy="0 0 0" />
-                <geometry>
-                  <mesh filename="package://talos_description/meshes/gripper/gripper_motor_single_collision.STL" scale="1 1 1"/>
+                  <mesh filename="package://talos_description/meshes/gripper/gripper_motor_single.dae" scale="1 1 1"/>
+                </geometry>
+                <material name="Orange"/>
+              </visual>
+              <collision>
+                <origin xyz="0 0 0" rpy="0 0 0" />
+                <geometry>
+                  <mesh filename="package://talos_description/meshes/gripper/gripper_motor_single_collision.dae" scale="1 1 1"/>
                 </geometry>
               </collision>
@@ -159,5 +159,5 @@
                 <origin xyz="0 0 0" rpy="0 0 0" />
                 <geometry>
-                  <mesh filename="package://talos_description/meshes/gripper/inner_single.STL" scale="1 1 1"/>
+                  <mesh filename="package://talos_description/meshes/gripper/inner_single.dae" scale="1 1 1"/>
                 </geometry>
               <material name="Orange"/>
@@ -166,5 +166,5 @@
                 <origin xyz="0 0 0" rpy="0 0 0" />
                 <geometry>
-                  <mesh filename="package://talos_description/meshes/gripper/inner_single_collision.STL" scale="1 1 1"/>
+                  <mesh filename="package://talos_description/meshes/gripper/inner_single_collision.dae" scale="1 1 1"/>
                 </geometry>
               </collision>
@@ -184,12 +184,12 @@
                 <origin xyz="0 0 0" rpy="0 0 0" />
                 <geometry>
-                  <mesh filename="package://talos_description/meshes/gripper/fingertip.STL" scale="1 1 1"/>
-                </geometry>
-              <material name="DarkGrey"/>
-              </visual>
-              <collision>
-                <origin xyz="0 0 0" rpy="0 0 0" />
-                <geometry>
-                  <mesh filename="package://talos_description/meshes/gripper/fingertip_collision.STL" scale="1 1 1"/>
+                  <mesh filename="package://talos_description/meshes/gripper/fingertip.dae" scale="1 1 1"/>
+                </geometry>
+              <material name="Black"/>
+              </visual>
+              <collision>
+                <origin xyz="0 0 0" rpy="0 0 0" />
+                <geometry>
+                  <mesh filename="package://talos_description/meshes/gripper/fingertip_collision.dae" scale="1 1 1"/>
                 </geometry>
               </collision>

File: talos_description/urdf/head/head.urdf.xacro (robot description, xacro)
@@ -27,12 +27,12 @@
         <origin xyz="0 0 0" rpy="0 0 0" />
         <geometry>
-          <mesh filename="package://talos_description/meshes/head/head_1.stl" scale="1 1 1"/>
+          <mesh filename="package://talos_description/meshes/head/head_1.dae" scale="1 1 1"/>
         </geometry>
-        <material name="DarkGrey" />
+        <material name="Black" />
       </visual>
       <collision>
         <origin xyz="0 0 0" rpy="0 0 0" />
         <geometry>
-          <mesh filename="package://talos_description/meshes/head/head_1_collision.stl" scale="1 1 1"/>
+          <mesh filename="package://talos_description/meshes/head/head_1_collision.dae" scale="1 1 1"/>
         </geometry>
       </collision>
@@ -71,12 +71,12 @@
         <origin xyz="0 0 0" rpy="0 0 0" />
         <geometry>
-          <mesh filename="package://talos_description/meshes/head/head_2.stl" scale="1 1 1"/>
+          <mesh filename="package://talos_description/meshes/head/head_2.dae" scale="1 1 1"/>
         </geometry>
-        <material name="LightGrey" />
+        <material name="White" />
       </visual>
       <collision>
         <origin xyz="0 0 0" rpy="0 0 0" />
         <geometry>
-          <mesh filename="package://talos_description/meshes/head/head_2_collision.stl" scale="1 1 1"/>
+          <mesh filename="package://talos_description/meshes/head/head_2_collision.dae" scale="1 1 1"/>
         </geometry>
       </collision>
@@ -98,10 +98,8 @@
       <mu1>0.9</mu1>
       <mu2>0.9</mu2>
+      <material>Gazebo/White</material>
     </gazebo>
     <gazebo reference="${name}_joint">
        <implicitSpringDamper>1</implicitSpringDamper>
-    </gazebo>
-    <gazebo reference="${name}_link">
-      <material>Gazebo/White</material>
     </gazebo>
   </xacro:macro>

File: talos_description/urdf/leg/foot_collision_default.urdf.xacro (robot description, xacro)
@@ -5,5 +5,5 @@
             <origin xyz="0 0 0" rpy="0 0 0" />
             <geometry>
-                <mesh filename="package://talos_description/meshes/v2/ankle_X_collision.stl" scale="1 ${reflect*1} 1"/>
+                <mesh filename="package://talos_description/meshes/v2/ankle_X_collision.dae" scale="1 ${reflect*1} 1"/>
             </geometry>
         </collision>

File: talos_description/urdf/leg/leg.urdf.xacro (robot description, xacro)
@@ -15,12 +15,12 @@
         <origin rpy="0 0 0" xyz="0 0 0"/>
         <geometry>
-          <mesh filename="package://talos_description/meshes/v2/hip_z_lo_res.stl" scale="1 ${reflect*1} 1"/>
-        </geometry>
-        <material name="DarkGrey" />
-      </visual>
-      <collision>
-        <origin rpy="0 0 0" xyz="0 0 0"/>
-        <geometry>
-           <mesh filename="package://talos_description/meshes/v2/hip_z_collision.stl" scale="1 ${reflect*1} 1"/>
+          <mesh filename="package://talos_description/meshes/v2/hip_z_lo_res.dae" scale="1 ${reflect*1} 1"/>
+        </geometry>
+        <material name="Black" />
+      </visual>
+      <collision>
+        <origin rpy="0 0 0" xyz="0 0 0"/>
+        <geometry>
+           <mesh filename="package://talos_description/meshes/v2/hip_z_collision.dae" scale="1 ${reflect*1} 1"/>
         </geometry>
       </collision>
@@ -41,12 +41,12 @@
         <origin xyz="0 0 0.0" rpy="0  0  0" />
         <geometry>
-          <mesh filename="package://talos_description/meshes/v2/hip_x_lo_res.stl" scale="1 ${reflect*1} 1"/>
-        </geometry>
-        <material name="DarkGrey" />
+          <mesh filename="package://talos_description/meshes/v2/hip_x_lo_res.dae" scale="1 ${reflect*1} 1"/>
+        </geometry>
+        <material name="Black" />
       </visual>
       <collision>
         <origin xyz="0 0 0.0" rpy="0  0  0" />
         <geometry>
-          <mesh filename="package://talos_description/meshes/v2/hip_x_collision.stl" scale="1 ${reflect*1} 1"/>
+          <mesh filename="package://talos_description/meshes/v2/hip_x_collision.dae" scale="1 ${reflect*1} 1"/>
         </geometry>
       </collision>
@@ -67,12 +67,12 @@
         <origin rpy="0 0 0" xyz="0 0 0"/>
         <geometry>
-          <mesh filename="package://talos_description/meshes/v2/hip_y_lo_res.stl" scale="1 ${reflect*1} 1"/>
-        </geometry>
-        <material name="DarkGrey" />
-      </visual>
-      <collision>
-        <origin rpy="0 0 0" xyz="0 0 0"/>
-        <geometry>
-           <mesh filename="package://talos_description/meshes/v2/hip_y_collision.stl" scale="1 ${reflect*1} 1"/>
+          <mesh filename="package://talos_description/meshes/v2/hip_y_lo_res.dae" scale="1 ${reflect*1} 1"/>
+        </geometry>
+        <material name="Black" />
+      </visual>
+      <collision>
+        <origin rpy="0 0 0" xyz="0 0 0"/>
+        <geometry>
+           <mesh filename="package://talos_description/meshes/v2/hip_y_collision.dae" scale="1 ${reflect*1} 1"/>
         </geometry>
       </collision>
@@ -93,12 +93,12 @@
         <origin rpy="0 0 0" xyz="0 0 0"/>
         <geometry>
-          <mesh filename="package://talos_description/meshes/v2/knee_lo_res.stl" scale="1 ${reflect*1} 1"/>
-        </geometry>
-        <material name="DarkGrey" />
-      </visual>
-      <collision>
-        <origin rpy="0 0 0" xyz="0 0 0"/>
-        <geometry>
-           <mesh filename="package://talos_description/meshes/v2/knee_collision.stl" scale="1 ${reflect*1} 1"/>
+          <mesh filename="package://talos_description/meshes/v2/knee_lo_res.dae" scale="1 ${reflect*1} 1"/>
+        </geometry>
+        <material name="Black" />
+      </visual>
+      <collision>
+        <origin rpy="0 0 0" xyz="0 0 0"/>
+        <geometry>
+           <mesh filename="package://talos_description/meshes/v2/knee_collision.dae" scale="1 ${reflect*1} 1"/>
         </geometry>
       </collision>
@@ -120,12 +120,12 @@
         <origin xyz="0 0 0.0" rpy="0 0 0" />
         <geometry>
-          <mesh filename="package://talos_description/meshes/v2/ankle_Y_lo_res.stl" scale="1 ${reflect*1} 1"/>
-        </geometry>
-        <material name="Grey" />
+          <mesh filename="package://talos_description/meshes/v2/ankle_Y_lo_res.dae" scale="1 ${reflect*1} 1"/>
+        </geometry>
+        <material name="White" />
       </visual>
       <collision>
         <origin xyz="0 0 0.0" rpy="0 0 0" />
         <geometry>
-          <mesh filename="package://talos_description/meshes/v2/ankle_Y_collision.stl" scale="1 ${reflect*1} 1"/>
+          <mesh filename="package://talos_description/meshes/v2/ankle_Y_collision.dae" scale="1 ${reflect*1} 1"/>
         </geometry>
       </collision>
@@ -146,7 +146,7 @@
         <origin rpy="0 0 0" xyz="0 0 0"/>
         <geometry>
-          <mesh filename="package://talos_description/meshes/v2/ankle_X_lo_res.stl" scale="1 ${reflect*1} 1"/>
-        </geometry>
-        <material name="Grey" />
+          <mesh filename="package://talos_description/meshes/v2/ankle_X_lo_res.dae" scale="1 ${reflect*1} 1"/>
+        </geometry>
+        <material name="White" />
       </visual>
       <xacro:talos_foot_collision />

File: talos_description/urdf/materials.urdf.xacro (robot description, xacro)
@@ -32,3 +32,6 @@
     <color rgba="1.0 0.5 0.0 1.0"/>
   </material>
+  <material name="Black">
+    <color rgba="0.0 0.0 0.0 1.0"/>
+  </material>
 </robot>

File: talos_description/urdf/sensors/orbbec_astra_pro.urdf.xacro (robot description, xacro)
@@ -35,9 +35,6 @@
         <origin xyz="0 0 0" rpy="0 0 0"/>
         <geometry>
-          <mesh filename="package://talos_description/meshes/sensors/orbbec/orbbec.STL" />
+          <mesh filename="package://talos_description/meshes/sensors/orbbec/orbbec.dae" />
         </geometry>
-        <material name="DarkGrey">
-          <color rgba="0.5 0.5 0.5 1"/>
-        </material>
       </visual>
       <collision>
