Commit message: Use DAE with texture for color

File: talos_description/urdf/torso/torso.urdf.xacro (robot description, xacro)
@@ -25,12 +25,11 @@
         <origin xyz="0 0 0" rpy="0 0 0" />
         <geometry>
-          <mesh filename="package://talos_description/meshes/torso/torso_2.STL" scale="1 1 1"/>
+          <mesh filename="package://talos_description/meshes/torso/torso_2.dae" scale="1 1 1"/>
         </geometry>
-        <material name="LightGrey" />
       </visual>
       <collision>
         <origin xyz="0 0 0" rpy="0 0 0" />
         <geometry>
-          <mesh filename="package://talos_description/meshes/torso/torso_2_collision.STL" scale="1 1 1"/>
+          <mesh filename="package://talos_description/meshes/torso/torso_2_collision.dae" scale="1 1 1"/>
         </geometry>
       </collision>
@@ -44,12 +43,11 @@
         <origin xyz="0 0 0" rpy="0 0 0" />
         <geometry>
-          <mesh filename="package://talos_description/meshes/torso/torso_1.STL" scale="1 1 1"/>
+          <mesh filename="package://talos_description/meshes/torso/torso_1.dae" scale="1 1 1"/>
         </geometry>
-        <material name="LightGrey" />
       </visual>
       <collision>
         <origin xyz="0 0 0" rpy="0 0 0" />
         <geometry>
-          <mesh filename="package://talos_description/meshes/torso/torso_1.STL" scale="1 1 1"/>
+          <mesh filename="package://talos_description/meshes/torso/torso_1.dae" scale="1 1 1"/>
         </geometry>
       </collision>
@@ -78,12 +76,11 @@
         <origin xyz="0 0 0" rpy="0 0 0" />
         <geometry>
-          <mesh filename="package://talos_description/meshes/torso/base_link.STL" scale="1 1 1"/>
+          <mesh filename="package://talos_description/meshes/torso/base_link.dae" scale="1 1 1"/>
         </geometry>
-        <material name="LightGrey" />
       </visual>
       <collision>
         <origin xyz="0 0 0" rpy="0 0 0" />
         <geometry>
-          <mesh filename="package://talos_description/meshes/torso/base_link_collision.STL" scale="1 1 1"/>
+          <mesh filename="package://talos_description/meshes/torso/base_link_collision.dae" scale="1 1 1"/>
         </geometry>
       </collision>
@@ -109,12 +106,15 @@
         <mu1>0.9</mu1>
         <mu2>0.9</mu2>
+        <material>Gazebo/White</material>
     </gazebo>
     <gazebo reference="${name}_2_link">
         <mu1>0.9</mu1>
         <mu2>0.9</mu2>
+        <material>Gazebo/White</material>
     </gazebo>
     <gazebo reference="base_link">
         <mu1>0.9</mu1>
         <mu2>0.9</mu2>
+        <material>Gazebo/White</material>
     </gazebo>
     <gazebo reference="${name}_1_joint">

Commit message: Lower body calibration

File: talos_description/urdf/arm/arm.urdf.xacro (robot description, xacro)
@@ -25,5 +25,10 @@
   <xacro:property name="arm_eps"            value="0.02" />
   <xacro:macro name="talos_arm" params="name parent side reflect">
-    <xacro:include filename="$(find talos_description_calibration)/urdf/calibration/arm_${side}.xacro" />
+    <xacro:unless value="$(arg test)">
+      <xacro:include filename="$(find talos_description_calibration)/urdf/calibration/arm_${side}.xacro" />
+    </xacro:unless>
+    <xacro:if value="$(arg test)">
+      <xacro:include filename="$(find talos_description)/test/calibration/arm_${side}.xacro" />
+    </xacro:if>
     <!--************************-->
     <!--        SHOULDER        -->

File: talos_description/urdf/arm/wrist.urdf.xacro (robot description, xacro)
@@ -22,5 +22,10 @@
   <xacro:property name="wrist_eps"          value="0.02" />
   <xacro:macro name="talos_wrist" params="name parent side reflect">
-    <xacro:include filename="$(find talos_description_calibration)/urdf/calibration/arm_${side}.xacro" />
+    <xacro:unless value="$(arg test)">
+      <xacro:include filename="$(find talos_description_calibration)/urdf/calibration/arm_${side}.xacro" />
+    </xacro:unless>
+    <xacro:if value="$(arg test)">
+      <xacro:include filename="$(find talos_description)/test/calibration/arm_${side}.xacro" />
+    </xacro:if>
     <!--************************-->
     <!--        WRIST           -->

File: talos_description/urdf/head/head.urdf.xacro (robot description, xacro)
@@ -12,5 +12,10 @@
   <xacro:include filename="$(find talos_description)/urdf/head/head.transmission.xacro" />
   <xacro:include filename="$(find talos_description)/urdf/sensors/orbbec_astra_pro.urdf.xacro" />
-  <xacro:include filename="$(find talos_description_calibration)/urdf/calibration/calibration_constants.urdf.xacro" />
+  <xacro:unless value="$(arg test)">
+    <xacro:include filename="$(find talos_description_calibration)/urdf/calibration/calibration_constants.urdf.xacro" />
+  </xacro:unless>
+  <xacro:if value="$(arg test)">
+    <xacro:include filename="$(find talos_description)/test/calibration/calibration_constants.urdf.xacro" />
+  </xacro:if>
   <!--Constant parameters-->
   <xacro:property name="head_friction" value="1.0" />

File: talos_description/urdf/leg/leg.urdf.xacro (robot description, xacro)
@@ -9,4 +9,10 @@
   <xacro:property name="leg_damping"      value="0.0" />
   <xacro:macro name="talos_leg" params="prefix reflect">
+    <xacro:unless value="$(arg test)">
+      <xacro:include filename="$(find talos_description_calibration)/urdf/calibration/leg_${prefix}.xacro" />
+    </xacro:unless>
+    <xacro:if value="$(arg test)">
+      <xacro:include filename="$(find talos_description)/test/calibration/leg_${prefix}.xacro" />
+    </xacro:if>
     <!-- Joint hip_z (mesh link) : child link hip_x -> parent link base_link -->
     <link name="leg_${prefix}_1_link">
@@ -29,6 +35,6 @@
       <parent link="base_link"/>
       <child link="leg_${prefix}_1_link"/>
-      <origin xyz="-0.02 ${reflect*0.08500} -0.27105"
-              rpy="${0.00000 * deg_to_rad} ${0.00000 * deg_to_rad} ${0.00000 * deg_to_rad}"/>
+      <origin xyz="${-0.02 + leg_1_joint_x_offset} ${reflect*0.08500 + leg_1_joint_y_offset} ${-0.27105 + leg_1_joint_z_offset}"
+              rpy="${0.00000 * deg_to_rad + leg_1_joint_roll_offset} ${0.00000 * deg_to_rad + leg_1_joint_pitch_offset} ${0.00000 * deg_to_rad + leg_1_joint_yaw_offset}"/>
       <axis xyz="0 0 1" />
       <limit lower="${(-55.0 + 35.0*reflect)*deg_to_rad}" upper="${(55.0 + 35.0*reflect)*deg_to_rad}" effort="100" velocity="3.87" />
@@ -55,6 +61,6 @@
       <parent link="leg_${prefix}_1_link"/>
       <child link="leg_${prefix}_2_link"/>
-      <origin xyz="0.00000 0.00000 0.00000"
-              rpy="${0.00000 * deg_to_rad} ${0.00000 * deg_to_rad} ${0.00000 * deg_to_rad}"/>
+      <origin xyz="${0.00000 + leg_2_joint_x_offset} ${0.00000 + leg_2_joint_y_offset} ${0.00000 + leg_2_joint_z_offset}"
+              rpy="${0.00000 * deg_to_rad + leg_2_joint_roll_offset} ${0.00000 * deg_to_rad + leg_2_joint_pitch_offset} ${0.00000 * deg_to_rad + leg_2_joint_yaw_offset}"/>
       <axis xyz="1 0 0" />
       <limit lower="-0.5236" upper="0.5236" effort="160" velocity="5.8" />
@@ -81,6 +87,6 @@
       <parent link="leg_${prefix}_2_link"/>
       <child link="leg_${prefix}_3_link"/>
-      <origin xyz="0.00000 0.00000 0.00000"
-              rpy="${0.00000 * deg_to_rad} ${0.00000 * deg_to_rad} ${0.00000 * deg_to_rad}"/>
+      <origin xyz="${0.00000 + leg_3_joint_x_offset} ${0.00000 + leg_3_joint_y_offset} ${0.00000 + leg_3_joint_z_offset}"
+              rpy="${0.00000 * deg_to_rad + leg_3_joint_roll_offset} ${0.00000 * deg_to_rad + leg_3_joint_pitch_offset} ${0.00000 * deg_to_rad + leg_3_joint_yaw_offset}"/>
       <axis xyz="0 1 0" />
       <limit lower="-2.095" upper="0.7" effort="160" velocity="5.8" />
@@ -107,6 +113,6 @@
       <parent link="leg_${prefix}_3_link"/>
       <child link="leg_${prefix}_4_link"/>
-      <origin xyz="0.00000 0.00000 -0.38000"
-              rpy="${0.00000 * deg_to_rad} ${0.00000 * deg_to_rad} ${0.00000 * deg_to_rad}"/>
+      <origin xyz="${0.00000 + leg_4_joint_x_offset} ${0.00000 + leg_4_joint_y_offset} ${-0.38000 + leg_4_joint_z_offset}"
+              rpy="${0.00000 * deg_to_rad + leg_4_joint_roll_offset} ${0.00000 * deg_to_rad + leg_4_joint_pitch_offset} ${0.00000 * deg_to_rad + leg_4_joint_yaw_offset}"/>
       <axis xyz="0 1 0" />
       <limit lower="0" upper="2.618" effort="400" velocity="7" />
@@ -134,6 +140,6 @@
       <parent link="leg_${prefix}_4_link"/>
       <child link="leg_${prefix}_5_link"/>
-      <origin xyz="0.00000 0.00000 -0.32500"
-              rpy="${0.00000 * deg_to_rad} ${0.00000 * deg_to_rad} ${0.00000 * deg_to_rad}"/>
+      <origin xyz="${0.00000 + leg_5_joint_x_offset} ${0.00000 + leg_5_joint_y_offset} ${-0.32500 + leg_5_joint_z_offset}"
+              rpy="${0.00000 * deg_to_rad + leg_5_joint_roll_offset} ${0.00000 * deg_to_rad + leg_5_joint_pitch_offset} ${0.00000 * deg_to_rad + leg_5_joint_yaw_offset}"/>
       <axis xyz="0 1 0" />
       <limit lower="-1.27" upper="0.68" effort="160" velocity="5.8" />
@@ -155,6 +161,6 @@
       <parent link="leg_${prefix}_5_link"/>
       <child link="leg_${prefix}_6_link"/>
-      <origin xyz="0.00000 0.00000 0.00000"
-              rpy="${0.00000 * deg_to_rad} ${0.00000 * deg_to_rad} ${0.00000 * deg_to_rad}"/>
+      <origin xyz="${0.00000 + leg_6_joint_x_offset} ${0.00000 + leg_6_joint_y_offset} ${0.00000 + leg_6_joint_z_offset}"
+              rpy="${0.00000 * deg_to_rad + leg_6_joint_roll_offset} ${0.00000 * deg_to_rad + leg_6_joint_pitch_offset} ${0.00000 * deg_to_rad + leg_6_joint_yaw_offset}"/>
       <axis xyz="1 0 0" />
       <limit lower="-0.5236" upper="0.5236" effort="100" velocity="4.8" />

File: talos_description/urdf/torso/torso.urdf.xacro (robot description, xacro)
@@ -12,5 +12,10 @@
   <xacro:include filename="$(find talos_description)/urdf/torso/torso.transmission.xacro" />
   <xacro:include filename="$(find talos_description)/urdf/sensors/imu.urdf.xacro" />
-  <xacro:include filename="$(find talos_description_calibration)/urdf/calibration/calibration_constants.urdf.xacro" />
+  <xacro:unless value="$(arg test)">
+    <xacro:include filename="$(find talos_description_calibration)/urdf/calibration/calibration_constants.urdf.xacro" />
+  </xacro:unless>
+  <xacro:if value="$(arg test)">
+    <xacro:include filename="$(find talos_description)/test/calibration/calibration_constants.urdf.xacro" />
+  </xacro:if>
  <!--Constant parameters-->
   <xacro:property name="torso_max_vel"  value="5.4" />

Commit message: Make modifications for the UEDIN markers

File: talos_description/urdf/arm/arm.urdf.xacro (robot description, xacro)
@@ -143,5 +143,5 @@
       <parent link="${name}_${side}_3_link" />
       <child link="${name}_${side}_4_link" />
-      <origin xyz="${0.02000 + arm_4_joint_x_offset} ${0.00000 + arm_4_joint_y_offset} ${-0.27300 + arm_4_joint_z_offset}"
+      <origin xyz="${0.02000 + arm_4_joint_x_offset} ${0.00000 + arm_4_joint_y_offset} ${-0.2782 + arm_4_joint_z_offset}"
               rpy="${0.00000 * deg_to_rad + arm_4_joint_roll_offset} ${0.00000 * deg_to_rad + arm_4_joint_pitch_offset} ${0.00000 * deg_to_rad + arm_4_joint_yaw_offset}"/>
       <axis xyz="0 1 0" />

File: talos_description/urdf/head/head.urdf.xacro (robot description, xacro)
@@ -46,6 +46,6 @@
       <parent link="${parent}"/>
       <child link="${name}_link"/>
-      <origin xyz="${0.02000 + head_1_joint_x_offset} ${0.00000 + head_1_joint_y_offset} ${0.32100 + head_1_joint_z_offset}"
-              rpy="${0.00000 * deg_to_rad + head_1_joint_roll_offset} ${0.00000 * deg_to_rad + head_1_joint_pitch_offset} ${0.00000 * deg_to_rad + head_1_joint_yaw_offset}"/>
+      <origin xyz="${0.0 + head_1_joint_x_offset} ${0.0 + head_1_joint_y_offset} ${0.316 + head_1_joint_z_offset}"
+              rpy="${0.0 * deg_to_rad + head_1_joint_roll_offset} ${0.0 * deg_to_rad + head_1_joint_pitch_offset} ${0.0 * deg_to_rad + head_1_joint_yaw_offset}"/>
       <axis xyz="0 1 0" />
       <limit lower="${-12.00000 * deg_to_rad}" upper="${45.00000 * deg_to_rad}" effort="8.0" velocity="${head_max_vel}" />
@@ -90,8 +90,8 @@
       <parent link="${parent}"/>
       <child link="${name}_link"/>
-      <origin xyz="${0.00000 + head_2_joint_x_offset} ${0.00000 + head_2_joint_y_offset} ${0.00000 + head_2_joint_z_offset}"
-              rpy="${0.00000 * deg_to_rad + head_2_joint_roll_offset} ${0.00000 * deg_to_rad + head_2_joint_pitch_offset} ${0.00000 * deg_to_rad + head_2_joint_yaw_offset}"/>
+      <origin xyz="${0.0 + head_2_joint_x_offset} ${0.0 + head_2_joint_y_offset} ${0.0 + head_2_joint_z_offset}"
+              rpy="${0.0 * deg_to_rad + head_2_joint_roll_offset} ${0.0 * deg_to_rad + head_2_joint_pitch_offset} ${0.0 * deg_to_rad + head_2_joint_yaw_offset}"/>
       <axis xyz="0 0 1" />
-      <limit lower="${-75.00000 * deg_to_rad}" upper="${75.00000 * deg_to_rad}" effort="4.0" velocity="${head_max_vel}" />
+      <limit lower="${-75.0 * deg_to_rad}" upper="${75.0 * deg_to_rad}" effort="4.0" velocity="${head_max_vel}" />
       <dynamics damping="${head_damping}" friction="${head_friction}"/>
        <!-- <safety_controller k_position="20"

File: talos_description/urdf/sensors/orbbec_astra_pro.urdf.xacro (robot description, xacro)
@@ -58,5 +58,5 @@
     <!-- frames of the depth sensor -->
     <joint name="${name}_depth_joint" type="fixed">
-      <origin xyz="0.0 0.03751 0.0" rpy="0 0 0" />
+      <origin xyz="0.0033 0.0 0.0" rpy="0 0 0" />
       <parent link="${name}_link" />
       <child link="${name}_depth_frame"/>
@@ -71,5 +71,5 @@
     <!-- frames of the rgb sensor -->
     <joint name="${name}_rgb_joint" type="fixed">
-      <origin xyz="0.0 0.01251 0.0" rpy="0 0 0" />
+      <origin xyz="0.033 -0.025 0.0" rpy="0 0 0" />
       <parent link="${name}_link" />
       <child link="${name}_rgb_frame"/>

File: talos_description_calibration/urdf/calibration/calibration_constants.urdf.xacro (robot description, xacro)
@@ -11,7 +11,7 @@
   <xacro:include filename="$(find talos_description_calibration)/urdf/deg_to_rad.xacro" />
   <!--Constant parameters-->
-  <xacro:property name="camera_position_x" value="0.066" />
-  <xacro:property name="camera_position_y" value="0.0" />
-  <xacro:property name="camera_position_z" value="0.1982" />
+  <xacro:property name="camera_position_x" value="0.0621" />
+  <xacro:property name="camera_position_y" value="0.0375" />
+  <xacro:property name="camera_position_z" value="0.1832" />
   <xacro:property name="camera_orientation_r" value="0.0" />
   <xacro:property name="camera_orientation_p" value="0.0" />

File: talos_description_inertial/urdf/inertial.xacro (robot description, xacro)
@@ -31,7 +31,7 @@
   <xacro:macro name="arm_left_4_link_inertial">
     <inertial>
-      <mass value="0.877346"/>
-      <inertia ixx="0.00251207716" ixy="0.00010070062" ixz="-0.00032788214" iyy="0.00275869324" iyz="0.00040022227" izz="0.00120735959" />
-      <origin rpy="0 0 0" xyz="-0.00742138 -0.0213895 -0.03312656"/>
+      <mass value="0.815675"/>
+      <inertia ixx="0.00299913" ixy="-0.00009333" ixz="0.0003389" iyy="0.00303994" iyz="-0.0004233" izz="0.00126248" />
+      <origin rpy="0 0 0" xyz="-0.00810404 -0.01944328 -0.03329237"/>
     </inertial>
   </xacro:macro>
@@ -80,7 +80,7 @@
   <xacro:macro name="arm_right_4_link_inertial">
     <inertial>
-      <mass value="0.877346"/>
-      <inertia ixx="0.00251207716" ixy="-0.00010070062" ixz="-0.00032788214" iyy="0.00275869324" iyz="-0.00040022227" izz="0.00120735959" />
-      <origin rpy="0 0 0" xyz="-0.00742138 0.0213895 -0.03312656"/>
+      <mass value="0.815675"/>
+      <inertia ixx="0.00299913" ixy="-0.00009333" ixz="0.0003389" iyy="0.00303994" iyz="-0.0004233" izz="0.00126248" />
+      <origin rpy="0 0 0" xyz="-0.00810404 -0.01944328 -0.03329237"/>
     </inertial>
   </xacro:macro>
@@ -227,14 +227,14 @@
   <xacro:macro name="head_1_link_inertial">
     <inertial>
-      <mass value="0.73746"/>
-      <inertia ixx="0.00224878584" ixy="4.69375e-06" ixz="8.55557e-05" iyy="0.00111158492" iyz="-4.132536e-05" izz="0.00205225921" />
-      <origin rpy="0 0 0" xyz="-0.00157211 -0.00157919 0.02175767"/>
+      <mass value="0.645847"/>
+      <inertia ixx="0.00162283" ixy="0.00000775" ixz="-0.00007338" iyy="0.00101072" iyz="-0.0001584" izz="0.00155812" />
+      <origin rpy="0 0 0" xyz="-0.00170599 0.00951995 0.02791276"/>
     </inertial>
   </xacro:macro>
   <xacro:macro name="head_2_link_inertial">
     <inertial>
-      <mass value="1.443954"/>
-      <inertia ixx="0.01084624339" ixy="1.050889e-05" ixz="0.00041594252" iyy="0.0109569176" iyz="2.367831e-05" izz="0.00571698895" />
-      <origin rpy="0 0 0" xyz="0.01002657 5.218e-05 0.14136068"/>
+      <mass value="1.297575"/>
+      <inertia ixx="0.01045038" ixy="0.00011521" ixz="-0.00021127" iyy="0.0099128" iyz="0.00107457" izz="0.0057925" />
+      <origin rpy="0 0 0" xyz="0.01425088 -0.00602046 0.13890363"/>
     </inertial>
   </xacro:macro>
@@ -255,7 +255,7 @@
   <xacro:macro name="leg_left_1_link_inertial">
     <inertial>
-      <mass value="1.845591"/>
-      <inertia ixx="0.00541533521" ixy="-0.00015428714" ixz="0.00131612622" iyy="0.00848624936" iyz="-1.906103e-05" izz="0.00474512541" />
-      <origin rpy="0 0 0" xyz="0.02247868 0.00106736 0.03130665"/>
+      <mass value="2.235009"/>
+      <inertia ixx="0.01049849" ixy="0.00004097" ixz="0.00009771" iyy="0.00534086" iyz="-0.0011949" izz="0.00708595" />
+      <origin rpy="0 0 0" xyz="0.08472839 -0.10997434 0.01705898"/>
     </inertial>
   </xacro:macro>
@@ -297,7 +297,7 @@
   <xacro:macro name="leg_right_1_link_inertial">
     <inertial>
-      <mass value="1.845591"/>
-      <inertia ixx="0.00541533521" ixy="0.00015428714" ixz="0.00131612622" iyy="0.00848624936" iyz="1.906103e-05" izz="0.00474512541" />
-      <origin rpy="0 0 0" xyz="0.02247868 -0.00106736 0.03130665"/>
+      <mass value="2.235009"/>
+      <inertia ixx="0.01049849" ixy="0.00004097" ixz="0.00009771" iyy="0.00534086" iyz="-0.0011949" izz="0.00708595" />
+      <origin rpy="0 0 0" xyz="0.08472839 -0.10997434 0.01705898"/>
     </inertial>
   </xacro:macro>

Commit message: Add detachable gripper base link to the arm_7_link

File: talos_description/urdf/arm/arm.urdf.xacro (robot description, xacro)
@@ -188,5 +188,5 @@
     <!--        WRIST           -->
     <!--************************-->
-     <xacro:talos_wrist name="arm" parent="${name}_${side}_4_link" side="${side}" reflect="${reflect}" />
+     <xacro:talos_wrist name="arm" parent="${name}_${side}_4_link" side="${side}" reflect="${reflect}" gripper_type="detachable"/>
     <!-- extensions -->
     <xacro:include filename="$(find talos_description)/urdf/arm/${side}_arm.transmissions.urdf.xacro" />

File: talos_description/urdf/arm/wrist.urdf.xacro (robot description, xacro)
@@ -21,5 +21,5 @@
   <xacro:property name="wrist_3_max_effort"   value="8.0" />
   <xacro:property name="wrist_eps"          value="0.02" />
-  <xacro:macro name="talos_wrist" params="name parent side reflect">
+  <xacro:macro name="talos_wrist" params="name parent side reflect gripper_type">
     <xacro:unless value="$(arg test)">
       <xacro:include filename="$(find talos_description_calibration)/urdf/calibration/arm_${side}.xacro" />
@@ -90,9 +90,9 @@
     </joint>
     <link name="${name}_${side}_7_link">
-      <xacro:call macro="${name}_${side}_7_link_inertial" />
+      <xacro:call macro="${name}_${side}_7_link_inertial" gripper_type="${gripper_type}"/>
       <visual>
         <origin xyz="0 0 0" rpy="0 0 0" />
         <geometry>
-          <mesh filename="package://talos_description/meshes/arm/arm_7.STL" scale="1 ${reflect} 1"/>
+          <mesh filename="package://talos_description/meshes/arm/arm_7_${gripper_type}.STL" scale="1 ${reflect} 1"/>
         </geometry>
         <material name="DarkGrey" />

File: talos_description_inertial/urdf/inertial.xacro (robot description, xacro)
@@ -50,10 +50,19 @@
     </inertial>
   </xacro:macro>
-  <xacro:macro name="arm_left_7_link_inertial">
-    <inertial>
-      <mass value="0.308441"/>
-      <inertia ixx="0.00030894317" ixy="-1.58687e-06" ixz="1.73418e-06" iyy="0.00021886181" iyz="-1.221167e-05" izz="0.00017519492" />
-      <origin rpy="0 0 0" xyz="0.007525 0.001378 -0.02463"/>
-    </inertial>
+  <xacro:macro name="arm_left_7_link_inertial" params="gripper_type">
+    <xacro:if value="${gripper_type == 'classic'}">
+      <inertial>
+        <mass value="0.308441"/>
+        <inertia ixx="0.00030894317" ixy="-1.58687e-06" ixz="1.73418e-06" iyy="0.00021886181" iyz="-1.221167e-05" izz="0.00017519492" />
+        <origin rpy="0 0 0" xyz="0.007525 0.001378 -0.02463"/>
+      </inertial>
+    </xacro:if>
+    <xacro:if value="${gripper_type == 'detachable'}">
+      <inertial>
+        <mass value="0.31314"/>
+        <origin xyz="-0.0029817 -0.00046512 -0.052845" rpy="0 0 0" />
+        <inertia ixx="0.00030716" ixy="2.8257E-06" ixz="-7.0302E-06" iyy="0.00023544" iyz="-5.7534E-06" izz="0.00028541" />
+      </inertial>
+    </xacro:if>
   </xacro:macro>
   <xacro:macro name="arm_right_1_link_inertial">
@@ -99,10 +108,19 @@
     </inertial>
   </xacro:macro>
-  <xacro:macro name="arm_right_7_link_inertial">
-    <inertial>
-      <mass value="0.308441"/>
-      <inertia ixx="0.00030894317" ixy="1.58687e-06" ixz="1.73418e-06" iyy="0.00021886181" iyz="1.221167e-05" izz="0.00017519492" />
-      <origin rpy="0 0 0" xyz="0.007525 -0.001378 -0.02463"/>
-    </inertial>
+  <xacro:macro name="arm_right_7_link_inertial" params="gripper_type">
+    <xacro:if value="${gripper_type == 'classic'}">
+      <inertial>
+        <mass value="0.308441"/>
+        <inertia ixx="0.00030894317" ixy="1.58687e-06" ixz="1.73418e-06" iyy="0.00021886181" iyz="1.221167e-05" izz="0.00017519492" />
+        <origin rpy="0 0 0" xyz="0.007525 -0.001378 -0.02463"/>
+      </inertial>
+    </xacro:if>
+    <xacro:if value="${gripper_type == 'detachable'}">
+      <inertial>
+        <mass value="0.31314"/>
+        <origin xyz="-0.0029817 0.00046512 -0.052845" rpy="0 0 0" />
+        <inertia ixx="0.00030716" ixy="-2.8257E-06" ixz="-7.0302E-06" iyy="0.00023544" iyz="5.7534E-06" izz="0.00028541" />
+      </inertial>
+    </xacro:if>
   </xacro:macro>
   <xacro:macro name="base_link_inertial">
