Commit message: Add gripper top and bottom camera links

File: talos_description/urdf/arm/arm.urdf.xacro (robot description, xacro)
@@ -188,5 +188,5 @@
     <!--        WRIST           -->
     <!--************************-->
-     <xacro:talos_wrist name="arm" parent="${name}_${side}_4_link" side="${side}" reflect="${reflect}" gripper_type="detachable"/>
+     <xacro:talos_wrist name="arm" parent="${name}_${side}_4_link" side="${side}" reflect="${reflect}" gripper_type="detachable" gripper_camera="true"/>
     <!-- extensions -->
     <xacro:include filename="$(find talos_description)/urdf/arm/${side}_arm.transmissions.urdf.xacro" />

File: talos_description/urdf/arm/wrist.urdf.xacro (robot description, xacro)
@@ -21,5 +21,5 @@
   <xacro:property name="wrist_3_max_effort"   value="8.0" />
   <xacro:property name="wrist_eps"          value="0.02" />
-  <xacro:macro name="talos_wrist" params="name parent side reflect gripper_type">
+  <xacro:macro name="talos_wrist" params="name parent side reflect gripper_type gripper_camera">
     <xacro:unless value="$(arg test)">
       <xacro:include filename="$(find talos_description_calibration)/urdf/calibration/arm_${side}.xacro" />
@@ -118,4 +118,62 @@
                           soft_upper_limit="${40.00000 * deg_to_rad - eps_radians}" /> -->
     </joint>
+    <xacro:if value="${gripper_camera}">
+      <link name="${name}_${side}_wrist_left_camera_link">
+        <inertial>
+          <origin xyz="0.01021 -0.00042075 -0.00034305" rpy="0 0 0" />
+          <mass value="0.030268" />
+          <inertia ixx="4.4282E-05" ixy="-1.6339E-07" ixz="7.9036E-06" iyy="3.4321E-05" iyz="3.6964E-07" izz="1.7371E-05" />
+        </inertial>
+        <visual>
+          <origin xyz="0 0 0" rpy="0 0 0" />
+          <geometry>
+            <mesh filename="package://talos_arm_tool_changer/meshes/camera_left_wrist_link.STL" />
+          </geometry>
+          <material name="">
+            <color rgba="0.29804 0.29804 0.29804 1" />
+          </material>
+        </visual>
+        <collision>
+          <origin xyz="0 0 0" rpy="0 0 0" />
+          <geometry>
+            <mesh filename="package://talos_arm_tool_changer/meshes/camera_left_wrist_link.STL" />
+          </geometry>
+        </collision>
+      </link>
+      <joint name="${name}_${side}_wrist_left_camera_joint" type="fixed">
+        <origin xyz="0.11239 0 -0.12048" rpy="-3.1415925371051 1.0472025163988 -3.14159251909337" />
+        <parent link="${name}_${side}_7_link" />
+        <child link="${name}_${side}_wrist_left_camera_link" />
+        <axis xyz="0 0 0" />
+      </joint>
+      <link name="${name}_${side}_wrist_right_camera_link">
+        <inertial>
+          <origin xyz="0.01021 -0.00042075 -0.00034305" rpy="0 0 0" />
+          <mass value="0.030268" />
+          <inertia ixx="4.4282E-05" ixy="-1.6339E-07" ixz="7.9036E-06" iyy="3.4321E-05" iyz="3.6964E-07" izz="1.7371E-05" />
+        </inertial>
+        <visual>
+          <origin xyz="0 0 0" rpy="0 0 0" />
+          <geometry>
+            <mesh filename="package://talos_arm_tool_changer/meshes/camera_right_wrist_link.STL" />
+          </geometry>
+          <material name="">
+            <color rgba="0.29804 0.29804 0.29804 1" />
+          </material>
+        </visual>
+        <collision>
+          <origin xyz="0 0 0" rpy="0 0 0" />
+          <geometry>
+            <mesh filename="package://talos_arm_tool_changer/meshes/camera_right_wrist_link.STL" />
+          </geometry>
+        </collision>
+      </link>
+      <joint name="${name}_${side}_wrist_right_camera_joint" type="fixed">
+        <origin xyz="-0.11119 0 -0.12048" rpy="-3.1415925371051 1.0472025163988 0" />
+        <parent link="${name}_${side}_7_link" />
+        <child link="${name}_${side}_wrist_right_camera_link" />
+        <axis xyz="0 0 0" />
+      </joint>
+    </xacro:if>
     <gazebo reference="${name}_${side}_5_link">
       <mu1>0.9</mu1>
