Commit message: Add gripper_mount_type and gripper_camera arguments and properties

File: talos_description/urdf/arm/arm.urdf.xacro (robot description, xacro)
@@ -24,5 +24,5 @@
   <xacro:property name="arm_4_max_effort"   value="70.0" />
   <xacro:property name="arm_eps"            value="0.02" />
-  <xacro:macro name="talos_arm" params="name parent side reflect">
+  <xacro:macro name="talos_arm" params="name parent side reflect gripper_mount_type">
     <xacro:unless value="$(arg test)">
       <xacro:include filename="$(find talos_description_calibration)/urdf/calibration/arm_${side}.xacro" />
@@ -188,5 +188,5 @@
     <!--        WRIST           -->
     <!--************************-->
-     <xacro:talos_wrist name="arm" parent="${name}_${side}_4_link" side="${side}" reflect="${reflect}" gripper_type="detachable" gripper_camera="true"/>
+     <xacro:talos_wrist name="arm" parent="${name}_${side}_4_link" side="${side}" reflect="${reflect}" gripper_mount_type="$(arg gripper_mount_type)"/>
     <!-- extensions -->
     <xacro:include filename="$(find talos_description)/urdf/arm/${side}_arm.transmissions.urdf.xacro" />

File: talos_description/urdf/arm/wrist.urdf.xacro (robot description, xacro)
@@ -21,5 +21,5 @@
   <xacro:property name="wrist_3_max_effort"   value="8.0" />
   <xacro:property name="wrist_eps"          value="0.02" />
-  <xacro:macro name="talos_wrist" params="name parent side reflect gripper_type gripper_camera">
+  <xacro:macro name="talos_wrist" params="name parent side reflect gripper_mount_type ">
     <xacro:unless value="$(arg test)">
       <xacro:include filename="$(find talos_description_calibration)/urdf/calibration/arm_${side}.xacro" />
@@ -90,9 +90,9 @@
     </joint>
     <link name="${name}_${side}_7_link">
-      <xacro:call macro="${name}_${side}_7_link_inertial" gripper_type="${gripper_type}"/>
+      <xacro:call macro="${name}_${side}_7_link_inertial" gripper_mount_type="${gripper_mount_type}"/>
       <visual>
         <origin xyz="0 0 0" rpy="0 0 0" />
         <geometry>
-          <mesh filename="package://talos_description/meshes/arm/arm_7_${gripper_type}.STL" scale="1 ${reflect} 1"/>
+          <mesh filename="package://talos_description/meshes/arm/arm_7_${gripper_mount_type}.STL" scale="1 ${reflect} 1"/>
         </geometry>
         <material name="DarkGrey" />
@@ -118,62 +118,4 @@
                           soft_upper_limit="${40.00000 * deg_to_rad - eps_radians}" /> -->
     </joint>
-    <xacro:if value="${gripper_camera}">
-      <link name="${name}_${side}_wrist_left_camera_link">
-        <inertial>
-          <origin xyz="0.01021 -0.00042075 -0.00034305" rpy="0 0 0" />
-          <mass value="0.030268" />
-          <inertia ixx="4.4282E-05" ixy="-1.6339E-07" ixz="7.9036E-06" iyy="3.4321E-05" iyz="3.6964E-07" izz="1.7371E-05" />
-        </inertial>
-        <visual>
-          <origin xyz="0 0 0" rpy="0 0 0" />
-          <geometry>
-            <mesh filename="package://talos_arm_tool_changer/meshes/camera_left_wrist_link.STL" />
-          </geometry>
-          <material name="">
-            <color rgba="0.29804 0.29804 0.29804 1" />
-          </material>
-        </visual>
-        <collision>
-          <origin xyz="0 0 0" rpy="0 0 0" />
-          <geometry>
-            <mesh filename="package://talos_arm_tool_changer/meshes/camera_left_wrist_link.STL" />
-          </geometry>
-        </collision>
-      </link>
-      <joint name="${name}_${side}_wrist_left_camera_joint" type="fixed">
-        <origin xyz="0.11239 0 -0.12048" rpy="-3.1415925371051 1.0472025163988 -3.14159251909337" />
-        <parent link="${name}_${side}_7_link" />
-        <child link="${name}_${side}_wrist_left_camera_link" />
-        <axis xyz="0 0 0" />
-      </joint>
-      <link name="${name}_${side}_wrist_right_camera_link">
-        <inertial>
-          <origin xyz="0.01021 -0.00042075 -0.00034305" rpy="0 0 0" />
-          <mass value="0.030268" />
-          <inertia ixx="4.4282E-05" ixy="-1.6339E-07" ixz="7.9036E-06" iyy="3.4321E-05" iyz="3.6964E-07" izz="1.7371E-05" />
-        </inertial>
-        <visual>
-          <origin xyz="0 0 0" rpy="0 0 0" />
-          <geometry>
-            <mesh filename="package://talos_arm_tool_changer/meshes/camera_right_wrist_link.STL" />
-          </geometry>
-          <material name="">
-            <color rgba="0.29804 0.29804 0.29804 1" />
-          </material>
-        </visual>
-        <collision>
-          <origin xyz="0 0 0" rpy="0 0 0" />
-          <geometry>
-            <mesh filename="package://talos_arm_tool_changer/meshes/camera_right_wrist_link.STL" />
-          </geometry>
-        </collision>
-      </link>
-      <joint name="${name}_${side}_wrist_right_camera_joint" type="fixed">
-        <origin xyz="-0.11119 0 -0.12048" rpy="-3.1415925371051 1.0472025163988 0" />
-        <parent link="${name}_${side}_7_link" />
-        <child link="${name}_${side}_wrist_right_camera_link" />
-        <axis xyz="0 0 0" />
-      </joint>
-    </xacro:if>
     <gazebo reference="${name}_${side}_5_link">
       <mu1>0.9</mu1>

File: talos_description/urdf/gripper/gripper.urdf.xacro (robot description, xacro)
@@ -5,7 +5,37 @@
   <xacro:include filename="$(find talos_description)/urdf/gripper/gripper.transmission.xacro" />
   <xacro:include filename="$(find talos_description)/urdf/gripper/gripper.gazebo.xacro" />
-  <xacro:macro name="talos_gripper" params="name parent reflect">
-            <link name="${name}_base_link">
-              <xacro:call macro="${name}_base_link_inertial" />
+  <xacro:macro name="talos_gripper" params="name side parent reflect gripper_camera">
+            <xacro:if value="${gripper_camera}">
+              <link name="${name}_${side}_gripper_camera_link">
+                <inertial>
+                  <origin xyz="0.01021 -0.00042075 -0.00034305" rpy="0 0 0" />
+                  <mass value="0.030268" />
+                  <inertia ixx="4.4282E-05" ixy="-1.6339E-07" ixz="7.9036E-06" iyy="3.4321E-05" iyz="3.6964E-07" izz="1.7371E-05" />
+                </inertial>
+                <visual>
+                  <origin xyz="0 0 0" rpy="0 0 0" />
+                  <geometry>
+                    <mesh filename="package://talos_description/meshes/gripper/gripper_camera_mount_link.STL" />
+                  </geometry>
+                  <material name="">
+                    <color rgba="0.29804 0.29804 0.29804 1" />
+                  </material>
+                </visual>
+                <collision>
+                  <origin xyz="0 0 0" rpy="0 0 0" />
+                  <geometry>
+                    <mesh filename="package://talos_description/meshes/gripper/gripper_camera_mount_link.STL" />
+                  </geometry>
+                </collision>
+              </link>
+              <joint name="${name}_${side}_wrist_left_camera_joint" type="fixed">
+                <origin xyz="0.11239 0 -0.12048" rpy="-3.1415925371051 1.0472025163988 -3.14159251909337" />
+                <parent link="arm_${side}_7_link"/>
+                <child link="${name}_${side}_gripper_camera_link" />
+                <axis xyz="0 0 0" />
+              </joint>
+            </xacro:if>
+            <link name="${name}_${side}_base_link">
+              <xacro:call macro="${name}_${side}_base_link_inertial" />
               <visual>
                 <origin xyz="0 0 0" rpy="0 0 0" />
@@ -22,13 +52,13 @@
               </collision>
             </link>
-            <joint name="${name}_base_link_joint" type="fixed">
+            <joint name="${name}_${side}_base_link_joint" type="fixed">
               <parent link="${parent}"/>
-              <child link="${name}_base_link"/>
+              <child link="${name}_${side}_base_link"/>
               <origin xyz="0.00000 0.0 -0.02875"
                       rpy="${0.00000 * deg_to_rad} ${0.00000 * deg_to_rad} ${0.00000 * deg_to_rad}"/>
               <axis xyz="0 0 0" />
             </joint>
-            <link name="${name}_motor_double_link">
-              <xacro:call macro="${name}_motor_double_link_inertial" />
+            <link name="${name}_${side}_motor_double_link">
+              <xacro:call macro="${name}_${side}_motor_double_link_inertial" />
               <visual>
                 <origin xyz="0 0 0" rpy="0 0 0" />
@@ -45,7 +75,7 @@
               </collision>
             </link>
-            <joint name="${name}_joint" type="revolute">
-              <parent link="${name}_base_link"/>
-              <child link="${name}_motor_double_link"/>
+            <joint name="${name}_${side}_joint" type="revolute">
+              <parent link="${name}_${side}_base_link"/>
+              <child link="${name}_${side}_motor_double_link"/>
               <origin xyz="0.0 0.02025 -0.03"
                       rpy="${0.0 * deg_to_rad} ${0.0 * deg_to_rad} ${0.0 * deg_to_rad}"/>
@@ -54,6 +84,6 @@
               <dynamics friction="1.0" damping="1.0"/>
             </joint>
-            <link name="${name}_inner_double_link">
-              <xacro:call macro="${name}_inner_double_link_inertial" />
+            <link name="${name}_${side}_inner_double_link">
+              <xacro:call macro="${name}_${side}_inner_double_link_inertial" />
               <visual>
                 <origin xyz="0 0 0" rpy="0 0 0" />
@@ -70,15 +100,15 @@
               </collision>
             </link>
-            <joint name="${name}_inner_double_joint" type="revolute">
-              <parent link="${name}_base_link"/>
-              <child link="${name}_inner_double_link"/>
+            <joint name="${name}_${side}_inner_double_joint" type="revolute">
+              <parent link="${name}_${side}_base_link"/>
+              <child link="${name}_${side}_inner_double_link"/>
               <origin xyz="0.00000 0.00525 -0.05598"
                       rpy="${0.00000 * deg_to_rad} ${0.00000 * deg_to_rad} ${0.00000 * deg_to_rad}"/>
               <axis xyz="1 0 0" />
               <limit lower="${-60.0 * deg_to_rad}" upper="${0.0 * deg_to_rad}" effort="100.0" velocity="1.0" />
-              <mimic joint="${name}_joint" multiplier="${1.0}" offset="0.0" />
-            </joint>
-            <link name="${name}_fingertip_1_link">
-              <xacro:call macro="${name}_fingertip_1_link_inertial" />
+              <mimic joint="${name}_${side}_joint" multiplier="${1.0}" offset="0.0" />
+            </joint>
+            <link name="${name}_${side}_fingertip_1_link">
+              <xacro:call macro="${name}_${side}_fingertip_1_link_inertial" />
               <visual>
                 <origin xyz="0 0 0" rpy="0 0 0" />
@@ -95,15 +125,15 @@
               </collision>
             </link>
-            <joint name="${name}_fingertip_1_joint" type="revolute">
-              <parent link="${name}_inner_double_link"/>
-              <child link="${name}_fingertip_1_link"/>
+            <joint name="${name}_${side}_fingertip_1_joint" type="revolute">
+              <parent link="${name}_${side}_inner_double_link"/>
+              <child link="${name}_${side}_fingertip_1_link"/>
               <origin xyz="0.03200 0.04589 -0.06553"
                       rpy="${0.00000 * deg_to_rad} ${0.00000 * deg_to_rad} ${0.00000 * deg_to_rad}"/>
               <axis xyz="1 0 0" />
               <limit lower="${0.0 * deg_to_rad}" upper="${60.0 * deg_to_rad}" effort="100.0" velocity="1.0" />
-              <mimic joint="${name}_joint" multiplier="${-1.0}" offset="0.0" />
-            </joint>
-            <link name="${name}_fingertip_2_link">
-              <xacro:call macro="${name}_fingertip_2_link_inertial" />
+              <mimic joint="${name}_${side}_joint" multiplier="${-1.0}" offset="0.0" />
+            </joint>
+            <link name="${name}_${side}_fingertip_2_link">
+              <xacro:call macro="${name}_${side}_fingertip_2_link_inertial" />
               <visual>
                 <origin xyz="0 0 0" rpy="0 0 0" />
@@ -120,15 +150,15 @@
               </collision>
             </link>
-            <joint name="${name}_fingertip_2_joint" type="revolute">
-              <parent link="${name}_inner_double_link"/>
-              <child link="${name}_fingertip_2_link"/>
+            <joint name="${name}_${side}_fingertip_2_joint" type="revolute">
+              <parent link="${name}_${side}_inner_double_link"/>
+              <child link="${name}_${side}_fingertip_2_link"/>
               <origin xyz="-0.03200 0.04589 -0.06553"
                       rpy="${0.00000 * deg_to_rad} ${0.00000 * deg_to_rad} ${0.00000 * deg_to_rad}"/>
               <axis xyz="1 0 0" />
               <limit lower="${0.0 * deg_to_rad}" upper="${60.0 * deg_to_rad}" effort="100.0" velocity="1.0" />
-              <mimic joint="${name}_joint" multiplier="${-1.0}" offset="0.0" />
-            </joint>
-            <link name="${name}_motor_single_link">
-              <xacro:call macro="${name}_motor_single_link_inertial" />
+              <mimic joint="${name}_${side}_joint" multiplier="${-1.0}" offset="0.0" />
+            </joint>
+            <link name="${name}_${side}_motor_single_link">
+              <xacro:call macro="${name}_${side}_motor_single_link_inertial" />
               <visual>
                 <origin xyz="0 0 0" rpy="0 0 0" />
@@ -145,15 +175,15 @@
               </collision>
             </link>
-            <joint name="${name}_motor_single_joint" type="revolute">
-              <parent link="${name}_base_link"/>
-              <child link="${name}_motor_single_link"/>
+            <joint name="${name}_${side}_motor_single_joint" type="revolute">
+              <parent link="${name}_${side}_base_link"/>
+              <child link="${name}_${side}_motor_single_link"/>
               <origin xyz="0.00000 -0.02025 -0.03000"
                       rpy="${0.00000 * deg_to_rad} ${0.00000 * deg_to_rad} ${0.00000 * deg_to_rad}"/>
               <axis xyz="1 0 0" />
               <limit lower="${0.0 * deg_to_rad}" upper="${60.0 * deg_to_rad}" effort="100.0" velocity="1.0" />
-              <mimic joint="${name}_joint" multiplier="${-1.0}" offset="0.0" />
-            </joint>
-            <link name="${name}_inner_single_link">
-              <xacro:call macro="${name}_inner_single_link_inertial" />
+              <mimic joint="${name}_${side}_joint" multiplier="${-1.0}" offset="0.0" />
+            </joint>
+            <link name="${name}_${side}_inner_single_link">
+              <xacro:call macro="${name}_${side}_inner_single_link_inertial" />
               <visual>
                 <origin xyz="0 0 0" rpy="0 0 0" />
@@ -170,15 +200,15 @@
               </collision>
             </link>
-            <joint name="${name}_inner_single_joint" type="revolute">
-              <parent link="${name}_base_link"/>
-              <child link="${name}_inner_single_link"/>
+            <joint name="${name}_${side}_inner_single_joint" type="revolute">
+              <parent link="${name}_${side}_base_link"/>
+              <child link="${name}_${side}_inner_single_link"/>
               <origin xyz="0.00000 -0.00525 -0.05598"
                       rpy="${0.00000 * deg_to_rad} ${0.00000 * deg_to_rad} ${0.00000 * deg_to_rad}"/>
               <axis xyz="1 0 0" />
               <limit lower="${0.0 * deg_to_rad}" upper="${60.0 * deg_to_rad}" effort="100.0" velocity="1.0" />
-              <mimic joint="${name}_joint" multiplier="${-1.0}" offset="0.0" />
-            </joint>
-            <link name="${name}_fingertip_3_link">
-              <xacro:call macro="${name}_fingertip_3_link_inertial" />
+              <mimic joint="${name}_${side}_joint" multiplier="${-1.0}" offset="0.0" />
+            </joint>
+            <link name="${name}_${side}_fingertip_3_link">
+              <xacro:call macro="${name}_${side}_fingertip_3_link_inertial" />
               <visual>
                 <origin xyz="0 0 0" rpy="0 0 0" />
@@ -195,22 +225,22 @@
               </collision>
             </link>
-            <joint name="${name}_fingertip_3_joint" type="revolute">
-              <parent link="${name}_inner_single_link"/>
-              <child link="${name}_fingertip_3_link"/>
+            <joint name="${name}_${side}_fingertip_3_joint" type="revolute">
+              <parent link="${name}_${side}_inner_single_link"/>
+              <child link="${name}_${side}_fingertip_3_link"/>
               <origin xyz="0.00000 -0.04589 -0.06553"
                       rpy="${0.00000 * deg_to_rad} ${0.00000 * deg_to_rad} ${180.00000 * deg_to_rad}"/>
               <axis xyz="1 0 0" />
               <limit lower="${0.0 * deg_to_rad}" upper="${60.0 * deg_to_rad}" effort="100.0" velocity="1.0" />
-              <mimic joint="${name}_joint" multiplier="${-1.0}" offset="0.0" />
+              <mimic joint="${name}_${side}_joint" multiplier="${-1.0}" offset="0.0" />
             </joint>
         <xacro:virtual_joints name="${name}" />
         <xacro:gripper_transmission name="${name}" reduction="1.0" />
         <!-- virtual mimic joints -->
-<!--         <xacro:gripper_virtual_transmission name="${name}_inner_double" reduction="1.0"/>
-        <xacro:gripper_virtual_transmission name="${name}_fingertip_1" reduction="1.0"/>
-        <xacro:gripper_virtual_transmission name="${name}_fingertip_2" reduction="1.0"/>
-        <xacro:gripper_virtual_transmission name="${name}_inner_single" reduction="1.0"/>
-        <xacro:gripper_virtual_transmission name="${name}_motor_single" reduction="1.0"/>
-        <xacro:gripper_virtual_transmission name="${name}_fingertip_3" reduction="1.0"/> -->
+<!--         <xacro:gripper_virtual_transmission name="${name}_${side}_inner_double" reduction="1.0"/>
+        <xacro:gripper_virtual_transmission name="${name}_${side}_fingertip_1" reduction="1.0"/>
+        <xacro:gripper_virtual_transmission name="${name}_${side}_fingertip_2" reduction="1.0"/>
+        <xacro:gripper_virtual_transmission name="${name}_${side}_inner_single" reduction="1.0"/>
+        <xacro:gripper_virtual_transmission name="${name}_${side}_motor_single" reduction="1.0"/>
+        <xacro:gripper_virtual_transmission name="${name}_${side}_fingertip_3" reduction="1.0"/> -->
   </xacro:macro>
 </robot>

File: talos_description/urdf/sensors/ftsensor.urdf.xacro (robot description, xacro)
@@ -8,5 +8,5 @@
 -->
 <robot xmlns:xacro="http://ros.org/wiki/xacro">
-  <xacro:macro name="ft_sensor" params="name parent side reflect">
+  <xacro:macro name="ft_sensor" params="name parent side reflect gripper_mount_type">
     <!--************************-->
     <!--        ft sensor       -->
@@ -31,5 +31,10 @@
       <parent link="${parent}" />
       <child link="${name}_${side}_ft_link" />
-      <origin xyz="0 0 -0.051" rpy="${0.0 * deg_to_rad} 0 ${(-180.0 + 90.0*reflect)* deg_to_rad}" />
+      <xacro:if value="${gripper_mount_type == 'detachable'}">
+        <origin xyz="0 0 -0.086" rpy="${0.0 * deg_to_rad} 0 ${(-180.0 + 90.0*reflect)* deg_to_rad}" />
+      </xacro:if>
+      <xacro:if value="${gripper_mount_type == 'classic'}">
+        <origin xyz="0 0 -0.051" rpy="${0.0 * deg_to_rad} 0 ${(-180.0 + 90.0*reflect)* deg_to_rad}" />
+      </xacro:if>
     </joint>
     <!--***********************-->

File: talos_description/urdf/talos_full_common.urdf.xacro (robot description, xacro)
@@ -28,10 +28,10 @@
   </xacro:if>
   <xacro:talos_head name="head" parent="torso_2_link" disable_gazebo_camera="$(arg disable_gazebo_camera)" head_type="$(arg head_type)"/>
-  <xacro:talos_arm name="arm" parent="torso_2_link" side="left" reflect="1" />
-  <xacro:talos_arm name="arm" parent="torso_2_link" side="right" reflect="-1" />
-  <xacro:ft_sensor name="wrist" parent="arm_right_7_link" side="right" reflect="1"  />
-  <xacro:ft_sensor name="wrist" parent="arm_left_7_link"  side="left"  reflect="-1" />
-  <xacro:talos_gripper name="gripper_left" parent="wrist_left_ft_tool_link" reflect="1" />
-  <xacro:talos_gripper name="gripper_right" parent="wrist_right_ft_tool_link" reflect="-1" />
+  <xacro:talos_arm name="arm" parent="torso_2_link" side="left" reflect="1" gripper_mount_type="$(arg gripper_mount_type)"/>
+  <xacro:talos_arm name="arm" parent="torso_2_link" side="right" reflect="-1" gripper_mount_type="$(arg gripper_mount_type)"/>
+  <xacro:ft_sensor name="wrist" parent="arm_right_7_link" side="right" reflect="1" gripper_mount_type="$(arg gripper_mount_type)" />
+  <xacro:ft_sensor name="wrist" parent="arm_left_7_link"  side="left"  reflect="-1" gripper_mount_type="$(arg gripper_mount_type)" />
+  <xacro:talos_gripper name="gripper" side="left" parent="wrist_left_ft_tool_link" reflect="1"  gripper_camera="$(arg gripper_camera)"/>
+  <xacro:talos_gripper name="gripper" side="right" parent="wrist_right_ft_tool_link" reflect="-1"  gripper_camera="$(arg gripper_camera)"/>
   <xacro:talos_leg prefix="left"  reflect="1" flexibility="$(arg flexibility)"/>
   <xacro:talos_leg prefix="right" reflect="-1" flexibility="$(arg flexibility)"/>

File: talos_description_inertial/urdf/inertial.xacro (robot description, xacro)
@@ -50,6 +50,6 @@
     </inertial>
   </xacro:macro>
-  <xacro:macro name="arm_left_7_link_inertial" params="gripper_type">
-    <xacro:if value="${gripper_type == 'classic'}">
+  <xacro:macro name="arm_left_7_link_inertial" params="gripper_mount_type">
+    <xacro:if value="${gripper_mount_type == 'classic'}">
       <inertial>
         <mass value="0.308441"/>
@@ -58,5 +58,5 @@
       </inertial>
     </xacro:if>
-    <xacro:if value="${gripper_type == 'detachable'}">
+    <xacro:if value="${gripper_mount_type == 'detachable'}">
       <inertial>
         <origin xyz="0.0020157 -0.00071287 -0.064959" rpy="0 0 0" />
@@ -108,6 +108,6 @@
     </inertial>
   </xacro:macro>
-  <xacro:macro name="arm_right_7_link_inertial" params="gripper_type">
-    <xacro:if value="${gripper_type == 'classic'}">
+  <xacro:macro name="arm_right_7_link_inertial" params="gripper_mount_type">
+    <xacro:if value="${gripper_mount_type == 'classic'}">
       <inertial>
         <mass value="0.308441"/>
@@ -116,5 +116,5 @@
       </inertial>
     </xacro:if>
-    <xacro:if value="${gripper_type == 'detachable'}">
+    <xacro:if value="${gripper_mount_type == 'detachable'}">
       <inertial>
         <origin xyz="0.0020157 0.00071287 -0.064959" rpy="0 0 0" />
