Commit message: [talos_description] factorize the symmetry in the capsule macro

File: talos_description/urdf/arm/arm.urdf.xacro (robot description, xacro)
@@ -44,10 +44,5 @@
       </visual>
       <xacro:if value="$(arg use_capsule_collision)">
-        <xacro:if value="${side == 'left'}">
-          <xacro:capsule-collision e1="-0.030119 0.141768 0.0465263" e2="-0.00429634 0.0157203 0.0513477" rad="0.076661652397679497" clen="0.12875612953621868" rpy="1.53256 0.201924 0.194397" mid="-0.0172077 0.0787443 0.048937" />
-        </xacro:if>
-        <xacro:if value="${side == 'right'}">
-	  <xacro:capsule-collision e1="-0.030119 -0.141768 0.0465263" e2="-0.00429634 -0.0157203 0.0513477" rad="0.076661652397679497" clen="0.12875612953621868" rpy="-1.53256 0.201924 -0.194397" mid="-0.0172077 -0.0787443 0.048937" />
-        </xacro:if>
+        <xacro:capsule-collision e1="-0.030119 0.141768 0.0465263" e2="-0.00429634 0.0157203 0.0513477" rad="0.076661652397679497" clen="0.12875612953621868" rpy="1.53256 0.201924 0.194397" mid="-0.0172077 0.0787443 0.048937" reflect="${reflect}" />
       </xacro:if>
       <xacro:unless value="$(arg use_capsule_collision)">
@@ -83,10 +78,5 @@
       </visual>
       <xacro:if value="$(arg use_capsule_collision)">
-        <xacro:if value="${side == 'left'}">
-          <xacro:capsule-collision e1="-8.22104e-05 0.00124357 -0.107621" e2="0.0268691 0.000255834 -0.00293965" rad="0.082464320229024751" clen="0.10809965507805776" rpy="0.00943534 0.251977 0.00119509" mid="0.0133935 0.000749701 -0.0552803" />
-        </xacro:if>
-        <xacro:if value="${side == 'right'}">
-	  <xacro:capsule-collision e1="-8.22104e-05 -0.00124357 -0.107621" e2="0.0268691 -0.000255834 -0.00293965" rad="0.082464320229024751" clen="0.10809965507805776" rpy="-0.00943534 0.251977 -0.00119509" mid="0.0133935 -0.000749701 -0.0552803" />
-        </xacro:if>
+        <xacro:capsule-collision e1="-8.22104e-05 0.00124357 -0.107621" e2="0.0268691 0.000255834 -0.00293965" rad="0.082464320229024751" clen="0.10809965507805776" rpy="0.00943534 0.251977 0.00119509" mid="0.0133935 0.000749701 -0.0552803" reflect="${reflect}" />
       </xacro:if>
       <xacro:unless value="$(arg use_capsule_collision)">
@@ -122,10 +112,5 @@
       </visual>
       <xacro:if value="$(arg use_capsule_collision)">
-        <xacro:if value="${side == 'left'}">
-          <xacro:capsule-collision e1="0.0012938 0.00577828 -0.203827" e2="0.0206547 0.0332832 -0.277413" rad="0.077010074599207598" clen="0.080908820017687497" rpy="-2.78389 0.241638 -1.1828" mid="0.0109743 0.0195307 -0.24062" />
-        </xacro:if>
-        <xacro:if value="${side == 'right'}">
-	  <xacro:capsule-collision e1="0.0012938 -0.00577828 -0.203827" e2="0.0206547 -0.0332832 -0.277413" rad="0.077010074599207598" clen="0.080908820017687497" rpy="2.78389 0.241638 1.1828" mid="0.0109743 -0.0195307 -0.24062" />
-        </xacro:if>
+        <xacro:capsule-collision e1="0.0012938 0.00577828 -0.203827" e2="0.0206547 0.0332832 -0.277413" rad="0.077010074599207598" clen="0.080908820017687497" rpy="-2.78389 0.241638 -1.1828" mid="0.0109743 0.0195307 -0.24062" reflect="${reflect}" />
       </xacro:if>
       <xacro:unless value="$(arg use_capsule_collision)">
@@ -164,10 +149,5 @@
       </visual>
       <xacro:if value="$(arg use_capsule_collision)">
-        <xacro:if value="${side == 'left'}">
-	  <xacro:capsule-collision e1="-0.020217 -0.00152238 -0.0600083" e2="-0.000255625 -0.0316283 0.0000811275" rad="0.061638573989565293" clen="0.07011106838940788" rpy="0.464462 0.288704 0.0687292" mid="-0.0102363 -0.0165753 -0.0299636" />
-        </xacro:if>
-        <xacro:if value="${side == 'right'}">
-	  <xacro:capsule-collision e1="-0.020217 0.00152238 -0.0600083" e2="-0.000255625 0.0316283 0.0000811275" rad="0.061638573989565293" clen="0.07011106838940788" rpy="-0.464462 0.288704 -0.0687292" mid="-0.0102363 0.0165753 -0.0299636" />
-        </xacro:if>
+        <xacro:capsule-collision e1="-0.020217 -0.00152238 -0.0600083" e2="-0.000255625 -0.0316283 0.0000811275" rad="0.061638573989565293" clen="0.07011106838940788" rpy="0.464462 0.288704 0.0687292" mid="-0.0102363 -0.0165753 -0.0299636" reflect="${reflect}" />
       </xacro:if>
       <xacro:unless value="$(arg use_capsule_collision)">

File: talos_description/urdf/arm/wrist.urdf.xacro (robot description, xacro)
@@ -41,10 +41,5 @@
       </visual>
       <xacro:if value="$(arg use_capsule_collision)">
-        <xacro:if value="${side == 'left'}">
-	  <xacro:capsule-collision e1="-2.13964e-05 0.000999035 0.0358616" e2="0.000145615 0.0012191 0.121451" rad="0.077412213480368891" clen="0.085589949413547098" rpy="-0.00257122 0.0019513 -2.50861e-06" mid="6.21094e-05 0.00110907 0.0786563" />
-        </xacro:if>
-        <xacro:if value="${side == 'right'}">
-	  <xacro:capsule-collision e1="-2.13964e-05 -0.000999035 0.0358616" e2="0.000145615 -0.0012191 0.121451" rad="0.077412213480368891" clen="0.085589949413547098" rpy="0.00257122 0.0019513 2.50861e-06" mid="6.21094e-05 -0.00110907 0.0786563" />
-        </xacro:if>
+        <xacro:capsule-collision e1="-2.13964e-05 0.000999035 0.0358616" e2="0.000145615 0.0012191 0.121451" rad="0.077412213480368891" clen="0.085589949413547098" rpy="-0.00257122 0.0019513 -2.50861e-06" mid="6.21094e-05 0.00110907 0.0786563" reflect="${reflect}" />
       </xacro:if>
       <xacro:unless value="$(arg use_capsule_collision)">
@@ -80,10 +75,5 @@
       </visual>
       <xacro:if value="$(arg use_capsule_collision)">
-        <xacro:if value="${side == 'left'}">
-	  <xacro:capsule-collision e1="3.71733e-07 -0.000248227 -0.00766634" e2="5.46154e-05 -8.61821e-05 0.00107298" rad="0.044402592090813625" clen="0.0087409825962203314" rpy="-0.0185399 0.00620572 -5.75286e-05" mid="2.74936e-05 -0.000167204 -0.00329668" />
-        </xacro:if>
-        <xacro:if value="${side == 'right'}">
-	  <xacro:capsule-collision e1="3.71733e-07 0.000248227 -0.00766634" e2="5.46154e-05 8.61821e-05 0.00107298" rad="0.044402592090813625" clen="0.0087409825962203314" rpy="0.0185399 0.00620572 5.75286e-05" mid="2.74936e-05 0.000167204 -0.00329668" />
-        </xacro:if>
+        <xacro:capsule-collision e1="3.71733e-07 -0.000248227 -0.00766634" e2="5.46154e-05 -8.61821e-05 0.00107298" rad="0.044402592090813625" clen="0.0087409825962203314" rpy="-0.0185399 0.00620572 -5.75286e-05" mid="2.74936e-05 -0.000167204 -0.00329668" reflect="${reflect}" />
       </xacro:if>
       <xacro:unless value="$(arg use_capsule_collision)">
@@ -119,10 +109,5 @@
       </visual>
       <xacro:if value="$(arg use_capsule_collision)">
-        <xacro:if value="${side == 'left'}">
-	  <xacro:capsule-collision e1="-3.67844e-05 -8.9312e-05 -0.0167866" e2="1.80245e-05 -1.49283e-05 -0.0702192" rad="0.048804145966408037" clen="0.05343267786175529" rpy="-3.1402 0.00102576 -1.27005" mid="-9.37996e-06 -5.21201e-05 -0.0435029" />
-        </xacro:if>
-        <xacro:if value="${side == 'right'}">
-	  <xacro:capsule-collision e1="-3.67844e-05 8.9312e-05 -0.0167866" e2="1.80245e-05 1.49283e-05 -0.0702192" rad="0.048804145966408037" clen="0.05343267786175529" rpy="3.1402 0.00102576 1.27005" mid="-9.37996e-06 5.21201e-05 -0.0435029" />
-        </xacro:if>
+        <xacro:capsule-collision e1="-3.67844e-05 -8.9312e-05 -0.0167866" e2="1.80245e-05 -1.49283e-05 -0.0702192" rad="0.048804145966408037" clen="0.05343267786175529" rpy="-3.1402 0.00102576 -1.27005" mid="-9.37996e-06 -5.21201e-05 -0.0435029" reflect="${reflect}" />
       </xacro:if>
       <xacro:unless value="$(arg use_capsule_collision)">

File: talos_description/urdf/capsule_collision.xacro (robot description, xacro)
@@ -8,21 +8,27 @@
 -->
 <robot xmlns:xacro="http://ros.org/wiki/xacro">
-  <xacro:macro name="capsule-collision" params="e1 e2 rad clen rpy mid">
+  <xacro:macro name="capsule-collision" params="e1 e2 rad clen rpy mid reflect:=1">
+    <!-- Old API: e1, e2, rpy and mid are space-separated strings ("x y z"), reflect multiplies Y and first/third RPY -->
+    <xacro:property name="e1_list" value="${e1.split()}" />
+    <xacro:property name="e2_list" value="${e2.split()}" />
+    <xacro:property name="rpy_list" value="${rpy.split()}" />
+    <xacro:property name="mid_list" value="${mid.split()}" />
+    <xacro:property name="rf" value="${float(reflect)}" />
     <collision>
-      <origin rpy="${rpy}" xyz="${e1}" />
+      <origin rpy="${float(rpy_list[0])*rf} ${rpy_list[1]} ${float(rpy_list[2])*rf}" xyz="${e1_list[0]} ${float(e1_list[1])*rf} ${e1_list[2]}" />
       <geometry>
-	<sphere radius="${rad}" />
+    	<sphere radius="${rad}" />
       </geometry>
     </collision>
     <collision>
-      <origin rpy="${rpy}" xyz="${mid}" />
+      <origin rpy="${float(rpy_list[0])*rf} ${rpy_list[1]} ${float(rpy_list[2])*rf}" xyz="${mid_list[0]} ${float(mid_list[1])*rf} ${mid_list[2]}" />
       <geometry>
-	<cylinder length="${clen}" radius="${rad}" />
+    	<cylinder length="${clen}" radius="${rad}" />
       </geometry>
     </collision>
     <collision>
-      <origin rpy="${rpy}" xyz="${e2}" />
+      <origin rpy="${float(rpy_list[0])*rf} ${rpy_list[1]} ${float(rpy_list[2])*rf}" xyz="${e2_list[0]} ${float(e2_list[1])*rf} ${e2_list[2]}" />
       <geometry>
-	<sphere radius="${rad}" />
+    	<sphere radius="${rad}" />
       </geometry>
     </collision>

File: talos_description/urdf/gripper/gripper.urdf.xacro (robot description, xacro)
@@ -28,10 +28,5 @@
               </visual>
               <xacro:if value="$(arg use_capsule_collision)">
-                <xacro:if value="${name == 'gripper_left'}">
-                  <xacro:capsule-collision e1="-0.00141404 0.0132339 -0.0265828" e2="-0.00133643 -0.0137463 -0.0261142" rad="0.060646620008233225" clen="0.026984385527609595" rpy="1.55343 0.00287592 0.00282641" mid="-0.00137524 -0.00025619 -0.0263485" />
-                </xacro:if>
-                <xacro:if value="${name == 'gripper_right'}">
-                  <xacro:capsule-collision e1="-0.00141404 0.0132339 -0.0265828" e2="-0.00133643 -0.0137463 -0.0261142" rad="0.060646620008233225" clen="0.026984385527609595" rpy="1.55343 0.00287592 0.00282641" mid="-0.00137524 -0.00025619 -0.0263485" />
-                </xacro:if>
+                <xacro:capsule-collision e1="-0.00141404 0.0132339 -0.0265828" e2="-0.00133643 -0.0137463 -0.0261142" rad="0.060646620008233225" clen="0.026984385527609595" rpy="1.55343 0.00287592 0.00282641" mid="-0.00137524 -0.00025619 -0.0263485" />
               </xacro:if>
               <xacro:unless value="$(arg use_capsule_collision)">
@@ -61,10 +56,5 @@
               </visual>
               <xacro:if value="$(arg use_capsule_collision)">
-                <xacro:if value="${name == 'gripper_left'}">
-		  <xacro:capsule-collision e1="-0.0265616 0.0150351 -0.0244879" e2="0.0170994 0.0176648 -0.0189716" rad="0.056117638554986304" clen="0.044086614202536976" rpy="-0.444846 1.43174 -0.388469" mid="-0.00473109 0.0163499 -0.0217297" />
-                </xacro:if>
-                <xacro:if value="${name == 'gripper_right'}">
-                  <xacro:capsule-collision e1="-0.0265616 0.0150351 -0.0244879" e2="0.0170994 0.0176648 -0.0189716" rad="0.056117638554986304" clen="0.044086614202536976" rpy="-0.444846 1.43174 -0.388469" mid="-0.00473109 0.0163499 -0.0217297" />
-                </xacro:if>
+                <xacro:capsule-collision e1="-0.0265616 0.0150351 -0.0244879" e2="0.0170994 0.0176648 -0.0189716" rad="0.056117638554986304" clen="0.044086614202536976" rpy="-0.444846 1.43174 -0.388469" mid="-0.00473109 0.0163499 -0.0217297" />
               </xacro:if>
               <xacro:unless value="$(arg use_capsule_collision)">
@@ -96,10 +86,5 @@
               </visual>
               <xacro:if value="$(arg use_capsule_collision)">
-                <xacro:if value="${name == 'gripper_left'}">
-		  <xacro:capsule-collision e1="-0.0179304 0.0279391 -0.034841" e2="0.0190611 0.0265842 -0.0355285" rad="0.048779412908590628" clen="0.03702274994466908" rpy="2.04039 1.52975 2.00344" mid="0.000565336 0.0272617 -0.0351848" />
-                </xacro:if>
-                <xacro:if value="${name == 'gripper_right'}">
-                  <xacro:capsule-collision e1="-0.0179304 0.0279391 -0.034841" e2="0.0190611 0.0265842 -0.0355285" rad="0.048779412908590628" clen="0.03702274994466908" rpy="2.04039 1.52975 2.00344" mid="0.000565336 0.0272617 -0.0351848" />
-                </xacro:if>
+                <xacro:capsule-collision e1="-0.0179304 0.0279391 -0.034841" e2="0.0190611 0.0265842 -0.0355285" rad="0.048779412908590628" clen="0.03702274994466908" rpy="2.04039 1.52975 2.00344" mid="0.000565336 0.0272617 -0.0351848" />
               </xacro:if>
               <xacro:unless value="$(arg use_capsule_collision)">
@@ -131,10 +116,5 @@
               </visual>
               <xacro:if value="$(arg use_capsule_collision)">
-                <xacro:if value="${name == 'gripper_left'}">
-		  <xacro:capsule-collision e1="-3.72021e-06 0.000302954 -0.026257" e2="-5.04286e-05 0.0140159 0.0163723" rad="0.016697853294401835" clen="0.044780558196911839" rpy="-0.311226 -0.00104305 0.000163635" mid="-2.70744e-05 0.00715944 -0.00494235" />
-                </xacro:if>
-                <xacro:if value="${name == 'gripper_right'}">
-		  <xacro:capsule-collision e1="-3.72021e-06 0.000302954 -0.026257" e2="-5.04286e-05 0.0140159 0.0163723" rad="0.016697853294401835" clen="0.044780558196911839" rpy="-0.311226 -0.00104305 0.000163635" mid="-2.70744e-05 0.00715944 -0.00494235" />
-                </xacro:if>
+          		  <xacro:capsule-collision e1="-3.72021e-06 0.000302954 -0.026257" e2="-5.04286e-05 0.0140159 0.0163723" rad="0.016697853294401835" clen="0.044780558196911839" rpy="-0.311226 -0.00104305 0.000163635" mid="-2.70744e-05 0.00715944 -0.00494235" />
               </xacro:if>
               <xacro:unless value="$(arg use_capsule_collision)">
@@ -166,5 +146,5 @@
               </visual>
               <xacro:if value="$(arg use_capsule_collision)">
-		<xacro:capsule-collision e1="-3.72021e-06 0.000302954 -0.026257" e2="-5.04286e-05 0.0140159 0.0163723" rad="0.016697853294401835" clen="0.044780558196911839" rpy="-0.311226 -0.00104305 0.000163635" mid="-2.70744e-05 0.00715944 -0.00494235" />
+                <xacro:capsule-collision e1="-3.72021e-06 0.000302954 -0.026257" e2="-5.04286e-05 0.0140159 0.0163723" rad="0.016697853294401835" clen="0.044780558196911839" rpy="-0.311226 -0.00104305 0.000163635" mid="-2.70744e-05 0.00715944 -0.00494235" />
               </xacro:if>
               <xacro:unless value="$(arg use_capsule_collision)">
@@ -196,5 +176,5 @@
               </visual>
               <xacro:if value="$(arg use_capsule_collision)">
-		<xacro:capsule-collision e1="-0.00541609 -0.00889752 -0.0121105" e2="0.0100479 -0.0148793 -0.0200314" rad="0.060566804043534143" clen="0.018375470004515674" rpy="2.49478 1.00016 2.04115" mid="0.00231593 -0.0118884 -0.0160709" />
+                <xacro:capsule-collision e1="-0.00541609 -0.00889752 -0.0121105" e2="0.0100479 -0.0148793 -0.0200314" rad="0.060566804043534143" clen="0.018375470004515674" rpy="2.49478 1.00016 2.04115" mid="0.00231593 -0.0118884 -0.0160709" />
               </xacro:if>
               <xacro:unless value="$(arg use_capsule_collision)">

File: talos_description/urdf/head/head.urdf.xacro (robot description, xacro)
@@ -30,5 +30,5 @@
       </visual>
       <xacro:if value="$(arg use_capsule_collision)">
-	<xacro:capsule-collision e1="9.25184e-05 -2.39435e-05 -0.000765958" e2="-0.0116532 0.000267479 0.0600432" rad="0.082632032931063207" clen="0.061933815385056032" rpy="-0.00479238 -0.190806 0.000458601" mid="-0.00578036 0.000121768 0.0296386" />
+        <xacro:capsule-collision e1="9.25184e-05 -2.39435e-05 -0.000765958" e2="-0.0116532 0.000267479 0.0600432" rad="0.082632032931063207" clen="0.061933815385056032" rpy="-0.00479238 -0.190806 0.000458601" mid="-0.00578036 0.000121768 0.0296386" />
       </xacro:if>
       <xacro:unless value="$(arg use_capsule_collision)">

File: talos_description/urdf/leg/leg.urdf.xacro (robot description, xacro)
@@ -72,10 +72,5 @@
       </visual>
       <xacro:if value="$(arg use_capsule_collision)">
-        <xacro:if value="${prefix == 'left'}">
-	  <xacro:capsule-collision e1="0.00653137 -0.00107636 0.0620231" e2="0.0148595 0.000151801 0.00431736" rad="0.10038884516307987" clen="0.058316498699378369" rpy="-3.12031 0.1433 -2.84723" mid="0.0106955 -0.000462282 0.0331702" />
-        </xacro:if>
-        <xacro:if value="${ prefix == 'right'}">
-	  <xacro:capsule-collision e1="0.00653137 0.00107636 0.0620231" e2="0.0148595 -0.000151801 0.00431736" rad="0.10038884516307987" clen="0.058316498699378369" rpy="3.12031 0.1433 2.84723" mid="0.0106955 0.000462282 0.0331702" />
-        </xacro:if>
+        <xacro:capsule-collision e1="0.00653137 -0.00107636 0.0620231" e2="0.0148595 0.000151801 0.00431736" rad="0.10038884516307987" clen="0.058316498699378369" rpy="-3.12031 0.1433 -2.84723" mid="0.0106955 -0.000462282 0.0331702" reflect="${reflect}" />
       </xacro:if>
       <xacro:unless value="$(arg use_capsule_collision)">
@@ -121,10 +116,5 @@
       </visual>
       <xacro:if value="$(arg use_capsule_collision)">
-        <xacro:if value="${prefix == 'left'}">
-	  <xacro:capsule-collision e1="-0.0163525 -0.0136729 0.000327785" e2="-0.0177494 0.072721 0.00192874" rad="0.065228014094609946" clen="0.086420044518244921" rpy="-1.55227 -0.0161651 0.0158683" mid="-0.0170509 0.029524 0.00112826" />
-        </xacro:if>
-        <xacro:if value="${prefix == 'right'}">
-		<xacro:capsule-collision e1="-0.0163525 0.0136729 0.000327785" e2="-0.0177494 -0.072721 0.00192874" rad="0.065228014094609946" clen="0.086420044518244921" rpy="1.55227 -0.0161651 -0.0158683" mid="-0.0170509 -0.029524 0.00112826" />
-        </xacro:if>
+        <xacro:capsule-collision e1="-0.0163525 -0.0136729 0.000327785" e2="-0.0177494 0.072721 0.00192874" rad="0.065228014094609946" clen="0.086420044518244921" rpy="-1.55227 -0.0161651 0.0158683" mid="-0.0170509 0.029524 0.00112826" reflect="${reflect}" />
       </xacro:if>
       <xacro:unless value="$(arg use_capsule_collision)">
@@ -157,10 +147,5 @@
       </visual>
       <xacro:if value="$(arg use_capsule_collision)">
-        <xacro:if value="${prefix == 'left'}">
-	  <xacro:capsule-collision e1="0.00475684 0.0387611 -0.305131" e2="0.0048036 0.0612963 -0.0132432" rad="0.14557912147210253" clen="0.29275626620252521" rpy="-0.077052 0.00015972 -6.15642e-06" mid="0.00478022 0.0500287 -0.159187" />
-        </xacro:if>
-        <xacro:if value="${prefix == 'right'}">
-	  <xacro:capsule-collision e1="0.00475684 -0.0387611 -0.305131" e2="0.0048036 -0.0612963 -0.0132432" rad="0.14557912147210253" clen="0.29275626620252521" rpy="0.077052 0.00015972 6.15642e-06" mid="0.00478022 -0.0500287 -0.159187" />
-        </xacro:if>
+        <xacro:capsule-collision e1="0.00475684 0.0387611 -0.305131" e2="0.0048036 0.0612963 -0.0132432" rad="0.14557912147210253" clen="0.29275626620252521" rpy="-0.077052 0.00015972 -6.15642e-06" mid="0.00478022 0.0500287 -0.159187" reflect="${reflect}" />
       </xacro:if>
       <xacro:unless value="$(arg use_capsule_collision)">
@@ -193,10 +178,5 @@
       </visual>
       <xacro:if value="$(arg use_capsule_collision)">
-        <xacro:if value="${prefix == 'left'}">
-	  <xacro:capsule-collision e1="0.00163993 0.0368989 -0.301909" e2="5.69681e-05 0.0588976 -0.00805678" rad="0.1184924950609377" clen="0.29467833417874939" rpy="-0.0747239 -0.00537185 0.000200797" mid="0.000848448 0.0478982 -0.154983" />
-        </xacro:if>
-        <xacro:if value="${prefix == 'right'}">
-	  <xacro:capsule-collision e1="0.00163993 -0.0368989 -0.301909" e2="5.69681e-05 -0.0588976 -0.00805678" rad="0.1184924950609377" clen="0.29467833417874939" rpy="0.0747239 -0.00537185 -0.000200797" mid="0.000848448 -0.0478982 -0.154983" />
-        </xacro:if>
+        <xacro:capsule-collision e1="0.00163993 0.0368989 -0.301909" e2="5.69681e-05 0.0588976 -0.00805678" rad="0.1184924950609377" clen="0.29467833417874939" rpy="-0.0747239 -0.00537185 0.000200797" mid="0.000848448 0.0478982 -0.154983" reflect="${reflect}" />
       </xacro:if>
       <xacro:unless value="$(arg use_capsule_collision)">
@@ -230,10 +210,5 @@
       </visual>
       <xacro:if value="$(arg use_capsule_collision)">
-        <xacro:if value="${prefix == 'left'}">
-	  <xacro:capsule-collision e1="-0.0304137 0.105995 0.00632637" e2="0.00663845 -0.0117406 -0.00301129" rad="0.056285651716761462" clen="0.12378102303209611" rpy="1.64994 0.303997 0.32863" mid="-0.0118876 0.0471272 0.00165754" />
-        </xacro:if>
-        <xacro:if value="${prefix == 'right'}">
-	  <xacro:capsule-collision e1="-0.0304137 -0.105995 0.00632637" e2="0.00663845 0.0117406 -0.00301129" rad="0.056285651716761462" clen="0.12378102303209611" rpy="-1.64994 0.303997 -0.32863" mid="-0.0118876 -0.0471272 0.00165754" />
-        </xacro:if>
+        <xacro:capsule-collision e1="-0.0304137 0.105995 0.00632637" e2="0.00663845 -0.0117406 -0.00301129" rad="0.056285651716761462" clen="0.12378102303209611" rpy="1.64994 0.303997 0.32863" mid="-0.0118876 0.0471272 0.00165754" reflect="${reflect}" />
       </xacro:if>
       <xacro:unless value="$(arg use_capsule_collision)">
