Commit message: Clean fake crane link, fix imu orientation.

File: talos_description/urdf/crane/crane.urdf.xacro (robot description, xacro)
@@ -38,11 +38,5 @@
       <parent link="${parent}" />
       <child link="crane_link" />
-      <origin xyz="0.003 0.0 0.4"
-          rpy="0.0  0.0  ${(90.0)* deg_to_rad}"/>
-      <!--
-      <axis xyz="0 1 0" />
-      <limit lower="${(-90)* deg_to_rad}" upper="${(90.0)* deg_to_rad}" effort="0.0" velocity="0.0" />
-      -->
-      <axis xyz="0 1 0" />
+      <origin xyz="0.003 0.0 0.4" rpy="0.0  0.0  0.0"/>
       <limit lower="0.0" upper="0.0" effort="0.0" velocity="0.0" />
       <dynamics friction="0.0" damping="0.0"/>

File: talos_description/urdf/torso/torso.urdf.xacro (robot description, xacro)
@@ -121,5 +121,5 @@
     </joint>
   <xacro:talos_imu name="imu" parent="${name}_2_link" update_rate="100.0">
-    <origin xyz="0.04925 0 0.078" rpy="${180.0*deg_to_rad} 0 ${90.0*deg_to_rad}"/>
+    <origin xyz="0.04925 0 0.078" rpy="${180.0*deg_to_rad} 0 ${-90.0*deg_to_rad}"/>
   </xacro:talos_imu>
   <gazebo reference="${name}_1_link">
