Commit message: Add head and camera calibration offsets

File: talos_description/urdf/head/head.transmission.xacro (robot description, xacro)
@@ -9,5 +9,5 @@
 <robot xmlns:xacro="http://ros.org/wiki/xacro">
   <xacro:macro name="talos_head_differential_transmission"
-               params="name number1 number2 act_reduction1 act_reduction2 jnt_reduction1 jnt_reduction2" >
+               params="name number1 number2 act_reduction1 act_reduction2 jnt_reduction1 jnt_reduction2 offset_value_1 offset_value_2" >
     <transmission name="talos_trans">
       <type>transmission_interface/HalfDifferentialTransmission</type>
@@ -22,5 +22,5 @@
       <joint name="${name}_${number1}_joint">
         <role>joint1</role>
-        <offset>0.0</offset>
+        <offset>${offset_value_1}</offset>
         <mechanicalReduction>${jnt_reduction1}</mechanicalReduction>
         <hardwareInterface>hardware_interface/PositionJointInterface</hardwareInterface>
@@ -29,5 +29,5 @@
       <joint name="${name}_${number2}_joint">
         <role>joint2</role>
-        <offset>0.0</offset>
+        <offset>${offset_value_2}</offset>
         <mechanicalReduction>${jnt_reduction2}</mechanicalReduction>
         <hardwareInterface>hardware_interface/PositionJointInterface</hardwareInterface>

File: talos_description/urdf/head/head.urdf.xacro (robot description, xacro)
@@ -12,4 +12,5 @@
   <xacro:include filename="$(find talos_description)/urdf/head/head.transmission.xacro" />
   <xacro:include filename="$(find talos_description)/urdf/sensors/orbbec_astra_pro.urdf.xacro" />
+  <xacro:include filename="$(find talos_description_calibration)/urdf/calibration/calibration_constants.urdf.xacro" />
   <!--Constant parameters-->
   <xacro:property name="head_friction" value="1.0" />
@@ -122,5 +123,5 @@
     <xacro:orbbec_astra_pro name="rgbd" parent="${name}_2">
       <!-- Pose of sensor frame wrt to base -->
-      <origin xyz="0.066 0.0 0.1982" rpy="0 0 0"/>
+      <origin xyz="${camera_position_x} ${camera_position_y} ${camera_position_z}" rpy="${camera_orientation_r} ${camera_orientation_p} ${camera_orientation_y}" />
       <!-- Pose of optical frame wrt to sensor -->
       <origin xyz="0 0 0" rpy="${-90 * deg_to_rad} 0 ${-90 * deg_to_rad}"/>
@@ -128,5 +129,6 @@
     <xacro:talos_head_differential_transmission name="${name}" number1="1" number2="2"
                                                 act_reduction1="1.0" act_reduction2="1.0"
-                                                jnt_reduction1="1.0" jnt_reduction2="2.0" />
+                                                jnt_reduction1="1.0" jnt_reduction2="2.0"
+                                                offset_value_1="${head_1_joint_offset}" offset_value_2="${head_2_joint_offset}"/>
   </xacro:macro>
 </robot>
