Commit message: MoveIt and play_motion config files

File: talos_description/urdf/head/head.urdf.xacro (robot description, xacro)
@@ -49,5 +49,5 @@
               rpy="${0.00000 * deg_to_rad} ${0.00000 * deg_to_rad} ${0.00000 * deg_to_rad}"/>
       <axis xyz="0 1 0" />
-      <limit lower="${-15.00000 * deg_to_rad}" upper="${45.00000 * deg_to_rad}" effort="1.0" velocity="1.0" />
+      <limit lower="${-15.00000 * deg_to_rad}" upper="${45.00000 * deg_to_rad}" effort="8.0" velocity="1.0" />
       <dynamics damping="${head_damping}" friction="${head_friction}"/>
        <!-- <safety_controller k_position="20"
@@ -99,5 +99,5 @@
               rpy="${0.00000 * deg_to_rad} ${0.00000 * deg_to_rad} ${0.00000 * deg_to_rad}"/>
       <axis xyz="0 0 1" />
-      <limit lower="${-75.00000 * deg_to_rad}" upper="${75.00000 * deg_to_rad}" effort="1.0" velocity="1.0" />
+      <limit lower="${-75.00000 * deg_to_rad}" upper="${75.00000 * deg_to_rad}" effort="4.0" velocity="1.0" />
       <dynamics damping="${head_damping}" friction="${head_friction}"/>
        <!-- <safety_controller k_position="20"

Commit message: Use orbbec pro with correct resolution in simulation

File: talos_description/urdf/head/head.urdf.xacro (robot description, xacro)
@@ -120,10 +120,10 @@
     <xacro:talos_head_1 name="${name}_1" parent="${parent}" />
     <xacro:talos_head_2 name="${name}_2" parent="${name}_1_link"/>
-    <xacro:xtion_pro_live name="rgbd" parent="${name}_2">
+    <xacro:orbbec_astra_pro name="rgbd" parent="${name}_2">
       <!-- Pose of sensor frame wrt to base -->
       <origin xyz="0.066 0.0 0.1982" rpy="0 0 0"/>
       <!-- Pose of optical frame wrt to sensor -->
       <origin xyz="0 0 0" rpy="${-90 * deg_to_rad} 0 ${-90 * deg_to_rad}"/>
-    </xacro:xtion_pro_live>
+    </xacro:orbbec_astra_pro>
     <xacro:talos_head_differential_transmission name="${name}" number1="1" number2="2"
                                                 act_reduction1="1.0" act_reduction2="1.0"

File: talos_description/urdf/sensors/orbbec_astra_pro.urdf.xacro (robot description, xacro)
@@ -18,7 +18,7 @@
 -->
 <robot xmlns:xacro="http://ros.org/wiki/xacro">
-  <xacro:include filename="$(find talos_description)/urdf/sensors/xtion_pro_live.gazebo.xacro" />
+  <xacro:include filename="$(find talos_description)/urdf/sensors/orbbec_astra_pro.gazebo.xacro" />
   <!-- Macro -->
-  <xacro:macro name="xtion_pro_live" params="name parent *origin *optical_origin">
+  <xacro:macro name="orbbec_astra_pro" params="name parent *origin *optical_origin">
     <!-- frames in the center of the camera -->
     <joint name="${name}_joint" type="fixed">
@@ -95,5 +95,5 @@
     <link name="${name}_rgb_optical_frame"/>
     <!-- extensions -->
-    <xacro:xtion_pro_live_rgbd_camera_gazebo name="${name}" />
+    <xacro:orbbec_astra_pro_rgbd_camera_gazebo name="${name}" />
   </xacro:macro>
 </robot>

Commit message: New inertials of the torso (incorrectly generated earlier) & head.

File: talos_description/urdf/head/head.urdf.xacro (robot description, xacro)
@@ -24,9 +24,9 @@
     <link name="${name}_link">
       <inertial>
-        <origin xyz="0.00120 0.00145 0.02165" rpy="0.00000 0.00000 0.00000"/>
-        <mass value="0.65988"/>
-        <inertia ixx="0.00122100000" ixy="-0.00000400000" ixz="0.00007000000"
-                 iyy="0.00092400000" iyz="-0.00004100000"
-                 izz="0.00103300000"/>
+        <origin xyz="-0.00157211000 -0.00157919000 0.02175767000" rpy="0.00000000000 0.00000000000 0.00000000000"/>
+        <mass value="0.73746000000"/>
+        <inertia ixx="0.00224878584" ixy="0.00000469375" ixz="0.00008555570"
+                 iyy="0.00111158492" iyz="-0.00004132536"
+                 izz="0.00205225921"/>
       </inertial>
       <visual>
@@ -47,5 +47,5 @@
       <parent link="${parent}"/>
       <child link="${name}_link"/>
-      <origin xyz="0.00000 0.00000 0.31600"
+      <origin xyz="0.02000 0.00000 0.32100"
               rpy="${0.00000 * deg_to_rad} ${0.00000 * deg_to_rad} ${0.00000 * deg_to_rad}"/>
       <axis xyz="0 1 0" />
@@ -74,9 +74,9 @@
     <link name="${name}_link">
       <inertial>
-        <origin xyz="-0.01036 -0.00037 0.13778" rpy="0.00000 0.00000 0.00000"/>
-        <mass value="1.40353"/>
-        <inertia ixx="0.00722500000" ixy="-0.00002500000" ixz="0.00032900000"
-                 iyy="0.00687300000" iyz="0.00004400000"
-                 izz="0.00437300000"/>
+        <origin xyz="0.01002657000 0.00005218000 0.14136068000" rpy="0.00000000000 0.00000000000 0.00000000000"/>
+        <mass value="1.44395400000"/>
+        <inertia ixx="0.01084624339" ixy="0.00001050889" ixz="0.00041594252"
+                 iyy="0.01095691760" iyz="0.00002367831"
+                 izz="0.00571698895"/>
       </inertial>
       <visual>

File: talos_description/urdf/torso/torso.urdf.xacro (robot description, xacro)
@@ -22,9 +22,9 @@
     <link name="${name}_2_link">
       <inertial>
-        <origin xyz="-0.04636 -0.00099 0.14528" rpy="0.00000 0.00000 0.00000"/>
-        <mass value="16.97403"/>
-        <inertia ixx="0.44372634000" ixy="-0.00069132000" ixz="0.01218206000"
-                 iyy="0.29985761000" iyz="0.00019623000"
-                 izz="0.32201555000"/>
+        <origin xyz="-0.04635630000 -0.00099023000 0.14528050000" rpy="0.00000000000 0.00000000000 0.00000000000"/>
+        <mass value="16.97403000000"/>
+        <inertia ixx="0.44372633826" ixy="0.00069132133" ixz="-0.01218206353"
+                 iyy="0.29985760680" iyz="-0.00019623338"
+                 izz="0.32201554742"/>
       </inertial>
       <visual>
@@ -47,9 +47,9 @@
     <link name="${name}_1_link">
       <inertial>
-        <origin xyz="0.00078 0.00004 -0.01782" rpy="0.00000 0.00000 0.00000"/>
-        <mass value="2.29466"/>
-        <inertia ixx="0.00638508000" ixy="0.00000007000" ixz="0.00003066000"
-                 iyy="0.00410256000" iyz="0.00000147000"
-                 izz="0.00622969000"/>
+        <origin xyz="0.00078223000 0.00003528000 -0.01782457000" rpy="0.00000000000 0.00000000000 0.00000000000"/>
+        <mass value="2.29465800000"/>
+        <inertia ixx="0.00638508087" ixy="-0.00000007107" ixz="-0.00003065592"
+                 iyy="0.00410256102" iyz="-0.00000146946"
+                 izz="0.00622968815"/>
       </inertial>
       <visual>
@@ -86,9 +86,9 @@
     <link name="base_link">
       <inertial>
-        <origin xyz="-0.05709 0.00153 -0.07625" rpy="0.00000 0.00000 0.00000"/>
-        <mass value="15.36284"/>
-        <inertia ixx="0.20105076000" ixy="-0.00023245000" ixz="-0.00401677000"
-                 iyy="0.08411497000" iyz="0.00087207000"
-                 izz="0.23189084000"/>
+        <origin xyz="-0.05709419000 0.00153054000 -0.07625210000" rpy="0.00000000000 0.00000000000 0.00000000000"/>
+        <mass value="15.36284000000"/>
+        <inertia ixx="0.20105075811" ixy="0.00023244734" ixz="0.00401677280"
+                 iyy="0.08411496729" iyz="-0.00087206649"
+                 izz="0.23189084140"/>
       </inertial>
       <visual>

Commit message: fixed head velocity

File: talos_description/urdf/head/head.urdf.xacro (robot description, xacro)
@@ -44,5 +44,5 @@
               rpy="${0.00000 * deg_to_rad} ${0.00000 * deg_to_rad} ${0.00000 * deg_to_rad}"/>
       <axis xyz="0 1 0" />
-      <limit lower="${-12.00000 * deg_to_rad}" upper="${45.00000 * deg_to_rad}" effort="8.0" velocity="1.0" />
+      <limit lower="${-12.00000 * deg_to_rad}" upper="${45.00000 * deg_to_rad}" effort="8.0" velocity="${head_max_vel}" />
       <dynamics damping="${head_damping}" friction="${head_friction}"/>
        <!-- <safety_controller k_position="20"
@@ -88,5 +88,5 @@
               rpy="${0.00000 * deg_to_rad} ${0.00000 * deg_to_rad} ${0.00000 * deg_to_rad}"/>
       <axis xyz="0 0 1" />
-      <limit lower="${-75.00000 * deg_to_rad}" upper="${75.00000 * deg_to_rad}" effort="4.0" velocity="1.0" />
+      <limit lower="${-75.00000 * deg_to_rad}" upper="${75.00000 * deg_to_rad}" effort="4.0" velocity="${head_max_vel}" />
       <dynamics damping="${head_damping}" friction="${head_friction}"/>
        <!-- <safety_controller k_position="20"

Commit message: Enable 6D calibration of arm, head and torso joints.

File: talos_description/urdf/head/head.urdf.xacro (robot description, xacro)
@@ -41,6 +41,6 @@
       <parent link="${parent}"/>
       <child link="${name}_link"/>
-      <origin xyz="0.02000 0.00000 0.32100"
-              rpy="${0.00000 * deg_to_rad} ${0.00000 * deg_to_rad} ${0.00000 * deg_to_rad}"/>
+      <origin xyz="${0.02000 + head_1_joint_x_offset} ${0.00000 + head_1_joint_y_offset} ${0.32100 + head_1_joint_z_offset}"
+              rpy="${0.00000 * deg_to_rad + head_1_joint_roll_offset} ${0.00000 * deg_to_rad + head_1_joint_pitch_offset} ${0.00000 * deg_to_rad + head_1_joint_yaw_offset}"/>
       <axis xyz="0 1 0" />
       <limit lower="${-12.00000 * deg_to_rad}" upper="${45.00000 * deg_to_rad}" effort="8.0" velocity="${head_max_vel}" />
@@ -85,6 +85,6 @@
       <parent link="${parent}"/>
       <child link="${name}_link"/>
-      <origin xyz="0.00000 0.00000 0.00000"
-              rpy="${0.00000 * deg_to_rad} ${0.00000 * deg_to_rad} ${0.00000 * deg_to_rad}"/>
+      <origin xyz="${0.00000 + head_2_joint_x_offset} ${0.00000 + head_2_joint_y_offset} ${0.00000 + head_2_joint_z_offset}"
+              rpy="${0.00000 * deg_to_rad + head_2_joint_roll_offset} ${0.00000 * deg_to_rad + head_2_joint_pitch_offset} ${0.00000 * deg_to_rad + head_2_joint_yaw_offset}"/>
       <axis xyz="0 0 1" />
       <limit lower="${-75.00000 * deg_to_rad}" upper="${75.00000 * deg_to_rad}" effort="4.0" velocity="${head_max_vel}" />

Commit message: added head version argument in the head urdf xacro

File: talos_description/urdf/head/head.urdf.xacro (robot description, xacro)
@@ -18,4 +18,5 @@
   <xacro:property name="head_max_vel"  value="3.0" />
   <xacro:property name="head_eps"      value="0.02" />
+  <xacro:property name="head_version"  default="default" />
   <!--************************-->
   <!--     HEAD_1 (TILT)      -->
@@ -109,10 +110,12 @@
     <xacro:talos_head_1 name="${name}_1" parent="${parent}" />
     <xacro:talos_head_2 name="${name}_2" parent="${name}_1_link"/>
-    <xacro:orbbec_astra_pro name="rgbd" parent="${name}_2" disable_gazebo="${disable_gazebo_camera}">
-      <!-- Pose of sensor frame wrt to base -->
-      <origin xyz="${camera_position_x} ${camera_position_y} ${camera_position_z}" rpy="${camera_orientation_r} ${camera_orientation_p} ${camera_orientation_y}" />
-      <!-- Pose of optical frame wrt to sensor -->
-      <origin xyz="0 0 0" rpy="${-90 * deg_to_rad} 0 ${-90 * deg_to_rad}"/>
-    </xacro:orbbec_astra_pro>
+    <xacro:if value="${head_version == 'default'}">
+      <xacro:orbbec_astra_pro name="rgbd" parent="${name}_2" disable_gazebo="${disable_gazebo_camera}">
+        <!-- Pose of sensor frame wrt to base -->
+        <origin xyz="${camera_position_x} ${camera_position_y} ${camera_position_z}" rpy="${camera_orientation_r} ${camera_orientation_p} ${camera_orientation_y}" />
+        <!-- Pose of optical frame wrt to sensor -->
+        <origin xyz="0 0 0" rpy="${-90 * deg_to_rad} 0 ${-90 * deg_to_rad}"/>
+      </xacro:orbbec_astra_pro>
+    </xacro:if>
     <xacro:talos_head_differential_transmission name="${name}" number1="1" number2="2"
                                                 act_reduction1="1.0" act_reduction2="1.0"

Commit message: added the conditions for the new lidar head version with intel t265, d435, and ouster lidar

File: talos_description/urdf/head/head.urdf.xacro (robot description, xacro)
@@ -118,4 +118,26 @@
       </xacro:orbbec_astra_pro>
     </xacro:if>
+    <xacro:if value="${head_version == 'lidar'}">
+      <!--File includes-->
+      <xacro:include filename="$(find realsense2_description)/urdf/_d435.urdf.xacro" />
+      <xacro:include filename="$(find realsense2_description)/urdf/_t265.urdf.xacro" />
+      <xacro:include filename="$(find talos_description)/urdf/sensors/OS1-64.urdf.xacro"/>
+      <!-- Intel D435 Camera -->
+      <sensor_d435 parent="${name}_2_link" name="${name}_d435_camera" topics_ns="${name}_d435_camera">
+        <origin xyz="0.074 0.0 0.135"
+                rpy="0.0 ${45.0 * deg_to_rad} 0.0"/>
+      </sensor_d435>
+      <!-- Intel T265 Camera -->
+      <sensor_t265 parent="${name}_2_link" name="${name}_t265_camera" topics_ns="${name}_t265_camera">
+        <origin xyz="0.109 0.0 0.196"
+                rpy="0.0 ${5.0 * deg_to_rad} 0.0"/>
+      </sensor_t265>
+      <!-- Ouster Lidar -->
+      <OS1-64 parent="${name}_2_link" name="${name}_os1_sensor" hz="10" samples="220">
+        <origin xyz="0.015 0.0 0.285"
+                rpy="0 0 0" />
+      </OS1-64>
+    </xacro:if>
+    <!-- Transmission -->
     <xacro:talos_head_differential_transmission name="${name}" number1="1" number2="2"
                                                 act_reduction1="1.0" act_reduction2="1.0"

Commit message: Fix the argument to the TALOS head macro

File: talos_description/urdf/head/head.urdf.xacro (robot description, xacro)
@@ -18,5 +18,4 @@
   <xacro:property name="head_max_vel"  value="3.0" />
   <xacro:property name="head_eps"      value="0.02" />
-  <xacro:property name="head_version"  default="default" />
   <!--************************-->
   <!--     HEAD_1 (TILT)      -->
@@ -107,8 +106,8 @@
     </gazebo>
   </xacro:macro>
-  <xacro:macro name="talos_head" params="name parent disable_gazebo_camera:=false">
+  <xacro:macro name="talos_head" params="name parent disable_gazebo_camera:=false head_type:=default">
     <xacro:talos_head_1 name="${name}_1" parent="${parent}" />
     <xacro:talos_head_2 name="${name}_2" parent="${name}_1_link"/>
-    <xacro:if value="${head_version == 'default'}">
+    <xacro:if value="${head_type == 'default'}">
       <xacro:orbbec_astra_pro name="rgbd" parent="${name}_2" disable_gazebo="${disable_gazebo_camera}">
         <!-- Pose of sensor frame wrt to base -->
@@ -118,5 +117,5 @@
       </xacro:orbbec_astra_pro>
     </xacro:if>
-    <xacro:if value="${head_version == 'lidar'}">
+    <xacro:if value="${head_type == 'lidar'}">
       <!--File includes-->
       <xacro:include filename="$(find realsense2_description)/urdf/_d435.urdf.xacro" />

File: talos_description/urdf/sensors/OS1-64.urdf.xacro (robot description, xacro)
@@ -18,5 +18,5 @@
          <origin xyz="0 0 0.0365" rpy="0 0 0" />
          <geometry>
- 	        <cylinder radius="0.04" length="0.073"/>
+          <cylinder radius="0.04" length="0.073"/>
          </geometry>
       </collision>
@@ -24,5 +24,5 @@
          <origin xyz="0 0 0.0" rpy="0 0 1.5707" />
          <geometry>
-	         <mesh filename="package://talos_description/meshes/sensors/ouster/os1_64.dae" />
+           <mesh filename="package://talos_description/meshes/sensors/ouster/os1_64.dae" />
            <!-- <cylinder length="0.073" radius="0.04" /> -->
          </geometry>

File: talos_description/urdf/talos_full_common.urdf.xacro (robot description, xacro)
@@ -27,5 +27,5 @@
     <xacro:crane parent="torso_2_link"/>
   </xacro:if>
-  <xacro:talos_head name="head" parent="torso_2_link" disable_gazebo_camera="$(arg disable_gazebo_camera)"/>
+  <xacro:talos_head name="head" parent="torso_2_link" disable_gazebo_camera="$(arg disable_gazebo_camera)" head_type="$(arg head_type)"/>
   <xacro:talos_arm name="arm" parent="torso_2_link" side="left" reflect="1" />
   <xacro:talos_arm name="arm" parent="torso_2_link" side="right" reflect="-1" />

Commit message: Update head xacro to use the new meshes

File: talos_description/urdf/head/head.urdf.xacro (robot description, xacro)
@@ -65,5 +65,5 @@
   <!--      HEAD_2 (PAN)      -->
   <!--************************-->
-  <xacro:macro name="talos_head_2" params="name parent">
+  <xacro:macro name="talos_head_2" params="name parent type:=default">
     <link name="${name}_link">
       <xacro:call macro="${name}_link_inertial" />
@@ -71,5 +71,5 @@
         <origin xyz="0 0 0" rpy="0 0 0" />
         <geometry>
-          <mesh filename="package://talos_description/meshes/head/head_2.stl" scale="1 1 1"/>
+          <mesh filename="package://talos_description/meshes/head/head_2_${type}.stl" scale="1 1 1"/>
         </geometry>
         <material name="LightGrey" />
@@ -78,5 +78,5 @@
         <origin xyz="0 0 0" rpy="0 0 0" />
         <geometry>
-          <mesh filename="package://talos_description/meshes/head/head_2_collision.stl" scale="1 1 1"/>
+          <mesh filename="package://talos_description/meshes/head/head_2_${type}_collision.stl" scale="1 1 1"/>
         </geometry>
       </collision>
@@ -108,5 +108,5 @@
   <xacro:macro name="talos_head" params="name parent disable_gazebo_camera:=false head_type:=default">
     <xacro:talos_head_1 name="${name}_1" parent="${parent}" />
-    <xacro:talos_head_2 name="${name}_2" parent="${name}_1_link"/>
+    <xacro:talos_head_2 name="${name}_2" parent="${name}_1_link" type="${head_type}"/>
     <xacro:if value="${head_type == 'default'}">
       <xacro:orbbec_astra_pro name="rgbd" parent="${name}_2" disable_gazebo="${disable_gazebo_camera}">

Commit message: Fix head and torso calibration

File: talos_description/urdf/head/head.urdf.xacro (robot description, xacro)
@@ -142,5 +142,5 @@
                                                 act_reduction1="1.0" act_reduction2="1.0"
                                                 jnt_reduction1="1.0" jnt_reduction2="2.0"
-                                                offset_value_1="${head_1_joint_offset}" offset_value_2="${head_2_joint_offset}"/>
+                                                offset_value_1="${head_1_joint_pitch_offset}" offset_value_2="${head_2_joint_yaw_offset}"/>
   </xacro:macro>
 </robot>

File: talos_description/urdf/torso/torso.urdf.xacro (robot description, xacro)
@@ -93,6 +93,6 @@
       <parent link="${name}_1_link"/>
       <child link="${name}_2_link"/>
-      <origin xyz="${0.0 + torso_1_joint_x_offset} ${0.0 + torso_1_joint_y_offset} ${0.0 + torso_1_joint_z_offset}"
-              rpy="${0.00000 * deg_to_rad + torso_1_joint_roll_offset} ${0.00000 * deg_to_rad + torso_1_joint_pitch_offset} ${0.00000 * deg_to_rad + torso_1_joint_yaw_offset}"/>
+      <origin xyz="${0.0 + torso_2_joint_x_offset} ${0.0 + torso_2_joint_y_offset} ${0.0 + torso_2_joint_z_offset}"
+              rpy="${0.00000 * deg_to_rad + torso_2_joint_roll_offset} ${0.00000 * deg_to_rad + torso_2_joint_pitch_offset} ${0.00000 * deg_to_rad + torso_2_joint_yaw_offset}"/>
       <axis xyz="0 1 0" />
       <limit lower="${-13.0 * deg_to_rad}" upper="${42.0 * deg_to_rad}"

File: talos_description_calibration/urdf/calibration/calibration_constants.urdf.xacro (robot description, xacro)
@@ -31,6 +31,4 @@
   <xacro:property name="arm_right_6_joint_offset" value="0.0" />
   <xacro:property name="arm_right_7_joint_offset" value="0.0" />
-  <xacro:property name="head_1_joint_offset" value="0.0" />
-  <xacro:property name="head_2_joint_offset" value="0.0" />
   <xacro:property name="head_1_joint_x_offset"     value="0.0" />
   <xacro:property name="head_1_joint_y_offset"     value="0.0" />
