Commit message: increase the size of the foot collision model

File: talos_description/urdf/leg/foot_collision_default.urdf.xacro (robot description, xacro)
@@ -5,5 +5,5 @@
             <origin xyz="0 0 0" rpy="0 0 0" />
             <geometry>
-                <mesh filename="package://talos_description/meshes/v2/ankle_X_collision.stl" scale="1 ${reflect*1} 1"/>
+                <mesh filename="package://talos_description/meshes/v2/ankle_X_collision.stl" scale="1.15 ${reflect*1.15} 1"/>
             </geometry>
         </collision>

Commit message: Don't increase y foot collision mesh so much

File: talos_description/urdf/leg/foot_collision_default.urdf.xacro (robot description, xacro)
@@ -5,5 +5,5 @@
             <origin xyz="0 0 0" rpy="0 0 0" />
             <geometry>
-                <mesh filename="package://talos_description/meshes/v2/ankle_X_collision.stl" scale="1.15 ${reflect*1.15} 1"/>
+                <mesh filename="package://talos_description/meshes/v2/ankle_X_collision.stl" scale="1.15 ${reflect*1.05} 1"/>
             </geometry>
         </collision>
