Commit message: increased effort limit in torso joint, use mesh collision for the feet.

File: talos_description/urdf/leg/leg.urdf.xacro (robot description, xacro)
@@ -185,12 +185,11 @@
         <material name="Grey" />
       </visual>
+      <collision>
+        <origin xyz="0 0 0" rpy="0 0 0" />
+        <geometry>
+          <mesh filename="package://talos_description/meshes/v2/ankle_X_collision.stl" scale="1 ${reflect*1} 1"/>
+        </geometry>
+      </collision>
       <!--
-      <collision>
-        <origin xyz="0 0 0" rpy="0 0 0" />
-        <geometry>
-          <mesh filename="package://talos_description/meshes/v2/ankle_X_collision.stl" scale="1 ${reflect*1} 1"/>
-        </geometry>
-      </collision>
-      -->
        <collision>
         <origin xyz="0 0 -0.1" rpy="0 0 0" />
@@ -199,4 +198,5 @@
         </geometry>
       </collision>
+      -->
     </link>
     <joint name="leg_${prefix}_6_joint" type="revolute">

File: talos_description/urdf/torso/torso.urdf.xacro (robot description, xacro)
@@ -14,5 +14,5 @@
  <!--Constant parameters-->
   <xacro:property name="torso_max_vel"  value="5.4" />
-  <xacro:property name="torso_max_effort"  value="78.0" />
+  <xacro:property name="torso_max_effort"  value="120.0" />
   <xacro:property name="torso_eps"      value="0.02" />
   <xacro:macro name="talos_torso" params="name">

Commit message: Revert "increased effort limit in torso joint, use mesh collision for the feet."
This reverts commit 79da15cf0422f552dae87f6bb7ccacd83059989f.

File: talos_description/urdf/leg/leg.urdf.xacro (robot description, xacro)
@@ -185,4 +185,5 @@
         <material name="Grey" />
       </visual>
+      <!--
       <collision>
         <origin xyz="0 0 0" rpy="0 0 0" />
@@ -191,5 +192,5 @@
         </geometry>
       </collision>
-      <!--
+      -->
        <collision>
         <origin xyz="0 0 -0.1" rpy="0 0 0" />
@@ -198,5 +199,4 @@
         </geometry>
       </collision>
-      -->
     </link>
     <joint name="leg_${prefix}_6_joint" type="revolute">

File: talos_description/urdf/torso/torso.urdf.xacro (robot description, xacro)
@@ -14,5 +14,5 @@
  <!--Constant parameters-->
   <xacro:property name="torso_max_vel"  value="5.4" />
-  <xacro:property name="torso_max_effort"  value="120.0" />
+  <xacro:property name="torso_max_effort"  value="78.0" />
   <xacro:property name="torso_eps"      value="0.02" />
   <xacro:macro name="talos_torso" params="name">

Commit message: Leg urdf: updated inertial parameters

File: talos_description/urdf/leg/leg.urdf.xacro (robot description, xacro)
@@ -12,9 +12,9 @@
     <link name="leg_${prefix}_1_link">
       <inertial>
-        <origin xyz="0.02320 ${reflect*-0.00009} 0.04949" rpy="0.00000 0.00000 0.00000"/>
-        <mass value="1.88569"/>
-        <inertia ixx="0.00384800000" ixy="${reflect*0.00003200000}" ixz="-0.00082600000"
-                 iyy="0.00599400000" iyz="${reflect*0.00007800000}"
-                 izz="0.00322200000"/>
+        <origin xyz="0.02247868000 ${reflect*0.00106736000} 0.03130665000" rpy="0.00000000000 0.00000000000 0.00000000000"/>
+        <mass value="1.84559100000"/>
+        <inertia ixx="0.00541533521" ixy="${reflect*-0.00015428714}" ixz="0.00131612622"
+                 iyy="0.00848624936" iyz="${reflect*-0.00001906103}"
+                 izz="0.00474512541"/>
       </inertial>
       <visual>
@@ -44,9 +44,9 @@
     <link name="leg_${prefix}_2_link">
       <inertial>
-        <origin xyz="0.01583 -0.00021 0.00619" rpy="0.00000 0.00000 0.00000"/>
-        <mass value="2.37607"/>
-        <inertia ixx="0.00342100000" ixy="${reflect*-0.00011300000}" ixz="-0.00022500000"
-                 iyy="0.00402400000" iyz="${reflect*-0.00003100000}"
-                 izz="0.00416400000"/>
+        <origin xyz="-0.00704703000 ${reflect*0.02592659000} 0.00273385000" rpy="0.00000000000 0.00000000000 0.00000000000"/>
+        <mass value="1.49095200000"/>
+        <inertia ixx="0.00497152259" ixy="${reflect*-0.00013113580}" ixz="-0.00000486648"
+                 iyy="0.00190550993" iyz="${reflect*0.00004585381}"
+                 izz="0.00474289754"/>
       </inertial>
       <visual>
@@ -76,9 +76,9 @@
     <link name="leg_${prefix}_3_link">
       <inertial>
-        <origin xyz="0.00658 ${reflect*0.06563} -0.17278" rpy="0.00000 0.00000 0.00000"/>
-        <mass value="6.82734"/>
-        <inertia ixx="0.12390600000" ixy="${reflect*-0.00041200000}" ixz="-0.00205900000"
-                 iyy="0.10844700000" iyz="${reflect*0.01672500000}"
-                 izz="0.02781200000"/>
+        <origin xyz="0.00585230000 ${reflect*0.06369670000} -0.18339564000" rpy="0.00000000000 0.00000000000 0.00000000000"/>
+        <mass value="6.23987100000"/>
+        <inertia ixx="0.15337403915" ixy="${reflect*0.00068913396}" ixz="0.00168034366"
+                 iyy="0.13648139346" iyz="${reflect*-0.02187635445}"
+                 izz="0.03001594885"/>
       </inertial>
       <visual>
@@ -108,9 +108,9 @@
     <link name="leg_${prefix}_4_link">
       <inertial>
-        <origin xyz="0.01520 ${reflect*0.02331} -0.12063" rpy="0.00000 0.00000 0.00000"/>
-        <mass value="3.63668"/>
-        <inertia ixx="0.03531500000" ixy="${reflect*0.00002900000}" ixz="-0.00016600000"
-                 iyy="0.02933600000" iyz="${reflect*-0.00130500000}"
-                 izz="0.01174000000"/>
+        <origin xyz="0.01317717000 ${reflect*0.02917508000} -0.11594602000" rpy="0.00000000000 0.00000000000 0.00000000000"/>
+        <mass value="3.75995100000"/>
+        <inertia ixx="0.04287677484" ixy="${reflect*0.00043705397}" ixz="0.00078292368"
+                 iyy="0.03598906971" iyz="${reflect*0.00037717694i}"
+                 izz="0.01364791564"/>
       </inertial>
       <visual>
@@ -139,10 +139,11 @@
     <!-- Joint ankle_y (mesh link) : child link ankle_x -> parent link knee -->
     <link name="leg_${prefix}_5_link">
-      <inertial>
-        <origin xyz="-0.01106 ${reflect*0.04708} 0.05271" rpy="0.00000 0.00000 0.00000"/>
-        <mass value="1.24433"/>
-        <inertia ixx="0.01148700000" ixy="${reflect*-0.00068600000}" ixz="-0.00052600000"
-                 iyy="0.00952600000" iyz="${reflect*0.00263300000}"
-                 izz="0.00390800000"/>
+      <!-- XXX AS: this link has moving lever and inertial parameters should slightly vary depending on configuration. XXX -->
+      <inertial>
+        <origin xyz="-0.01400838000 ${reflect*0.04180064000} 0.03820186000" rpy="0.00000000000 0.00000000000 0.00000000000"/>
+        <mass value="1.29096000000"/>
+        <inertia ixx="0.01143430819" ixy="${reflect*0.00096978273}" ixz="0.00039976581"
+                 iyy="0.00888974312" iyz="${reflect*-0.00277808667}"
+                 izz="0.00506373875"/>
       </inertial>
       <visual>
@@ -172,9 +173,9 @@
     <link name="leg_${prefix}_6_link">
       <inertial>
-        <origin xyz="-0.02087 ${reflect*-0.00019} -0.06059" rpy="0.00000 0.00000 0.00000"/>
-        <mass value="1.59457"/>
-        <inertia ixx="0.00383800000" ixy="${reflect*0.00001600000}" ixz="-0.00104100000"
-                 iyy="0.00657200000" iyz="${reflect*-0.00001700000}"
-                 izz="0.00504400000"/>
+        <origin xyz="-0.02034668000 ${reflect*-0.00051514000} -0.05987428000" rpy="0.00000000000 0.00000000000 0.00000000000"/>
+        <mass value="1.59777300000"/>
+        <inertia ixx="0.00439027267" ixy="${reflect*-0.00006743674}" ixz="0.00113816363"
+                 iyy="0.00743063029" iyz="${reflect*0.00003943143}"
+                 izz="0.00550906699"/>
       </inertial>
       <visual>
@@ -201,8 +202,8 @@
         <origin xyz="0.0 0.0 0.0" rpy="0 0 0"/>
         <mass value="0.01" />
-         <inertia ixx="0.0001"  ixy="0.0"  ixz="0.0" iyy="0.0001" iyz="0.0" izz="0.0001" />
-      </inertial>
-     </link>
-     <joint name="leg_${prefix}_sole_fix_joint" type="fixed">
+        <inertia ixx="0.0001"  ixy="0.0"  ixz="0.0" iyy="0.0001" iyz="0.0" izz="0.0001" />
+      </inertial>
+    </link>
+    <joint name="leg_${prefix}_sole_fix_joint" type="fixed">
       <parent link="leg_${prefix}_6_link" />
       <child link="${prefix}_sole_link" />

Commit message: Indentation & comments.

File: talos_description/urdf/leg/leg.urdf.xacro (robot description, xacro)
@@ -58,5 +58,5 @@
       </visual>
       <collision>
-      <origin xyz="0 0 0.0" rpy="0  0  0" />
+        <origin xyz="0 0 0.0" rpy="0  0  0" />
         <geometry>
           <mesh filename="package://talos_description/meshes/v2/hip_x_collision.stl" scale="1 ${reflect*1} 1"/>

File: talos_description/urdf/torso/torso.urdf.xacro (robot description, xacro)
@@ -70,4 +70,5 @@
       <parent link="base_link"/>
       <child link="${name}_1_link"/>
+      <!-- XXX AS: The kinematic chain order for the torso was reversed manually. This value does not match the CAD model. XXX -->
       <origin xyz="0.0 0.0 0.0722"
               rpy="${0.00000 * deg_to_rad} ${0.00000 * deg_to_rad} ${0.00000 * deg_to_rad}"/>
@@ -120,26 +121,28 @@
                           soft_upper_limit="${75.00000 * deg_to_rad - eps_radians}" /> -->
     </joint>
-  <xacro:talos_imu name="imu" parent="${name}_2_link" update_rate="100.0">
-    <origin xyz="0.04925 0 0.078" rpy="${180.0*deg_to_rad} 0 ${-90.0*deg_to_rad}"/>
-  </xacro:talos_imu>
-  <gazebo reference="${name}_1_link">
-     <mu1>0.9</mu1>
-     <mu2>0.9</mu2>
-   </gazebo>
-   <gazebo reference="${name}_2_link">
-     <mu1>0.9</mu1>
-     <mu2>0.9</mu2>
-   </gazebo>
-   <gazebo reference="base_link">
-     <mu1>0.9</mu1>
-     <mu2>0.9</mu2>
-   </gazebo>
-   <gazebo reference="${name}_1_joint">
-      <implicitSpringDamper>1</implicitSpringDamper>
-   </gazebo>
-   <gazebo reference="${name}_2_joint">
-     <implicitSpringDamper>1</implicitSpringDamper>
-     <provideFeedback>1</provideFeedback>
-   </gazebo>
+    <xacro:talos_imu name="imu" parent="${name}_2_link" update_rate="100.0">
+        <!-- TODO AS: match model & sensor -->
+        <!-- <origin xyz="0.04925 0 0.078" rpy="${180.0*deg_to_rad} 0 ${-90.0*deg_to_rad}"/>-->
+        <origin xyz="0.04925 0 0.078" rpy="${180.0*deg_to_rad} 0 ${0.0*deg_to_rad}"/>
+    </xacro:talos_imu>
+    <gazebo reference="${name}_1_link">
+        <mu1>0.9</mu1>
+        <mu2>0.9</mu2>
+    </gazebo>
+    <gazebo reference="${name}_2_link">
+        <mu1>0.9</mu1>
+        <mu2>0.9</mu2>
+    </gazebo>
+    <gazebo reference="base_link">
+        <mu1>0.9</mu1>
+        <mu2>0.9</mu2>
+    </gazebo>
+    <gazebo reference="${name}_1_joint">
+        <implicitSpringDamper>1</implicitSpringDamper>
+    </gazebo>
+    <gazebo reference="${name}_2_joint">
+        <implicitSpringDamper>1</implicitSpringDamper>
+        <provideFeedback>1</provideFeedback>
+    </gazebo>
     <!-- extensions -->
     <xacro:talos_torso_differential_transmission name="${name}" number1="1" number2="2"

Commit message: Increase max effort for the knees

File: talos_description/urdf/leg/leg.urdf.xacro (robot description, xacro)
@@ -110,5 +110,5 @@
               rpy="${0.00000 * deg_to_rad} ${0.00000 * deg_to_rad} ${0.00000 * deg_to_rad}"/>
       <axis xyz="0 1 0" />
-      <limit lower="0" upper="2.618" effort="300" velocity="7" />
+      <limit lower="0" upper="2.618" effort="400" velocity="7" />
       <dynamics friction="${leg_friction}" damping="${leg_damping}"/>
     </joint>

Commit message: Add hip flexibility option in xacro file

File: talos_description/urdf/leg/leg.urdf.xacro (robot description, xacro)
@@ -9,5 +9,5 @@
   <xacro:property name="leg_friction"     value="0.0" />
   <xacro:property name="leg_damping"      value="0.0" />
-  <xacro:macro name="talos_leg" params="prefix reflect">
+  <xacro:macro name="talos_leg" params="prefix reflect flexibility:=false">
     <xacro:unless value="$(arg test)">
       <xacro:include filename="$(find talos_description_calibration)/urdf/calibration/leg_${prefix}.xacro" />
@@ -16,5 +16,52 @@
       <xacro:include filename="$(find talos_description)/test/calibration/leg_${prefix}.xacro" />
     </xacro:if>
-    <!-- Joint hip_z (mesh link) : child link hip_x -> parent link base_link -->
+    <xacro:if value="${flexibility}">
+  <!-- Joint flex_hip_y (mesh link) : child link flex_hip_x -> parent link base_link -->
+    <link name="leg_${prefix}_flex_1_link">
+    <inertial>
+      <origin rpy="0. 0. 0." xyz="0. 0. 0."/>
+      <mass value="0.0000"/>
+      <inertia ixx="0." ixy="0." ixz="-0." iyy="0." iyz="0." izz="0."/>
+    </inertial>
+    <visual>
+      <origin rpy="0 0 0" xyz="0 0 0"/>
+      <geometry>
+        <cylinder length="0.001" radius="0.1"/>
+      </geometry>
+      <material name="LightGrey"/>
+    </visual>
+  </link>
+  <joint name="leg_${prefix}_flex_1_joint" type="revolute">
+    <parent link="base_link"/>
+    <child link="leg_${prefix}_flex_1_link"/>
+    <origin rpy="0.0 0.0 0.0" xyz="-0.02 ${reflect*0.085} -0.18105"/>
+    <axis xyz="0 1 0"/>
+    <limit effort="100" lower="-0.349065850399" upper="1.57079632679" velocity="3.87"/>
+    <dynamics damping="0.0" friction="0.0"/>
+  </joint>
+  <!-- Joint flex_hip_x (mesh link) : child link hip_z -> parent link flex_hip_y -->
+  <link name="leg_${prefix}_flex_2_link">
+    <inertial>
+      <origin rpy="0. 0. 0." xyz="0. 0. 0."/>
+      <mass value="0."/>
+      <inertia ixx="0." ixy="0." ixz="-0." iyy="0." iyz="0." izz="0."/>
+    </inertial>
+    <visual>
+      <origin rpy="0 0 0" xyz="0 0 0"/>
+      <geometry>
+        <cylinder length="0.001" radius="0.1"/>
+      </geometry>
+      <material name="LightGrey"/>
+    </visual>
+  </link>
+  <joint name="leg_${prefix}_flex_2_joint" type="revolute">
+    <parent link="leg_${prefix}_flex_1_link"/>
+    <child link="leg_${prefix}_flex_2_link"/>
+    <origin rpy="0.0 0.0 0.0" xyz="-0.000 0.000 -0.0000"/>
+    <axis xyz="1 0 0"/>
+    <limit effort="100" lower="-0.349065850399" upper="1.57079632679" velocity="3.87"/>
+    <dynamics damping="0.0" friction="0.0"/>
+  </joint>
+    </xacro:if>
     <link name="leg_${prefix}_1_link">
       <xacro:call macro="leg_${prefix}_1_link_inertial" />
@@ -33,6 +80,12 @@
       </collision>
     </link>
+    <!-- Joint hip_z (mesh link) : child link hip_x -> parent link base_link -->
     <joint name="leg_${prefix}_1_joint" type="revolute">
-      <parent link="base_link"/>
+      <xacro:if value="${flexibility}">
+      	<parent link="leg_${prefix}_flex_2_link"/>
+      </xacro:if>
+      <xacro:unless value="${flexibility}">
+      	<parent link="base_link"/>
+      </xacro:unless>
       <child link="leg_${prefix}_1_link"/>
       <origin xyz="${-0.02 + leg_1_joint_x_offset} ${reflect*0.08500 + leg_1_joint_y_offset} ${-0.27105 + leg_1_joint_z_offset}"

File: talos_description/urdf/talos_full_common.urdf.xacro (robot description, xacro)
@@ -34,6 +34,6 @@
   <xacro:talos_gripper name="gripper_left" parent="wrist_left_ft_tool_link" reflect="1" />
   <xacro:talos_gripper name="gripper_right" parent="wrist_right_ft_tool_link" reflect="-1" />
-  <xacro:talos_leg prefix="left"  reflect="1" />
-  <xacro:talos_leg prefix="right" reflect="-1" />
+  <xacro:talos_leg prefix="left"  reflect="1" flexibility="true"/>
+  <xacro:talos_leg prefix="right" reflect="-1" flexibility="true"/>
   <!-- Macro to have the add-on links specific to each TALOS -->
   <xacro:talos_addons />

Commit message: Fix xacro for flexibility

File: talos_description/urdf/leg/leg.urdf.xacro (robot description, xacro)
@@ -37,5 +37,5 @@
     <origin rpy="0.0 0.0 0.0" xyz="-0.02 ${reflect*0.085} -0.18105"/>
     <axis xyz="0 1 0"/>
-    <limit effort="100" lower="-0.349065850399" upper="1.57079632679" velocity="3.87"/>
+    <limit effort="100" lower="-1.57" upper="1.57" velocity="100"/>
     <dynamics damping="0.0" friction="0.0"/>
   </joint>
@@ -60,5 +60,5 @@
     <origin rpy="0.0 0.0 0.0" xyz="-0.000 0.000 -0.0000"/>
     <axis xyz="1 0 0"/>
-    <limit effort="100" lower="-0.349065850399" upper="1.57079632679" velocity="3.87"/>
+    <limit effort="100" lower="-1.57" upper="1.57" velocity="100"/>
     <dynamics damping="0.0" friction="0.0"/>
   </joint>
@@ -81,11 +81,7 @@
     </link>
     <!-- Joint hip_z (mesh link) : child link hip_x -> parent link base_link -->
+    <xacro:unless value="${flexibility}">
     <joint name="leg_${prefix}_1_joint" type="revolute">
-      <xacro:if value="${flexibility}">
-      	<parent link="leg_${prefix}_flex_2_link"/>
-      </xacro:if>
-      <xacro:unless value="${flexibility}">
-      	<parent link="base_link"/>
-      </xacro:unless>
+      <parent link="base_link"/>
       <child link="leg_${prefix}_1_link"/>
       <origin xyz="${-0.02 + leg_1_joint_x_offset} ${reflect*0.08500 + leg_1_joint_y_offset} ${-0.27105 + leg_1_joint_z_offset}"
@@ -95,4 +91,15 @@
       <dynamics friction="${leg_friction}" damping="${leg_damping}"/>
     </joint>
+    </xacro:unless>
+    <xacro:if value="${flexibility}">
+    <joint name="leg_${prefix}_1_joint" type="revolute">
+      <parent link="leg_${prefix}_flex_2_link"/>
+      <child link="leg_${prefix}_1_link"/>
+      <origin rpy="0.0 0.0 0.0" xyz="0.00 0.000 -0.090"/>
+      <axis xyz="0 0 1" />
+      <limit lower="${(-55.0 + 35.0*reflect)*deg_to_rad}" upper="${(55.0 + 35.0*reflect)*deg_to_rad}" effort="100" velocity="3.87" />
+      <dynamics friction="${leg_friction}" damping="${leg_damping}"/>
+    </joint>
+    </xacro:if>
     <!-- Joint hip_x (mesh link) : child link hip_y -> parent link hip_z -->
     <link name="leg_${prefix}_2_link">
@@ -307,4 +314,26 @@
     <material>Gazebo/White</material>
   </gazebo>
+  <xacro:if value="${flexibility}">
+   <gazebo reference="leg_${prefix}_flex_1_link">
+     <mu1>0.9</mu1>
+     <mu2>0.9</mu2>
+   </gazebo>
+   <gazebo reference="leg_${prefix}_flex_2_link">
+     <mu1>0.9</mu1>
+     <mu2>0.9</mu2>
+   </gazebo>
+   <gazebo reference="leg_${prefix}_flex_1_joint">
+      <implicitSpringDamper>1</implicitSpringDamper>
+   </gazebo>
+   <gazebo reference="leg_${prefix}_flex_2_joint">
+      <implicitSpringDamper>1</implicitSpringDamper>
+   </gazebo>
+  <gazebo reference="leg_${prefix}_flex_1_link">
+    <material>Gazebo/FlatBlack</material>
+  </gazebo>
+  <gazebo reference="leg_${prefix}_flex_2_link">
+    <material>Gazebo/FlatBlack</material>
+  </gazebo>
+  </xacro:if>
   </xacro:macro>
 </robot>

Commit message: increase torque limit of the flexibility

File: talos_description/urdf/leg/leg.urdf.xacro (robot description, xacro)
@@ -37,5 +37,5 @@
     <origin rpy="0.0 0.0 0.0" xyz="-0.02 ${reflect*0.085} -0.18105"/>
     <axis xyz="0 1 0"/>
-    <limit effort="100" lower="-1.57" upper="1.57" velocity="100"/>
+    <limit effort="500" lower="-1.57" upper="1.57" velocity="100"/>
     <dynamics damping="0.0" friction="0.0"/>
   </joint>
@@ -60,5 +60,5 @@
     <origin rpy="0.0 0.0 0.0" xyz="-0.000 0.000 -0.0000"/>
     <axis xyz="1 0 0"/>
-    <limit effort="100" lower="-1.57" upper="1.57" velocity="100"/>
+    <limit effort="500" lower="-1.57" upper="1.57" velocity="100"/>
     <dynamics damping="0.0" friction="0.0"/>
   </joint>

Commit message: Add very small mass and inertia to flexibility links (because of issue in pybullet with null values for inertia)

File: talos_description/urdf/leg/leg.urdf.xacro (robot description, xacro)
@@ -21,6 +21,6 @@
     <inertial>
       <origin rpy="0. 0. 0." xyz="0. 0. 0."/>
-      <mass value="0.0000"/>
-      <inertia ixx="0." ixy="0." ixz="-0." iyy="0." iyz="0." izz="0."/>
+      <mass value="1.0E-6"/>
+      <inertia ixx="1.0E-6" ixy="0." ixz="-0." iyy="1.0E-6" iyz="0." izz="1.0E-6"/>
     </inertial>
     <visual>
@@ -44,6 +44,6 @@
     <inertial>
       <origin rpy="0. 0. 0." xyz="0. 0. 0."/>
-      <mass value="0."/>
-      <inertia ixx="0." ixy="0." ixz="-0." iyy="0." iyz="0." izz="0."/>
+      <mass value="1.0E-6"/>
+      <inertia ixx="1.0E-6" ixy="0." ixz="-0." iyy="1.0E-6" iyz="0." izz="1.0E-6"/>
     </inertial>
     <visual>

Commit message: change the leg cameras parent link to leg_6_joint

File: talos_description/urdf/leg/leg.urdf.xacro (robot description, xacro)
@@ -239,5 +239,5 @@
       </link>
       <joint name="support_front_${prefix}_joint" type="fixed">
-        <parent link="leg_${prefix}_5_link"/>
+        <parent link="leg_${prefix}_6_link"/>
         <child link="support_front_${prefix}_camera_link"/>
         <origin xyz="0.1125 0 -0.064"
@@ -249,5 +249,5 @@
       </link>
       <joint name="support_rear_${prefix}_joint" type="fixed">
-        <parent link="leg_${prefix}_5_link"/>
+        <parent link="leg_${prefix}_6_link"/>
         <child link="support_rear_${prefix}_camera_link"/>
         <origin xyz="-0.1313 0 -0.064"
