Commit message: Invert torso joints order. Check base_link

File: talos_description/urdf/torso/torso.urdf.xacro (robot description, xacro)
@@ -68,11 +68,11 @@
     </link>
     <joint name="${name}_1_joint" type="revolute">
-      <parent link="${name}_2_link"/>
+      <parent link="base_link"/>
       <child link="${name}_1_link"/>
-      <origin xyz="0.0 0.0 0.0"
+      <origin xyz="0.0 0.0 0.0722"
               rpy="${0.00000 * deg_to_rad} ${0.00000 * deg_to_rad} ${0.00000 * deg_to_rad}"/>
-      <axis xyz="0 1 0" />
-      <limit lower="${-45.0 * deg_to_rad}" upper="${15.0 * deg_to_rad}"
-             effort="${torso_max_effort}" velocity="${torso_max_vel}"/>
+      <axis xyz="0 0 1" />
+      <limit lower="${-75.00000 * deg_to_rad}" upper="${75.00000 * deg_to_rad}"
+             effort="${torso_max_effort}" velocity="${torso_max_vel}" />
       <dynamics damping="1.0" friction="1.0"/>
       <!-- <safety_controller k_position="20"
@@ -108,10 +108,10 @@
     <joint name="${name}_2_joint" type="revolute">
       <parent link="${name}_1_link"/>
-      <child link="base_link"/>
-      <origin xyz="0.0 0.0 -0.0722"
+      <child link="${name}_2_link"/>
+      <origin xyz="0.0 0.0 0.0"
               rpy="${0.00000 * deg_to_rad} ${0.00000 * deg_to_rad} ${0.00000 * deg_to_rad}"/>
-      <axis xyz="0 0 1" />
-      <limit lower="${-75.00000 * deg_to_rad}" upper="${75.00000 * deg_to_rad}"
-             effort="${torso_max_effort}" velocity="${torso_max_vel}" />
+      <axis xyz="0 1 0" />
+      <limit lower="${-15.0 * deg_to_rad}" upper="${45.0 * deg_to_rad}"
+             effort="${torso_max_effort}" velocity="${torso_max_vel}"/>
       <dynamics friction="1.0" damping="1.0"/>
       <!-- <safety_controller k_position="20"

Commit message: Fix imu tf and frame

File: talos_description/urdf/torso/torso.urdf.xacro (robot description, xacro)
@@ -121,5 +121,5 @@
     </joint>
   <xacro:talos_imu name="imu" parent="${name}_2_link" update_rate="100.0">
-    <origin xyz="0.04925 0 0.078" rpy="${180.0*deg_to_rad} 0 ${-90.0*deg_to_rad}"/>
+    <origin xyz="0.04925 0 0.078" rpy="${180.0*deg_to_rad} 0 ${90.0*deg_to_rad}"/>
   </xacro:talos_imu>
   <gazebo reference="${name}_1_link">

Commit message: Updated dynamic parameters of the torso.

File: talos_description/urdf/torso/torso.urdf.xacro (robot description, xacro)
@@ -22,9 +22,9 @@
     <link name="${name}_2_link">
       <inertial>
-        <origin xyz="-0.04551 -0.00053 0.16386" rpy="0.00000 0.00000 0.00000"/>
-        <mass value="17.55011"/>
-        <inertia ixx="0.37376900000" ixy="0.00063900000" ixz="0.01219600000"
-                 iyy="0.24790200000" iyz="0.00000700000"
-                 izz="0.28140400000"/>
+        <origin xyz="-0.02069 -0.00224 0.14214" rpy="0.00000 0.00000 0.00000"/>
+        <mass value="18.05564"/>
+        <inertia ixx="0.48557589000" ixy="-0.00187823000" ixz="0.00665087000"
+                 iyy="0.32765320000" iyz="0.00292274000"
+                 izz="0.33966948000"/>
       </inertial>
       <visual>
@@ -47,9 +47,9 @@
     <link name="${name}_1_link">
       <inertial>
-        <origin xyz="0.00013 -0.00001 -0.01306" rpy="0.00000 0.00000 0.00000"/>
-        <mass value="3.02433"/>
-        <inertia ixx="0.00759400000" ixy="0.00000100000" ixz="-0.00004800000"
-                 iyy="0.00429200000" iyz="-0.00000100000"
-                 izz="0.00749700000"/>
+        <origin xyz="0.00078 0.00004 -0.01782" rpy="0.00000 0.00000 0.00000"/>
+        <mass value="2.29466"/>
+        <inertia ixx="0.00638508000" ixy="0.00000007000" ixz="0.00003066000"
+                 iyy="0.00410256000" iyz="0.00000147000"
+                 izz="0.00622969000"/>
       </inertial>
       <visual>
@@ -86,9 +86,9 @@
     <link name="base_link">
       <inertial>
-        <origin xyz="-0.08222 0.00838 -0.07261" rpy="0.00000 0.00000 0.00000"/>
-        <mass value="13.53810"/>
-        <inertia ixx="0.06989000000" ixy="-0.00011700000" ixz="0.00023000000"
-                 iyy="0.03998200000" iyz="-0.00132500000"
-                 izz="0.08234500000"/>
+        <origin xyz="-0.05709 0.00153 -0.07625" rpy="0.00000 0.00000 0.00000"/>
+        <mass value="15.36284"/>
+        <inertia ixx="0.20105076000" ixy="-0.00023245000" ixz="-0.00401677000"
+                 iyy="0.08411497000" iyz="0.00087207000"
+                 izz="0.23189084000"/>
       </inertial>
       <visual>

Commit message: torso_link_1 inertial parameters (now ok)

File: talos_description/urdf/torso/torso.urdf.xacro (robot description, xacro)
@@ -22,9 +22,9 @@
     <link name="${name}_2_link">
       <inertial>
-        <origin xyz="-0.02069 -0.00224 0.14214" rpy="0.00000 0.00000 0.00000"/>
-        <mass value="18.05564"/>
-        <inertia ixx="0.48557589000" ixy="-0.00187823000" ixz="0.00665087000"
-                 iyy="0.32765320000" iyz="0.00292274000"
-                 izz="0.33966948000"/>
+        <origin xyz="-0.04636 -0.00099 0.14528" rpy="0.00000 0.00000 0.00000"/>
+        <mass value="16.97403"/>
+        <inertia ixx="0.44372634000" ixy="-0.00069132000" ixz="0.01218206000"
+                 iyy="0.29985761000" iyz="0.00019623000"
+                 izz="0.32201555000"/>
       </inertial>
       <visual>

Commit message: Fix IMU orientation (again)

File: talos_description/urdf/torso/torso.urdf.xacro (robot description, xacro)
@@ -122,5 +122,5 @@
     </joint>
     <xacro:talos_imu name="imu" parent="${name}_2_link" update_rate="100.0">
-        <origin xyz="0.04925 0 0.078" rpy="${180.0*deg_to_rad} 0 ${-90.0*deg_to_rad}"/>
+        <origin xyz="0.04925 0 0.078" rpy="${180.0*deg_to_rad} 0 ${90.0*deg_to_rad}"/>
     </xacro:talos_imu>
     <gazebo reference="${name}_1_link">

Commit message: Add configurable imu rpy offsets

File: talos_description/urdf/torso/torso.urdf.xacro (robot description, xacro)
@@ -12,4 +12,5 @@
   <xacro:include filename="$(find talos_description)/urdf/torso/torso.transmission.xacro" />
   <xacro:include filename="$(find talos_description)/urdf/sensors/imu.urdf.xacro" />
+  <xacro:include filename="$(find talos_description_calibration)/urdf/calibration/calibration_constants.urdf.xacro" />
  <!--Constant parameters-->
   <xacro:property name="torso_max_vel"  value="5.4" />
@@ -104,5 +105,6 @@
     </joint>
     <xacro:talos_imu name="imu" parent="${name}_2_link" update_rate="100.0">
-        <origin xyz="0.04925 0 0.078" rpy="${180.0*deg_to_rad} 0 ${90.0*deg_to_rad}"/>
+    <origin xyz="0.04925 0 0.078"
+	    rpy="${(180.0 + torso_imu_roll_offset)*deg_to_rad} ${(0.0 + torso_imu_pitch_offset)*deg_to_rad} ${(90.0 + torso_imu_pitch_offset)*deg_to_rad}"/>
     </xacro:talos_imu>
     <gazebo reference="${name}_1_link">

File: talos_description_calibration/urdf/calibration/calibration_constants.urdf.xacro (robot description, xacro)
@@ -33,3 +33,7 @@
   <xacro:property name="head_1_joint_offset" value="0.0" />
   <xacro:property name="head_2_joint_offset" value="0.0" />
+  <!-- Torso rpy offsets in degrees -->
+  <xacro:property name="torso_imu_roll_offset" value="0.0" />
+  <xacro:property name="torso_imu_pitch_offset" value="0.0" />
+  <xacro:property name="torso_imu_yaw_offset" value="0.0" />
 </robot>

Commit message: Add configurable imu xyz

File: talos_description/urdf/torso/torso.urdf.xacro (robot description, xacro)
@@ -105,5 +105,5 @@
     </joint>
     <xacro:talos_imu name="imu" parent="${name}_2_link" update_rate="100.0">
-    <origin xyz="0.04925 0 0.078"
+    <origin xyz="${0.04925 + torso_imu_x_offset} ${0.0 + torso_imu_y_offset} ${0.078 + torso_imu_z_offset}"
 	    rpy="${(180.0 + torso_imu_roll_offset)*deg_to_rad} ${(0.0 + torso_imu_pitch_offset)*deg_to_rad} ${(90.0 + torso_imu_pitch_offset)*deg_to_rad}"/>
     </xacro:talos_imu>

File: talos_description_calibration/urdf/calibration/calibration_constants.urdf.xacro (robot description, xacro)
@@ -33,4 +33,7 @@
   <xacro:property name="head_1_joint_offset" value="0.0" />
   <xacro:property name="head_2_joint_offset" value="0.0" />
+  <xacro:property name="torso_imu_x_offset" value="0.0" />
+  <xacro:property name="torso_imu_y_offset" value="0.0" />
+  <xacro:property name="torso_imu_z_offset" value="0.0" />
   <!-- Torso rpy offsets in degrees -->
   <xacro:property name="torso_imu_roll_offset" value="0.0" />
